File: solenoid_10/solenoid_10.kicad_sch (KiCad schematic)
At the start: 7 parts, among them J1 Conn_01x12_Pin

Commit message: Added test points for all channels
Parts:
- added TP10: CH8, symbol Connector:TestPoint
- added TP11: CH9, symbol Connector:TestPoint
- added TP12: CH10, symbol Connector:TestPoint
- added TP3: CH1, symbol Connector:TestPoint
- added TP4: CH2, symbol Connector:TestPoint
- added TP5: CH3, symbol Connector:TestPoint
- added TP6: CH4, symbol Connector:TestPoint
- added TP7: CH5, symbol Connector:TestPoint
- added TP8: CH6, symbol Connector:TestPoint
- added TP9: CH7, symbol Connector:TestPoint
Connections:
- net CH10_IN: now also TP12.1
- net CH1_IN: now also TP3.1
- net CH2_IN: now also TP4.1
- net CH3_IN: now also TP5.1
- net CH4_IN: now also TP6.1
- net CH5_IN: now also TP7.1
- net CH6_IN: now also TP8.1
- net CH7_IN: now also TP9.1
- net CH8_IN: now also TP10.1
- net CH9_IN: now also TP11.1
Other:
- removed sheet solenoid_channel2
- note added: "Test Points"
- moved on the sheet: TP1, TP2

Commit message: Duplicated channel sheet for all 10 channels.
Other:
- added sheet solenoid_channel10 (solenoid_channel.kicad_sch)
- added sheet solenoid_channel2 (solenoid_channel.kicad_sch)
- added sheet solenoid_channel3 (solenoid_channel.kicad_sch)
- added sheet solenoid_channel4 (solenoid_channel.kicad_sch)
- added sheet solenoid_channel5 (solenoid_channel.kicad_sch)
- added sheet solenoid_channel6 (solenoid_channel.kicad_sch)
- added sheet solenoid_channel7 (solenoid_channel.kicad_sch)
- added sheet solenoid_channel8 (solenoid_channel.kicad_sch)
- added sheet solenoid_channel9 (solenoid_channel.kicad_sch)
- note added: "Solenoid Channels"
- moved on the sheet: TP1, TP10, TP11, TP12, TP2, TP3, TP4, TP5, TP6, TP7, TP8, TP9

Commit message: Ran annotation on entire schematic
Parts:
- renumbered LED4 to LED1, LED5 to LED2, R3 to R1, R4 to R2
Changed lines of the file:
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@@
 		(on_board yes)
 		(dnp no)
-		(property "Reference" "LED4"
+		(property "Reference" "LED1"
 			(at 23.622 108.204 0)
 			(effects
@@
 			(project ""
 				(path "/434e6819-69f9-43cf-b2a3-58457aa05675"
-					(reference "LED4")
+					(reference "LED1")
 					(unit 1)
 				)
@@
 		(dnp no)
 		(fields_autoplaced yes)
-		(property "Reference" "R4"
+		(property "Reference" "R2"
 			(at 35.56 130.81 90)
 			(effects
@@
 			(project "solenoid_10"
 				(path "/434e6819-69f9-43cf-b2a3-58457aa05675"
-					(reference "R4")
+					(reference "R2")
 					(unit 1)
 				)
@@
 		(on_board yes)
 		(dnp no)
-		(property "Reference" "LED5"
+		(property "Reference" "LED2"
 			(at 24.892 129.286 0)
 			(effects
@@
 			(project "solenoid_10"
 				(path "/434e6819-69f9-43cf-b2a3-58457aa05675"
-					(reference "LED5")
+					(reference "LED2")
 					(unit 1)
 				)
@@
 		(dnp no)
 		(fields_autoplaced yes)
-		(property "Reference" "#PWR03"
+		(property "Reference" "#PWR02"
 			(at 44.45 121.92 0)
 			(effects
@@
 			(project "solenoid_10"
 				(path "/434e6819-69f9-43cf-b2a3-58457aa05675"
-					(reference "#PWR03")
+					(reference "#PWR02")
 					(unit 1)
 				)
@@
 		(dnp no)
 		(fields_autoplaced yes)
-		(property "Reference" "R3"
+		(property "Reference" "R1"
 			(at 35.56 109.22 90)
 			(effects
@@
 			(project "solenoid_10"
 				(path "/434e6819-69f9-43cf-b2a3-58457aa05675"
-					(reference "R3")
+					(reference "R1")
 					(unit 1)
 				)
@@
 		(dnp no)
 		(fields_autoplaced yes)
-		(property "Reference" "#PWR04"
+		(property "Reference" "#PWR03"
 			(at 44.45 143.51 0)
 			(effects
@@
 			(project "solenoid_10"
 				(path "/434e6819-69f9-43cf-b2a3-58457aa05675"
-					(reference "#PWR04")
-					(unit 1)
-				)
+					(reference "#PWR03")
+					(unit 1)
+				)

Commit message: Ran electrical rule check, fixed power flag for ground.
Changed lines of the file:
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@@
 		(color 0 0 0 0)
 	)
+	(junction
+		(at 39.37 87.63)
+		(diameter 0)
+		(color 0 0 0 0)
+	)
 	(wire
 		(pts
@@
 	(wire
 		(pts
+			(xy 39.37 87.63) (xy 39.37 90.17)
+		)
+		(stroke
+			(width 0)
+			(type default)
+		)
+	)
+	(wire
+		(pts
 			(xy 31.75 58.42) (xy 45.72 58.42)
 		)
@@
 	(wire
 		(pts
-			(xy 39.37 81.28) (xy 39.37 90.17)
+			(xy 39.37 81.28) (xy 39.37 87.63)
 		)
 		(stroke
@@
 					(unit 1)
 				)
+			)
+		)
+	)
+	(symbol
+		(lib_id "power:PWR_FLAG")
+		(at 39.37 87.63 90)
+		(unit 1)
+		(exclude_from_sim no)
+		(in_bom yes)
+		(on_board yes)
+		(dnp no)
+		(fields_autoplaced yes)
+		(property "Reference" "#FLG03"
+			(at 37.465 87.63 0)
+			(effects
+				(font
+					(size 1.27 1.27)
+				)
+				(hide yes)
+			)
+		)
+		(property "Value" "PWR_FLAG"
+			(at 35.56 87.6299 90)
+			(effects
+				(font
+					(size 1.27 1.27)
+				)
+				(justify left)
+			)
+		)
+		(property "Footprint" ""
+			(at 39.37 87.63 0)
+			(effects
+				(font
+					(size 1.27 1.27)
+				)
+				(hide yes)
+			)
+		)
+		(property "Datasheet" "~"
+			(at 39.37 87.63 0)
+			(effects
+				(font
+					(size 1.27 1.27)
+				)
+				(hide yes)
+			)
+		)
+		(property "Description" "Special symbol for telling ERC where power comes from"
+			(at 39.37 87.63 0)
+			(effects
+				(font
+					(size 1.27 1.27)
+				)
+				(hide yes)
+			)
+		)
+		(pin "1"
+		)
+		(instances
+			(project ""
+				(path "/434e6819-69f9-43cf-b2a3-58457aa05675"
+					(reference "#FLG03")
+					(unit 1)
+				)

Commit message: Added jlcpcb numbers and footprints for most components.
Parts:
- J1, LED1, LED2: now left out of the parts list
- R1, R2: footprint (none) -> Resistor_SMD:R_0805_2012Metric_Pad1.20x1.40mm_HandSolder; JLCPCB (none) -> C17379; now left out of the parts list
- TP1, TP10, TP11, TP12, TP2, TP3, TP4, TP5, TP6, TP7, TP8, TP9: footprint (none) -> TestPoint:TestPoint_Pad_1.0x1.0mm; now left out of the parts list
Changed lines of the file:
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@@
 		(unit 1)
 		(exclude_from_sim no)
-		(in_bom yes)
+		(in_bom no)
 		(on_board yes)
 		(dnp no)
@@
 			)
 		)
+		(property "JLCPCB" ""
+			(at 26.67 115.57 0)
+			(effects
+				(font
+					(size 1.27 1.27)
+				)
+			)
+		)
 		(pin "1"
 		)
@@
 		(unit 1)
 		(exclude_from_sim no)
-		(in_bom yes)
+		(in_bom no)
 		(on_board yes)
 		(dnp no)
@@
 			)
 		)
-		(property "Footprint" ""
+		(property "Footprint" "TestPoint:TestPoint_Pad_1.0x1.0mm"
 			(at 182.88 57.15 0)
 			(effects
@@
 			)
 		)
+		(property "JLCPCB" ""
+			(at 182.88 62.23 0)
+			(effects
+				(font
+					(size 1.27 1.27)
+				)
+			)
+		)
 		(pin "1"
 		)
@@
 		(unit 1)
 		(exclude_from_sim no)
-		(in_bom yes)
+		(in_bom no)
 		(on_board yes)
 		(dnp no)
@@
 			)
 		)
-		(property "Footprint" ""
+		(property "Footprint" "TestPoint:TestPoint_Pad_1.0x1.0mm"
 			(at 182.88 80.01 0)
 			(effects
@@
 			)
 		)
+		(property "JLCPCB" ""
+			(at 182.88 85.09 0)
+			(effects
+				(font
+					(size 1.27 1.27)
+				)
+			)
+		)
 		(pin "1"
 		)
@@
 		(unit 1)
 		(exclude_from_sim no)
-		(in_bom yes)
+		(in_bom no)
 		(on_board yes)
 		(dnp no)
@@
 			)
 		)
-		(property "Footprint" ""
+		(property "Footprint" "TestPoint:TestPoint_Pad_1.0x1.0mm"
 			(at 182.88 118.11 0)
 			(effects
@@
 			)
 		)
+		(property "JLCPCB" ""
+			(at 182.88 123.19 0)
+			(effects
+				(font
+					(size 1.27 1.27)
+				)
+			)
+		)
 		(pin "1"
 		)
@@
 		(unit 1)
 		(exclude_from_sim no)
-		(in_bom yes)
+		(in_bom no)
 		(on_board yes)
 		(dnp no)
@@
 			)
 		)
-		(property "Footprint" ""
+		(property "Footprint" "Resistor_SMD:R_0805_2012Metric_Pad1.20x1.40mm_HandSolder"
 			(at 35.56 137.16 0)
 			(effects
@@
 			)
 		)
+		(property "JLCPCB" "C17379"
+			(at 35.56 137.16 0)
+			(effects
+				(font
+					(size 1.27 1.27)
+				)
+			)
+		)
 		(pin "2"
 		)
@@
 		(unit 1)
 		(exclude_from_sim no)
-		(in_bom yes)
+		(in_bom no)
 		(on_board yes)
 		(dnp no)
@@
 			)
 		)
-		(property "Footprint" ""
+		(property "Footprint" "TestPoint:TestPoint_Pad_1.0x1.0mm"
 			(at 182.88 95.25 0)
 			(effects
@@
 			)
 		)
+		(property "JLCPCB" ""
+			(at 182.88 100.33 0)
+			(effects
+				(font
+					(size 1.27 1.27)
+				)
+			)
+		)
 		(pin "1"
 		)
@@
 		(unit 1)
 		(exclude_from_sim no)
-		(in_bom yes)
+		(in_bom no)
 		(on_board yes)
 		(dnp no)
@@
 			)
 		)
-		(property "Footprint" ""
+		(property "Footprint" "TestPoint:TestPoint_Pad_1.0x1.0mm"
 			(at 182.88 49.53 0)
 			(effects
@@
 			)
 		)
+		(property "JLCPCB" ""
+			(at 182.88 54.61 0)
+			(effects
+				(font
+					(size 1.27 1.27)
+				)
+			)
+		)
 		(pin "1"
 		)
@@
 		(unit 1)
 		(exclude_from_sim no)
-		(in_bom yes)
+		(in_bom no)
 		(on_board yes)
 		(dnp no)
@@
 			)
 		)
-		(property "Footprint" ""
+		(property "Footprint" "TestPoint:TestPoint_Pad_1.0x1.0mm"
 			(at 182.88 64.77 0)
 			(effects
@@
 			)
 		)
+		(property "JLCPCB" ""
+			(at 182.88 69.85 0)
+			(effects
+				(font
+					(size 1.27 1.27)
+				)
+			)
+		)
 		(pin "1"
 		)
@@
 		(unit 1)
 		(exclude_from_sim no)
-		(in_bom yes)
+		(in_bom no)
 		(on_board yes)
 		(dnp no)
@@
 			)
 		)
+		(property "JLCPCB" ""
+			(at 26.67 137.16 0)
+			(effects
+				(font
+					(size 1.27 1.27)
+				)
+			)
+		)
 		(pin "1"
 		)
@@
 		(unit 1)
 		(exclude_from_sim no)
-		(in_bom yes)
+		(in_bom no)
 		(on_board yes)
 		(dnp no)
@@
 			)
 		)
-		(property "Footprint" ""
+		(property "Footprint" "TestPoint:TestPoint_Pad_1.0x1.0mm"
 			(at 182.88 110.49 0)
 			(effects
@@
 			)
 		)
+		(property "JLCPCB" ""
+			(at 182.88 115.57 0)
+			(effects
+				(font
+					(size 1.27 1.27)
+				)
+			)
+		)
 		(pin "1"
 		)
@@
 		(unit 1)
 		(exclude_from_sim no)
-		(in_bom yes)
+		(in_bom no)
 		(on_board yes)
 		(dnp no)
@@
 			)
 		)
-		(property "Footprint" ""
+		(property "Footprint" "Resistor_SMD:R_0805_2012Metric_Pad1.20x1.40mm_HandSolder"
 			(at 35.56 115.57 0)
 			(effects
@@
 			)
 		)
+		(property "JLCPCB" "C17379"
+			(at 35.56 115.57 0)
+			(effects
+				(font
+					(size 1.27 1.27)
+				)
+			)
+		)
 		(pin "2"
 		)
@@
 		(unit 1)
 		(exclude_from_sim no)
-		(in_bom yes)
+		(in_bom no)
 		(on_board yes)
 		(dnp no)
@@
 			)
 		)
-		(property "Footprint" ""
+		(property "Footprint" "TestPoint:TestPoint_Pad_1.0x1.0mm"
 			(at 182.88 87.63 0)
 			(effects
@@
 			)
 		)
+		(property "JLCPCB" ""
+			(at 182.88 92.71 0)
+			(effects
+				(font
+					(size 1.27 1.27)
+				)
+			)
+		)
 		(pin "1"
 		)
@@
 		(unit 1)
 		(exclude_from_sim no)
-		(in_bom yes)
+		(in_bom no)
 		(on_board yes)
 		(dnp no)
@@
 			)
 		)
-		(property "Footprint" ""
+		(property "Footprint" "TestPoint:TestPoint_Pad_1.0x1.0mm"
 			(at 182.88 41.91 0)
 			(effects
@@
 			)
 		)
+		(property "JLCPCB" ""
+			(at 182.88 46.99 0)
+			(effects
+				(font
+					(size 1.27 1.27)
+				)
+			)
+		)
 		(pin "1"
 		)
@@
 		(unit 1)
 		(exclude_from_sim no)
-		(in_bom yes)
+		(in_bom no)
 		(on_board yes)
 		(dnp no)
@@
 			)
 		)
-		(property "Footprint" ""
+		(property "Footprint" "TestPoint:TestPoint_Pad_1.0x1.0mm"
 			(at 182.88 102.87 0)
 			(effects
@@
 			)
 		)
+		(property "JLCPCB" ""
+			(at 182.88 107.95 0)
+			(effects
+				(font
+					(size 1.27 1.27)
+				)
+			)
+		)
 		(pin "1"
 		)
@@
 		(unit 1)
 		(exclude_from_sim no)
-		(in_bom yes)
+		(in_bom no)
 		(on_board yes)
 		(dnp no)
@@
 			)
 		)
+		(property "JLCPCB" ""
+			(at 26.67 66.04 0)
+			(effects
+				(font
+					(size 1.27 1.27)
+				)
+			)
+		)
 		(pin "9"
 		)
@@
 		(unit 1)
 		(exclude_from_sim no)
-		(in_bom yes)
+		(in_bom no)
 		(on_board yes)
 		(dnp no)
@@
 			)
 		)
-		(property "Footprint" ""
+		(property "Footprint" "TestPoint:TestPoint_Pad_1.0x1.0mm"
 			(at 182.88 72.39 0)
 			(effects
@@
 			)
 		)
+		(property "JLCPCB" ""
+			(at 182.88 77.47 0)
+			(effects
+				(font
+					(size 1.27 1.27)
+				)
+			)
+		)
 		(pin "1"
 		)
@@
 		(unit 1)
 		(exclude_from_sim no)
-		(in_bom yes)
+		(in_bom no)
 		(on_board yes)
 		(dnp no)
@@
 			)
 		)
-		(property "Footprint" ""
+		(property "Footprint" "TestPoint:TestPoint_Pad_1.0x1.0mm"
 			(at 182.88 34.29 0)
 			(effects
@@
 			)
 		)
+		(property "JLCPCB" ""
+			(at 182.88 39.37 0)
+			(effects
+				(font
+					(size 1.27 1.27)
+				)
+			)
+		)

Commit message: Assigned footprint for m12 connector
Parts:
- J1: footprint (none) -> solenoid_fp:M12-P12A-GPBM12; JLCPCB (none) -> C7423418
Changed lines of the file:
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@@
 			)
 		)
-		(property "Footprint" ""
+		(property "Footprint" "solenoid_fp:M12-P12A-GPBM12"
 			(at 26.67 66.04 0)
 			(effects
@@
 			)
 		)
-		(property "JLCPCB" ""
+		(property "JLCPCB" "C7423418"
 			(at 26.67 66.04 0)
 			(effects
+				(font
+					(size 1.27 1.27)
+				)
+			)
+		)
+		(property "Purpose" ""
+			(at 26.67 66.04 0)
+			(effects

Commit message: Rarranged M12 pin to channel connections.
The changes allow better trace routing to minimize both length and the
EMI that could occur from routing traces accross each other.
Connections:
- net +24V: now also J1.2 (Pin_2); no longer J1.1 (Pin_1)
- net CH10_IN: now also J1.8 (Pin_8); no longer J1.11 (Pin_11)
- net CH1_IN: now also J1.7 (Pin_7); no longer J1.2 (Pin_2)
- net CH2_IN: now also J1.6 (Pin_6); no longer J1.3 (Pin_3)
- net CH3_IN: now also J1.5 (Pin_5); no longer J1.4 (Pin_4)
- net CH4_IN: now also J1.4 (Pin_4); no longer J1.5 (Pin_5)
- net CH5_IN: now also J1.1 (Pin_1); no longer J1.6 (Pin_6)
- net CH6_IN: now also J1.12 (Pin_12); no longer J1.7 (Pin_7)
- net CH7_IN: now also J1.11 (Pin_11); no longer J1.8 (Pin_8)
- net CH8_IN: now also J1.10 (Pin_10); no longer J1.9 (Pin_9)
- net CH9_IN: now also J1.9 (Pin_9); no longer J1.10 (Pin_10)
- net GND: now also J1.3 (Pin_3); no longer J1.12 (Pin_12)

Commit message: Updated sheet info/name and date on schematic main sheet.
Other:
- company: Home-Wood-Creations -> Homewood Creations
Changed lines of the file:
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@@
 	(title_block
 		(title "Solenoid_10")
-		(date "2025-04-09")
+		(date "2025-04-12")
 		(rev "0.1.0")
-		(company "Home-Wood-Creations")
+		(company "Homewood Creations")
 		(comment 1 "Author: Jake Goodwin")
 	)
