File: solenoid_10/solenoid_channel.kicad_sch (KiCad schematic)
At the start: 8 parts, among them J2 1217080-1, J3 1217080-1, Q1 AO4486

Commit message: Added 12v power supply section for testing.
Parts:
- renumbered Dsh1 to D2
Changed lines of the file:
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@@
 		(dnp no)
 		(fields_autoplaced yes)
-		(property "Reference" "Dsh1"
+		(property "Reference" "D2"
 			(at 146.05 78.74 0)
 			(effects
@@
 			(project "solenoid_10"
 				(path "/434e6819-69f9-43cf-b2a3-58457aa05675/22d9bef0-fbbf-4c96-a1de-b9073d4eab1a"
-					(reference "Dsh1")
+					(reference "D2")
 					(unit 1)
 				)

Commit message: Added hole for solenoid channel
Parts:
- added H1: solenoid_hole, symbol Mechanical:MountingHole
Changed lines of the file:
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@@
+	)
+	(symbol
+		(lib_id "Mechanical:MountingHole")
+		(at 139.7 45.72 0)
+		(unit 1)
+		(exclude_from_sim yes)
+		(in_bom no)
+		(on_board yes)
+		(dnp no)
+		(fields_autoplaced yes)
+		(property "Reference" "H1"
+			(at 142.24 44.4499 0)
+			(effects
+				(font
+					(size 1.27 1.27)
+				)
+				(justify left)
+			)
+		)
+		(property "Value" "solenoid_hole"
+			(at 142.24 46.9899 0)
+			(effects
+				(font
+					(size 1.27 1.27)
+				)
+				(justify left)
+			)
+		)
+		(property "Footprint" ""
+			(at 139.7 45.72 0)
+			(effects
+				(font
+					(size 1.27 1.27)
+				)
+				(hide yes)
+			)
+		)
+		(property "Datasheet" "~"
+			(at 139.7 45.72 0)
+			(effects
+				(font
+					(size 1.27 1.27)
+				)
+				(hide yes)
+			)
+		)
+		(property "Description" "Mounting Hole without connection"
+			(at 139.7 45.72 0)
+			(effects
+				(font
+					(size 1.27 1.27)
+				)
+				(hide yes)
+			)
+		)
+		(instances
+			(project ""
+				(path "/434e6819-69f9-43cf-b2a3-58457aa05675/22d9bef0-fbbf-4c96-a1de-b9073d4eab1a"
+					(reference "H1")
+					(unit 1)
+				)
+				(path "/434e6819-69f9-43cf-b2a3-58457aa05675/31dd3f1a-af55-40f0-ad15-494e6c90d7a9"
+					(reference "H2")
+					(unit 1)
+				)
+			)
+		)
 	)
 	(symbol

Commit message: swapped over to 1.8mm SMD led
Parts:
- removed LED1: LED_5mm, PCM_LED_THT_AKL:LED_D5.0mm, symbol PCM_LED_AKL:LED_5mm
- added LED6: LED_1.8mm_SMD, PCM_LED_SMD_AKL:LED_1.8mm_GullWing, symbol PCM_LED_AKL:LED_1.8mm_SMD
Connections:
- net 24V: now also LED6.2 (A)
- net at R1.2 (-): now also LED6.1 (K)
Other:
- moved on the sheet: R1
Changed lines of the file:
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@@
 	(wire
 		(pts
-			(xy 153.67 63.5) (xy 163.83 63.5)
+			(xy 160.02 63.5) (xy 163.83 63.5)
 		)
 		(stroke
@@
 		(pts
 			(xy 163.83 63.5) (xy 163.83 74.93)
+		)
+		(stroke
+			(width 0)
+			(type default)
+		)
+	)
+	(wire
+		(pts
+			(xy 149.86 63.5) (xy 143.51 63.5)
 		)
 		(stroke
@@
 	)
 	(symbol
+		(lib_id "PCM_LED_AKL:LED_1.8mm_SMD")
+		(at 139.7 63.5 0)
+		(unit 1)
+		(exclude_from_sim no)
+		(in_bom yes)
+		(on_board yes)
+		(dnp no)
+		(fields_autoplaced yes)
+		(property "Reference" "LED6"
+			(at 139.7 54.61 0)
+			(effects
+				(font
+					(size 1.27 1.27)
+				)
+			)
+		)
+		(property "Value" "LED_1.8mm_SMD"
+			(at 139.7 57.15 0)
+			(effects
+				(font
+					(size 1.27 1.27)
+				)
+			)
+		)
+		(property "Footprint" "PCM_LED_SMD_AKL:LED_1.8mm_GullWing"
+			(at 139.7 63.5 0)
+			(effects
+				(font
+					(size 1.27 1.27)
+				)
+				(hide yes)
+			)
+		)
+		(property "Datasheet" "~"
+			(at 139.7 63.5 0)
+			(effects
+				(font
+					(size 1.27 1.27)
+				)
+				(hide yes)
+			)
+		)
+		(property "Description" "LED, Generic 1.8mm SMD subminiature gull wing, Alternate KiCad Library"
+			(at 139.7 63.5 0)
+			(effects
+				(font
+					(size 1.27 1.27)
+				)
+				(hide yes)
+			)
+		)
+		(pin "1"
+		)
+		(pin "2"
+		)
+		(instances
+			(project "solenoid_10"
+				(path "/434e6819-69f9-43cf-b2a3-58457aa05675/22d9bef0-fbbf-4c96-a1de-b9073d4eab1a"
+					(reference "LED6")
+					(unit 1)
+				)
+				(path "/434e6819-69f9-43cf-b2a3-58457aa05675/31dd3f1a-af55-40f0-ad15-494e6c90d7a9"
+					(reference "LED7")
+					(unit 1)
+				)
+			)
+		)
+	)
+	(symbol
 		(lib_id "1217080-1:1217080-1")
 		(at 153.67 74.93 0)
@@
 	(symbol
 		(lib_id "PCM_Elektuur:R")
-		(at 148.59 63.5 270)
+		(at 154.94 63.5 270)
 		(unit 1)
 		(exclude_from_sim no)
@@
 		(fields_autoplaced yes)
 		(property "Reference" "R1"
-			(at 148.59 57.15 90)
+			(at 154.94 57.15 90)
 			(effects
 				(font
@@
 		)
 		(property "Value" "1k2"
-			(at 148.59 59.69 90)
+			(at 154.94 59.69 90)
 			(effects
 				(font
@@
 		)
 		(property "Footprint" ""
-			(at 148.59 63.5 0)
+			(at 154.94 63.5 0)
 			(effects
 				(font
@@
 		)
 		(property "Datasheet" ""
-			(at 148.59 63.5 0)
+			(at 154.94 63.5 0)
 			(effects
 				(font
@@
 		)
 		(property "Description" "resistor"
-			(at 148.59 63.5 0)
+			(at 154.94 63.5 0)
 			(effects
 				(font
@@
 		)
 		(property "Indicator" "+"
-			(at 151.765 60.325 0)
+			(at 158.115 60.325 0)
 			(effects
 				(font
@@
 		)
 		(property "Rating" "W"
-			(at 145.415 66.04 0)
+			(at 151.765 66.04 0)
 			(effects
 				(font
@@
 					(unit 1)
 				)
-			)
-		)
-	)
-	(symbol
-		(lib_id "PCM_LED_AKL:LED_5mm")
-		(at 139.7 63.5 0)
-		(unit 1)
-		(exclude_from_sim no)
-		(in_bom yes)
-		(on_board yes)
-		(dnp no)
-		(fields_autoplaced yes)
-		(property "Reference" "LED1"
-			(at 139.7 54.61 0)
-			(effects
-				(font
-					(size 1.27 1.27)
-				)
-			)
-		)
-		(property "Value" "LED_5mm"
-			(at 139.7 57.15 0)
-			(effects
-				(font
-					(size 1.27 1.27)
-				)
-			)
-		)
-		(property "Footprint" "PCM_LED_THT_AKL:LED_D5.0mm"
-			(at 139.7 63.5 0)
-			(effects
-				(font
-					(size 1.27 1.27)
-				)
-				(hide yes)
-			)
-		)
-		(property "Datasheet" "~"
-			(at 139.7 63.5 0)
-			(effects
-				(font
-					(size 1.27 1.27)
-				)
-				(hide yes)
-			)
-		)
-		(property "Description" "LED, Generic 5mm THT, Alternate KiCad Library"
-			(at 139.7 63.5 0)
-			(effects
-				(font
-					(size 1.27 1.27)
-				)
-				(hide yes)
-			)
-		)
-		(pin "1"
-		)
-		(pin "2"
-		)
-		(instances
-			(project "solenoid_10"
-				(path "/434e6819-69f9-43cf-b2a3-58457aa05675/22d9bef0-fbbf-4c96-a1de-b9073d4eab1a"
-					(reference "LED1")
-					(unit 1)
-				)
-				(path "/434e6819-69f9-43cf-b2a3-58457aa05675/31dd3f1a-af55-40f0-ad15-494e6c90d7a9"
-					(reference "LED3")
-					(unit 1)
-				)

Commit message: Duplicated channel sheet for all 10 channels.
Parts:
- renumbered H1 to H

Commit message: Added over-voltage and over-current protection to DCDC sheet.
Parts:
- renumbered H to H3
Changed lines of the file:
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@@
 		(dnp no)
 		(fields_autoplaced yes)
-		(property "Reference" "H"
+		(property "Reference" "H?"
 			(at 142.24 44.4499 0)
 			(effects
@@
 					(unit 1)
 				)
+				(path "/434e6819-69f9-43cf-b2a3-58457aa05675/22d9bef0-fbbf-4c96-a1de-b9073d4eab1a"
+					(reference "H?")
+					(unit 1)
+				)

Commit message: Added polyfuses to all channels
Parts:
- added F2: SMD1812P030TF/60, symbol Device:Polyfuse
Connections:
- net 24V: now also F2.1; no longer D2.1 (K), J3.1, J3.2, LED6.2 (A)
- new net: D2.1 (K), F2.2, J3.1, J3.2, LED6.2 (A)
Other:
- moved on the sheet: D2, H3, J2, J3, LED6, R1, S1
