File: solenoid_10/solenoid_channel.kicad_sch (KiCad schematic)
At the start: 10 parts, among them J2 1217080-1, J3 1217080-1, Q1 AO4486

Commit message: Reassigned TE footprint for all channels and set solenoid hole as M3 (3.2mm)
Parts:
- H1: footprint (none) -> MountingHole:MountingHole_3.2mm_M3_Pad_Via
- J2, J3: footprint 1217080-1:TE_1217080-1 -> solenoid_fp:TE_1217080-1
Changed lines of the file:
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@@
 			)
 		)
-		(property "Footprint" "1217080-1:TE_1217080-1"
+		(property "Footprint" "solenoid_fp:TE_1217080-1"
 			(at 153.67 66.04 0)
 			(effects
@@
 		)
 		(property "JLCPCB" ""
+			(at 153.67 66.04 0)
+			(effects
+				(font
+					(size 1.27 1.27)
+				)
+			)
+		)
+		(property "Purpose" ""
 			(at 153.67 66.04 0)
 			(effects
@@
 			)
 		)
-		(property "Footprint" "1217080-1:TE_1217080-1"
+		(property "Footprint" "solenoid_fp:TE_1217080-1"
 			(at 137.16 66.04 0)
 			(effects
@@
 		)
 		(property "JLCPCB" ""
+			(at 137.16 66.04 0)
+			(effects
+				(font
+					(size 1.27 1.27)
+				)
+			)
+		)
+		(property "Purpose" ""
 			(at 137.16 66.04 0)
 			(effects
@@
 			)
 		)
-		(property "Footprint" ""
+		(property "Footprint" "MountingHole:MountingHole_3.2mm_M3_Pad_Via"
 			(at 139.7 36.83 0)
 			(effects
@@
 			(at 139.7 36.83 0)
 			(effects
+				(font
+					(size 1.27 1.27)
+				)
+			)
+		)
+		(property "Purpose" ""
+			(at 139.7 36.83 0)
+			(effects

Commit message: changed to DIN965 3.2mm holes
Parts:
- H1: footprint MountingHole:MountingHole_3.2mm_M3_Pad_Via -> MountingHole:MountingHole_3.2mm_M3_DIN965
Changed lines of the file:
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@@
 			)
 		)
-		(property "Footprint" "MountingHole:MountingHole_3.2mm_M3_Pad_Via"
+		(property "Footprint" "MountingHole:MountingHole_3.2mm_M3_DIN965"
 			(at 139.7 36.83 0)
 			(effects

Commit message: Updated LED indicator with new JLCPCB number: C2286 for red led with 0603 footprint.
Parts:
- LED3: value LED_1.8mm_SMD -> KT-0603R; footprint PCM_LED_SMD_AKL:LED_1.8mm_GullWing -> PCM_LED_SMD_AKL:LED_0201_0603Metric_Pad0.64x0.40mm; JLCPCB (none) -> C2286
Changed lines of the file:
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@@
 			)
 		)
-		(property "Value" "LED_1.8mm_SMD"
+		(property "Value" "KT-0603R"
 			(at 139.7 48.26 0)
 			(effects
@@
 			)
 		)
-		(property "Footprint" "PCM_LED_SMD_AKL:LED_1.8mm_GullWing"
+		(property "Footprint" "PCM_LED_SMD_AKL:LED_0201_0603Metric_Pad0.64x0.40mm"
 			(at 139.7 54.61 0)
 			(effects
@@
 			)
 		)
-		(property "JLCPCB" ""
+		(property "JLCPCB" "C2286"
 			(at 139.7 54.61 0)
 			(effects
+				(font
+					(size 1.27 1.27)
+				)
+			)
+		)
+		(property "Purpose" ""
+			(at 139.7 54.61 0)
+			(effects

Commit message: changed solenoid holes from 3.2mm to 3.5mm
Parts:
- H1: footprint MountingHole:MountingHole_3.2mm_M3_DIN965 -> MountingHole:MountingHole_3.5mm
Changed lines of the file:
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@@
 			)
 		)
-		(property "Footprint" "MountingHole:MountingHole_3.2mm_M3_DIN965"
+		(property "Footprint" "MountingHole:MountingHole_3.5mm"
 			(at 139.7 36.83 0)
 			(effects

Commit message: changed all buttons to new footprint(with 3D model) and imported changes into PCB editor.
Parts:
- S1: footprint digikey-footprints:Switch_Tactile_THT_B3F-1xxx -> solenoid_fp:SW_TH_Tactile_Omron_B3F-10xx
Changed lines of the file:
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@@
 			)
 		)
-		(property "Footprint" "digikey-footprints:Switch_Tactile_THT_B3F-1xxx"
+		(property "Footprint" "solenoid_fp:SW_TH_Tactile_Omron_B3F-10xx"
 			(at 101.6 87.63 0)
 			(effects

Commit message: Updated netclass setup and fixed silkscreen sizing issue.
Parts:
- D1, F1, H1, J2, J3, Q1, R3, R4: now in the parts list
- LED3: footprint PCM_LED_SMD_AKL:LED_0201_0603Metric_Pad0.64x0.40mm -> PCM_LED_SMD_AKL:LED_0201_0603Metric; now in the parts list
- S1: footprint solenoid_fp:SW_TH_Tactile_Omron_B3F-10xx -> solenoid_fp:Switch_Tactile_THT_B3F-1xxx; now in the parts list
Changed lines of the file:
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@@
 		(unit 1)
 		(exclude_from_sim no)
-		(in_bom no)
+		(in_bom yes)
 		(on_board yes)
 		(dnp no)
@@
 		(unit 1)
 		(exclude_from_sim no)
-		(in_bom no)
+		(in_bom yes)
 		(on_board yes)
 		(dnp no)
@@
 		(unit 1)
 		(exclude_from_sim no)
-		(in_bom no)
+		(in_bom yes)
 		(on_board yes)
 		(dnp no)
@@
 			)
 		)
-		(property "Footprint" "PCM_LED_SMD_AKL:LED_0201_0603Metric_Pad0.64x0.40mm"
+		(property "Footprint" "PCM_LED_SMD_AKL:LED_0201_0603Metric"
 			(at 139.7 54.61 0)
 			(effects
@@
 		(unit 1)
 		(exclude_from_sim no)
-		(in_bom no)
+		(in_bom yes)
 		(on_board yes)
 		(dnp yes)
@@
 		(unit 1)
 		(exclude_from_sim no)
-		(in_bom no)
+		(in_bom yes)
 		(on_board yes)
 		(dnp no)
@@
 		(unit 1)
 		(exclude_from_sim no)
-		(in_bom no)
+		(in_bom yes)
 		(on_board yes)
 		(dnp yes)
@@
 		(unit 1)
 		(exclude_from_sim no)
-		(in_bom no)
+		(in_bom yes)
 		(on_board yes)
 		(dnp no)
@@
 		(unit 1)
 		(exclude_from_sim no)
-		(in_bom no)
+		(in_bom yes)
 		(on_board yes)
 		(dnp no)
@@
 			)
 		)
-		(property "Footprint" "solenoid_fp:SW_TH_Tactile_Omron_B3F-10xx"
+		(property "Footprint" "solenoid_fp:Switch_Tactile_THT_B3F-1xxx"
 			(at 101.6 87.63 0)
 			(effects
@@
 		(unit 1)
 		(exclude_from_sim yes)
-		(in_bom no)
+		(in_bom yes)
 		(on_board yes)
 		(dnp no)
@@
 		(unit 1)
 		(exclude_from_sim no)
-		(in_bom no)
+		(in_bom yes)
 		(on_board yes)
 		(dnp no)

Commit message: Solenoid_10, refactored input power and dc-dc converter
+ Removed crowbar circuit.
+ Added larger traces on input.
+ Added multiple copper fills for lower resistance.
+ Updated silkscreen textbox.
Other:
- company: (none) -> Homewood Creations
- title: (none) -> Solenoid_10
Changed lines of the file:
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@@
 	(generator_version "9.0")
 	(paper "A4")
+	(title_block
+		(title "Solenoid_10")
+		(rev "0.1.0")
+		(company "Homewood Creations")
+	)
 	(text_box "I_Hold: 0.3A\nI_Trip: 0.6A\nV_Max: 60V"
 		(exclude_from_sim no)

Commit message: Solenoid_10, updated cap and SOP-8 footprints and jlcpcb numbers.
+ Changed capacitor for one that has larger quantity in stock.
+ Updated footprints for MOSFET for default kicad style.
Parts:
- Q1: footprint PCM_Package_SO_AKL:SO-8_3.9x4.9mm_P1.27mm -> Package_SO:SOP-8_3.76x4.96mm_P1.27mm
Changed lines of the file:
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@@
 			)
 		)
-		(property "Footprint" "PCM_Package_SO_AKL:SO-8_3.9x4.9mm_P1.27mm"
+		(property "Footprint" "Package_SO:SOP-8_3.76x4.96mm_P1.27mm"
 			(at 158.75 93.98 0)
 			(effects
