File: solenoid_10/solenoid_channel.kicad_sch (KiCad schematic)
At the start: 10 parts, among them J2 1217080-1, J3 1217080-1, Q1 AO4486

Commit message: Solenoid_10, checked stock of more parts update fp.
+ Checked stock of Caps, LEDs, diodes and inductors.
+ Updated Footprints for better compat accross systems.
Parts:
- D1: footprint PCM_Diode_SMD_AKL:D_SOD-123F -> Diode_SMD:D_SOD-123F
- LED3: footprint PCM_LED_SMD_AKL:LED_0201_0603Metric -> LED_SMD:LED_0603_1608Metric
Changed lines of the file:
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@@
 			)
 		)
-		(property "Footprint" "PCM_Diode_SMD_AKL:D_SOD-123F"
+		(property "Footprint" "Diode_SMD:D_SOD-123F"
 			(at 146.05 76.2 0)
 			(effects
@@
 			)
 		)
-		(property "Footprint" "PCM_LED_SMD_AKL:LED_0201_0603Metric"
+		(property "Footprint" "LED_SMD:LED_0603_1608Metric"
 			(at 139.7 54.61 0)
 			(effects

Commit message: solenoid_10, refactored for manufacturing.
+ chagned cap to alternate that costs less for assembly.
+ marked more components as DNP
+ marked more components as no POS.
Parts:
- D1: JLCPCB C64898 -> (none); LCSC (none) -> C64898
- F1: JLCPCB C20995 -> (none); LCSC (none) -> C20995
- LED3: JLCPCB C2286 -> (none); LCSC (none) -> C2286
- Q1: JLCPCB C5125950 -> (none); LCSC (none) -> C5125950
- R3: JLCPCB C17673 -> (none); LCSC (none) -> C17673
- R4: JLCPCB C17379 -> (none); LCSC (none) -> C17379
- S1: JLCPCB C93157 -> (none); LCSC (none) -> C93157
Changed lines of the file:
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@@
 			)
 		)
-		(property "JLCPCB" "C17673"
-			(at 144.78 97.79 0)
-			(effects
-				(font
-					(size 1.27 1.27)
-				)
+		(property "LCSC" "C17673"
+			(at 144.78 97.79 90)
+			(effects
+				(font
+					(size 1.27 1.27)
+				)
+				(hide yes)
 			)
 		)
@@
 			)
 		)
-		(property "JLCPCB" "C64898"
+		(property "LCSC" "C64898"
 			(at 146.05 76.2 0)
 			(effects
@@
 					(size 1.27 1.27)
 				)
+				(hide yes)
 			)
 		)
@@
 			)
 		)
-		(property "JLCPCB" "C2286"
-			(at 139.7 54.61 0)
-			(effects
-				(font
-					(size 1.27 1.27)
-				)
-			)
-		)
 		(property "Purpose" ""
 			(at 139.7 54.61 0)
@@
 					(size 1.27 1.27)
 				)
+			)
+		)
+		(property "LCSC" "C2286"
+			(at 139.7 54.61 0)
+			(effects
+				(font
+					(size 1.27 1.27)
+				)
+				(hide yes)
 			)
 		)
@@
 				(justify bottom)
 				(hide yes)
-			)
-		)
-		(property "JLCPCB" ""
-			(at 153.67 66.04 0)
-			(effects
-				(font
-					(size 1.27 1.27)
-				)
 			)
 		)
@@
 			)
 		)
-		(property "JLCPCB" "C17379"
-			(at 154.94 54.61 0)
-			(effects
-				(font
-					(size 1.27 1.27)
-				)
+		(property "LCSC" "C17379"
+			(at 154.94 54.61 90)
+			(effects
+				(font
+					(size 1.27 1.27)
+				)
+				(hide yes)
 			)
 		)
@@
 			)
 		)
-		(property "JLCPCB" ""
-			(at 137.16 66.04 0)
-			(effects
-				(font
-					(size 1.27 1.27)
-				)
-			)
-		)
 		(property "Purpose" ""
 			(at 137.16 66.04 0)
@@
 			)
 		)
-		(property "JLCPCB" "C5125950"
+		(property "LCSC" "C5125950"
 			(at 153.67 96.52 0)
 			(effects
@@
 					(size 1.27 1.27)
 				)
+				(hide yes)
 			)
 		)
@@
 			)
 		)
-		(property "JLCPCB" "C93157"
-			(at 106.68 92.71 0)
-			(effects
-				(font
-					(size 1.27 1.27)
-				)
+		(property "LCSC" "C93157"
+			(at 106.68 92.71 90)
+			(effects
+				(font
+					(size 1.27 1.27)
+				)
+				(hide yes)
 			)
 		)
@@
 			)
 		)
-		(property "JLCPCB" ""
-			(at 139.7 36.83 0)
-			(effects
-				(font
-					(size 1.27 1.27)
-				)
-			)
-		)
 		(property "Purpose" ""
 			(at 139.7 36.83 0)
@@
 			)
 		)
-		(property "JLCPCB" "C20995"
-			(at 107.95 66.04 0)
-			(effects
-				(font
-					(size 1.27 1.27)
-				)
-			)
-		)
+		(property "LCSC" "C20995"
+			(at 107.95 66.04 90)
+			(effects
+				(font
+					(size 1.27 1.27)
+				)
+				(hide yes)
+			)
+		)

Commit message: solenoid_10, updated to fix the XL1509 IC, rotation by -90 for pick and place.
Parts:
- H1: now not fitted; now left out of the parts list
- J2, J3: now left out of the parts list
Changed lines of the file:
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@@
 		(unit 1)
 		(exclude_from_sim no)
-		(in_bom yes)
+		(in_bom no)
 		(on_board yes)
 		(dnp yes)
@@
 		(unit 1)
 		(exclude_from_sim no)
-		(in_bom yes)
+		(in_bom no)
 		(on_board yes)
 		(dnp yes)
@@
 		(unit 1)
 		(exclude_from_sim yes)
-		(in_bom yes)
+		(in_bom no)
 		(on_board yes)
-		(dnp no)
+		(dnp yes)
 		(fields_autoplaced yes)
 		(property "Reference" "H1"
