File: solenoid_10/solenoid_10.kicad_pcb (KiCad board)
At the start: 4 copper layers, 319.8 x 25 mm, 127 parts, among them J1 Conn_01x12_Pin, J10 1217080-1, J11 1217080-1, J12 1217080-1, J13 1217080-1, J14 1217080-1, J15 1217080-1, J16 1217080-1, J17 1217080-1, J18 1217080-1, J19 1217080-1, J2 1217080-1, J20 1217080-1, J21 1217080-1, J3 1217080-1, J4 1217080-1, J5 1217080-1, J6 1217080-1, J7 1217080-1, J8 1217080-1, J9 1217080-1, Q1 AO4486, Q10 AO4486, Q11 AO4486, Q2 BT148W-600R, Q3 AO4486, Q4 AO4486, Q5 AO4486, Q6 AO4486, Q7 AO4486, Q8 AO4486, Q9 AO4486, U1 XL1509-5.0

Commit message: updated shape of PCB to allow lower label area.
Parts:
- moved F8 20.0 mm to (251.9, 79.0)
- moved LED9 20.0 mm to (251.6, 86.7)
- moved Q7 20.0 mm to (240.9, 79.8)
- moved R17 20.0 mm to (251.6, 89.2)
- moved D1 20.0 mm to (119.7, 70.2)
- moved H1 20.0 mm to (119.7, 76.1)
- moved J2 20.0 mm to (114.2, 71.8)
- moved J3 20.0 mm to (125.2, 71.8)
- moved D10 20.0 mm to (303.7, 70.2)
- moved D11 20.0 mm to (326.6, 70.2)
- moved D3 20.0 mm to (142.7, 70.2)
- moved D4 20.0 mm to (165.7, 70.2)
- moved D5 20.0 mm to (188.7, 70.2)
- moved D6 20.0 mm to (211.7, 70.2)
- moved D7 20.0 mm to (234.7, 70.2)
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Other:
- board size 319.8 x 25 mm -> 297 x 29 mm

Commit message: widened out board.
Parts:
- moved TP4 62.8 mm to (74.9, 62.6)
- moved TP5 60.5 mm to (76.5, 54.6)
- moved TP6 55.3 mm to (73.4, 37.0)
- moved TP8 49.8 mm to (70.5, 46.5)
- moved TP7 46.3 mm to (62.3, 56.8)
- moved TP9 39.7 mm to (61.1, 40.7)
- moved TP10 22.5 mm to (45.9, 42.1)
- moved TP11 13.6 mm to (37.4, 34.4)
Other:
- board size 297 x 29 mm -> 297 x 37.5 mm
- board text removed: "50mm from point is starting of channels"
Changed lines of the file:
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@@
 	(footprint "TestPoint:TestPoint_Pad_1.0x1.0mm"
 		(layer "F.Cu")
-		(at 21.34 38.3)
+		(at 70.45 46.45)
 		(descr "SMD rectangular pad as test Point, square 1.0mm side length")
 		(tags "test point SMD pad rectangle square")
@@
 	(footprint "TestPoint:TestPoint_Pad_1.0x1.0mm"
 		(layer "F.Cu")
-		(at 21.34 35.25)
+		(at 62.3 56.75)
 		(descr "SMD rectangular pad as test Point, square 1.0mm side length")
 		(tags "test point SMD pad rectangle square")
@@
 	(footprint "TestPoint:TestPoint_Pad_1.0x1.0mm"
 		(layer "F.Cu")
-		(at 18.29 41.35)
+		(at 73.375 36.95)
 		(descr "SMD rectangular pad as test Point, square 1.0mm side length")
 		(tags "test point SMD pad rectangle square")
@@
 		)
 		(property "Value" "CH4"
-			(at -2.29 6.05 0)
-			(layer "B.Fab")
+			(at 0.01 2.15 180)
+			(layer "F.Fab")
 			(effects
 				(font
@@
 					(thickness 0.15)
 				)
-				(justify mirror)
 			)
 		)
@@
 	(footprint "TestPoint:TestPoint_Pad_1.0x1.0mm"
 		(layer "F.Cu")
-		(at 21.34 41.35)
+		(at 61.075 40.675)
 		(descr "SMD rectangular pad as test Point, square 1.0mm side length")
 		(tags "test point SMD pad rectangle square")
@@
 		)
 		(property "Value" "CH7"
-			(at -0.14 3.75 0)
-			(layer "B.Fab")
+			(at -0.075 2.225 180)
+			(layer "F.Fab")
 			(effects
 				(font
@@
 					(thickness 0.15)
 				)
-				(justify mirror)
 			)
 		)
@@
 	(footprint "TestPoint:TestPoint_Pad_1.0x1.0mm"
 		(layer "F.Cu")
-		(at 24.39 35.25)
+		(at 45.85 42.125)
 		(descr "SMD rectangular pad as test Point, square 1.0mm side length")
 		(tags "test point SMD pad rectangle square")
@@
 		)
 		(property "Value" "CH10"
-			(at -19.19 2.05 0)
-			(layer "B.Fab")
+			(at 0.01 2.05 180)
+			(layer "F.Fab")
 			(effects
 				(font
@@
 					(thickness 0.15)
 				)
-				(justify mirror)
 			)
 		)
@@
 	(footprint "TestPoint:TestPoint_Pad_1.0x1.0mm"
 		(layer "F.Cu")
-		(at 18.29 35.25)
+		(at 74.875 62.575)
 		(descr "SMD rectangular pad as test Point, square 1.0mm side length")
 		(tags "test point SMD pad rectangle square")
@@
 	(footprint "TestPoint:TestPoint_Pad_1.0x1.0mm"
 		(layer "F.Cu")
-		(at 18.29 38.3)
+		(at 76.55 54.65)
 		(descr "SMD rectangular pad as test Point, square 1.0mm side length")
 		(tags "test point SMD pad rectangle square")
@@
 	(footprint "TestPoint:TestPoint_Pad_1.0x1.0mm"
 		(layer "F.Cu")
-		(at 24.39 38.3)
+		(at 37.425 34.375)
 		(descr "SMD rectangular pad as test Point, square 1.0mm side length")
 		(tags "test point SMD pad rectangle square")
@@
 	(gr_rect
 		(start 39.8 66.75)
-		(end 336.8 95.75)
+		(end 336.8 104.25)
 		(stroke
 			(width 0.05)
@@
 		(layer "Edge.Cuts")
 	)
-	(gr_text "50mm from point is starting of channels"
-		(at 39.5 97.8 0)
-		(layer "F.Cu")
-		(effects
-			(font
-				(size 1.5 1.5)
-				(thickness 0.3)
-				(bold yes)
-			)
-			(justify left bottom)
-		)
-	)
 	(group ""

Commit message: updated footprint and layout of pcb
ssh-keygen -t ed25519 -C "your_email@example.com"#   (use "git pull" to update your local branch)
Parts:
- moved TP12 314.2 mm to (333.8, 96.0)
- moved TP11 273.4 mm to (303.8, 96.0)
- moved TP10 242.2 mm to (281.8, 97.0)
- moved TP9 211.1 mm to (264.8, 96.0)
- moved TP8 172.6 mm to (235.8, 96.0)
- moved F2 156.1 mm to (244.8, 105.8)
- moved TP7 154.6 mm to (211.8, 96.0)
- moved Q2 152.8 mm to (254.8, 107.0)
- moved TP6 135.9 mm to (195.8, 96.0)
- moved DZ1 133.2 mm to (228.1, 105.0)
- moved C3 133.0 mm to (235.8, 106.0)
- moved C2 127.7 mm to (200.6, 104.2)
- moved L1 127.7 mm to (217.3, 106.4)
- moved R5 127.7 mm to (223.6, 103.1)
- moved U1 127.7 mm to (207.9, 106.5)
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Other:
- board size 297 x 37.5 mm -> 233 x 48.5 mm
- board text added: "M62/63"
- board text added: "M64/65"
Changed lines of the file:
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@@
 			(psa4output no)
 			(plot_black_and_white yes)
-			(plotinvisibletext no)
 			(sketchpadsonfab no)
 			(plotpadnumbers no)
@@
 	(footprint "TestPoint:TestPoint_Pad_1.0x1.0mm"
 		(layer "F.Cu")
-		(at 70.45 46.45)
+		(at 235.8 96)
 		(descr "SMD rectangular pad as test Point, square 1.0mm side length")
 		(tags "test point SMD pad rectangle square")
@@
 	(footprint "PCM_Diode_SMD_AKL:D_SOD-123"
 		(layer "F.Cu")
-		(at 97.625 87 90)
+		(at 223.695 107.475 90)
 		(descr "SOD-123, Alternate KiCad Library")
 		(tags "SOD-123")
@@
 	(footprint "TestPoint:TestPoint_Pad_1.0x1.0mm"
 		(layer "F.Cu")
-		(at 62.3 56.75)
+		(at 211.8 96)
 		(descr "SMD rectangular pad as test Point, square 1.0mm side length")
 		(tags "test point SMD pad rectangle square")
@@
 	(footprint "PCM_Capacitor_SMD_US_Handsoldering_AKL:C_Elec_10x10.2"
 		(layer "F.Cu")
-		(at 65.425 83.725 -90)
+		(at 186.8 105 -90)
 		(descr "SMD capacitor, aluminum electrolytic nonpolar, 10.0x10.2mm, Alternate KiCad Library")
 		(tags "capacitor electrolyic nonpolar")
@@
 	(footprint "PCM_LED_SMD_AKL:LED_1.8mm_GullWing"
 		(layer "F.Cu")
-		(at 79.75 74.75)
+		(at 166.8 104)
 		(descr "1.8mm subminiature LED, Gull wing leads, 1.8mm diameter, https://www.tme.eu/Document/4f49387584433289ec12a23aabbb9450/OSXX212411C-TR7_VER.A.3.2.pdf, Alternate KiCad Library")
 		(tags "LED gull wing 1.8mm subminiature")
@@
 	(footprint "Diode_SMD:D_SOD-323_HandSoldering"
 		(layer "F.Cu")
-		(at 97.525 78.7 -90)
+		(at 228.125 105.05 -90)
 		(descr "SOD-323")
 		(tags "SOD-323")
@@
 	(footprint "TestPoint:TestPoint_Pad_1.0x1.0mm"
 		(layer "F.Cu")
-		(at 61.25 69.175)
+		(at 174.8 105)
 		(descr "SMD rectangular pad as test Point, square 1.0mm side length")
 		(tags "test point SMD pad rectangle square")
@@
 	(footprint "Capacitor_SMD:C_0805_2012Metric_Pad1.18x1.45mm_HandSolder"
 		(layer "F.Cu")
-		(at 74.575 83.725 -90)
+		(at 200.645 104.2 -90)
 		(descr "Capacitor SMD 0805 (2012 Metric), square (rectangular) end terminal, IPC_7351 nominal with elongated pad for handsoldering. (Body size source: IPC-SM-782 page 76, https://www.pcb-3d.com/wordpress/wp-content/uploads/ipc-sm-782a_amendment_1_and_2.pdf, https://docs.google.com/spreadsheets/d/1BsfQQcO9C6DZCsRaXUlFlo91Tg2WpOkGARC1WS5S8t0/edit?usp=sharing), generated with kicad-footprint-generator")
 		(tags "capacitor handsolder")
@@
 	(footprint "TestPoint:TestPoint_Pad_1.0x1.0mm"
 		(layer "F.Cu")
-		(at 73.375 36.95)
+		(at 195.8 96)
 		(descr "SMD rectangular pad as test Point, square 1.0mm side length")
 		(tags "test point SMD pad rectangle square")
@@
 	(footprint "TestPoint:TestPoint_Pad_1.0x1.0mm"
 		(layer "F.Cu")
-		(at 56.3 69.05)
+		(at 174.8 100)
 		(descr "SMD rectangular pad as test Point, square 1.0mm side length")
 		(tags "test point SMD pad rectangle square")
@@
 	(footprint "PCM_Package_TO_SOT_SMD_AKL:SOT-223-3_TabPin2"
 		(layer "F.Cu")
-		(at 104.95 77.3)
+		(at 254.8 107)
 		(descr "module CMS SOT223 4 pins, Alternate KiCad Library")
 		(tags "CMS SOT")
@@
 	(footprint "PCM_LED_SMD_AKL:LED_1.8mm_GullWing"
 		(layer "F.Cu")
-		(at 67.45 74.825)
+		(at 154.5 104.075)
 		(descr "1.8mm subminiature LED, Gull wing leads, 1.8mm diameter, https://www.tme.eu/Document/4f49387584433289ec12a23aabbb9450/OSXX212411C-TR7_VER.A.3.2.pdf, Alternate KiCad Library")
 		(tags "LED gull wing 1.8mm subminiature")
@@
 	(footprint "Package_SO:SOIC-8_3.9x4.9mm_P1.27mm"
 		(layer "F.Cu")
-		(at 81.825 86 -90)
+		(at 207.895 106.475 -90)
 		(descr "SOIC, 8 Pin (JEDEC MS-012AA, https://www.analog.com/media/en/package-pcb-resources/package/pkg_pdf/soic_narrow-r/r_8.pdf), generated with kicad-footprint-generator ipc_gullwing_generator.py")
 		(tags "SOIC SO")
@@
 	(footprint "Capacitor_SMD:CP_Elec_6.3x5.8"
 		(layer "F.Cu")
-		(at 104.35 85.925 -90)
+		(at 235.8 106 -90)
 		(descr "SMD capacitor, aluminum electrolytic, Nichicon, 6.3x5.8mm")
 		(tags "capacitor electrolytic")
@@
 	(footprint "Resistor_SMD:R_0805_2012Metric_Pad1.20x1.40mm_HandSolder"
 		(layer "F.Cu")
-		(at 62.075 74.85)
+		(at 149.125 104.1)
 		(descr "Resistor SMD 0805 (2012 Metric), square (rectangular) end terminal, IPC_7351 nominal with elongated pad for handsoldering. (Body size source: IPC-SM-782 page 72, https://www.pcb-3d.com/wordpress/wp-content/uploads/ipc-sm-782a_amendment_1_and_2.pdf), generated with kicad-footprint-generator")
 		(tags "resistor handsolder")
@@
 	(footprint "Resistor_SMD:R_0805_2012Metric_Pad1.20x1.40mm_HandSolder"
 		(layer "F.Cu")
-		(at 74.35 74.8)
+		(at 161.4 104.05)
 		(descr "Resistor SMD 0805 (2012 Metric), square (rectangular) end terminal, IPC_7351 nominal with elongated pad for handsoldering. (Body size source: IPC-SM-782 page 72, https://www.pcb-3d.com/wordpress/wp-content/uploads/ipc-sm-782a_amendment_1_and_2.pdf), generated with kicad-footprint-generator")
 		(tags "resistor handsolder")
@@
 	(footprint "TestPoint:TestPoint_Pad_1.0x1.0mm"
 		(layer "F.Cu")
-		(at 61.075 40.675)
+		(at 264.8 96)
 		(descr "SMD rectangular pad as test Point, square 1.0mm side length")
 		(tags "test point SMD pad rectangle square")
@@
 	(footprint "solenoid_fp:M12-P12A-GPBM12"
 		(layer "F.Cu")
-		(at 49.8 80.2)
+		(at 129.57 103.2)
 		(property "Reference" "J1"
 			(at 0 -0.5 0)
@@
 		)
 		(property "Value" "Conn_01x12_Pin"
-			(at 0 1 0)
+			(at -9.83 -3.2 0)
 			(unlocked yes)
 			(layer "F.Fab")
@@
 	(footprint "TestPoint:TestPoint_Pad_1.0x1.0mm"
 		(layer "F.Cu")
-		(at 45.85 42.125)
+		(at 281.8 97)
 		(descr "SMD rectangular pad as test Point, square 1.0mm side length")
 		(tags "test point SMD pad rectangle square")
@@
 	(footprint "TestPoint:TestPoint_Pad_1.0x1.0mm"
 		(layer "F.Cu")
-		(at 24.39 41.35)
+		(at 333.8 96)
 		(descr "SMD rectangular pad as test Point, square 1.0mm side length")
 		(tags "test point SMD pad rectangle square")
@@
 	(footprint "TestPoint:TestPoint_Pad_1.0x1.0mm"
 		(layer "F.Cu")
-		(at 74.875 62.575)
+		(at 142.8 96)
 		(descr "SMD rectangular pad as test Point, square 1.0mm side length")
 		(tags "test point SMD pad rectangle square")
@@
 	(footprint "TestPoint:TestPoint_Pad_1.0x1.0mm"
 		(layer "F.Cu")
-		(at 76.55 54.65)
+		(at 172.8 96)
 		(descr "SMD rectangular pad as test Point, square 1.0mm side length")
 		(tags "test point SMD pad rectangle square")
@@
 	(footprint "TestPoint:TestPoint_Pad_1.0x1.0mm"
 		(layer "F.Cu")
-		(at 65.825 69.225)
+		(at 174.8 110)
 		(descr "SMD rectangular pad as test Point, square 1.0mm side length")
 		(tags "test point SMD pad rectangle square")
@@
 	(footprint "Fuse:Fuse_1812_4532Metric_Pad1.30x3.40mm_HandSolder"
 		(layer "F.Cu")
-		(at 91.2 77.925 90)
+		(at 244.8 105.775 90)
 		(descr "Fuse SMD 1812 (4532 Metric), square (rectangular) end terminal, IPC_7351 nominal with elongated pad for handsoldering. (Body size source: https://www.nikhef.nl/pub/departments/mt/projects/detectorR_D/dtddice/ERJ2G.pdf), generated with kicad-footprint-generator")
 		(tags "fuse handsolder")
@@
 	(footprint "Resistor_SMD:R_0805_2012Metric_Pad1.20x1.40mm_HandSolder"
 		(layer "F.Cu")
-		(at 97.55 82.65 -90)
+		(at 223.62 103.125 -90)
 		(descr "Resistor SMD 0805 (2012 Metric), square (rectangular) end terminal, IPC_7351 nominal with elongated pad for handsoldering. (Body size source: IPC-SM-782 page 72, https://www.pcb-3d.com/wordpress/wp-content/uploads/ipc-sm-782a_amendment_1_and_2.pdf), generated with kicad-footprint-generator")
 		(tags "resistor handsolder")
 		(property "Reference" "R5"
-			(at 0 -1.65 90)
+			(at 5.875 -6.18 90)
 			(layer "F.SilkS")
 			(effects
@@
 		)
 		(property "Value" "1k"
-			(at 0 1.65 90)
+			(at 5.875 -2.88 90)
 			(layer "F.Fab")
 			(effects
@@
 		)
 		(fp_text user "${REFERENCE}"
-			(at 0 0 90)
+			(at 5.875 -4.53 90)
 			(layer "F.Fab")
 			(effects
@@
 	(footprint "Inductor_SMD:L_Bourns_SRP7028A_7.3x6.6mm"
 		(layer "F.Cu")
-		(at 91.2 85.9 90)
+		(at 217.27 106.375 90)
 		(descr "Shielded Power Inductors (https://www.bourns.com/docs/product-datasheets/srp7028a.pdf)")
 		(tags "Shielded Inductors Bourns SMD SRP7028A")
@@
 	(footprint "TestPoint:TestPoint_Pad_1.0x1.0mm"
 		(layer "F.Cu")
-		(at 37.425 34.375)
+		(at 303.8 96)
 		(descr "SMD rectangular pad as test Point, square 1.0mm side length")
 		(tags "test point SMD pad rectangle square")
@@
 	)
 	(gr_rect
-		(start 39.8 66.75)
-		(end 336.8 104.25)
+		(start 106.7 64.75)
+		(end 339.7 113.25)
 		(stroke
 			(width 0.05)
@@
 		(layer "Edge.Cuts")
 	)
+	(gr_text "M64/65"
+		(at 135.8 66 0)
+		(layer "F.SilkS")
+		(effects
+			(font
+				(size 1.5 2)
+				(thickness 0.1875)
+			)
+			(justify left)
+		)
+	)
+	(gr_text "M62/63"
+		(at 112.8 66 0)
+		(layer "F.SilkS")
+		(effects
+			(font
+				(size 1.5 2)
+				(thickness 0.1875)
+			)
+			(justify left)
+		)
+	)
 	(group ""

Commit message: Added a ground plane to pcb.
Routing:
- added copper zone on In1.Cu, net GND
Changed lines of the file:
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@@
+		)
+	)
+	(zone
+		(net 2)
+		(net_name "GND")
+		(layer "In1.Cu")
+		(hatch edge 0.5)
+		(connect_pads
+			(clearance 0.5)
+		)
+		(min_thickness 0.25)
+		(filled_areas_thickness no)
+		(fill yes
+			(thermal_gap 0.5)
+			(thermal_bridge_width 0.5)
+		)
+		(polygon
+			(pts
+				(xy 107.3 65.5) (xy 107.3 112.5) (xy 339.3 112.5) (xy 339.3 65.5)
+			)
 		)
 	)

Commit message: Added power plane for the +24V net.
Routing:
- added copper zone on In2.Cu, net /+24V
Changed lines of the file:
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@@
+		)
+	)
+	(zone
+		(net 1)
+		(net_name "/+24V")
+		(layer "In2.Cu")
+		(hatch edge 0.5)
+		(priority 1)
+		(connect_pads
+			(clearance 0.5)
+		)
+		(min_thickness 0.25)
+		(filled_areas_thickness no)
+		(fill
+			(thermal_gap 0.5)
+			(thermal_bridge_width 0.5)
+		)
+		(polygon
+			(pts
+				(xy 107.3 65.5) (xy 107.3 112.5) (xy 339.3 112.5) (xy 339.3 65.5)
+			)
 		)
 	)

Commit message: Added traces to channel 1. Move test points to channel locations.
Parts:
- moved TP3 63.1 mm to (113.8, 94.0)
- moved TP12 13.6 mm to (320.3, 94.0)
- moved TP5 13.2 mm to (159.8, 94.0)
- moved TP6 13.2 mm to (182.8, 94.0)
- moved TP9 13.2 mm to (251.8, 94.0)
- moved TP10 7.62 mm to (274.8, 94.0)
- moved TP8 7.28 mm to (228.8, 94.0)
- moved TP11 6.32 mm to (297.8, 94.0)
- moved TP4 6.32 mm to (136.8, 94.0)
- moved TP7 6.32 mm to (205.8, 94.0)
Routing:
- net /solenoid_channel1/solenoid_P: track 0.00 -> 22.9 mm
- net /solenoid_channel1/solenoid_N: track 0.00 -> 16.3 mm
- net /CH1_IN: track 0.00 -> 9.14 mm
- net Net-(Q1-G): track 0.00 -> 7.21 mm
- net /VGATE: track 0.00 -> 6.50 mm
- net GND: track 0.00 -> 3.95 mm, vias 0 -> 1
- net Net-(LED3-K): track 0.00 -> 3.15 mm
- net /+24V: track 0.00 -> 1.28 mm, vias 0 -> 1

Commit message: Added LED/TP labels for 24v and 5v nets.
Parts:
- moved TP1 23.0 mm to (154.3, 110.5)
- moved TP2 9.71 mm to (166.8, 110.5)
Routing:
- net /+24V: track 1.28 -> 4.16 mm, vias 1 -> 3
- net GND: track 3.95 -> 6.30 mm, vias 1 -> 3
- net Net-(LED2-K): track 0.00 -> 1.97 mm
- net Net-(LED1-K): track 0.00 -> 1.94 mm
- net /VGATE: track 6.50 -> 8.00 mm, vias 0 -> 1
Other:
- board text added: "+24V"
- board text added: "+5V"
Changed lines of the file:
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@@
 	(footprint "TestPoint:TestPoint_Pad_1.0x1.0mm"
 		(layer "F.Cu")
-		(at 174.8 105)
+		(at 166.8 110.5)
 		(descr "SMD rectangular pad as test Point, square 1.0mm side length")
 		(tags "test point SMD pad rectangle square")
@@
 	(footprint "TestPoint:TestPoint_Pad_1.0x1.0mm"
 		(layer "F.Cu")
-		(at 174.8 100)
+		(at 154.3 110.5)
 		(descr "SMD rectangular pad as test Point, square 1.0mm side length")
 		(tags "test point SMD pad rectangle square")
@@
 		)
 	)
+	(gr_text "+5V"
+		(at 163.8 108 0)
+		(layer "F.SilkS")
+		(effects
+			(font
+				(size 1.5 1.5)
+				(thickness 0.3)
+				(bold yes)
+			)
+			(justify left bottom)
+		)
+	)
+	(gr_text "+24V"
+		(at 150.8 108 0)
+		(layer "F.SilkS")
+		(effects
+			(font
+				(size 1.5 1.5)
+				(thickness 0.3)
+				(bold yes)
+			)
+			(justify left bottom)
+		)
+	)
 	(gr_text "M62/63"
 		(at 112.8 66 0)
@@
 	)
 	(segment
+		(start 156.95 104.075)
+		(end 158.225 104.075)
+		(width 0.2)
+		(layer "F.Cu")
+		(net 1)
+	)
+	(segment
+		(start 154.3 110.5)
+		(end 152.8 110.5)
+		(width 0.2)
+		(layer "F.Cu")
+		(net 1)
+	)
+	(segment
+		(start 158.225 104.075)
+		(end 158.3 104)
+		(width 0.2)
+		(layer "F.Cu")
+		(net 1)
+	)
+	(segment
 		(start 113.913375 80.113375)
 		(end 113.8 80)
@@
 		(net 1)
 	)
+	(via
+		(at 152.8 110.5)
+		(size 0.6)
+		(drill 0.3)
+		(layers "F.Cu" "B.Cu")
+		(net 1)
+	)
+	(via
+		(at 158.3 104)
+		(size 0.6)
+		(drill 0.3)
+		(layers "F.Cu" "B.Cu")
+		(net 1)
+	)
 	(segment
 		(start 125.228375 82.3845)
@@
 	)
 	(segment
+		(start 148.125 104.1)
+		(end 146.9 104.1)
+		(width 0.5)
+		(layer "F.Cu")
+		(net 2)
+	)
+	(segment
 		(start 123.958375 82.3845)
 		(end 126.498375 82.3845)
@@
 		(net 2)
 	)
+	(segment
+		(start 159.3 104)
+		(end 159.35 104.05)
+		(width 0.5)
+		(layer "F.Cu")
+		(net 2)
+	)
+	(segment
+		(start 160.4 104.05)
+		(end 159.35 104.05)
+		(width 0.5)
+		(layer "F.Cu")
+		(net 2)
+	)
 	(via
 		(at 125.3 81)
@@
 		(net 2)
 	)
+	(via
+		(at 146.8 104)
+		(size 0.5)
+		(drill 0.3)
+		(layers "F.Cu" "B.Cu")
+		(net 2)
+	)
+	(via
+		(at 159.35 104.05)
+		(size 0.5)
+		(drill 0.3)
+		(layers "F.Cu" "B.Cu")
+		(net 2)
+	)
 	(segment
 		(start 113.913375 76.7845)
@@
 	)
 	(segment
+		(start 166.8 110.5)
+		(end 165.3 110.5)
+		(width 0.2)
+		(layer "F.Cu")
+		(net 26)
+	)
+	(via
+		(at 165.3 110.5)
+		(size 0.6)
+		(drill 0.3)
+		(layers "F.Cu" "B.Cu")
+		(net 26)
+	)
+	(segment
 		(start 120.088375 83.1595)
 		(end 119.738375 82.8095)
@@
 	)
 	(segment
+		(start 152.05 104.075)
+		(end 150.15 104.075)
+		(width 0.2)
+		(layer "F.Cu")
+		(net 37)
+	)
+	(segment
+		(start 150.15 104.075)
+		(end 150.125 104.1)
+		(width 0.2)
+		(layer "F.Cu")
+		(net 37)
+	)
+	(segment
+		(start 162.45 104)
+		(end 162.4 104.05)
+		(width 0.2)
+		(layer "F.Cu")
+		(net 38)
+	)
+	(segment
+		(start 164.35 104)
+		(end 162.45 104)
+		(width 0.2)
+		(layer "F.Cu")
+		(net 38)
+	)
+	(segment

Commit message: ran ch1/2 tp traces, added +24v & GND pin connection from m12 footprint.
Routing:
- net /CH1_IN: track 9.14 -> 28.8 mm
- net /CH2_IN: track 0.00 -> 12.4 mm
- net GND: track 6.30 -> 11.0 mm, vias 3 -> 5
- net /+24V: track 4.16 -> 8.43 mm, vias 3 -> 5
- net /VGATE: track 8.00 -> 6.50 mm, vias 1 -> 0
Changed lines of the file:
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@@
+	)
+	(segment
+		(start 186.8 100.6)
+		(end 186.8 103.5)
+		(width 0.2)
+		(layer "F.Cu")
+		(net 1)
+	)
+	(segment
+		(start 129.57 100.73)
+		(end 129.57 102.1)
+		(width 0.2)
+		(layer "F.Cu")
+		(net 1)
 	)
 	(segment
@@
 	)
 	(via
+		(at 186.8 103.5)
+		(size 0.6)
+		(drill 0.3)
+		(layers "F.Cu" "B.Cu")
+		(net 1)
+	)
+	(via
 		(at 113.8 80)
 		(size 0.6)
@@
 	)
 	(via
+		(at 129.57 100.73)
+		(size 0.6)
+		(drill 0.3)
+		(layers "F.Cu" "B.Cu")
+		(net 1)
+	)
+	(via
 		(at 152.8 110.5)
 		(size 0.6)
@@
 		(layers "F.Cu" "B.Cu")
 		(net 1)
+	)
+	(segment
+		(start 131 99.3)
+		(end 131.3 99)
+		(width 0.5)
+		(layer "F.Cu")
+		(net 2)
+	)
+	(segment
+		(start 186.8 109.4)
+		(end 186.8 106.5)
+		(width 0.5)
+		(layer "F.Cu")
+		(net 2)
 	)
 	(segment
@@
 	)
 	(segment
+		(start 131 100.68)
+		(end 131 99.3)
+		(width 0.5)
+		(layer "F.Cu")
+		(net 2)
+	)
+	(segment
 		(start 159.3 104)
 		(end 159.35 104.05)
@@
 	)
 	(via
+		(at 131.3 99)
+		(size 0.5)
+		(drill 0.3)
+		(layers "F.Cu" "B.Cu")
+		(net 2)
+	)
+	(via
 		(at 159.35 104.05)
+		(size 0.5)
+		(drill 0.3)
+		(layers "F.Cu" "B.Cu")
+		(net 2)
+	)
+	(via
+		(at 186.8 106.5)
 		(size 0.5)
 		(drill 0.3)
@@
 	)
 	(segment
-		(start 166.8 110.5)
-		(end 165.3 110.5)
-		(width 0.2)
-		(layer "F.Cu")
-		(net 26)
-	)
-	(via
-		(at 165.3 110.5)
-		(size 0.6)
-		(drill 0.3)
-		(layers "F.Cu" "B.Cu")
-		(net 26)
+		(start 130.52 102.469562)
+		(end 136.8 96.189562)
+		(width 0.2)
+		(layer "F.Cu")
+		(net 31)
+	)
+	(segment
+		(start 130.52 103.75)
+		(end 130.52 102.469562)
+		(width 0.2)
+		(layer "F.Cu")
+		(net 31)
+	)
+	(segment
+		(start 136.8 96.189562)
+		(end 136.8 94)
+		(width 0.2)
+		(layer "F.Cu")
+		(net 31)
 	)
 	(segment
@@
 		(width 0.2)
 		(layer "F.Cu")
+		(net 35)
+	)
+	(segment
+		(start 128.62 103.75)
+		(end 128.62 102.469562)
+		(width 0.2)
+		(layer "F.Cu")
+		(net 35)
+	)
+	(segment
+		(start 128.62 102.469562)
+		(end 120.150438 94)
+		(width 0.2)
+		(layer "F.Cu")
+		(net 35)
+	)
+	(segment
+		(start 120.150438 94)
+		(end 113.8 94)
+		(width 0.2)
+		(layer "F.Cu")
