File: solenoid_10/solenoid_10.kicad_pcb (KiCad board)
At the start: 4 copper layers, 233 x 48.5 mm, 127 parts, among them J1 Conn_01x12_Pin, J10 1217080-1, J11 1217080-1, J12 1217080-1, J13 1217080-1, J14 1217080-1, J15 1217080-1, J16 1217080-1, J17 1217080-1, J18 1217080-1, J19 1217080-1, J2 1217080-1, J20 1217080-1, J21 1217080-1, J3 1217080-1, J4 1217080-1, J5 1217080-1, J6 1217080-1, J7 1217080-1, J8 1217080-1, J9 1217080-1, Q1 AO4486, Q10 AO4486, Q11 AO4486, Q2 BT148W-600R, Q3 AO4486, Q4 AO4486, Q5 AO4486, Q6 AO4486, Q7 AO4486, Q8 AO4486, Q9 AO4486, U1 XL1509-5.0

Commit message: Added correct M-Codes for all channels. Added M12 label.
Other:
- board text added: "M12 CONN:"
- board text added: "M66/67"
- board text added: "M68/69"
- board text added: "M70/71"
- board text added: "M72/73"
- board text added: "M74/75"
- board text added: "M76/77"
- board text added: "M78/79"
- board text added: "M80/81"
Changed lines of the file:
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@@
 		(layer "Edge.Cuts")
 	)
-	(gr_text "M64/65"
+	(gr_text "M12 CONN:"
+		(at 111.8 103.2 0)
+		(layer "F.SilkS")
+		(effects
+			(font
+				(size 1 1)
+				(thickness 0.1)
+			)
+			(justify left bottom)
+		)
+	)
+	(gr_text "M68/69"
 		(at 181.8 66 0)
 		(layer "F.SilkS")
@@
 		)
 	)
-	(gr_text "M64/65"
+	(gr_text "M78/79"
 		(at 296.3 66 0)
 		(layer "F.SilkS")
@@
 		)
 	)
-	(gr_text "M64/65"
+	(gr_text "M70/71"
 		(at 204.8 66 0)
 		(layer "F.SilkS")
@@
 		)
 	)
-	(gr_text "M64/65"
+	(gr_text "M80/81"
 		(at 319.3 66 0)
 		(layer "F.SilkS")
@@
 		)
 	)
-	(gr_text "M64/65"
+	(gr_text "M74/75"
 		(at 250.8 66 0)
 		(layer "F.SilkS")
@@
 		)
 	)
-	(gr_text "M64/65"
+	(gr_text "M66/67"
 		(at 158.8 66 0)
 		(layer "F.SilkS")
@@
 		)
 	)
-	(gr_text "M64/65"
+	(gr_text "M72/73"
 		(at 227.8 66 0)
 		(layer "F.SilkS")
@@
 		)
 	)
-	(gr_text "M64/65"
+	(gr_text "M76/77"
 		(at 273.8 66 0)
 		(layer "F.SilkS")

Commit message: finished indicator traces and channels traces.
Routing:
- net /solenoid_channel4/solenoid_N: track 16.3 -> 36.0 mm
- net /solenoid_channel3/solenoid_N: track 16.3 -> 36.0 mm
- net /solenoid_channel1/solenoid_N: track 16.3 -> 36.0 mm
- net /solenoid_channel6/solenoid_N: track 16.3 -> 35.8 mm
- net /solenoid_channel5/solenoid_N: track 16.3 -> 35.8 mm
- net /solenoid_channel2/solenoid_N: track 16.3 -> 35.8 mm
- net /solenoid_channel7/solenoid_N: track 16.3 -> 35.8 mm
- net /solenoid_channel9/solenoid_N: track 16.3 -> 35.8 mm
- net /solenoid_channel8/solenoid_N: track 16.3 -> 35.8 mm
- net /solenoid_channel10/solenoid_N: track 16.3 -> 35.8 mm
- net /CH10_IN: track 212.3 -> 223.7 mm
- net /CH4_IN: track 63.1 -> 74.4 mm
- net /CH3_IN: track 40.9 -> 52.2 mm
- net /CH5_IN: track 88.1 -> 99.4 mm
- net /CH2_IN: track 19.8 -> 31.1 mm
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
Commit message: updated led in PCB
Parts:
- LED1, LED2: value LED_1.8mm_SMD -> KT-0603R; footprint PCM_LED_SMD_AKL:LED_1.8mm_GullWing -> PCM_LED_SMD_AKL:LED_0603_1608Metric_Pad1.05x0.95mm
- LED10, LED11, LED12, LED3, LED4, LED5, LED6, LED7, LED8, LED9: value LED_1.8mm_SMD -> KT-0603R; footprint PCM_LED_SMD_AKL:LED_1.8mm_GullWing -> PCM_LED_SMD_AKL:LED_0201_0603Metric_Pad0.64x0.40mm

Commit message: updated PCB from shcematic, imported new mounting holes.
Parts:
- added H11: 4.5mm, MountingHole:MountingHole_4.5mm, F.Cu at (77.2, 90.8)
- added H12: 4.5mm, MountingHole:MountingHole_4.5mm, F.Cu at (77.2, 101.3)
- H1, H10, H2, H3, H4, H5, H6, H7, H8, H9: footprint MountingHole:MountingHole_3.2mm_M3_DIN965 -> MountingHole:MountingHole_3.5mm

Commit message: Appended change.
Parts:
- S1, S10, S2, S3, S4, S5, S6, S7, S8, S9: footprint digikey-footprints:Switch_Tactile_THT_B3F-1xxx -> solenoid_fp:SW_TH_Tactile_Omron_B3F-10xx
Routing:
- net /VGATE: track 81.4 -> 16.4 mm
- net /CH6_IN: track 121.6 -> 128.1 mm
- net /CH9_IN: track 197.9 -> 204.4 mm
- net /CH8_IN: track 172.0 -> 178.5 mm
- net /CH7_IN: track 146.5 -> 153.0 mm
- net /CH5_IN: track 99.4 -> 105.9 mm
- net /CH4_IN: track 74.4 -> 80.9 mm
- net /CH3_IN: track 52.2 -> 58.7 mm
- net /CH1_IN: track 37.0 -> 43.5 mm
- net /CH10_IN: track 223.7 -> 230.2 mm
- net /CH2_IN: track 31.1 -> 37.6 mm

Commit message: Removed old custom footprint and setup the new model for M12 along with 3D model.
Parts:
- removed J1: Conn_01x12_Pin, solenoid_fp:M12-P12A-GPBM12
- added J22: M12-P12A-GPBM12, solenoid_fp:TE_T4140012121-000, F.Cu at (129.8, 103.0)

Commit message: Positioned M12 mounting holes +-14mm from center of M12 connector at Y: 103
Parts:
- moved H12 72.4 mm to (149.7, 103.1)
- moved H11 36.3 mm to (111.4, 103.0)
- moved LED1 15.0 mm to (169.5, 104.1)
- moved LED2 15.0 mm to (181.8, 104.0)
- moved R1 15.0 mm to (164.1, 104.1)
- moved R2 15.0 mm to (176.4, 104.0)
- moved TP1 15.0 mm to (169.3, 110.5)
- moved TP2 15.0 mm to (181.8, 110.5)
- moved J22 0.25 mm to (130.0, 103.0)
Changed lines of the file:
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@@
 	(footprint "PCM_LED_SMD_AKL:LED_0603_1608Metric_Pad1.05x0.95mm"
 		(layer "F.Cu")
-		(at 166.8 104)
+		(at 181.8 104)
 		(descr "LED SMD 0603 (1608 Metric), square (rectangular) end terminal, IPC_7351 nominal, (Body size source: http://www.tortai-tech.com/upload/download/2011102023233369053.pdf), generated with kicad-footprint-generator")
 		(tags "LED handsolder")
@@
 	(footprint "TestPoint:TestPoint_Pad_1.0x1.0mm"
 		(layer "F.Cu")
-		(at 166.8 110.5)
+		(at 181.8 110.5)
 		(descr "SMD rectangular pad as test Point, square 1.0mm side length")
 		(tags "test point SMD pad rectangle square")
@@
 	(footprint "TestPoint:TestPoint_Pad_1.0x1.0mm"
 		(layer "F.Cu")
-		(at 154.3 110.5)
+		(at 169.3 110.5)
 		(descr "SMD rectangular pad as test Point, square 1.0mm side length")
 		(tags "test point SMD pad rectangle square")
@@
 	(footprint "MountingHole:MountingHole_4.5mm"
 		(layer "F.Cu")
-		(at 77.25 90.75)
+		(at 111.375 103)
 		(descr "Mounting Hole 4.5mm, no annular")
 		(tags "mounting hole 4.5mm no annular")
@@
 	(footprint "PCM_LED_SMD_AKL:LED_0603_1608Metric_Pad1.05x0.95mm"
 		(layer "F.Cu")
-		(at 154.5 104.075)
+		(at 169.5 104.075)
 		(descr "LED SMD 0603 (1608 Metric), square (rectangular) end terminal, IPC_7351 nominal, (Body size source: http://www.tortai-tech.com/upload/download/2011102023233369053.pdf), generated with kicad-footprint-generator")
 		(tags "LED handsolder")
@@
 	(footprint "Resistor_SMD:R_0805_2012Metric_Pad1.20x1.40mm_HandSolder"
 		(layer "F.Cu")
-		(at 149.125 104.1)
+		(at 164.125 104.1)
 		(descr "Resistor SMD 0805 (2012 Metric), square (rectangular) end terminal, IPC_7351 nominal with elongated pad for handsoldering. (Body size source: IPC-SM-782 page 72, https://www.pcb-3d.com/wordpress/wp-content/uploads/ipc-sm-782a_amendment_1_and_2.pdf), generated with kicad-footprint-generator")
 		(tags "resistor handsolder")
@@
 	(footprint "Resistor_SMD:R_0805_2012Metric_Pad1.20x1.40mm_HandSolder"
 		(layer "F.Cu")
-		(at 161.4 104.05)
+		(at 176.4 104.05)
 		(descr "Resistor SMD 0805 (2012 Metric), square (rectangular) end terminal, IPC_7351 nominal with elongated pad for handsoldering. (Body size source: IPC-SM-782 page 72, https://www.pcb-3d.com/wordpress/wp-content/uploads/ipc-sm-782a_amendment_1_and_2.pdf), generated with kicad-footprint-generator")
 		(tags "resistor handsolder")
@@
 	(footprint "solenoid_fp:TE_T4140012121-000"
 		(layer "F.Cu")
-		(at 129.75 103.05 -45)
+		(at 130 103 -45)
 		(property "Reference" "J22"
 			(at -0.325 -10.885 135)
@@
 	(footprint "MountingHole:MountingHole_4.5mm"
 		(layer "F.Cu")
-		(at 77.25 101.3)
+		(at 149.65 103.1)
 		(descr "Mounting Hole 4.5mm, no annular")
 		(tags "mounting hole 4.5mm no annular")
@@
 	)
 	(gr_text "+5V"
-		(at 163.8 108 0)
+		(at 178.8 108 0)
 		(layer "F.SilkS")
 		(effects
@@
 	)
 	(gr_text "+24V"
-		(at 150.8 108 0)
+		(at 165.8 108 0)
 		(layer "F.SilkS")
 		(effects
@@
 	)
 	(segment
-		(start 156.95 104.075)
-		(end 158.225 104.075)
+		(start 171.95 104.075)
+		(end 173.225 104.075)
 		(width 0.2)
 		(layer "F.Cu")
@@
 	)
 	(segment
-		(start 154.3 110.5)
-		(end 152.8 110.5)
+		(start 169.3 110.5)
+		(end 167.8 110.5)
 		(width 0.2)
 		(layer "F.Cu")
@@
 	)
 	(segment
-		(start 158.225 104.075)
-		(end 158.3 104)
+		(start 173.225 104.075)
+		(end 173.3 104)
 		(width 0.2)
 		(layer "F.Cu")
@@
 	)
 	(via
-		(at 152.8 110.5)
+		(at 167.8 110.5)
 		(size 0.6)
 		(drill 0.3)
@@
 	)
 	(via
-		(at 158.3 104)
+		(at 173.3 104)
 		(size 0.6)
 		(drill 0.3)
@@
 	)
 	(segment
-		(start 148.125 104.1)
-		(end 146.9 104.1)
+		(start 163.125 104.1)
+		(end 161.9 104.1)
 		(width 0.5)
 		(layer "F.Cu")
@@
 	)
 	(segment
-		(start 159.3 104)
-		(end 159.35 104.05)
+		(start 174.3 104)
+		(end 174.35 104.05)
 		(width 0.5)
 		(layer "F.Cu")
@@
 	)
 	(segment
-		(start 160.4 104.05)
-		(end 159.35 104.05)
+		(start 175.4 104.05)
+		(end 174.35 104.05)
 		(width 0.5)
 		(layer "F.Cu")
@@
 	)
 	(via
-		(at 146.8 104)
+		(at 161.8 104)
 		(size 0.5)
 		(drill 0.3)
@@
 	)
 	(via
-		(at 159.35 104.05)
+		(at 174.35 104.05)
 		(size 0.5)
 		(drill 0.3)
@@
 	)
 	(segment
-		(start 152.05 104.075)
-		(end 150.15 104.075)
+		(start 167.05 104.075)
+		(end 165.15 104.075)
 		(width 0.2)
 		(layer "F.Cu")
@@
 	)
 	(segment
-		(start 150.15 104.075)
-		(end 150.125 104.1)
+		(start 165.15 104.075)
+		(end 165.125 104.1)
 		(width 0.2)
 		(layer "F.Cu")
@@
 	)
 	(segment
-		(start 162.45 104)
-		(end 162.4 104.05)
+		(start 177.45 104)
+		(end 177.4 104.05)
 		(width 0.2)
 		(layer "F.Cu")
@@
 	)
 	(segment
-		(start 164.35 104)
-		(end 162.45 104)
+		(start 179.35 104)
+		(end 177.45 104)
 		(width 0.2)
 		(layer "F.Cu")

Commit message: cleaned up silkscren refernce numbers, re-routed channel 1 and moved Mosfet for hole spacing.
Parts:
- moved H12 3.65 mm to (146.0, 103.0)
- moved H11 2.62 mm to (114.0, 103.0)
- moved Q1 1.00 mm to (126.9, 79.8)
Routing:
- net Net-(Q1-G): track 7.21 -> 8.34 mm
- net /solenoid_channel1/solenoid_P: track 22.9 -> 23.7 mm
Changed lines of the file:
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@@
 	(footprint "PCM_Package_SO_AKL:SO-8_3.9x4.9mm_P1.27mm"
 		(layer "F.Cu")
-		(at 125.863375 79.8095 90)
+		(at 126.863375 79.8095 90)
 		(descr "SO, 8 Pin (https://www.nxp.com/docs/en/data-sheet/PCF8523.pdf), Alternate KiCad Library")
 		(tags "SO SO")
@@
 	(footprint "MountingHole:MountingHole_4.5mm"
 		(layer "F.Cu")
-		(at 111.375 103)
+		(at 114 103)
 		(descr "Mounting Hole 4.5mm, no annular")
 		(tags "mounting hole 4.5mm no annular")
@@
 		(at 130 103 -45)
 		(property "Reference" "J22"
-			(at -0.325 -10.885 135)
+			(at -7.778175 -7.778175 0)
 			(layer "F.SilkS")
 			(effects
@@
 	(footprint "MountingHole:MountingHole_4.5mm"
 		(layer "F.Cu")
-		(at 149.65 103.1)
+		(at 146 103)
 		(descr "Mounting Hole 4.5mm, no annular")
 		(tags "mounting hole 4.5mm no annular")
@@
 	(gr_rect
 		(start 184.8 97)
-		(end 260.3 112.5)
+		(end 260.3 112)
 		(stroke
 			(width 0.1)
@@
 	)
 	(gr_text "M12 CONN:"
-		(at 111.8 103.2 0)
+		(at 108.8 111.5 0)
 		(layer "F.SilkS")
 		(effects
@@
 		)
 	)
-	(table
-		(column_count 1)
+	(gr_text_box "10CH Solenoid Breakout\nVersion 0.1.0\nHomewood Creations"
+		(start 260.8 96.875)
+		(end 295.8 112.125)
+		(margins 1.0025 1.0025 1.0025 1.0025)
 		(layer "F.SilkS")
-		(border
-			(external yes)
-			(header yes)
-			(stroke
-				(width 0.1)
-				(type solid)
-			)
-		)
-		(separators
-			(rows yes)
-			(cols yes)
-			(stroke
-				(width 0.1)
-				(type solid)
+		(effects
+			(font
+				(size 1 1)
+				(thickness 0.1)
 			)
+			(justify left top)
 		)
-		(column_widths 30.5)
-		(row_heights 3.5 3.5 8.5)
-		(cells
-			(table_cell "M12 10CH Solenoid Breakout"
-				(start 260.8 97)
-				(end 291.3 100.5)
-				(margins 1.0025 1.0025 1.0025 1.0025)
-				(span 1 1)
-				(layer "F.SilkS")
-				(effects
-					(font
-						(size 1.27 1.27)
-					)
-					(justify left)
-				)
-			)
-			(table_cell "Version: 0.1.0"
-				(start 260.8 100.5)
-				(end 291.3 104)
-				(margins 1.0025 1.0025 1.0025 1.0025)
-				(span 1 1)
-				(layer "F.SilkS")
-				(effects
-					(font
-						(size 1.27 1.27)
-					)
-					(justify left)
-				)
-			)
-			(table_cell "Homewood Creations"
-				(start 260.8 104)
-				(end 291.3 112.5)
-				(margins 1.0025 1.0025 1.0025 1.0025)
-				(span 1 1)
-				(layer "F.SilkS")
-				(effects
-					(font
-						(size 1.27 1.27)
-					)
-					(justify left)
-				)
-			)
+		(border yes)
+		(stroke
+			(width 0.1)
+			(type solid)
 		)
 	)
@@
 	)
 	(segment
-		(start 125.228375 82.3845)
-		(end 125.228375 81.071625)
+		(start 215.958376 82.3845)
+		(end 218.498376 82.3845)
 		(width 0.5)
 		(layer "F.Cu")
@@
 	)
 	(segment
-		(start 215.958376 82.3845)
-		(end 218.498376 82.3845)
+		(start 124.958375 82.3845)
+		(end 127.498375 82.3845)
 		(width 0.5)
 		(layer "F.Cu")
@@
 	)
 	(segment
+		(start 126.228375 82.3845)
+		(end 126.228375 81.078375)
+		(width 0.5)
+		(layer "F.Cu")
+		(net 2)
+	)
+	(segment
 		(start 309.228376 81.071625)
 		(end 309.300001 81)
@@
 	)
 	(segment
-		(start 123.958375 82.3845)
-		(end 126.498375 82.3845)
-		(width 0.5)
-		(layer "F.Cu")
-		(net 2)
-	)
-	(segment
-		(start 125.228375 81.071625)
-		(end 125.3 81)
-		(width 0.5)
-		(layer "F.Cu")
-		(net 2)
-	)
-	(segment
 		(start 263.228376 82.3845)
 		(end 263.228376 81.071625)
@@
 	)
 	(segment
+		(start 126.228375 81.078375)
+		(end 126.2 81.05)
+		(width 0.5)
+		(layer "F.Cu")
+		(net 2)
+	)
+	(segment
 		(start 200.645 106.155)
 		(end 200.3 106.5)
@@
 	)
 	(via
-		(at 125.3 81)
-		(size 0.5)
-		(drill 0.3)
-		(layers "F.Cu" "B.Cu")
-		(net 2)
-	)
-	(via
 		(at 240.300001 81)
 		(size 0.5)
@@
 		(net 2)
 	)
+	(via
+		(at 126.2 81.05)
+		(size 0.5)
+		(drill 0.3)
+		(layers "F.Cu" "B.Cu")
+		(net 2)
+	)
 	(segment
 		(start 218.3 103.65)
@@
 	)
 	(segment
-		(start 116.063375 86.6595)
-		(end 116.063375 78.9345)
+		(start 115.914375 78.7855)
+		(end 113.913375 76.7845)
 		(width 0.2)
 		(layer "F.Cu")
@@
 	)
 	(segment
-		(start 116.063375 78.9345)
-		(end 113.913375 76.7845)
+		(start 114.020875 86.6595)
+		(end 115.914375 84.766)
+		(width 0.2)
+		(layer "F.Cu")
+		(net 4)
+	)
+	(segment
+		(start 115.914375 84.766)
+		(end 115.914375 78.7855)
 		(width 0.2)
 		(layer "F.Cu")
@@
 	)
 	(segment
+		(start 124.958375 77.2345)
+		(end 128.768375 77.2345)
+		(width 0.2)
+		(layer "F.Cu")
+		(net 5)
+	)
+	(segment
 		(start 125.213375 74.2995)
 		(end 125.213375 69.2195)
@@
 	)
 	(segment
-		(start 123.958375 77.2345)
-		(end 125.228375 77.2345)
-		(width 0.2)
-		(layer "F.Cu")
-		(net 5)
-	)
-	(segment
 		(start 121.113375 70.1595)
 		(end 124.273375 70.1595)
@@
 	)
 	(segment
-		(start 125.228375 76.571625)
-		(end 125.213375 76.556625)
-		(width 0.2)
-		(layer "F.Cu")
-		(net 5)
-	)
-	(segment
-		(start 126.498375 77.2345)
-		(end 125.228375 77.2345)
+		(start 124.958375 74.5545)
+		(end 125.213375 74.2995)
 		(width 0.2)
 		(layer "F.Cu")
@@
 	)
 	(segment
-		(start 126.498375 77.2345)
-		(end 127.768375 77.2345)
+		(start 124.958375 77.2345)
+		(end 124.958375 74.5545)
 		(width 0.2)
 		(layer "F.Cu")
@@
 	)
 	(segment
-		(start 125.213375 76.556625)
-		(end 125.213375 74.2995)
-		(width 0.2)
-		(layer "F.Cu")
-		(net 5)
-	)
-	(segment
-		(start 125.228375 77.2345)
-		(end 125.228375 76.571625)
-		(width 0.2)
-		(layer "F.Cu")
-		(net 5)
-	)
-	(segment
 		(start 208.53 104)
 		(end 208.53 103.653032)
@@
 	)
 	(segment
-		(start 112.613375 88.1095)
-		(end 111.163375 86.6595)
+		(start 112.613375 87.252)
+		(end 113.205875 86.6595)
 		(width 0.2)
 		(layer "F.Cu")
@@
 	(segment
 		(start 112.613375 89.2095)
-		(end 112.613375 88.1095)
+		(end 112.613375 87.252)
 		(width 0.2)
 		(layer "F.Cu")
@@
 	)
 	(segment
-		(start 121.738375 82.8095)
-		(end 122.489375 83.5605)
+		(start 128.768375 82.3845)
+		(end 128.768375 83.259499)
 		(width 0.2)
 		(layer "F.Cu")
@@
 	)
 	(segment
-		(start 127.768375 83.031625)
-		(end 127.768375 82.3845)
+		(start 128.467374 83.5605)
+		(end 122.489375 83.5605)
 		(width 0.2)
 		(layer "F.Cu")
@@
 	(segment
 		(start 122.489375 83.5605)
-		(end 127.2395 83.5605)
+		(end 121.738375 82.8095)
 		(width 0.2)
 		(layer "F.Cu")
@@
 	)
 	(segment
-		(start 127.2395 83.5605)
-		(end 127.768375 83.031625)
+		(start 128.768375 83.259499)
+		(end 128.467374 83.5605)
 		(width 0.2)
 		(layer "F.Cu")
