File: solenoid_10/solenoid_10.kicad_pcb (KiCad board)
At the start: 4 copper layers, 233 x 48.5 mm, 129 parts, among them J10 1217080-1, J11 1217080-1, J12 1217080-1, J13 1217080-1, J14 1217080-1, J15 1217080-1, J16 1217080-1, J17 1217080-1, J18 1217080-1, J19 1217080-1, J2 1217080-1, J20 1217080-1, J21 1217080-1, J22 M12-P12A-GPBM12, J3 1217080-1, J4 1217080-1, J5 1217080-1, J6 1217080-1, J7 1217080-1, J8 1217080-1, J9 1217080-1, Q1 AO4486, Q10 AO4486, Q11 AO4486, Q2 BT148W-600R, Q3 AO4486, Q4 AO4486, Q5 AO4486, Q6 AO4486, Q7 AO4486, Q8 AO4486, Q9 AO4486, U1 XL1509-5.0

Commit message: replicated channel 1 layout accross channels 2-10
Parts:
- moved Q10 1.00 mm to (310.9, 79.8)
- moved Q11 1.00 mm to (333.7, 79.8)
- moved Q3 1.00 mm to (149.9, 79.8)
- moved Q4 1.00 mm to (172.9, 79.8)
- moved Q5 1.00 mm to (195.9, 79.8)
- moved Q6 1.00 mm to (218.9, 79.8)
- moved Q7 1.00 mm to (241.9, 79.8)
- moved Q8 1.00 mm to (264.9, 79.8)
- moved Q9 1.00 mm to (287.9, 79.8)
Routing:
- net /solenoid_channel3/solenoid_N: track 0.00 -> 36.1 mm
- net /solenoid_channel2/solenoid_N: track 0.00 -> 36.1 mm
- net /solenoid_channel6/solenoid_N: track 0.00 -> 36.1 mm
- net /solenoid_channel5/solenoid_N: track 0.00 -> 36.1 mm
- net /solenoid_channel4/solenoid_N: track 0.00 -> 36.1 mm
- net /solenoid_channel7/solenoid_N: track 0.00 -> 36.1 mm
- net /solenoid_channel9/solenoid_N: track 0.00 -> 36.1 mm
- net /solenoid_channel8/solenoid_N: track 0.00 -> 36.1 mm
- net /solenoid_channel10/solenoid_N: track 0.00 -> 36.1 mm
- net GND: track 23.4 -> 58.4 mm, vias 11 -> 20
- net /solenoid_channel6/solenoid_P: track 0.00 -> 23.7 mm
- net /solenoid_channel3/solenoid_P: track 0.00 -> 23.7 mm
- net /solenoid_channel2/solenoid_P: track 0.00 -> 23.7 mm
- net /solenoid_channel7/solenoid_P: track 0.00 -> 23.7 mm
- net /solenoid_channel5/solenoid_P: track 0.00 -> 23.7 mm
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
Commit message: adjusted the hole position to account for blade offset.
Parts:
- moved H1 1.59 mm to (120.2, 77.6)
Routing:
- net /solenoid_channel1/solenoid_N: track 36.1 -> 35.1 mm
Changed lines of the file:
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@@
 		(allow_soldermask_bridges_in_footprints no)
 		(tenting front back)
-		(grid_origin 106.8 65)
+		(grid_origin 106.7 64.75)
 		(pcbplotparams
 			(layerselection 0x00000000_00000000_55555555_5755f5ff)
@@
 	(footprint "MountingHole:MountingHole_3.5mm"
 		(layer "F.Cu")
-		(at 119.713375 76.0845)
+		(at 120.182 77.609)
 		(descr "Mounting Hole 3.5mm, no annular")
 		(tags "mounting hole 3.5mm no annular")
@@
 	)
 	(segment
-		(start 118.787375 85.6355)
-		(end 118.787375 80.7255)
+		(start 121.113375 70.1595)
+		(end 124.273375 70.1595)
 		(width 0.2)
 		(layer "F.Cu")
@@
 	)
 	(segment
-		(start 118.787375 80.7255)
+		(start 124.958375 74.5545)
 		(end 125.213375 74.2995)
 		(width 0.2)
@@
 	)
 	(segment
-		(start 121.113375 70.1595)
-		(end 124.273375 70.1595)
+		(start 124.958375 79.141625)
+		(end 124.958375 77.2345)
 		(width 0.2)
 		(layer "F.Cu")
@@
 	)
 	(segment
-		(start 124.958375 74.5545)
-		(end 125.213375 74.2995)
+		(start 122.5 81.6)
+		(end 124.958375 79.141625)
 		(width 0.2)
 		(layer "F.Cu")
@@
 	)
 	(segment
-		(start 114.613375 89.2095)
-		(end 115.213375 89.2095)
+		(start 124.958375 77.2345)
+		(end 124.958375 74.5545)
 		(width 0.2)
 		(layer "F.Cu")
@@
 	)
 	(segment
-		(start 124.958375 77.2345)
-		(end 124.958375 74.5545)
+		(start 118.837375 84.9855)
+		(end 118.837375 82.12434)
 		(width 0.2)
 		(layer "F.Cu")
@@
 	)
 	(segment
-		(start 115.213375 89.2095)
-		(end 118.787375 85.6355)
+		(start 114.613375 89.2095)
+		(end 118.837375 84.9855)
 		(width 0.2)
 		(layer "F.Cu")
@@
 		(width 0.2)
 		(layer "F.Cu")
+		(net 5)
+	)
+	(segment
+		(start 114.613375 89.2095)
+		(end 115.213375 89.2095)
+		(width 0.2)
+		(layer "F.Cu")
+		(net 5)
+	)
+	(segment
+		(start 118.837375 82.12434)
+		(end 119.361715 81.6)
+		(width 0.2)
+		(layer "F.Cu")
+		(net 5)
+	)
+	(segment
+		(start 119.361715 81.6)
+		(end 122.5 81.6)
+		(width 0.2)
+		(layer "F.Cu")

Commit message: updated the switch pin numbering/footprints
Parts:
- moved H10 1.59 mm to (327.1, 77.6)
- moved H7 1.59 mm to (258.2, 77.6)
- moved H8 1.59 mm to (281.2, 77.6)
- moved H9 1.59 mm to (304.2, 77.6)
- moved H2 1.59 mm to (143.2, 77.6)
- moved H3 1.59 mm to (166.2, 77.6)
- moved H4 1.59 mm to (189.2, 77.6)
- moved H5 1.59 mm to (212.2, 77.6)
- moved H6 1.59 mm to (235.2, 77.6)
Routing:
- net /CH2_IN: track 28.7 -> 30.8 mm
- net /solenoid_channel9/solenoid_N: track 36.1 -> 35.1 mm
- net /solenoid_channel8/solenoid_N: track 36.1 -> 35.1 mm
- net /solenoid_channel3/solenoid_N: track 36.1 -> 35.1 mm
- net /solenoid_channel10/solenoid_N: track 36.1 -> 35.1 mm
- net /solenoid_channel2/solenoid_N: track 36.1 -> 35.1 mm
- net /solenoid_channel6/solenoid_N: track 36.1 -> 35.1 mm
- net /solenoid_channel5/solenoid_N: track 36.1 -> 35.1 mm
- net /solenoid_channel4/solenoid_N: track 36.1 -> 35.1 mm
- net /solenoid_channel7/solenoid_N: track 36.1 -> 35.1 mm

Commit message: ran the updated channel traces.
Routing:
- net /CH10_IN: track 221.2 -> 230.5 mm
- net /CH6_IN: track 119.2 -> 128.1 mm
- net /CH5_IN: track 97.0 -> 105.9 mm
- net /CH4_IN: track 72.0 -> 80.9 mm
- net /CH3_IN: track 49.9 -> 58.7 mm
- net /CH9_IN: track 195.5 -> 204.4 mm
- net /CH8_IN: track 169.6 -> 178.5 mm
- net /CH7_IN: track 144.1 -> 153.0 mm
- net /CH2_IN: track 30.8 -> 37.6 mm
Changed lines of the file:
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@@
+	)
+	(segment
+		(start 251.8 94)
+		(end 258.088376 87.711625)
+		(width 0.2)
+		(layer "F.Cu")
+		(net 27)
 	)
 	(segment
@@
 	)
 	(segment
+		(start 212.088375 87.711625)
+		(end 212.088376 87.711625)
+		(width 0.2)
+		(layer "F.Cu")
+		(net 28)
+	)
+	(segment
 		(start 212.088376 83.1595)
 		(end 211.738376 82.8095)
@@
 	)
 	(segment
+		(start 205.8 94)
+		(end 212.088375 87.711625)
+		(width 0.2)
+		(layer "F.Cu")
+		(net 28)
+	)
+	(segment
 		(start 204.8 95)
 		(end 205.8 94)
@@
 	)
 	(segment
+		(start 297.8 94)
+		(end 304.088375 87.711625)
+		(width 0.2)
+		(layer "F.Cu")
+		(net 29)
+	)
+	(segment
 		(start 229.8 97)
 		(end 230.8 96)
@@
 	)
 	(segment
+		(start 304.088375 87.711625)
+		(end 304.088376 87.711625)
+		(width 0.2)
+		(layer "F.Cu")
+		(net 29)
+	)
+	(segment
 		(start 182.8 97.5)
 		(end 183.3 97)
@@
 	)
 	(segment
+		(start 274.8 94)
+		(end 281.088375 87.711625)
+		(width 0.2)
+		(layer "F.Cu")
+		(net 30)
+	)
+	(segment
 		(start 281.088376 87.711625)
 		(end 281.088376 85.3095)
@@
 	)
 	(segment
+		(start 281.088375 87.711625)
+		(end 281.088376 87.711625)
+		(width 0.2)
+		(layer "F.Cu")
+		(net 30)
+	)
+	(segment
 		(start 143.0701 97)
 		(end 182.3671 97)
@@
 	)
 	(segment
+		(start 143.088375 87.711625)
+		(end 143.088376 87.711625)
+		(width 0.2)
+		(layer "F.Cu")
+		(net 31)
+	)
+	(segment
 		(start 143.088376 87.711625)
 		(end 143.088376 85.3095)
@@
 	)
 	(segment
+		(start 136.8 94)
+		(end 143.088375 87.711625)
+		(width 0.2)
+		(layer "F.Cu")
+		(net 31)
+	)
+	(segment
 		(start 143.088376 89.8095)
 		(end 149.588376 89.8095)
@@
 	)
 	(segment
-		(start 136.8 94)
-		(end 138.886076 94)
-		(width 0.2)
-		(layer "F.Cu")
-		(net 31)
-	)
-	(segment
 		(start 149.588376 85.3095)
 		(end 143.088376 85.3095)
@@
 	)
 	(segment
+		(start 235.088375 87.711625)
+		(end 235.088376 87.711625)
+		(width 0.2)
+		(layer "F.Cu")
+		(net 32)
+	)
+	(segment
 		(start 235.088376 83.1595)
 		(end 234.738376 82.8095)
@@
 	)
 	(segment
+		(start 228.8 94)
+		(end 235.088375 87.711625)
+		(width 0.2)
+		(layer "F.Cu")
+		(net 32)
+	)
+	(segment
 		(start 235.088376 89.8095)
 		(end 241.588376 89.8095)
@@
 	)
 	(segment
+		(start 182.8 94)
+		(end 189.088375 87.711625)
+		(width 0.2)
+		(layer "F.Cu")
+		(net 33)
+	)
+	(segment
 		(start 195.588376 85.3095)
 		(end 189.088376 85.3095)
@@
 	)
 	(segment
+		(start 189.088375 87.711625)
+		(end 189.088376 87.711625)
+		(width 0.2)
+		(layer "F.Cu")
+		(net 33)
+	)
+	(segment
 		(start 132.09 101.77)
 		(end 136.03 101.77)
@@
 	)
 	(segment
+		(start 326.963376 87.711625)
+		(end 326.963376 87.686624)
+		(width 0.2)
+		(layer "F.Cu")
+		(net 34)
+	)
+	(segment
 		(start 302.3 94)
 		(end 320.3 94)
@@
 	)
 	(segment
-		(start 326.963376 87.711625)
+		(start 326.963376 87.686624)
 		(end 326.963376 85.3095)
 		(width 0.2)
@@
 	)
 	(segment
+		(start 320.3 94)
+		(end 320.65 94)
+		(width 0.2)
+		(layer "F.Cu")
+		(net 34)
+	)
+	(segment
 		(start 126.045 105.195983)
 		(end 128.447017 107.598)
@@
 	)
 	(segment
+		(start 320.65 94)
+		(end 326.963376 87.686624)
+		(width 0.2)
+		(layer "F.Cu")
+		(net 34)
+	)
+	(segment
 		(start 298.8 97.5)
 		(end 302.3 94)
@@
 	)
 	(segment
+		(start 159.8 94)
+		(end 166.088375 87.711625)
+		(width 0.2)
+		(layer "F.Cu")
+		(net 36)
+	)
+	(segment
 		(start 166.088376 83.1595)
 		(end 165.738376 82.8095)
 		(width 0.2)
 		(layer "F.Cu")
+		(net 36)
+	)
+	(segment
+		(start 166.088375 87.711625)
+		(end 166.088376 87.711625)
+		(width 0.2)
+		(layer "F.Cu")

Commit message: Spaced out vias in channel setup.
Routing:
- net (no net): track 0.00 -> 65.0 mm
- net GND: track 58.4 -> 72.1 mm
- net /+24V: track 22.1 -> 31.7 mm
- net /CH1_IN: track 43.5 -> 37.0 mm
- net /CH6_IN: track 128.1 -> 121.6 mm
- net /CH5_IN: track 105.9 -> 99.4 mm
- net /CH4_IN: track 80.9 -> 74.4 mm
- net /CH9_IN: track 204.4 -> 197.9 mm
- net /CH3_IN: track 58.7 -> 52.3 mm
- net /CH2_IN: track 37.6 -> 31.1 mm
- net /CH8_IN: track 178.5 -> 172.1 mm
- net /CH7_IN: track 153.0 -> 146.5 mm
- net /CH10_IN: track 230.5 -> 224.0 mm

Commit message: Updated netclass setup and fixed silkscreen sizing issue.
Parts:
- LED1, LED2: footprint PCM_LED_SMD_AKL:LED_0603_1608Metric_Pad1.05x0.95mm -> PCM_LED_SMD_AKL:LED_0603_1608Metric
- LED10, LED11, LED12, LED3, LED4, LED5, LED6, LED7, LED8, LED9: footprint PCM_LED_SMD_AKL:LED_0201_0603Metric_Pad0.64x0.40mm -> PCM_LED_SMD_AKL:LED_0201_0603Metric
- S1, S10, S2, S3, S4, S5, S6, S7, S8, S9: footprint solenoid_fp:SW_TH_Tactile_Omron_B3F-10xx -> solenoid_fp:Switch_Tactile_THT_B3F-1xxx
- moved TP4 2.20 mm to (139.0, 94.0)
Connections:
- S1 pad 3: (no net) -> /VGATE
- S1 pad 4: (no net) -> /VGATE
- S10 pad 3: (no net) -> /VGATE
- S10 pad 4: (no net) -> /VGATE
- S2 pad 3: (no net) -> /VGATE
- S2 pad 4: (no net) -> /VGATE
- S3 pad 3: (no net) -> /VGATE
- S3 pad 4: (no net) -> /VGATE
- S4 pad 3: (no net) -> /VGATE
- S4 pad 4: (no net) -> /VGATE
- S5 pad 3: (no net) -> /VGATE
- S5 pad 4: (no net) -> /VGATE
- S6 pad 3: (no net) -> /VGATE
- S6 pad 4: (no net) -> /VGATE
- S7 pad 3: (no net) -> /VGATE
- S7 pad 4: (no net) -> /VGATE
- S8 pad 3: (no net) -> /VGATE
- S8 pad 4: (no net) -> /VGATE
- S9 pad 3: (no net) -> /VGATE
- S9 pad 4: (no net) -> /VGATE
Routing:
- net /VGATE: track 16.4 -> 81.4 mm
- net (no net): track 65.0 -> 0.00 mm
- net GND: track 72.1 -> 80.5 mm
- net /CH2_IN: track 31.1 -> 28.5 mm
- net /+24V: track 31.7 -> 34.2 mm
- net Net-(LED2-K): track 1.97 -> 3.62 mm
- net Net-(LED1-K): track 1.94 -> 3.55 mm

Commit message: updated minimum TH setting to 0.15
Routing:
- net GND: track 80.5 -> 81.2 mm
Changed lines of the file:
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@@
-	)
-	(segment
-		(start 191.3 109.4)
-		(end 191.3 106.5)
-		(width 0.5)
-		(layer "F.Cu")
-		(net 2)
 	)
 	(segment
@@
 	)
 	(segment
+		(start 191.3 109.4)
+		(end 191.3 105.9)
+		(width 0.5)
+		(layer "F.Cu")
+		(net 2)
+	)
+	(segment
 		(start 211.2 108.95)
 		(end 211.65 109.4)
@@
 	)
 	(segment
+		(start 191.3 105.9)
+		(end 191.35 105.85)
+		(width 0.5)
+		(layer "F.Cu")
+		(net 2)
+	)
+	(segment
 		(start 216.958376 82.3845)
 		(end 219.498376 82.3845)
@@
 	)
 	(via
-		(at 191.3 106.5)
-		(size 0.5)
-		(drill 0.3)
+		(at 191.35 105.85)
+		(size 0.5)
+		(drill 0.3)

Commit message: All clearances, vias and track now passing DRC checks.
Routing:
- net /+24V: track 34.2 -> 39.6 mm, vias 16 -> 17
- net /CH2_IN: track 28.5 -> 31.8 mm
- net /VGATE: track 81.4 -> 84.5 mm, vias 0 -> 2
- net GND: track 81.2 -> 78.8 mm, vias 20 -> 19
- added copper zone on B.Cu, net /VGATE
