File: solenoid_10/dc_dc_psu.kicad_sch (KiCad schematic)
At the start: 6 parts, among them U2 XL1509-5.0

Commit message: Added over-voltage and over-current protection to DCDC sheet.
Parts:
- added DZ1: BZT52-C5V6, PCM_Diode_SMD_AKL:D_SOD-123, symbol PCM_Diode_Zener_AKL:BZT52-C5V6
- added F1: SMD1812P075TF/33, symbol Device:Polyfuse
- added Q12: BT148W-600R, PCM_Package_TO_SOT_SMD_AKL:SOT-223-3_TabPin2, symbol PCM_Thyristor_AKL:BT148W-600R
- added R23: 1k, symbol PCM_Elektuur:R
Connections:
- net +5V: now also DZ1.1 (K), F1.2, Q12.2 (A); no longer C5.1, L1.2, U2.3 (FB)
- net GND: now also Q12.1 (K), R23.2 (-)
- new net: DZ1.2 (A), Q12.3 (G), R23.1 (+)
- new net Feedback: C5.1, F1.1, L1.2, U2.3 (FB)
Other:
- note added: "DC-DC buck converter 5.0V Output"
- note added: "Over-Voltage & Over-Current Crowbar"
- moved on the sheet: C3, C4, C5, D3, L1, U2

Commit message: Ran annotation on entire schematic
Parts:
- renumbered C4 to C1, C3 to C2, C5 to C3, D3 to D2, F1 to F2, Q12 to Q2, R23 to R5, U2 to U1
Changed lines of the file:
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@@
 		(dnp no)
 		(fields_autoplaced yes)
-		(property "Reference" "D3"
+		(property "Reference" "D2"
 			(at 129.54 54.2924 90)
 			(effects
@@
 			(project ""
 				(path "/434e6819-69f9-43cf-b2a3-58457aa05675/a48983fa-5ca6-467e-9e84-c08993af2c43"
-					(reference "D3")
+					(reference "D2")
 					(unit 1)
 				)
@@
 		(dnp no)
 		(fields_autoplaced yes)
-		(property "Reference" "F1"
+		(property "Reference" "F2"
 			(at 177.8 44.45 90)
 			(effects
@@
 			(project ""
 				(path "/434e6819-69f9-43cf-b2a3-58457aa05675/a48983fa-5ca6-467e-9e84-c08993af2c43"
-					(reference "F1")
+					(reference "F2")
 					(unit 1)
 				)
@@
 		(on_board yes)
 		(dnp no)
-		(property "Reference" "Q12"
+		(property "Reference" "Q2"
 			(at 224.79 60.9601 90)
 			(effects
@@
 			(project ""
 				(path "/434e6819-69f9-43cf-b2a3-58457aa05675/a48983fa-5ca6-467e-9e84-c08993af2c43"
-					(reference "Q12")
+					(reference "Q2")
 					(unit 1)
 				)
@@
 		(on_board yes)
 		(dnp no)
-		(property "Reference" "C5"
+		(property "Reference" "C3"
 			(at 156.21 53.7209 0)
 			(effects
@@
 			(project "solenoid_10"
 				(path "/434e6819-69f9-43cf-b2a3-58457aa05675/a48983fa-5ca6-467e-9e84-c08993af2c43"
-					(reference "C5")
+					(reference "C3")
 					(unit 1)
 				)
@@
 		(dnp no)
 		(fields_autoplaced yes)
-		(property "Reference" "R23"
+		(property "Reference" "R5"
 			(at 199.39 68.5799 0)
 			(effects
@@
 			(project ""
 				(path "/434e6819-69f9-43cf-b2a3-58457aa05675/a48983fa-5ca6-467e-9e84-c08993af2c43"
-					(reference "R23")
+					(reference "R5")
 					(unit 1)
 				)
@@
 		(on_board yes)
 		(dnp no)
-		(property "Reference" "C4"
+		(property "Reference" "C1"
 			(at 54.61 54.9909 0)
 			(effects
@@
 			(project ""
 				(path "/434e6819-69f9-43cf-b2a3-58457aa05675/a48983fa-5ca6-467e-9e84-c08993af2c43"
-					(reference "C4")
+					(reference "C1")
 					(unit 1)
 				)
@@
 		(dnp no)
 		(fields_autoplaced yes)
-		(property "Reference" "#PWR06"
+		(property "Reference" "#PWR05"
 			(at 95.25 86.36 0)
 			(effects
@@
 			(project ""
 				(path "/434e6819-69f9-43cf-b2a3-58457aa05675/a48983fa-5ca6-467e-9e84-c08993af2c43"
-					(reference "#PWR06")
+					(reference "#PWR05")
 					(unit 1)
 				)
@@
 		(dnp no)
 		(fields_autoplaced yes)
-		(property "Reference" "#FLG03"
+		(property "Reference" "#FLG02"
 			(at 250.19 46.355 0)
 			(effects
@@
 			(project ""
 				(path "/434e6819-69f9-43cf-b2a3-58457aa05675/a48983fa-5ca6-467e-9e84-c08993af2c43"
-					(reference "#FLG03")
+					(reference "#FLG02")
 					(unit 1)
 				)
@@
 		(dnp no)
 		(fields_autoplaced yes)
-		(property "Reference" "U2"
+		(property "Reference" "U1"
 			(at 95.25 45.72 0)
 			(effects
@@
 			(project "solenoid_10"
 				(path "/434e6819-69f9-43cf-b2a3-58457aa05675/a48983fa-5ca6-467e-9e84-c08993af2c43"
-					(reference "U2")
+					(reference "U1")
 					(unit 1)
 				)
@@
 		(dnp no)
 		(fields_autoplaced yes)
-		(property "Reference" "C3"
+		(property "Reference" "C2"
 			(at 67.31 55.8799 0)
 			(effects
@@
 			(project ""
 				(path "/434e6819-69f9-43cf-b2a3-58457aa05675/a48983fa-5ca6-467e-9e84-c08993af2c43"
-					(reference "C3")
-					(unit 1)
-				)
+					(reference "C2")
+					(unit 1)
+				)

Commit message: Added jlcpcb numbers and footprints for most components.
Parts:
- C1: footprint (none) -> PCM_Capacitor_SMD_US_Handsoldering_AKL:C_Elec_10x10.2; JLCPCB (none) -> C19606; now left out of the parts list
- C2: footprint (none) -> Capacitor_SMD:C_0805_2012Metric_Pad1.18x1.45mm_HandSolder; JLCPCB (none) -> C1738; now left out of the parts list
- C3: footprint (none) -> Capacitor_SMD:CP_Elec_6.3x5.8; JLCPCB (none) -> C2943990; now left out of the parts list
- D2: footprint PCM_Diode_SMD_AKL:D_SMC -> PCM_Diode_SMD_AKL:D_SOD-123; JLCPCB (none) -> C908230; now left out of the parts list
- DZ1: footprint PCM_Diode_SMD_AKL:D_SOD-123 -> Diode_SMD:D_SOD-323_HandSoldering; JLCPCB (none) -> C313486; now left out of the parts list
- F2: footprint (none) -> Fuse:Fuse_1812_4532Metric_Pad1.30x3.40mm_HandSolder; JLCPCB (none) -> C20997; now left out of the parts list
- L1: footprint (none) -> Inductor_SMD:L_Bourns_SRP7028A_7.3x6.6mm; JLCPCB (none) -> C2894721; now left out of the parts list
- Q2: JLCPCB (none) -> C256433; now left out of the parts list
- R5: footprint (none) -> Resistor_SMD:R_0805_2012Metric_Pad1.20x1.40mm_HandSolder; JLCPCB (none) -> C17513; now left out of the parts list
- U1: JLCPCB (none) -> C2902368; now left out of the parts list
Changed lines of the file:
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@@
 		(unit 1)
 		(exclude_from_sim no)
-		(in_bom yes)
+		(in_bom no)
 		(on_board yes)
 		(dnp no)
@@
 			)
 		)
-		(property "Footprint" "PCM_Diode_SMD_AKL:D_SMC"
+		(property "Footprint" "PCM_Diode_SMD_AKL:D_SOD-123"
 			(at 127 55.88 0)
 			(effects
@@
 			)
 		)
+		(property "JLCPCB" "C908230"
+			(at 127 55.88 0)
+			(effects
+				(font
+					(size 1.27 1.27)
+				)
+			)
+		)
 		(pin "2"
 		)
@@
 		(unit 1)
 		(exclude_from_sim no)
-		(in_bom yes)
+		(in_bom no)
 		(on_board yes)
 		(dnp no)
@@
 			)
 		)
-		(property "Footprint" ""
+		(property "Footprint" "Fuse:Fuse_1812_4532Metric_Pad1.30x3.40mm_HandSolder"
 			(at 182.88 49.53 0)
 			(effects
@@
 			)
 		)
+		(property "JLCPCB" "C20997"
+			(at 177.8 50.8 0)
+			(effects
+				(font
+					(size 1.27 1.27)
+				)
+			)
+		)
 		(pin "1"
 		)
@@
 		(unit 1)
 		(exclude_from_sim no)
-		(in_bom yes)
+		(in_bom no)
 		(on_board yes)
 		(dnp no)
@@
 			)
 		)
+		(property "JLCPCB" "C256433"
+			(at 222.25 59.69 0)
+			(effects
+				(font
+					(size 1.27 1.27)
+				)
+			)
+		)
 		(pin "1"
 		)
@@
 		(unit 1)
 		(exclude_from_sim no)
-		(in_bom yes)
+		(in_bom no)
 		(on_board yes)
 		(dnp no)
@@
 			)
 		)
-		(property "Footprint" ""
+		(property "Footprint" "Capacitor_SMD:CP_Elec_6.3x5.8"
 			(at 153.3652 59.69 0)
 			(effects
@@
 			)
 		)
+		(property "JLCPCB" "C2943990"
+			(at 152.4 55.88 0)
+			(effects
+				(font
+					(size 1.27 1.27)
+				)
+			)
+		)
 		(pin "1"
 		)
@@
 		(unit 1)
 		(exclude_from_sim no)
-		(in_bom yes)
+		(in_bom no)
 		(on_board yes)
 		(dnp no)
@@
 			)
 		)
-		(property "Footprint" ""
+		(property "Footprint" "Resistor_SMD:R_0805_2012Metric_Pad1.20x1.40mm_HandSolder"
 			(at 196.85 69.85 0)
 			(effects
@@
 			)
 		)
+		(property "JLCPCB" "C17513"
+			(at 196.85 69.85 0)
+			(effects
+				(font
+					(size 1.27 1.27)
+				)
+			)
+		)
 		(pin "2"
 		)
@@
 		(unit 1)
 		(exclude_from_sim no)
-		(in_bom yes)
+		(in_bom no)
 		(on_board yes)
 		(dnp no)
@@
 			)
 		)
-		(property "Footprint" ""
+		(property "Footprint" "PCM_Capacitor_SMD_US_Handsoldering_AKL:C_Elec_10x10.2"
 			(at 51.7652 60.96 0)
 			(effects
@@
 				)
 				(hide yes)
+			)
+		)
+		(property "JLCPCB" "C19606"
+			(at 50.8 57.15 0)
+			(effects
+				(font
+					(size 1.27 1.27)
+				)
 			)
 		)
@@
 		(unit 1)
 		(exclude_from_sim no)
-		(in_bom yes)
+		(in_bom no)
 		(on_board yes)
 		(dnp no)
@@
 			)
 		)
-		(property "Footprint" ""
+		(property "Footprint" "Inductor_SMD:L_Bourns_SRP7028A_7.3x6.6mm"
 			(at 133.35 50.8 0)
 			(effects
@@
 				)
 				(hide yes)
+			)
+		)
+		(property "JLCPCB" "C2894721"
+			(at 133.35 50.8 0)
+			(effects
+				(font
+					(size 1.27 1.27)
+				)
 			)
 		)
@@
 		(unit 1)
 		(exclude_from_sim no)
-		(in_bom yes)
+		(in_bom no)
 		(on_board yes)
 		(dnp no)
@@
 			)
 		)
+		(property "JLCPCB" "C2902368"
+			(at 95.25 55.88 0)
+			(effects
+				(font
+					(size 1.27 1.27)
+				)
+			)
+		)
 		(pin "5"
 		)
@@
 		(unit 1)
 		(exclude_from_sim no)
-		(in_bom yes)
+		(in_bom no)
 		(on_board yes)
 		(dnp no)
@@
 			)
 		)
-		(property "Footprint" ""
+		(property "Footprint" "Capacitor_SMD:C_0805_2012Metric_Pad1.18x1.45mm_HandSolder"
 			(at 64.4652 60.96 0)
 			(effects
@@
 			)
 		)
+		(property "JLCPCB" "C1738"
+			(at 63.5 57.15 0)
+			(effects
+				(font
+					(size 1.27 1.27)
+				)
+			)
+		)
 		(pin "1"
 		)
@@
 		(unit 1)
 		(exclude_from_sim no)
-		(in_bom yes)
+		(in_bom no)
 		(on_board yes)
 		(dnp no)
@@
 			)
 		)
-		(property "Footprint" "PCM_Diode_SMD_AKL:D_SOD-123"
+		(property "Footprint" "Diode_SMD:D_SOD-323_HandSoldering"
 			(at 196.85 55.88 0)
 			(effects
@@
 			)
 		)
+		(property "JLCPCB" "C313486"
+			(at 196.85 55.88 0)
+			(effects
+				(font
+					(size 1.27 1.27)
+				)
+			)
+		)

Commit message: Updated netclass setup and fixed silkscreen sizing issue.
Parts:
- C1, C2, C3, D2, DZ1, F2, L1, Q2, R5, U1: now in the parts list
Changed lines of the file:
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@@
 		(unit 1)
 		(exclude_from_sim no)
-		(in_bom no)
+		(in_bom yes)
 		(on_board yes)
 		(dnp no)
@@
 		(unit 1)
 		(exclude_from_sim no)
-		(in_bom no)
+		(in_bom yes)
 		(on_board yes)
 		(dnp no)
@@
 		(unit 1)
 		(exclude_from_sim no)
-		(in_bom no)
+		(in_bom yes)
 		(on_board yes)
 		(dnp no)
@@
 		(unit 1)
 		(exclude_from_sim no)
-		(in_bom no)
+		(in_bom yes)
 		(on_board yes)
 		(dnp no)
@@
 		(unit 1)
 		(exclude_from_sim no)
-		(in_bom no)
+		(in_bom yes)
 		(on_board yes)
 		(dnp no)
@@
 		(unit 1)
 		(exclude_from_sim no)
-		(in_bom no)
+		(in_bom yes)
 		(on_board yes)
 		(dnp no)
@@
 		(unit 1)
 		(exclude_from_sim no)
-		(in_bom no)
+		(in_bom yes)
 		(on_board yes)
 		(dnp no)
@@
 		(unit 1)
 		(exclude_from_sim no)
-		(in_bom no)
+		(in_bom yes)
 		(on_board yes)
 		(dnp no)
@@
 		(unit 1)
 		(exclude_from_sim no)
-		(in_bom no)
+		(in_bom yes)
 		(on_board yes)
 		(dnp no)
@@
 		(unit 1)
 		(exclude_from_sim no)
-		(in_bom no)
-		(on_board yes)
-		(dnp no)
+		(in_bom yes)
+		(on_board yes)
+		(dnp no)

Commit message: Solenoid_10, refactored input power and dc-dc converter
+ Removed crowbar circuit.
+ Added larger traces on input.
+ Added multiple copper fills for lower resistance.
+ Updated silkscreen textbox.
Parts:
- removed DZ1: BZT52-C5V6, Diode_SMD:D_SOD-323_HandSoldering, symbol PCM_Diode_Zener_AKL:BZT52-C5V6
- removed F2: SMD1812P075TF/33, Fuse:Fuse_1812_4532Metric_Pad1.30x3.40mm_HandSolder, symbol Device:Polyfuse
- removed Q2: BT148W-600R, PCM_Package_TO_SOT_SMD_AKL:SOT-223-3_TabPin2, symbol PCM_Thyristor_AKL:BT148W-600R
- removed R5: 1k, Resistor_SMD:R_0805_2012Metric_Pad1.20x1.40mm_HandSolder, symbol PCM_Elektuur:R
- added NT1: NetTie_2, NetTie:NetTie-2_SMD_Pad0.5mm, symbol Device:NetTie_2
Connections:
- net +5V: now also C3.1, L1.2, NT1.2
- net Feedback: now also NT1.1; no longer C3.1, L1.2
Other:
- note removed: "Over-Voltage & Over-Current Crowbar"
- company: (none) -> Homewood Creations
- title: (none) -> Solenoid_10

Commit message: Solenoid_10, updated cap and SOP-8 footprints and jlcpcb numbers.
+ Changed capacitor for one that has larger quantity in stock.
+ Updated footprints for MOSFET for default kicad style.
Parts:
- C1: footprint PCM_Capacitor_SMD_US_Handsoldering_AKL:C_Elec_10x10.2 -> Capacitor_SMD:CP_Elec_10x10; JLCPCB C19606 -> C3032175
Changed lines of the file:
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@@
 			)
 		)
-		(property "Footprint" "PCM_Capacitor_SMD_US_Handsoldering_AKL:C_Elec_10x10.2"
+		(property "Footprint" "Capacitor_SMD:CP_Elec_10x10"
 			(at 51.7652 60.96 0)
 			(effects
@@
 			)
 		)
-		(property "JLCPCB" "C19606"
+		(property "JLCPCB" "C3032175"
 			(at 50.8 57.15 0)
 			(effects

Commit message: Solenoid_10, checked stock of more parts update fp.
+ Checked stock of Caps, LEDs, diodes and inductors.
+ Updated Footprints for better compat accross systems.
Parts:
- D2: footprint PCM_Diode_SMD_AKL:D_SOD-123 -> Diode_SMD:D_SOD-123
Changed lines of the file:
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@@
 			)
 		)
-		(property "Footprint" "PCM_Diode_SMD_AKL:D_SOD-123"
+		(property "Footprint" "Diode_SMD:D_SOD-123"
 			(at 127 55.88 0)
 			(effects

Commit message: solenoid_10, refactored for manufacturing.
+ chagned cap to alternate that costs less for assembly.
+ marked more components as DNP
+ marked more components as no POS.
Parts:
- C1: JLCPCB C3032175 -> (none); LCSC (none) -> C2895745
- C2: JLCPCB C1738 -> (none); LCSC (none) -> C1738
- C3: JLCPCB C2943990 -> (none); LCSC (none) -> C2943990
- D2: JLCPCB C908230 -> (none); LCSC (none) -> C908230
- L1: JLCPCB C2894721 -> (none); LCSC (none) -> C2894721
- U1: JLCPCB C2902368 -> (none); LCSC (none) -> C2902368
Changed lines of the file:
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@@
 			)
 		)
-		(property "JLCPCB" "C908230"
-			(at 127 55.88 0)
-			(effects
-				(font
-					(size 1.27 1.27)
-				)
+		(property "LCSC" "C908230"
+			(at 127 55.88 90)
+			(effects
+				(font
+					(size 1.27 1.27)
+				)
+				(hide yes)
 			)
 		)
@@
 			)
 		)
-		(property "JLCPCB" "C2943990"
+		(property "LCSC" "C2943990"
 			(at 152.4 55.88 0)
 			(effects
@@
 					(size 1.27 1.27)
 				)
+				(hide yes)
 			)
 		)
@@
 			)
 		)
-		(property "JLCPCB" "C3032175"
+		(property "LCSC" "C2895745"
 			(at 50.8 57.15 0)
 			(effects
@@
 					(size 1.27 1.27)
 				)
+				(hide yes)
 			)
 		)
@@
 			)
 		)
-		(property "JLCPCB" "C2894721"
-			(at 133.35 50.8 0)
-			(effects
-				(font
-					(size 1.27 1.27)
-				)
+		(property "LCSC" "C2894721"
+			(at 133.35 50.8 90)
+			(effects
+				(font
+					(size 1.27 1.27)
+				)
+				(hide yes)
 			)
 		)
@@
 			)
 		)
-		(property "JLCPCB" "C2902368"
+		(property "LCSC" "C2902368"
 			(at 95.25 55.88 0)
 			(effects
@@
 					(size 1.27 1.27)
 				)
+				(hide yes)
 			)
 		)
@@
 			)
 		)
-		(property "JLCPCB" "C1738"
+		(property "LCSC" "C1738"
 			(at 63.5 57.15 0)
 			(effects
@@
 					(size 1.27 1.27)
 				)
-			)
-		)
+				(hide yes)
+			)
+		)
