File: solenoid_10/dc_dc_psu.kicad_sch (KiCad schematic)
At the start: 7 parts, among them U1 XL1509-5.0

Commit message: Fixed bug with enable pin on solenoid 10 board design.
Connections:
- net +24V_IN: no longer U1.4 (~{EN})
- no-connect marks 0 -> 1
