File: mega_shield/mega_connector.kicad_sch (KiCad schematic)
At the start: 1 part

Commit message: Added Y-axis uc labels and sheet pins
Connections:
- net Y_PED: now reaches A1.A14
- net Y_EN: now reaches A1.A2
- net Y_STEP: now reaches A1.A6
- net Y_DIR: now reaches A1.A7
- net Y_LIM_MIN: now reaches A1.D14 (D14/TX3)
- net Y_LIM_MAX: now reaches A1.D15 (D15/RX3)
- net Y_ERR: now reaches A1.D20 (D20/SDA)
Changed lines of the file:
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@@
+		)
+	)
+	(hierarchical_label "Y_DIR"
+		(shape output)
+		(at 106.68 92.71 180)
+		(effects
+			(font
+				(size 1.27 1.27)
+			)
+			(justify right)
+		)
+	)
+	(hierarchical_label "Y_LIM_MIN"
+		(shape input)
+		(at 106.68 59.69 180)
+		(effects
+			(font
+				(size 1.27 1.27)
+			)
+			(justify right)
 		)
 	)
@@
 			)
 			(justify left)
+		)
+	)
+	(hierarchical_label "Y_ERR"
+		(shape input)
+		(at 106.68 62.23 180)
+		(effects
+			(font
+				(size 1.27 1.27)
+			)
+			(justify right)
 		)
 	)
@@
 		(shape input)
 		(at 88.9 128.27 180)
+		(effects
+			(font
+				(size 1.27 1.27)
+			)
+			(justify right)
+		)
+	)
+	(hierarchical_label "Y_LIM_MAX"
+		(shape input)
+		(at 106.68 57.15 180)
 		(effects
 			(font
@@
 		)
 	)
+	(hierarchical_label "Y_EN"
+		(shape output)
+		(at 106.68 80.01 180)
+		(effects
+			(font
+				(size 1.27 1.27)
+			)
+			(justify right)
+		)
+	)
+	(hierarchical_label "Y_PED"
+		(shape input)
+		(at 106.68 110.49 180)
+		(effects
+			(font
+				(size 1.27 1.27)
+			)
+			(justify right)
+		)
+	)
 	(hierarchical_label "X_EN"
 		(shape output)
@@
 		)
 	)
+	(hierarchical_label "Y_STEP"
+		(shape output)
+		(at 106.68 90.17 180)
+		(effects
+			(font
+				(size 1.27 1.27)
+			)
+			(justify right)
+		)
+	)

Commit message: Added Z-axis uc labels and sheet pins.
Connections:
- net Z_EN: now reaches A1.A8
- net Z_PED: now reaches A1.D13
- net Z_LIM_MIN: now reaches A1.D18 (D18/TX1)
- net Z_ERR: now reaches A1.D19 (D19/RX1)
- net Z_LIM_MAX: now reaches A1.D32
- net Z_STEP: now reaches A1.D46
- net Z_DIR: now reaches A1.D48
Changed lines of the file:
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@@
+		)
+	)
+	(hierarchical_label "Z_PED"
+		(shape input)
+		(at 172.72 69.85 0)
+		(effects
+			(font
+				(size 1.27 1.27)
+			)
+			(justify left)
+		)
+	)
+	(hierarchical_label "Z_EN"
+		(shape output)
+		(at 106.68 95.25 180)
+		(effects
+			(font
+				(size 1.27 1.27)
+			)
+			(justify right)
 		)
 	)
@@
 		)
 	)
+	(hierarchical_label "Z_LIM_MAX"
+		(shape input)
+		(at 172.72 97.79 0)
+		(effects
+			(font
+				(size 1.27 1.27)
+			)
+			(justify left)
+		)
+	)
+	(hierarchical_label "Z_LIM_MIN"
+		(shape input)
+		(at 106.68 49.53 180)
+		(effects
+			(font
+				(size 1.27 1.27)
+			)
+			(justify right)
+		)
+	)
 	(hierarchical_label "Y_LIM_MIN"
 		(shape input)
@@
 		)
 	)
+	(hierarchical_label "Z_DIR"
+		(shape output)
+		(at 172.72 138.43 0)
+		(effects
+			(font
+				(size 1.27 1.27)
+			)
+			(justify left)
+		)
+	)
+	(hierarchical_label "Z_STEP"
+		(shape output)
+		(at 172.72 133.35 0)
+		(effects
+			(font
+				(size 1.27 1.27)
+			)
+			(justify left)
+		)
+	)
+	(hierarchical_label "Z_ERR"
+		(shape input)
+		(at 106.68 46.99 180)
+		(effects
+			(font
+				(size 1.27 1.27)
+			)
+			(justify right)
+		)
+	)

Commit message: Added A-axis uc labels and sheet pins.
Connections:
- net A_ERR: now reaches A1.D11
- net A_EN: now reaches A1.D24
- net A_STEP: now reaches A1.D26
- net A_DIR: now reaches A1.D28
- net A_LIM_MAX: now reaches A1.D40
- net A_LIM_MIN: now reaches A1.D42
- net A_PED: now reaches A1.D50 (D50_MISO)
Changed lines of the file:
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@@
+		)
+	)
+	(hierarchical_label "A_STEP"
+		(shape output)
+		(at 172.72 82.55 0)
+		(effects
+			(font
+				(size 1.27 1.27)
+			)
+			(justify left)
 		)
 	)
@@
 		)
 	)
+	(hierarchical_label "A_ERR"
+		(shape input)
+		(at 172.72 64.77 0)
+		(effects
+			(font
+				(size 1.27 1.27)
+			)
+			(justify left)
+		)
+	)
+	(hierarchical_label "A_LIM_MAX"
+		(shape input)
+		(at 172.72 118.11 0)
+		(effects
+			(font
+				(size 1.27 1.27)
+			)
+			(justify left)
+		)
+	)
 	(hierarchical_label "Y_DIR"
 		(shape output)
@@
 		)
 	)
+	(hierarchical_label "A_LIM_MIN"
+		(shape input)
+		(at 172.72 123.19 0)
+		(effects
+			(font
+				(size 1.27 1.27)
+			)
+			(justify left)
+		)
+	)
 	(hierarchical_label "Z_LIM_MIN"
 		(shape input)
@@
 		)
 	)
+	(hierarchical_label "A_PED"
+		(shape input)
+		(at 172.72 143.51 0)
+		(effects
+			(font
+				(size 1.27 1.27)
+			)
+			(justify left)
+		)
+	)
 	(hierarchical_label "X_ERR"
 		(shape input)
@@
 		)
 	)
+	(hierarchical_label "A_EN"
+		(shape output)
+		(at 172.72 77.47 0)
+		(effects
+			(font
+				(size 1.27 1.27)
+			)
+			(justify left)
+		)
+	)
+	(hierarchical_label "A_DIR"
+		(shape output)
+		(at 172.72 87.63 0)
+		(effects
+			(font
+				(size 1.27 1.27)
+			)
+			(justify left)
+		)
+	)

Commit message: Added B-axis uc labels and sheet pins.
Connections:
- net B_LIM_MAX: now reaches A1.A5
- net B_ERR: now reaches A1.D12
- net B_EN: now reaches A1.D30
- net B_DIR: now reaches A1.D34
- net B_STEP: now reaches A1.D36
- net B_LIM_MIN: now reaches A1.D44
- net B_PED: now reaches A1.D52 (D52_SCK)
Changed lines of the file:
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@@
+		)
+	)
+	(hierarchical_label "B_PED"
+		(shape input)
+		(at 172.72 148.59 0)
+		(effects
+			(font
+				(size 1.27 1.27)
+			)
+			(justify left)
+		)
+	)
+	(hierarchical_label "B_EN"
+		(shape output)
+		(at 172.72 92.71 0)
+		(effects
+			(font
+				(size 1.27 1.27)
+			)
+			(justify left)
 		)
 	)
@@
 		)
 	)
+	(hierarchical_label "B_LIM_MAX"
+		(shape input)
+		(at 106.68 87.63 180)
+		(effects
+			(font
+				(size 1.27 1.27)
+			)
+			(justify right)
+		)
+	)
 	(hierarchical_label "X_PED"
 		(shape input)
@@
 		)
 	)
+	(hierarchical_label "B_DIR"
+		(shape output)
+		(at 172.72 102.87 0)
+		(effects
+			(font
+				(size 1.27 1.27)
+			)
+			(justify left)
+		)
+	)
 	(hierarchical_label "A_PED"
 		(shape input)
@@
 		)
 	)
+	(hierarchical_label "B_ERR"
+		(shape input)
+		(at 172.72 67.31 0)
+		(effects
+			(font
+				(size 1.27 1.27)
+			)
+			(justify left)
+		)
+	)
 	(hierarchical_label "A_DIR"
 		(shape output)
@@
 		(effects
 			(font
+				(size 1.27 1.27)
+			)
+			(justify left)
+		)
+	)
+	(hierarchical_label "B_LIM_MIN"
+		(shape input)
+		(at 172.72 128.27 0)
+		(effects
+			(font
+				(size 1.27 1.27)
+			)
+			(justify left)
+		)
+	)
+	(hierarchical_label "B_STEP"
+		(shape output)
+		(at 172.72 107.95 0)
+		(effects
+			(font

Commit message: Added C-axis uc labels and sheet pins.
Connections:
- net C_LIM_MIN: now reaches A1.A3
- net C_LIM_MAX: now reaches A1.A4
- net C_STEP: now reaches A1.D49
- net C_DIR: now reaches A1.D51 (D51_MOSI)
- net C_EN: now reaches A1.D53 (D53_CS)
Changed lines of the file:
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@@
+		)
+	)
+	(hierarchical_label "C_LIM_MIN"
+		(shape input)
+		(at 106.68 82.55 180)
+		(effects
+			(font
+				(size 1.27 1.27)
+			)
+			(justify right)
 		)
 	)
@@
 		)
 	)
+	(hierarchical_label "C_DIR"
+		(shape output)
+		(at 172.72 146.05 0)
+		(effects
+			(font
+				(size 1.27 1.27)
+			)
+			(justify left)
+		)
+	)
 	(hierarchical_label "B_EN"
 		(shape output)
@@
 		)
 	)
+	(hierarchical_label "C_LIM_MAX"
+		(shape input)
+		(at 106.68 85.09 180)
+		(effects
+			(font
+				(size 1.27 1.27)
+			)
+			(justify right)
+		)
+	)
 	(hierarchical_label "Y_LIM_MIN"
 		(shape input)
@@
 		)
 	)
+	(hierarchical_label "C_STEP"
+		(shape output)
+		(at 172.72 140.97 0)
+		(effects
+			(font
+				(size 1.27 1.27)
+			)
+			(justify left)
+		)
+	)
 	(hierarchical_label "B_STEP"
 		(shape output)
@@
 		)
 	)
+	(hierarchical_label "C_EN"
+		(shape output)
+		(at 172.72 151.13 0)
+		(effects
+			(font
+				(size 1.27 1.27)
+			)
+			(justify left)
+		)
+	)

Commit message: Added remaining uc labels and sheet pins.
Connections:
- net FEED_HOLD: now reaches A1.A10
- net CYCLE_START: now reaches A1.A11
- net SAFETY_DOOR: now reaches A1.A12
- net PROBE: now reaches A1.A15
- net RESET: now reaches A1.A9
- net RX0: now reaches A1.D0 (D0/RX0)
- net TX0: now reaches A1.D1 (D1/TX0)
- net COOL_FLOOD: now reaches A1.D10
- net OUT_5: now reaches A1.D16 (D16/TX2)
- net OUT_6: now reaches A1.D17 (D17/RX2)
- net OUT_8: now reaches A1.D33
- net OUT_3: now reaches A1.D35
- net OUT_1: now reaches A1.D37
- net OUT_7: now reaches A1.D39
- net SPIN_EN: now reaches A1.D4
- net OUT_9: now reaches A1.D41
- net OUT_10: now reaches A1.D43
- net OUT_11: now reaches A1.D45
- net OUT_12: now reaches A1.D47
- net SPIN_DIR: now reaches A1.D5
- net OUT_2: now reaches A1.D6
- net OUT_4: now reaches A1.D7
- net SPIN_PWM: now reaches A1.D8
- net COOL_MIST: now reaches A1.D9
- no-connect marks 0 -> 8
