File: mega_shield/mega_connector.kicad_sch (KiCad schematic)
At the start: 1 part

Commit message: mega_shield, ran DRC and ERC. Currently passing all tests/checks.
Parts:
- added J27, J28, J29, J30, J31: Conn_01x08_Pin, Connector_PinSocket_2.54mm:PinSocket_1x08_P2.54mm_Vertical, symbol Connector:Conn_01x08_Socket
- added J32: Conn_01x06_Socket, Connector_PinSocket_2.54mm:PinSocket_1x06_P2.54mm_Vertical, symbol Connector:Conn_01x06_Socket
- added J33: Conn_01x10_Socket, Connector_PinSocket_2.54mm:PinSocket_1x10_P2.54mm_Vertical, symbol Connector:Conn_01x10_Socket
- added J34: Conn_02x18_Odd_Even, Connector_PinSocket_2.54mm:PinSocket_2x18_P2.54mm_Vertical, symbol Connector_Generic:Conn_02x18_Odd_Even
Connections:
- no-connect marks 14 -> 106

Commit message: mega_shield, changed out 2.54mm pin headers for mega.
Parts:
- removed J27, J28, J29, J30, J31: Conn_01x08_Pin, Connector_PinSocket_2.54mm:PinSocket_1x08_P2.54mm_Vertical, symbol Connector:Conn_01x08_Socket
- removed J32: Conn_01x06_Socket, Connector_PinSocket_2.54mm:PinSocket_1x06_P2.54mm_Vertical, symbol Connector:Conn_01x06_Socket
- removed J33: Conn_01x10_Socket, Connector_PinSocket_2.54mm:PinSocket_1x10_P2.54mm_Vertical, symbol Connector:Conn_01x10_Socket
- added J27, J28, J29, J30, J35: Conn_01x08_Pin, Connector_PinHeader_2.54mm:PinHeader_1x08_P2.54mm_Vertical, symbol Connector:Conn_01x08_Pin
- added J31: Conn_01x06_Pin, Connector_PinHeader_2.54mm:PinHeader_1x06_P2.54mm_Vertical, symbol Connector:Conn_01x06_Pin
- added J32: Conn_01x10_Pin, Connector_PinHeader_2.54mm:PinHeader_1x10_P2.54mm_Vertical, symbol Connector:Conn_01x10_Pin
- J34: jlcpcb C2897419 -> C2894979
