File: mega_shield/mega_connector.kicad_sch (KiCad schematic)
At the start: 9 parts, among them J27 Conn_01x08_Pin, J28 Conn_01x08_Pin, J29 Conn_01x08_Pin, J30 Conn_01x08_Pin, J31 Conn_01x06_Pin, J32 Conn_01x10_Pin, J34 Conn_02x18_Odd_Even, J35 Conn_01x08_Pin

Commit message: Re-Annotated megashield, added the new totem pole driver JLCPCB numbers and imported into PCB.
Parts:
- renumbered J35 to J1, J28 to J2, J30 to J3, J34 to J4, J27 to J5, J29 to J6, J31 to J7, J32 to J8
Changed lines of the file:
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@@
 		(dnp yes)
 		(fields_autoplaced yes)
-		(property "Reference" "J31"
+		(property "Reference" "J7"
 			(at 46.355 83.82 0)
 			(show_name no)
@@
 			(project "mega_shield"
 				(path "/554fcf27-dc63-4666-abbc-7481d15942c4/02fc7425-ece1-4292-86d4-346700d4242c"
-					(reference "J31")
+					(reference "J7")
 					(unit 1)
 				)
@@
 		(dnp yes)
 		(fields_autoplaced yes)
-		(property "Reference" "J32"
+		(property "Reference" "J8"
 			(at 46.355 109.22 0)
 			(show_name no)
@@
 			(project "mega_shield"
 				(path "/554fcf27-dc63-4666-abbc-7481d15942c4/02fc7425-ece1-4292-86d4-346700d4242c"
-					(reference "J32")
+					(reference "J8")
 					(unit 1)
 				)
@@
 		(dnp yes)
 		(fields_autoplaced yes)
-		(property "Reference" "J28"
+		(property "Reference" "J2"
 			(at 26.035 58.42 0)
 			(show_name no)
@@
 			(project "mega_shield"
 				(path "/554fcf27-dc63-4666-abbc-7481d15942c4/02fc7425-ece1-4292-86d4-346700d4242c"
-					(reference "J28")
+					(reference "J2")
 					(unit 1)
 				)
@@
 		(dnp yes)
 		(fields_autoplaced yes)
-		(property "Reference" "J27"
+		(property "Reference" "J5"
 			(at 46.355 33.02 0)
 			(show_name no)
@@
 			(project "mega_shield"
 				(path "/554fcf27-dc63-4666-abbc-7481d15942c4/02fc7425-ece1-4292-86d4-346700d4242c"
-					(reference "J27")
+					(reference "J5")
 					(unit 1)
 				)
@@
 		(dnp yes)
 		(fields_autoplaced yes)
-		(property "Reference" "J29"
+		(property "Reference" "J6"
 			(at 46.355 58.42 0)
 			(show_name no)
@@
 			(project "mega_shield"
 				(path "/554fcf27-dc63-4666-abbc-7481d15942c4/02fc7425-ece1-4292-86d4-346700d4242c"
-					(reference "J29")
+					(reference "J6")
 					(unit 1)
 				)
@@
 		(dnp yes)
 		(fields_autoplaced yes)
-		(property "Reference" "J34"
+		(property "Reference" "J4"
 			(at 31.75 133.35 0)
 			(show_name no)
@@
 			(project "mega_shield"
 				(path "/554fcf27-dc63-4666-abbc-7481d15942c4/02fc7425-ece1-4292-86d4-346700d4242c"
-					(reference "J34")
+					(reference "J4")
 					(unit 1)
 				)
@@
 		(dnp yes)
 		(fields_autoplaced yes)
-		(property "Reference" "J30"
+		(property "Reference" "J3"
 			(at 26.035 83.82 0)
 			(show_name no)
@@
 			(project "mega_shield"
 				(path "/554fcf27-dc63-4666-abbc-7481d15942c4/02fc7425-ece1-4292-86d4-346700d4242c"
-					(reference "J30")
+					(reference "J3")
 					(unit 1)
 				)
@@
 		(dnp yes)
 		(fields_autoplaced yes)
-		(property "Reference" "J35"
+		(property "Reference" "J1"
 			(at 26.035 33.02 0)
 			(show_name no)
@@
 			(project "mega_shield"
 				(path "/554fcf27-dc63-4666-abbc-7481d15942c4/02fc7425-ece1-4292-86d4-346700d4242c"
-					(reference "J35")
+					(reference "J1")
 					(unit 1)
 				)
