File: mega_shield/mega_shield.kicad_sch (KiCad schematic)
At the start: 0 parts

Commit message: updated CS817x22HS value.
Other:
- added sheet servo_interface_ (servo_interface_.kicad_sch)
- added sheet spin_interface (spin_interface.kicad_sch)

Commit message: removed +36V connection from the M12 signal connector in the servo interface sheet.
Other:
- sheet servo_interface_ renamed servo_interface_X
- added sheet servo_interface_X1 (servo_interface_.kicad_sch)
Changed lines of the file:
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@@
 		(company "Homewood Creations")
+	)
+	(wire
+		(pts
+			(xy 306.07 86.36) (xy 342.9 86.36)
+		)
+		(stroke
+			(width 0)
+			(type default)
+		)
+	)
+	(wire
+		(pts
+			(xy 306.07 96.52) (xy 342.9 96.52)
+		)
+		(stroke
+			(width 0)
+			(type default)
+		)
+	)
+	(wire
+		(pts
+			(xy 306.07 93.98) (xy 342.9 93.98)
+		)
+		(stroke
+			(width 0)
+			(type default)
+		)
+	)
+	(wire
+		(pts
+			(xy 306.07 81.28) (xy 342.9 81.28)
+		)
+		(stroke
+			(width 0)
+			(type default)
+		)
+	)
+	(wire
+		(pts
+			(xy 306.07 83.82) (xy 342.9 83.82)
+		)
+		(stroke
+			(width 0)
+			(type default)
+		)
+	)
+	(wire
+		(pts
+			(xy 306.07 91.44) (xy 342.9 91.44)
+		)
+		(stroke
+			(width 0)
+			(type default)
+		)
 	)
 	(sheet
@@
 	)
 	(sheet
-		(at 342.9 76.2)
-		(size 21.59 21.59)
+		(at 342.9 100.33)
+		(size 21.59 17.78)
 		(exclude_from_sim no)
 		(in_bom yes)
 		(on_board yes)
 		(dnp no)
-		(fields_autoplaced yes)
 		(stroke
 			(width 0.1524)
@@
 			(color 0 0 0 0.0000)
 		)
-		(property "Sheetname" "servo_interface_"
-			(at 342.9 75.4884 0)
+		(property "Sheetname" "servo_interface_X1"
+			(at 342.646 99.822 0)
 			(effects
 				(font
@@
 		)
 		(property "Sheetfile" "servo_interface_.kicad_sch"
-			(at 342.9 98.3746 0)
+			(at 364.998 109.728 0)
+			(effects
+				(font
+					(size 1.27 1.27)
+				)
+				(justify left top)
+			)
+		)
+		(pin "ALARM" output
+			(at 342.9 106.68 180)
+			(effects
+				(font
+					(size 1.27 1.27)
+				)
+				(justify left)
+			)
+		)
+		(pin "DIR" input
+			(at 342.9 101.6 180)
+			(effects
+				(font
+					(size 1.27 1.27)
+				)
+				(justify left)
+			)
+		)
+		(pin "EN" input
+			(at 342.9 104.14 180)
+			(effects
+				(font
+					(size 1.27 1.27)
+				)
+				(justify left)
+			)
+		)
+		(pin "HOME" output
+			(at 342.9 111.76 180)
+			(effects
+				(font
+					(size 1.27 1.27)
+				)
+				(justify left)
+			)
+		)
+		(pin "PED" output
+			(at 342.9 114.3 180)
+			(effects
+				(font
+					(size 1.27 1.27)
+				)
+				(justify left)
+			)
+		)
+		(pin "STEP" input
+			(at 342.9 116.84 180)
+			(effects
+				(font
+					(size 1.27 1.27)
+				)
+				(justify left)
+			)
+		)
+		(pin "+5V_IN" input
+			(at 364.49 104.14 0)
+			(effects
+				(font
+					(size 1.27 1.27)
+				)
+				(justify right)
+			)
+		)
+		(pin "+36V_IN" input
+			(at 364.49 101.6 0)
+			(effects
+				(font
+					(size 1.27 1.27)
+				)
+				(justify right)
+			)
+		)
+		(instances
+			(project "mega_shield"
+				(path "/554fcf27-dc63-4666-abbc-7481d15942c4"
+					(page "4")
+				)
+			)
+		)
+	)
+	(sheet
+		(at 342.9 80.01)
+		(size 21.59 17.78)
+		(exclude_from_sim no)
+		(in_bom yes)
+		(on_board yes)
+		(dnp no)
+		(stroke
+			(width 0.1524)
+			(type solid)
+		)
+		(fill
+			(color 0 0 0 0.0000)
+		)
+		(property "Sheetname" "servo_interface_X"
+			(at 342.646 79.502 0)
+			(effects
+				(font
+					(size 1.27 1.27)
+				)
+				(justify left bottom)
+			)
+		)
+		(property "Sheetfile" "servo_interface_.kicad_sch"
+			(at 364.998 89.408 0)
 			(effects
 				(font
@@
 		)
 		(pin "+5V_IN" input
+			(at 364.49 83.82 0)
+			(effects
+				(font
+					(size 1.27 1.27)
+				)
+				(justify right)
+			)
+		)
+		(pin "+36V_IN" input
 			(at 364.49 81.28 0)
 			(effects
 				(font
-					(size 1.27 1.27)
-				)
-				(justify right)
-			)
-		)
-		(pin "+36V_IN" input
-			(at 364.49 78.74 0)
-			(effects
-				(font

Commit message: Created/connected 5 servo interfaces for axis(s) X, Y, Z, A and B. C is left unpopulated for now.
Other:
- sheet servo_interface_X1 renamed servo_interface_Y
- added sheet servo_interface_A (servo_interface_.kicad_sch)
- added sheet servo_interface_B (servo_interface_.kicad_sch)
- added sheet servo_interface_Z (servo_interface_.kicad_sch)

Commit message: Added empty solenoid interface sheet.
Other:
- added sheet solenoid_interface (solenoid_interface.kicad_sch)
Changed lines of the file:
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@@
+	)
+	(sheet
+		(at 190.5 114.3)
+		(size 13.97 12.7)
+		(exclude_from_sim no)
+		(in_bom yes)
+		(on_board yes)
+		(dnp no)
+		(fields_autoplaced yes)
+		(stroke
+			(width 0.1524)
+			(type solid)
+		)
+		(fill
+			(color 0 0 0 0.0000)
+		)
+		(property "Sheetname" "solenoid_interface"
+			(at 190.5 113.5884 0)
+			(effects
+				(font
+					(size 1.27 1.27)
+				)
+				(justify left bottom)
+			)
+		)
+		(property "Sheetfile" "solenoid_interface.kicad_sch"
+			(at 190.5 127.5846 0)
+			(effects
+				(font
+					(size 1.27 1.27)
+				)
+				(justify left top)
+			)
+		)
+		(instances
+			(project "mega_shield"
+				(path "/554fcf27-dc63-4666-abbc-7481d15942c4"
+					(page "9")
+				)
+			)
+		)
 	)
 	(sheet

Commit message: Imported sheet pins for solenoid interface sheet.
Other:
- sheet solenoid_interface ports: added +24V_IN, +5V_IN, SLND_1; removed none
Changed lines of the file:
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@@
 	)
 	(sheet
-		(at 190.5 114.3)
-		(size 13.97 12.7)
+		(at 181.61 114.3)
+		(size 21.59 38.1)
 		(exclude_from_sim no)
 		(in_bom yes)
@@
 		)
 		(property "Sheetname" "solenoid_interface"
-			(at 190.5 113.5884 0)
+			(at 181.61 113.5884 0)
 			(effects
 				(font
@@
 		)
 		(property "Sheetfile" "solenoid_interface.kicad_sch"
-			(at 190.5 127.5846 0)
+			(at 181.61 152.9846 0)
 			(effects
 				(font
@@
 			)
 		)
+		(pin "+5V_IN" input
+			(at 181.61 118.11 180)
+			(effects
+				(font
+					(size 1.27 1.27)
+				)
+				(justify left)
+			)
+		)
+		(pin "+24V_IN" input
+			(at 181.61 115.57 180)
+			(effects
+				(font
+					(size 1.27 1.27)
+				)
+				(justify left)
+			)
+		)
+		(pin "SLND_1" input
+			(at 203.2 115.57 0)
+			(effects
+				(font
+					(size 1.27 1.27)
+				)
+				(justify right)
+			)
+		)

Commit message: Added sheet labels for channels 1-10 to the solenoid interface sheet. Imported pins.
Other:
- sheet solenoid_interface ports: added SLND_10, SLND_2, SLND_3, SLND_4, SLND_5, SLND_6, SLND_7, SLND_8, SLND_9; removed none
Changed lines of the file:
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@@
+	(wire
+		(pts
+			(xy 203.2 124.46) (xy 242.57 124.46)
+		)
+		(stroke
+			(width 0)
+			(type default)
+		)
+	)
 	(wire
 		(pts
@@
 	(wire
 		(pts
+			(xy 203.2 139.7) (xy 242.57 139.7)
+		)
+		(stroke
+			(width 0)
+			(type default)
+		)
+	)
+	(wire
+		(pts
+			(xy 203.2 116.84) (xy 242.57 116.84)
+		)
+		(stroke
+			(width 0)
+			(type default)
+		)
+	)
+	(wire
+		(pts
 			(xy 306.07 104.14) (xy 342.9 104.14)
 		)
@@
 	(wire
 		(pts
+			(xy 203.2 119.38) (xy 242.57 119.38)
+		)
+		(stroke
+			(width 0)
+			(type default)
+		)
+	)
+	(wire
+		(pts
 			(xy 306.07 124.46) (xy 342.9 124.46)
 		)
@@
 	(wire
 		(pts
+			(xy 203.2 127) (xy 242.57 127)
+		)
+		(stroke
+			(width 0)
+			(type default)
+		)
+	)
+	(wire
+		(pts
 			(xy 381 165.1) (xy 364.49 165.1)
 		)
@@
 	(wire
 		(pts
+			(xy 203.2 121.92) (xy 242.57 121.92)
+		)
+		(stroke
+			(width 0)
+			(type default)
+		)
+	)
+	(wire
+		(pts
 			(xy 306.07 172.72) (xy 342.9 172.72)
 		)
@@
 	(wire
 		(pts
+			(xy 203.2 134.62) (xy 242.57 134.62)
+		)
+		(stroke
+			(width 0)
+			(type default)
+		)
+	)
+	(wire
+		(pts
 			(xy 381 83.82) (xy 381 104.14)
 		)
@@
 	(wire
 		(pts
+			(xy 203.2 132.08) (xy 242.57 132.08)
+		)
+		(stroke
+			(width 0)
+			(type default)
+		)
+	)
+	(wire
+		(pts
 			(xy 364.49 83.82) (xy 381 83.82)
 		)
@@
 	(wire
 		(pts
+			(xy 203.2 137.16) (xy 242.57 137.16)
+		)
+		(stroke
+			(width 0)
+			(type default)
+		)
+	)
+	(wire
+		(pts
 			(xy 306.07 121.92) (xy 342.9 121.92)
+		)
+		(stroke
+			(width 0)
+			(type default)
+		)
+	)
+	(wire
+		(pts
+			(xy 203.2 129.54) (xy 242.57 129.54)
 		)
 		(stroke
@@
 	)
 	(sheet
-		(at 181.61 114.3)
-		(size 21.59 38.1)
+		(at 181.61 115.57)
+		(size 21.59 34.29)
 		(exclude_from_sim no)
 		(in_bom yes)
@@
 		)
 		(property "Sheetname" "solenoid_interface"
-			(at 181.61 113.5884 0)
+			(at 181.61 114.8584 0)
 			(effects
 				(font
@@
 		)
 		(property "Sheetfile" "solenoid_interface.kicad_sch"
-			(at 181.61 152.9846 0)
+			(at 181.61 150.4446 0)
 			(effects
 				(font
@@
 		)
 		(pin "+5V_IN" input
-			(at 181.61 118.11 180)
+			(at 181.61 119.38 180)
 			(effects
 				(font
@@
 		)
 		(pin "+24V_IN" input
-			(at 181.61 115.57 180)
+			(at 181.61 116.84 180)
 			(effects
 				(font
@@
 		)
 		(pin "SLND_1" input
-			(at 203.2 115.57 0)
-			(effects
-				(font
+			(at 203.2 116.84 0)
+			(effects
+				(font
+					(size 1.27 1.27)
+				)
+				(justify right)
+			)
+		)
+		(pin "SLND_2" input
+			(at 203.2 119.38 0)
+			(effects
+				(font
+					(size 1.27 1.27)
+				)
+				(justify right)
+			)
+		)
+		(pin "SLND_3" input
+			(at 203.2 121.92 0)
+			(effects
+				(font
+					(size 1.27 1.27)
+				)
+				(justify right)
+			)
+		)
+		(pin "SLND_4" input
+			(at 203.2 124.46 0)
+			(effects
+				(font
+					(size 1.27 1.27)
+				)
+				(justify right)
+			)
+		)
+		(pin "SLND_5" input
+			(at 203.2 127 0)
+			(effects
+				(font
+					(size 1.27 1.27)
+				)
+				(justify right)
+			)
+		)
+		(pin "SLND_6" input
+			(at 203.2 129.54 0)
+			(effects
+				(font
+					(size 1.27 1.27)
+				)
+				(justify right)
+			)
+		)
+		(pin "SLND_7" input
+			(at 203.2 132.08 0)
+			(effects
+				(font
+					(size 1.27 1.27)
+				)
+				(justify right)
+			)
+		)
+		(pin "SLND_8" input
+			(at 203.2 134.62 0)
+			(effects
+				(font
+					(size 1.27 1.27)
+				)
+				(justify right)
+			)
+		)
+		(pin "SLND_9" input
+			(at 203.2 137.16 0)
+			(effects
+				(font
+					(size 1.27 1.27)
+				)
+				(justify right)
+			)
+		)
+		(pin "SLND_10" input
+			(at 203.2 139.7 0)
+			(effects
+				(font

Commit message: Added blank sheets for the door and IO module interfaces.
Other:
- added sheet IO_module_interface (IO_module_interface.kicad_sch)
- added sheet door_interface (door_interface.kicad_sch)
Changed lines of the file:
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@@
+	)
+	(sheet
+		(at 177.8 190.5)
+		(size 13.97 12.7)
+		(exclude_from_sim no)
+		(in_bom yes)
+		(on_board yes)
+		(dnp no)
+		(fields_autoplaced yes)
+		(stroke
+			(width 0.1524)
+			(type solid)
+		)
+		(fill
+			(color 0 0 0 0.0000)
+		)
+		(property "Sheetname" "IO_module_interface"
+			(at 177.8 189.7884 0)
+			(effects
+				(font
+					(size 1.27 1.27)
+				)
+				(justify left bottom)
+			)
+		)
+		(property "Sheetfile" "IO_module_interface.kicad_sch"
+			(at 177.8 203.7846 0)
+			(effects
+				(font
+					(size 1.27 1.27)
+				)
+				(justify left top)
+			)
+		)
+		(instances
+			(project "mega_shield"
+				(path "/554fcf27-dc63-4666-abbc-7481d15942c4"
+					(page "11")
+				)
+			)
+		)
 	)
 	(sheet
@@
 				)
 			)
+		)
+	)
+	(sheet
+		(at 177.8 165.1)
+		(size 12.7 12.7)
+		(exclude_from_sim no)
+		(in_bom yes)
+		(on_board yes)
+		(dnp no)
+		(fields_autoplaced yes)
+		(stroke
+			(width 0.1524)
+			(type solid)
+		)
+		(fill
+			(color 0 0 0 0.0000)
+		)
+		(property "Sheetname" "door_interface"
+			(at 177.8 164.3884 0)
+			(effects
+				(font
+					(size 1.27 1.27)
+				)
+				(justify left bottom)
+			)
+		)
+		(property "Sheetfile" "door_interface.kicad_sch"
+			(at 177.8 178.3846 0)
+			(effects
+				(font
+					(size 1.27 1.27)
+				)
+				(justify left top)
+			)
+		)
+		(instances
+			(project "mega_shield"
+				(path "/554fcf27-dc63-4666-abbc-7481d15942c4"
+					(page "10")
+				)
+			)

Commit message: Added sheet pins for door interface. Added +5v, +9v, +24v and +24V_Safe labels to main sheet.
Other:
- sheet door_interface ports: added +5V_IN, DOOR_OUT; removed none
