File: mega_shield/door_interface.kicad_sch (KiCad schematic)
At the start: 0 parts

Commit message: Added polyfuse protection for door interface 5V power input.
Parts:
- added F12: SMD1812P050TF, symbol Device:Polyfuse
- added LED11: LED_0603_Red, PCM_LED_SMD_AKL:LED_0603_1608Metric, symbol PCM_LED_AKL:LED_0603_Red
- added R32: 2k, symbol Device:R
Connections:
- net +5V_DOOR: now also F12.2, R32.2
- net +5V_IN: now also F12.1, LED11.2 (A)
- new net: LED11.1 (K), R32.1
Other:
- note added: "Fuse Indicator, turns on led when tripped"
- note added: "Polyfuse: I_Hold: 0.5A I_Trip: 1.0A V_Max: 15V"

Commit message: Added discrete non-inverting schmitt trigger outline and door indicator led.
Parts:
- added LED12: LED_0603_Red, PCM_LED_SMD_AKL:LED_0603_1608Metric, symbol PCM_LED_AKL:LED_0603_Red
- added R33, R34: R, symbol Device:R
- added R35: 300, symbol Device:R
- added U1: LM358DR, digikey-footprints:SOIC-8_W3.9mm, symbol dk_Linear-Amplifiers-Instrumentation-OP-Amps-Buffer-Amps:LM358DR
Connections:
- net +5V_DOOR: now also R35.2, U1.8 (VCC)
- net DOOR_FILT: now also R33.1
- net DOOR_OUT: now also LED12.1 (K), R34.2, U1.1
- new net: LED12.2 (A), R35.1
- new net: R33.2, R34.1, U1.3
- new net GND: U1.2, U1.4 (GND)
- no-connect marks 0 -> 5
Other:
- note added: "Door Indicator"
- note added: "Non-Inverting Schmitt Trigger"

Commit message: Added digital isolator to door interface
Parts:
- added C1, C42: 1u, symbol Device:C
- added U22: CS817x22HS, Package_SO:SOIC-8_3.9x4.9mm_P1.27mm, symbol mega_shield:CS817x20HS
Connections:
- net +5V_DOOR: now also C1.1, U22.1 (VDD1)
- net +5V_IN: now also C42.2, U22.8 (VDD2)
- net DOOR_IN: now also U22.2 (INA)
- net DOOR_OUT: now also U22.7 (OUTA)
- net GND: now also C1.2, C42.1, U22.4 (GND1), U22.5 (GND2)
- no-connect marks 5 -> 6
Other:
- note added: "Digitally Isolated Door Input(built in schmitt trigger for debouncing)"
- moved on the sheet: LED12, R33, R34, R35, U1A, U1B

Commit message: removed discrete trigger circuit.
Parts:
- removed R33, R34: R, symbol Device:R
- removed U1: LM358DR, digikey-footprints:SOIC-8_W3.9mm, symbol dk_Linear-Amplifiers-Instrumentation-OP-Amps-Buffer-Amps:LM358DR
Connections:
- no-connect marks 6 -> 1
Other:
- note removed: "Non-Inverting Schmitt Trigger"
- moved on the sheet: LED12, R35
