File: mega_shield/door_interface.kicad_sch (KiCad schematic)
At the start: 8 parts, among them U22 CS817x22HS

Commit message: Finished door interface sheet, added mosfet for door indicatior to maintain door signal level.
Parts:
- added Q1: 2SK3018, PCM_Package_TO_SOT_SMD_AKL:SOT-323_SC-70, symbol PCM_Transistor_MOSFET_AKL:2SK3018
Connections:
- net DOOR_OUT: now also Q1.1 (G); no longer LED12.1 (K)
- net GND: now also Q1.2 (S)
- new net: LED12.1 (K), Q1.3 (D)
Other:
- moved on the sheet: LED12
Changed lines of the file:
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@@
 	)
 	(rectangle
-		(start 228.6 50.8)
-		(end 257.81 91.44)
+		(start 215.9 50.8)
+		(end 257.81 97.79)
 		(stroke
 			(width 0)
@@
 	(text "Door Indicator"
 		(exclude_from_sim no)
-		(at 235.712 49.784 0)
+		(at 223.012 49.784 0)
 		(effects
 			(font
@@
 	)
 	(junction
-		(at 237.49 85.09)
-		(diameter 0)
-		(color 0 0 0 0)
-	)
-	(junction
 		(at 39.37 62.23)
 		(diameter 0)
@@
 	(wire
 		(pts
-			(xy 237.49 76.2) (xy 237.49 85.09)
-		)
-		(stroke
-			(width 0)
-			(type default)
-		)
-	)
-	(wire
-		(pts
-			(xy 237.49 62.23) (xy 237.49 68.58)
+			(xy 237.49 62.23) (xy 237.49 63.5)
 		)
 		(stroke
@@
 	(wire
 		(pts
-			(xy 212.09 85.09) (xy 237.49 85.09)
-		)
-		(stroke
-			(width 0)
-			(type default)
-		)
-	)
-	(wire
-		(pts
 			(xy 130.81 80.01) (xy 137.16 80.01)
 		)
@@
 	(wire
 		(pts
+			(xy 175.26 80.01) (xy 189.23 80.01)
+		)
+		(stroke
+			(width 0)
+			(type default)
+		)
+	)
+	(wire
+		(pts
 			(xy 35.56 62.23) (xy 39.37 62.23)
 		)
@@
 	(wire
 		(pts
-			(xy 237.49 85.09) (xy 262.89 85.09)
-		)
-		(stroke
-			(width 0)
-			(type default)
-		)
-	)
-	(wire
-		(pts
 			(xy 127 93.98) (xy 127 102.87)
 		)
@@
 	(wire
 		(pts
+			(xy 237.49 71.12) (xy 237.49 72.39)
+		)
+		(stroke
+			(width 0)
+			(type default)
+		)
+	)
+	(wire
+		(pts
 			(xy 52.07 74.93) (xy 58.42 74.93)
 		)
@@
 		(pts
 			(xy 39.37 62.23) (xy 50.8 62.23)
-		)
-		(stroke
-			(width 0)
-			(type default)
-		)
-	)
-	(wire
-		(pts
-			(xy 175.26 80.01) (xy 182.88 80.01)
 		)
 		(stroke
@@
 	(hierarchical_label "DOOR_OUT"
 		(shape output)
-		(at 182.88 80.01 0)
+		(at 231.14 78.74 180)
 		(effects
 			(font
 				(size 1.27 1.27)
 			)
-			(justify left)
+			(justify right)
 		)
 	)
@@
 	(hierarchical_label "DOOR_OUT"
 		(shape output)
-		(at 262.89 85.09 0)
+		(at 189.23 80.01 0)
 		(effects
 			(font
@@
 	(symbol
 		(lib_id "PCM_LED_AKL:LED_0603_Red")
-		(at 237.49 72.39 270)
+		(at 237.49 67.31 270)
 		(unit 1)
 		(exclude_from_sim no)
@@
 		(fields_autoplaced yes)
 		(property "Reference" "LED12"
-			(at 242.57 71.1199 90)
+			(at 242.57 66.0399 90)
 			(effects
 				(font
@@
 		)
 		(property "Value" "LED_0603_Red"
-			(at 242.57 73.6599 90)
+			(at 242.57 68.5799 90)
 			(effects
 				(font
@@
 		)
 		(property "Footprint" "PCM_LED_SMD_AKL:LED_0603_1608Metric"
-			(at 237.49 72.39 0)
+			(at 237.49 67.31 0)
 			(effects
 				(font
@@
 		)
 		(property "Datasheet" "~"
-			(at 237.49 72.39 0)
+			(at 237.49 67.31 0)
 			(effects
 				(font
@@
 		)
 		(property "Description" "Red SMD LED, 0603, Alternate KiCad Library"
-			(at 237.49 72.39 0)
+			(at 237.49 67.31 0)
 			(effects
 				(font
@@
 		)
 		(property "Purpose" ""
-			(at 237.49 72.39 0)
+			(at 237.49 67.31 0)
 			(effects
 				(font
@@
 		)
 		(property "jlcpcb" "C94743"
-			(at 237.49 72.39 0)
+			(at 237.49 67.31 0)
 			(effects
 				(font
@@
 	)
 	(symbol
+		(lib_id "PCM_Transistor_MOSFET_AKL:2SK3018")
+		(at 234.95 77.47 0)
+		(unit 1)
+		(exclude_from_sim no)
+		(in_bom yes)
+		(on_board yes)
+		(dnp no)
+		(fields_autoplaced yes)
+		(property "Reference" "Q1"
+			(at 241.3 76.1999 0)
+			(effects
+				(font
+					(size 1.27 1.27)
+				)
+				(justify left)
+			)
+		)
+		(property "Value" "2SK3018"
+			(at 241.3 78.7399 0)
+			(effects
+				(font
+					(size 1.27 1.27)
+				)
+				(justify left)
+			)
+		)
+		(property "Footprint" "PCM_Package_TO_SOT_SMD_AKL:SOT-323_SC-70"
+			(at 240.03 74.93 0)
+			(effects
+				(font
+					(size 1.27 1.27)
+				)
+				(hide yes)
+			)
+		)
+		(property "Datasheet" "https://www.tme.eu/Document/b7f69991697dc3f1bab7ef8aaf2c7541/2SK3018.pdf"
+			(at 234.95 77.47 0)
+			(effects
+				(font
+					(size 1.27 1.27)
+				)
+				(hide yes)
+			)
+		)
+		(property "Description" "SOT-323 N-MOSFET enchancement mode transistor, 30V, 100mA, 200mW, Alternate KiCAD Library"
+			(at 234.95 77.47 0)
+			(effects
+				(font
+					(size 1.27 1.27)
+				)
+				(hide yes)
+			)
+		)
+		(pin "3"
+		)
+		(pin "1"
+		)
+		(pin "2"
+		)
+		(instances
+			(project ""
+				(path "/554fcf27-dc63-4666-abbc-7481d15942c4/8e8f1c99-9a41-47b9-930d-77476c883f62"
+					(reference "Q1")
+					(unit 1)
+				)
+			)
+		)
+	)
+	(symbol
 		(lib_id "power:GND")
 		(at 143.51 62.23 0)
@@
 					(unit 1)
 				)
+			)
+		)
+	)
+	(symbol
+		(lib_id "power:GND")
+		(at 237.49 82.55 0)
+		(unit 1)
+		(exclude_from_sim no)
+		(in_bom yes)
+		(on_board yes)
+		(dnp no)
+		(fields_autoplaced yes)
+		(property "Reference" "#PWR0149"
+			(at 237.49 88.9 0)
+			(effects
+				(font
+					(size 1.27 1.27)
+				)
+				(hide yes)
+			)
+		)
+		(property "Value" "GND"
+			(at 237.49 87.63 0)
+			(effects
+				(font
+					(size 1.27 1.27)
+				)
+			)
+		)
+		(property "Footprint" ""
+			(at 237.49 82.55 0)
+			(effects
+				(font
+					(size 1.27 1.27)
+				)
+				(hide yes)
+			)
+		)
+		(property "Datasheet" ""
+			(at 237.49 82.55 0)
+			(effects
+				(font
+					(size 1.27 1.27)
+				)
+				(hide yes)
+			)
+		)
+		(property "Description" "Power symbol creates a global label with name \"GND\" , ground"
+			(at 237.49 82.55 0)
+			(effects
+				(font
+					(size 1.27 1.27)
+				)
+				(hide yes)
+			)
+		)
+		(pin "1"
+		)
+		(instances
+			(project "mega_shield"
+				(path "/554fcf27-dc63-4666-abbc-7481d15942c4/8e8f1c99-9a41-47b9-930d-77476c883f62"
+					(reference "#PWR0149")
+					(unit 1)
+				)

Commit message: Added the M83P connector for the door interface.
Parts:
- added J11: T4040014031-000, CONN3_T4040014031-000_TEC, symbol M8P3:T4040014031-000
Connections:
- net DOOR_IN: now also J11.4
- net GND: now also J11.3
- no-connect marks 2 -> 3
Other:
- note added: "M8P3 Door connector"
- moved on the sheet: C1, C42, F12, LED11, LED12, Q1, R32, R35, U22
