File: mega_shield/homing_interface_.kicad_sch (KiCad schematic)
At the start: 0 parts

Commit message: Added M83P connector to homing interface.
Parts:
- added J2: T4040014031-000, CONN3_T4040014031-000_TEC, symbol M8P3:T4040014031-000
Changed lines of the file:
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@@
+		)
+	)
+	(symbol
+		(lib_id "M8P3:T4040014031-000")
+		(at 184.15 95.25 0)
+		(unit 1)
+		(exclude_from_sim no)
+		(in_bom yes)
+		(on_board yes)
+		(dnp no)
+		(fields_autoplaced yes)
+		(property "Reference" "J2"
+			(at 198.12 96.5199 0)
+			(effects
+				(font
+					(size 1.524 1.524)
+				)
+				(justify left)
+			)
+		)
+		(property "Value" "T4040014031-000"
+			(at 198.12 99.0599 0)
+			(effects
+				(font
+					(size 1.524 1.524)
+				)
+				(justify left)
+			)
+		)
+		(property "Footprint" "CONN3_T4040014031-000_TEC"
+			(at 184.15 95.25 0)
+			(effects
+				(font
+					(size 1.27 1.27)
+					(italic yes)
+				)
+				(hide yes)
+			)
+		)
+		(property "Datasheet" "T4040014031-000"
+			(at 184.15 95.25 0)
+			(effects
+				(font
+					(size 1.27 1.27)
+					(italic yes)
+				)
+				(hide yes)
+			)
+		)
+		(property "Description" ""
+			(at 184.15 95.25 0)
+			(effects
+				(font
+					(size 1.27 1.27)
+				)
+				(hide yes)
+			)
+		)
+		(pin "3"
+		)
+		(pin "1"
+		)
+		(pin "4"
+		)
+		(instances
+			(project ""
+				(path "/554fcf27-dc63-4666-abbc-7481d15942c4/400d9ece-7151-4ceb-add7-34c828d7284c"
+					(reference "J2")
+					(unit 1)
+				)
+			)
 		)
 	)

Commit message: setup both min and max proximity sensor connections and voltage jumpers for each.
Parts:
- added C7, C8: 22u, symbol Device:C
- added J3: T4040014031-000, CONN3_T4040014031-000_TEC, symbol M8P3:T4040014031-000
- added J4, J5: Conn_01x03_Pin, symbol Connector:Conn_01x03_Pin
Connections:
- net LIM_MAX: now also J3.3
- net LIM_MIN: now also J2.3
- net V_Prox1: now reaches J2.1
- net V_Prox1: now also C7.1, J4.2 (Pin_2)
- net at J2.4: now also C7.2
- new net: C8.2, J3.4
- new net +24V_IN: J4.1 (Pin_1), J5.1 (Pin_1)
- new net +5V_IN: J4.3 (Pin_3), J5.3 (Pin_3)
- new net V_Prox2: C8.1, J3.1, J5.2 (Pin_2)
Other:
- note added: "Proximity Sensor 1 Voltage Selection Jumper"
- note added: "Proximity Sensor 2 Voltage Selection Jumper"
- moved on the sheet: J2

Commit message: removed the 3pin voltage jumper setup from the proximity sensor interface.
Parts:
- removed J4, J5: Conn_01x03_Pin, symbol Connector:Conn_01x03_Pin
Other:
- note removed: "Proximity Sensor 1 Voltage Selection Jumper"
- note removed: "Proximity Sensor 2 Voltage Selection Jumper"

Commit message: Adde note on sensor selection and reliability measures, adde homing interfaces for all servos.
Parts:
- added C38, C40: 1u, symbol Device:C
- added Q39, Q40: 2SK3018, PCM_Package_TO_SOT_SMD_AKL:SOT-323_SC-70, symbol PCM_Transistor_MOSFET_AKL:2SK3018
- added R29, R30: 1k, symbol Device:R
- added U20: CS817x22HS, Package_SO:SOIC-8_3.9x4.9mm_P1.27mm, symbol mega_shield:CS817x20HS
- renumbered C7 to C, J2 to J
Connections:
- net V_Prox2 is gone; now on net +24V_IN: C8.1, J3.1
- net +5V_IN: now also C40.2, U20.8 (VDD2)
- net LIM_MAX: now also Q40.2 (S), R30.2; no longer J3.3
- net LIM_MIN: now also Q39.2 (S), R29.2; no longer J.3
- net V_Prox1 renamed +24V_IN
- net +24V_IN: now also C38.1, U20.1 (VDD1)
- new net: Q39.1 (G), U20.7 (OUTA)
- new net: Q40.1 (G), U20.6 (OUTB)
- new net +5V_Servo: R29.1, R30.1
- new net GND: C38.2, C40.1, Q39.3 (D), Q40.3 (D), U20.4 (GND1), U20.5 (GND2)
- new net LIM_MAX_IN: J3.3, U20.3 (INB)
- new net LIM_MIN_IN: J.3, U20.2 (INA)
Other:
- note added: "Could add fuse here."
- note added: "Digitally Isolated Proximity sensors"
- note added: "M8P3 Min/Max limit connectors"
- note added: "Proximity Sensor supply"
- note added: "Sensor Info"
- moved on the sheet: C, C8, J, J3

Commit message: removed the I/O interface sheet from project.
Parts:
- renumbered C to C14, J to J4
Changed lines of the file:
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@@
 		(dnp no)
 		(fields_autoplaced yes)
-		(property "Reference" "C"
+		(property "Reference" "C?"
 			(at 88.9 44.4499 0)
 			(effects
@@
 				(path "/554fcf27-dc63-4666-abbc-7481d15942c4/298c55ac-606f-4a25-bd04-443d4dadcb78"
 					(reference "C14")
+					(unit 1)
+				)
+				(path "/554fcf27-dc63-4666-abbc-7481d15942c4/400d9ece-7151-4ceb-add7-34c828d7284c"
+					(reference "C?")
 					(unit 1)
 				)
@@
 		(dnp no)
 		(fields_autoplaced yes)
-		(property "Reference" "J"
+		(property "Reference" "J?"
 			(at 53.34 48.2599 0)
 			(effects
@@
 					(unit 1)
 				)
+				(path "/554fcf27-dc63-4666-abbc-7481d15942c4/400d9ece-7151-4ceb-add7-34c828d7284c"
+					(reference "J?")
+					(unit 1)
+				)

Commit message: Marked all MAX limit switch connectors as DNP(do not populate).
Parts:
- J3: now not fitted; now left out of the parts list
Changed lines of the file:
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@@
 		(unit 1)
 		(exclude_from_sim no)
-		(in_bom yes)
+		(in_bom no)
 		(on_board yes)
-		(dnp no)
+		(dnp yes)
 		(fields_autoplaced yes)
 		(property "Reference" "J3"
@@
 			)
 		)
+		(property "Purpose" ""
+			(at 67.31 62.23 0)
+			(effects
+				(font
+					(size 1.27 1.27)
+				)
+			)
+		)

Commit message: Added test points to the homing interfaces.
Parts:
- added TP66, TP71, TP76, TP81, TP86: TestPoint, symbol Connector:TestPoint
Connections:
- net +5V_Servo is gone; now on net +5V_IN: R29.1, R30.1
- net +24V_IN: now also TP66.1
- net LIM_MAX: now also TP86.1
- net LIM_MAX_IN: now also TP76.1
- net LIM_MIN: now also TP81.1
- net LIM_MIN_IN: now also TP71.1
Other:
- note added: "Homing Interface Test Points"

Commit message: Ran the annotation operation on all schematics.
Parts:
- renumbered C14 to C38, C8 to C39, C38 to C40, C40 to C41, J4 to J8, J3 to J9, Q39 to Q33, Q40 to Q34, R29 to R32, R30 to R33, TP66 to TP74, TP71 to TP75, TP81 to TP77, TP86 to TP78, U20 to U24
