File: mega_shield/homing_interface_.kicad_sch (KiCad schematic)
At the start: 15 parts, among them J8 T4040014031-000, J9 T4040014031-000, U14 4N35, U24 4N35

Commit message: re-annotating for entire schematic completed.
Parts:
- renumbered C38 to C18, C39 to C19, R67 to R22, R77 to R23, R68 to R24, R78 to R25, U24 to U15

Commit message: replicated layout of homing interfaces. Placed the homing interface into PCB.
Connections:
- net +24V_IN: no longer J9.1
- net LIM_MAX_IN: no longer J9.3
- net at C19.2: no longer J9.4
Other:
- moved on the sheet: J9
Changed lines of the file:
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@@
 	(symbol
 		(lib_id "M8P3:T4040014031-000")
-		(at 67.31 62.23 0)
+		(at 48.26 83.82 0)
 		(mirror y)
 		(unit 1)
@@
 		(fields_autoplaced yes)
 		(property "Reference" "J9"
-			(at 53.34 63.4999 0)
+			(at 34.29 85.0899 0)
 			(effects
 				(font
@@
 		)
 		(property "Value" "T4040014031-000"
-			(at 53.34 66.0399 0)
+			(at 34.29 87.6299 0)
 			(effects
 				(font
@@
 		)
 		(property "Footprint" "footprints:CONN3_T4040014031-000_TEC"
-			(at 67.31 62.23 0)
+			(at 48.26 83.82 0)
 			(effects
 				(font
@@
 		)
 		(property "Datasheet" "T4040014031-000"
-			(at 67.31 62.23 0)
+			(at 48.26 83.82 0)
 			(effects
 				(font
@@
 		)
 		(property "Description" ""
-			(at 67.31 62.23 0)
+			(at 48.26 83.82 0)
 			(effects
 				(font
@@
 		)
 		(property "Purpose" ""
-			(at 67.31 62.23 0)
+			(at 48.26 83.82 0)
 			(effects
 				(font
@@
 		)
 		(property "jlcpcb" "C19108956"
-			(at 67.31 62.23 0)
+			(at 48.26 83.82 0)
 			(effects
 				(font

Commit message: fixed issue with shcematic connector having moved in homing interface sheet.
Connections:
- net +24V_IN: now also J9.1
- net LIM_MAX_IN: now also J9.3
- net at C19.2: now also J9.4
Other:
- moved on the sheet: J9
Changed lines of the file:
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@@
 	(symbol
 		(lib_id "M8P3:T4040014031-000")
-		(at 48.26 83.82 0)
+		(at 67.31 62.23 0)
 		(mirror y)
 		(unit 1)
@@
 		(fields_autoplaced yes)
 		(property "Reference" "J9"
-			(at 34.29 85.0899 0)
+			(at 53.34 63.4999 0)
 			(effects
 				(font
@@
 		)
 		(property "Value" "T4040014031-000"
-			(at 34.29 87.6299 0)
+			(at 53.34 66.0399 0)
 			(effects
 				(font
@@
 		)
 		(property "Footprint" "footprints:CONN3_T4040014031-000_TEC"
-			(at 48.26 83.82 0)
+			(at 67.31 62.23 0)
 			(effects
 				(font
@@
 		)
 		(property "Datasheet" "T4040014031-000"
-			(at 48.26 83.82 0)
+			(at 67.31 62.23 0)
 			(effects
 				(font
@@
 		)
 		(property "Description" ""
-			(at 48.26 83.82 0)
+			(at 67.31 62.23 0)
 			(effects
 				(font
@@
 		)
 		(property "Purpose" ""
-			(at 48.26 83.82 0)
+			(at 67.31 62.23 0)
 			(effects
 				(font
@@
 		)
 		(property "jlcpcb" "C19108956"
-			(at 48.26 83.82 0)
+			(at 67.31 62.23 0)
 			(effects
 				(font

Commit message: mega_shield, Changed out all caps where needed for in-stock and lower cost parts.
+ Changed out for parts with higher stock.
+ Changed out for 0805 sized components.
+ Changed out for higher voltage.
+ Removed 22uF SMD caps for lower cost 10uF caps in parallel.
+ Updated diode footprint to SOD-123F

BOM cost reduced, and reliability improved.
Parts:
- added C20, C21: 10u/50V, Capacitor_SMD:C_0805_2012Metric_Pad1.18x1.45mm_HandSolder, symbol Device:C
- C18, C19: value 22u -> 10u/50V; footprint Capacitor_SMD:C_0805_2012Metric -> Capacitor_SMD:C_0805_2012Metric_Pad1.18x1.45mm_HandSolder; jlcpcb C6119901 -> C440198
Connections:
- net +24V_IN: now also C20.1, C21.1
- net at C19.2, J9.4: now also C21.2
- net at C18.2, J8.4: now also C20.2

Commit message: mega_shield, updated multiple resistors and added comments.
+ Updated optoisolator resistor value --> 15k for better protection.
+ Changed all resistors to 0805 footprints
+ Swapped out expensive values to standardized E24/E96.
+ Updated jlcpcb numbers for all resistors.
Parts:
- R22, R23: value 2k5 -> 15k; footprint Resistor_SMD:R_0201_0603Metric -> Resistor_SMD:R_0805_2012Metric_Pad1.20x1.40mm_HandSolder; jlcpcb C25804 -> C17475
- R24, R25: footprint Resistor_SMD:R_0201_0603Metric -> Resistor_SMD:R_0805_2012Metric_Pad1.20x1.40mm_HandSolder; jlcpcb C1226 -> C17557
Changed lines of the file:
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@@
+		)
+	)
+	(text_box "Assuming the input voltage is 24V~30V we need to current limit the I_f value for\nthe optoisolator to approximatly 2mA."
+		(exclude_from_sim no)
+		(at 139.7 109.22 0)
+		(size 72.39 10.16)
+		(margins 0.9525 0.9525 0.9525 0.9525)
+		(stroke
+			(width 0)
+			(type solid)
+		)
+		(fill
+			(type none)
+		)
+		(effects
+			(font
+				(size 1.27 1.27)
+			)
+			(justify left top)
 		)
 	)
@@
 			)
 		)
-		(property "Value" "2k5"
+		(property "Value" "15k"
 			(at 162.56 50.8 90)
 			(effects
@@
 			)
 		)
-		(property "Footprint" "Resistor_SMD:R_0201_0603Metric"
+		(property "Footprint" "Resistor_SMD:R_0805_2012Metric_Pad1.20x1.40mm_HandSolder"
 			(at 162.56 52.832 90)
 			(effects
@@
 			)
 		)
-		(property "jlcpcb" "C25804"
+		(property "jlcpcb" "C17475"
 			(at 162.56 54.61 0)
 			(effects
@@
 			)
 		)
-		(property "Footprint" "Resistor_SMD:R_0201_0603Metric"
+		(property "Footprint" "Resistor_SMD:R_0805_2012Metric_Pad1.20x1.40mm_HandSolder"
 			(at 186.182 88.9 90)
 			(effects
@@
 			)
 		)
-		(property "jlcpcb" "C1226"
+		(property "jlcpcb" "C17557"
 			(at 187.96 88.9 0)
 			(effects
@@
 			)
 		)
-		(property "Value" "2k5"
+		(property "Value" "15k"
 			(at 162.56 87.63 90)
 			(effects
@@
 			)
 		)
-		(property "Footprint" "Resistor_SMD:R_0201_0603Metric"
+		(property "Footprint" "Resistor_SMD:R_0805_2012Metric_Pad1.20x1.40mm_HandSolder"
 			(at 162.56 89.662 90)
 			(effects
@@
 			)
 		)
-		(property "jlcpcb" "C25804"
+		(property "jlcpcb" "C17475"
 			(at 162.56 91.44 0)
 			(effects
@@
 			)
 		)
-		(property "Footprint" "Resistor_SMD:R_0201_0603Metric"
+		(property "Footprint" "Resistor_SMD:R_0805_2012Metric_Pad1.20x1.40mm_HandSolder"
 			(at 186.182 52.07 90)
 			(effects
@@
 			)
 		)
-		(property "jlcpcb" "C1226"
+		(property "jlcpcb" "C17557"
 			(at 187.96 52.07 0)
 			(effects

Commit message: mega_shield, Set all test points to use the keystone 5000-5004 footprints.
Parts:
- TP74, TP75, TP76, TP77, TP78: footprint TestPoint:TestPoint_Pad_1.0x1.0mm -> TestPoint:TestPoint_Keystone_5000-5004_Miniature
Changed lines of the file:
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@@
 			)
 		)
-		(property "Footprint" "TestPoint:TestPoint_Pad_1.0x1.0mm"
+		(property "Footprint" "TestPoint:TestPoint_Keystone_5000-5004_Miniature"
 			(at 36.83 109.22 0)
 			(effects
@@
 			)
 		)
-		(property "Footprint" "TestPoint:TestPoint_Pad_1.0x1.0mm"
+		(property "Footprint" "TestPoint:TestPoint_Keystone_5000-5004_Miniature"
 			(at 36.83 116.84 0)
 			(effects
@@
 			)
 		)
-		(property "Footprint" "TestPoint:TestPoint_Pad_1.0x1.0mm"
+		(property "Footprint" "TestPoint:TestPoint_Keystone_5000-5004_Miniature"
 			(at 63.5 124.46 0)
 			(effects
@@
 			)
 		)
-		(property "Footprint" "TestPoint:TestPoint_Pad_1.0x1.0mm"
+		(property "Footprint" "TestPoint:TestPoint_Keystone_5000-5004_Miniature"
 			(at 36.83 124.46 0)
 			(effects
@@
 			)
 		)
-		(property "Footprint" "TestPoint:TestPoint_Pad_1.0x1.0mm"
+		(property "Footprint" "TestPoint:TestPoint_Keystone_5000-5004_Miniature"
 			(at 63.5 116.84 0)
 			(effects

Commit message: mega_shield, updated all 116 test points, changed values based on color code, added jlcpcb numbers and set footprints.
Parts:
- TP74, TP75, TP76: value TestPoint -> RH-5002; jlcpcb (none) -> C5199802; now in the parts list
- TP77, TP78: value TestPoint -> RH-5000; jlcpcb (none) -> C5277086; now in the parts list
Changed lines of the file:
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@@
 		(unit 1)
 		(exclude_from_sim no)
-		(in_bom no)
+		(in_bom yes)
 		(on_board yes)
 		(dnp no)
@@
 			)
 		)
-		(property "Value" "TestPoint"
+		(property "Value" "RH-5002"
 			(at 33.528 111.76 90)
 			(effects
@@
 		(property "Description" "test point"
 			(at 36.83 114.3 0)
+			(effects
+				(font
+					(size 1.27 1.27)
+				)
+				(hide yes)
+			)
+		)
+		(property "jlcpcb" "C5199802"
+			(at 36.83 114.3 90)
 			(effects
 				(font
@@
 		(unit 1)
 		(exclude_from_sim no)
-		(in_bom no)
+		(in_bom yes)
 		(on_board yes)
 		(dnp no)
@@
 			)
 		)
-		(property "Value" "TestPoint"
+		(property "Value" "RH-5002"
 			(at 33.528 119.38 90)
 			(effects
@@
 		(property "Description" "test point"
 			(at 36.83 121.92 0)
+			(effects
+				(font
+					(size 1.27 1.27)
+				)
+				(hide yes)
+			)
+		)
+		(property "jlcpcb" "C5199802"
+			(at 36.83 121.92 90)
 			(effects
 				(font
@@
 		(unit 1)
 		(exclude_from_sim no)
-		(in_bom no)
+		(in_bom yes)
 		(on_board yes)
 		(dnp no)
@@
 			)
 		)
-		(property "Value" "TestPoint"
+		(property "Value" "RH-5000"
 			(at 60.198 127 90)
 			(effects
@@
 		(property "Description" "test point"
 			(at 63.5 129.54 0)
+			(effects
+				(font
+					(size 1.27 1.27)
+				)
+				(hide yes)
+			)
+		)
+		(property "jlcpcb" "C5277086"
+			(at 63.5 129.54 90)
 			(effects
 				(font
@@
 		(unit 1)
 		(exclude_from_sim no)
-		(in_bom no)
+		(in_bom yes)
 		(on_board yes)
 		(dnp no)
@@
 			)
 		)
-		(property "Value" "TestPoint"
+		(property "Value" "RH-5002"
 			(at 33.528 127 90)
 			(effects
@@
 		(property "Description" "test point"
 			(at 36.83 129.54 0)
+			(effects
+				(font
+					(size 1.27 1.27)
+				)
+				(hide yes)
+			)
+		)
+		(property "jlcpcb" "C5199802"
+			(at 36.83 129.54 90)
 			(effects
 				(font
@@
 		(unit 1)
 		(exclude_from_sim no)
-		(in_bom no)
+		(in_bom yes)
 		(on_board yes)
 		(dnp no)
@@
 			)
 		)
-		(property "Value" "TestPoint"
+		(property "Value" "RH-5000"
 			(at 60.198 119.38 90)
 			(effects
@@
 			(effects
 				(font
+					(size 1.27 1.27)
+				)
+				(hide yes)
+			)
+		)
+		(property "jlcpcb" "C5277086"
+			(at 63.5 121.92 90)
+			(effects
+				(font

Commit message: mega_shield, Added all test point symbols and updated association of 3D models.
Parts:
- renumbered TP74 to TP80, TP75 to TP81, TP76 to TP82, TP77 to TP83, TP78 to TP84
