File: mega_shield/homing_interface_.kicad_sch (KiCad schematic)
At the start: 17 parts, among them J8 54-00277, J9 54-00277, U14 4N35, U15 4N35

Commit message: mega_shield, marked circular components as DNP, added jlcpcb numbers to 90degree terminal blocks.
Parts:
- J8, J9: now not fitted
Changed lines of the file:
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@@
 		(in_bom yes)
 		(on_board yes)
-		(dnp no)
+		(dnp yes)
 		(fields_autoplaced yes)
 		(property "Reference" "J8"
@@
 		(in_bom yes)
 		(on_board yes)
-		(dnp no)
+		(dnp yes)
 		(fields_autoplaced yes)
 		(property "Reference" "J9"

Commit message: mega_shield, re-annotated all components.
Parts:
- renumbered R22 to R44, R23 to R45, R24 to R46, R25 to R47
Changed lines of the file:
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@@
 		(dnp no)
 		(fields_autoplaced yes)
-		(property "Reference" "R22"
+		(property "Reference" "R44"
 			(at 162.56 48.26 90)
 			(effects
@@
 			(project "mega_shield"
 				(path "/554fcf27-dc63-4666-abbc-7481d15942c4/298c55ac-606f-4a25-bd04-443d4dadcb78"
-					(reference "R26")
+					(reference "R48")
 					(unit 1)
 				)
 				(path "/554fcf27-dc63-4666-abbc-7481d15942c4/400d9ece-7151-4ceb-add7-34c828d7284c"
-					(reference "R22")
+					(reference "R44")
 					(unit 1)
 				)
 				(path "/554fcf27-dc63-4666-abbc-7481d15942c4/64d796ae-634b-498c-8b87-bb3c7a5fb7ee"
-					(reference "R37")
+					(reference "R59")
 					(unit 1)
 				)
 				(path "/554fcf27-dc63-4666-abbc-7481d15942c4/a1009379-c1df-4080-8264-1d6ad70ed4b7"
-					(reference "R45")
+					(reference "R67")
 					(unit 1)
 				)
 				(path "/554fcf27-dc63-4666-abbc-7481d15942c4/cbf77838-d146-4db1-a0da-db3eb68b8af8"
-					(reference "R30")
+					(reference "R52")
 					(unit 1)
 				)
@@
 		(dnp no)
 		(fields_autoplaced yes)
-		(property "Reference" "R25"
+		(property "Reference" "R47"
 			(at 190.5 87.6299 0)
 			(effects
@@
 			(project "mega_shield"
 				(path "/554fcf27-dc63-4666-abbc-7481d15942c4/298c55ac-606f-4a25-bd04-443d4dadcb78"
-					(reference "R29")
+					(reference "R51")
 					(unit 1)
 				)
 				(path "/554fcf27-dc63-4666-abbc-7481d15942c4/400d9ece-7151-4ceb-add7-34c828d7284c"
-					(reference "R25")
+					(reference "R47")
 					(unit 1)
 				)
 				(path "/554fcf27-dc63-4666-abbc-7481d15942c4/64d796ae-634b-498c-8b87-bb3c7a5fb7ee"
-					(reference "R40")
+					(reference "R62")
 					(unit 1)
 				)
 				(path "/554fcf27-dc63-4666-abbc-7481d15942c4/a1009379-c1df-4080-8264-1d6ad70ed4b7"
-					(reference "R48")
+					(reference "R70")
 					(unit 1)
 				)
 				(path "/554fcf27-dc63-4666-abbc-7481d15942c4/cbf77838-d146-4db1-a0da-db3eb68b8af8"
-					(reference "R33")
+					(reference "R55")
 					(unit 1)
 				)
@@
 		(dnp no)
 		(fields_autoplaced yes)
-		(property "Reference" "R23"
+		(property "Reference" "R45"
 			(at 162.56 85.09 90)
 			(effects
@@
 			(project "mega_shield"
 				(path "/554fcf27-dc63-4666-abbc-7481d15942c4/298c55ac-606f-4a25-bd04-443d4dadcb78"
-					(reference "R27")
+					(reference "R49")
 					(unit 1)
 				)
 				(path "/554fcf27-dc63-4666-abbc-7481d15942c4/400d9ece-7151-4ceb-add7-34c828d7284c"
-					(reference "R23")
+					(reference "R45")
 					(unit 1)
 				)
 				(path "/554fcf27-dc63-4666-abbc-7481d15942c4/64d796ae-634b-498c-8b87-bb3c7a5fb7ee"
-					(reference "R38")
+					(reference "R60")
 					(unit 1)
 				)
 				(path "/554fcf27-dc63-4666-abbc-7481d15942c4/a1009379-c1df-4080-8264-1d6ad70ed4b7"
-					(reference "R46")
+					(reference "R68")
 					(unit 1)
 				)
 				(path "/554fcf27-dc63-4666-abbc-7481d15942c4/cbf77838-d146-4db1-a0da-db3eb68b8af8"
-					(reference "R31")
+					(reference "R53")
 					(unit 1)
 				)
@@
 		(dnp no)
 		(fields_autoplaced yes)
-		(property "Reference" "R24"
+		(property "Reference" "R46"
 			(at 190.5 50.7999 0)
 			(effects
@@
 			(project "mega_shield"
 				(path "/554fcf27-dc63-4666-abbc-7481d15942c4/298c55ac-606f-4a25-bd04-443d4dadcb78"
-					(reference "R28")
+					(reference "R50")
 					(unit 1)
 				)
 				(path "/554fcf27-dc63-4666-abbc-7481d15942c4/400d9ece-7151-4ceb-add7-34c828d7284c"
-					(reference "R24")
+					(reference "R46")
 					(unit 1)
 				)
 				(path "/554fcf27-dc63-4666-abbc-7481d15942c4/64d796ae-634b-498c-8b87-bb3c7a5fb7ee"
-					(reference "R39")
+					(reference "R61")
 					(unit 1)
 				)
 				(path "/554fcf27-dc63-4666-abbc-7481d15942c4/a1009379-c1df-4080-8264-1d6ad70ed4b7"
-					(reference "R47")
+					(reference "R69")
 					(unit 1)
 				)
 				(path "/554fcf27-dc63-4666-abbc-7481d15942c4/cbf77838-d146-4db1-a0da-db3eb68b8af8"
-					(reference "R32")
-					(unit 1)
-				)
+					(reference "R54")
+					(unit 1)
+				)

Commit message: mega_shield, updated all optocouple circuits to use new AEC-Q200 qualified resistor on inputs.
Parts:
- R44, R45: value 15k -> 2k7; jlcpcb C17475 -> C1854836
- R46, R47: value 220 -> 4k7; jlcpcb C17557 -> C17673
Connections:
- net +5V_IN: now also U14.5, U15.5; no longer R46.1, R47.1
- net GND: now also R46.2, R47.2; no longer U14.4, U15.4
- net LIM_MAX: now also R47.1, U15.4; no longer R47.2, U15.5
- net LIM_MIN: now also R46.1, U14.4; no longer R46.2, U14.5
Other:
- moved on the sheet: R44, R45, R46, R47, U14, U15

Commit message: mega_shield, passing all ERC(electrical rules check). Zero errors
+ Fixed missing symbols from defunct digikey lib.
+ Fixed created custom symbol for AO4486 NMOS.
+ Fixed all Power flag and pin conflicts.
+ Excluded passive/unspecified warnings/errors.
Parts:
- added NT3: NetTie_2, NetTie:NetTie-2_THT_Pad1.0mm, symbol Device:NetTie_2
Connections:
- net +24V_IN: now also NT3.1; no longer C19.1, C20.1, C21.1, C22.1, J8.1, J9.1, TP80.1
- new net V_Proxy: C19.1, C20.1, C21.1, C22.1, J8.1, J9.1, NT3.2, TP80.1

Commit message: mega_shield, rerouted and place components for spindle interface
Parts:
- removed NT3: NetTie_2, NetTie:NetTie-2_THT_Pad1.0mm, symbol Device:NetTie_2
Connections:
- net V_Proxy is gone; now on net +24V_IN: C19.1, C20.1, C21.1, C22.1, J8.1, J9.1, TP80.1
Changed lines of the file:
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@@
-	(wire
-		(pts
-			(xy 53.34 25.4) (xy 63.5 25.4)
-		)
-		(stroke
-			(width 0)
-			(type default)
-		)
-	)
 	(wire
 		(pts
@@
 	(wire
 		(pts
-			(xy 38.1 25.4) (xy 48.26 25.4)
+			(xy 38.1 25.4) (xy 63.5 25.4)
 		)
 		(stroke
@@
 					(unit 1)
 				)
-			)
-		)
-	)
-	(symbol
-		(lib_id "Device:NetTie_2")
-		(at 50.8 25.4 0)
-		(mirror x)
-		(unit 1)
-		(exclude_from_sim no)
-		(in_bom no)
-		(on_board yes)
-		(dnp no)
-		(property "Reference" "NT3"
-			(at 50.8 30.48 0)
-			(effects
-				(font
-					(size 1.27 1.27)
-				)
-			)
-		)
-		(property "Value" "NetTie_2"
-			(at 50.8 27.94 0)
-			(effects
-				(font
-					(size 1.27 1.27)
-				)
-			)
-		)
-		(property "Footprint" "NetTie:NetTie-2_THT_Pad1.0mm"
-			(at 50.8 25.4 0)
-			(effects
-				(font
-					(size 1.27 1.27)
-				)
-				(hide yes)
-			)
-		)
-		(property "Datasheet" "~"
-			(at 50.8 25.4 0)
-			(effects
-				(font
-					(size 1.27 1.27)
-				)
-				(hide yes)
-			)
-		)
-		(property "Description" "Net tie, 2 pins"
-			(at 50.8 25.4 0)
-			(effects
-				(font
-					(size 1.27 1.27)
-				)
-				(hide yes)
-			)
-		)
-		(pin "1"
-		)
-		(pin "2"
-		)
-		(instances
-			(project ""
-				(path "/554fcf27-dc63-4666-abbc-7481d15942c4/298c55ac-606f-4a25-bd04-443d4dadcb78"
-					(reference "NT4")
-					(unit 1)
-				)
-				(path "/554fcf27-dc63-4666-abbc-7481d15942c4/400d9ece-7151-4ceb-add7-34c828d7284c"
-					(reference "NT3")
-					(unit 1)
-				)
-				(path "/554fcf27-dc63-4666-abbc-7481d15942c4/64d796ae-634b-498c-8b87-bb3c7a5fb7ee"
-					(reference "NT6")
-					(unit 1)
-				)
-				(path "/554fcf27-dc63-4666-abbc-7481d15942c4/a1009379-c1df-4080-8264-1d6ad70ed4b7"
-					(reference "NT7")
-					(unit 1)
-				)
-				(path "/554fcf27-dc63-4666-abbc-7481d15942c4/cbf77838-d146-4db1-a0da-db3eb68b8af8"
-					(reference "NT5")
-					(unit 1)
-				)

Commit message: mega_shield, switched from 4N35 --> PC817, higher stock and 1/3 price. Started on M8P3 offset.
Parts:
- removed U14, U15: 4N35, Package_DIP:DIP-6_W7.62mm, symbol Isolator:4N35
- added U14, U15: PC817, Package_DIP:DIP-4_W7.62mm, symbol Isolator:PC817
Connections:
- net +5V_IN: now also U14.4, U15.4
- net GND: now also U14.2, U15.2
- net LIM_MAX: now also U15.3
- net LIM_MIN: now also U14.3
- net at R45.1: now also U15.1
- net at R44.1: now also U14.1
- no-connect marks 2 -> 0

Commit message: mega_shield, fixed up discrepencies in comments for test points. Added Axis names to silkscreen.
Parts:
- TP80, TP81, TP82: value RH-5002 -> 5002
Changed lines of the file:
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@@
 			)
 		)
-		(property "Value" "RH-5002"
+		(property "Value" "5002"
 			(at 31.75 106.68 0)
 			(effects
@@
 			)
 		)
-		(property "Value" "RH-5002"
+		(property "Value" "5002"
 			(at 31.75 115.824 0)
 			(effects
@@
 			)
 		)
-		(property "Value" "RH-5002"
+		(property "Value" "5002"
 			(at 31.75 124.46 0)
 			(effects
