File: mega_shield/spin_interface.kicad_sch (KiCad schematic)
At the start: 8 parts, among them U1 MCP6241RT-I-OT

Commit message: Added isolation to the spindler interface dir and en signals.
Parts:
- added C57, C58: 1u, symbol Device:C
- added Q7, Q8: 2SK3018, PCM_Package_TO_SOT_SMD_AKL:SOT-323_SC-70, symbol PCM_Transistor_MOSFET_AKL:2SK3018
- added R4, R5: 1k, symbol Device:R
- added U4: CS817x22HS, Package_SO:SOIC-8_3.9x4.9mm_P1.27mm, symbol mega_shield:CS817x20HS
Connections:
- net +5V_SPIN: now also C57.1, C58.2, R4.1, R5.1, U4.1 (VDD1), U4.8 (VDD2)
- net GND: now also C57.2, C58.1, Q7.3 (D), Q8.3 (D), U4.4 (GND1), U4.5 (GND2)
- net SPIN_DIR: now also U4.2 (INA)
- net SPIN_EN: now also U4.3 (INB)
- new net: Q8.1 (G), U4.6 (OUTB)
- new net: Q7.1 (G), U4.7 (OUTA)
- new net SPIN_DIR_OC: Q7.2 (S), R4.2
- new net SPIN_EN_OC: Q8.2 (S), R5.2
Other:
- note added: "Digitally Isolated Inputs"

Commit message: Added the spindle interface connector. Added original schematics note from Brandon.
Parts:
- added J2: 691311500004, 691311500004:691311500004, symbol wurth_4P:691311500004
Connections:
- net +5V_SPIN: now also J2.1
- net GND: now also J2.4
- net SPIN_DIR_OC: now also J2.2
- net SPIN_EN_OC: now also J2.3
Other:
- note added: "Spindle Connection"
- moved on the sheet: C53, C54, C55, C56, C57, C58, NT1, Q7, Q8, R1, R3, R4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

Commit message: Added test points to the spindle interface.
Parts:
- added TP91, TP92, TP93, TP94, TP95, TP96, TP97: TestPoint, symbol Connector:TestPoint
Connections:
- net +5V_SPIN: now also TP91.1, TP95.1
- net SPIN_DIR: now also TP93.1
- net SPIN_DIR_OC: now also TP96.1
- net SPIN_EN: now also TP94.1
- net SPIN_EN_OC: now also TP97.1
- net SPIN_PWM: now also TP92.1
Other:
- note added: "Spin Interface Test Points"

Commit message: updated spindle interface to use 5pin connector with one pin for the 10v or 5V connection.
Parts:
- removed J2: 691311500004, 691311500004:691311500004, symbol wurth_4P:691311500004
- added J11: 1757271, 1757271:PHOENIX_1757271, symbol TERM_BLOCK_HDR_5POS_5.08MM:1757271
Connections:
- net +5V_SPIN: no longer C53.2, C54.2, C56.2, C58.2, R4.1, R5.1, TP95.1, U1.1, U1.2 (V+), U1.4 (-), U4.8 (VDD2)
- net GND: now also J11.05
- net SPIN_DIR_OC: now also J11.03
- net SPIN_EN_OC: now also J11.04
- new net SPIN_SPEED: C53.2, C54.2, C56.2, C58.2, J11.01, J11.02, R4.1, R5.1, TP95.1, U1.1, U1.2 (V+), U1.4 (-), U4.8 (VDD2)
Changed lines of the file:
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@@
 	)
 	(rectangle
-		(start 139.7 25.4)
+		(start 129.54 25.4)
 		(end 179.07 50.8)
 		(stroke
@@
 	(wire
 		(pts
+			(xy 157.48 30.48) (xy 165.1 30.48)
+		)
+		(stroke
+			(width 0)
+			(type default)
+		)
+	)
+	(wire
+		(pts
 			(xy 105.41 95.25) (xy 101.6 95.25)
 		)
@@
 		)
 	)
-	(label "+5V_SPIN"
-		(at 207.01 81.28 0)
-		(effects
-			(font
-				(size 1.27 1.27)
-			)
-			(justify left bottom)
-		)
-	)
 	(label "SPIN_DIR_OC"
 		(at 165.1 35.56 0)
@@
 		)
 	)
-	(label "+5V_SPIN"
-		(at 228.6 77.47 0)
+	(label "V_SPIN"
+		(at 228.6 109.22 0)
 		(effects
 			(font
@@
 			)
 			(justify left bottom)
+		)
+	)
+	(label "V_SPIN"
+		(at 92.71 72.39 180)
+		(effects
+			(font
+				(size 1.27 1.27)
+			)
+			(justify right bottom)
 		)
 	)
@@
 		)
 	)
+	(label "V_SPIN"
+		(at 165.1 30.48 0)
+		(effects
+			(font
+				(size 1.27 1.27)
+			)
+			(justify left bottom)
+		)
+	)
 	(label "SPIN_DIR_OC"
 		(at 63.5 167.64 0)
@@
 		)
 	)
-	(label "+5V_SPIN"
-		(at 228.6 109.22 0)
-		(effects
-			(font
-				(size 1.27 1.27)
-			)
-			(justify left bottom)
-		)
-	)
 	(label "SPIN_SPEED"
 		(at 111.76 95.25 0)
@@
 	)
 	(label "+5V_SPIN"
-		(at 92.71 72.39 180)
-		(effects
-			(font
-				(size 1.27 1.27)
-			)
-			(justify right bottom)
-		)
-	)
-	(label "+5V_SPIN"
 		(at 38.1 152.4 0)
 		(effects
@@
 	(label "+5V_SPIN"
 		(at 58.42 34.29 0)
+		(effects
+			(font
+				(size 1.27 1.27)
+			)
+			(justify left bottom)
+		)
+	)
+	(label "V_SPIN"
+		(at 207.01 81.28 0)
+		(effects
+			(font
+				(size 1.27 1.27)
+			)
+			(justify left bottom)
+		)
+	)
+	(label "V_SPIN"
+		(at 228.6 77.47 0)
 		(effects
 			(font
@@
 	)
 	(symbol
-		(lib_id "wurth_4P:691311500004")
-		(at 152.4 38.1 90)
-		(mirror x)
-		(unit 1)
-		(exclude_from_sim no)
-		(in_bom yes)
-		(on_board yes)
-		(dnp no)
-		(property "Reference" "J2"
-			(at 153.67 46.99 90)
-			(effects
-				(font
-					(size 1.27 1.27)
-				)
-			)
-		)
-		(property "Value" "691311500004"
-			(at 153.67 44.45 90)
-			(effects
-				(font
-					(size 1.27 1.27)
-				)
-			)
-		)
-		(property "Footprint" "691311500004:691311500004"
-			(at 152.4 38.1 0)
-			(effects
-				(font
-					(size 1.27 1.27)
-				)
-				(justify bottom)
-				(hide yes)
-			)
-		)
-		(property "Datasheet" ""
-			(at 152.4 38.1 0)
-			(effects
-				(font
-					(size 1.27 1.27)
-				)
-				(hide yes)
-			)
-		)
-		(property "Description" ""
-			(at 152.4 38.1 0)
-			(effects
-				(font
-					(size 1.27 1.27)
-				)
-				(hide yes)
-			)
-		)
-		(pin "2"
-		)
-		(pin "1"
-		)
-		(pin "3"
-		)
-		(pin "4"
-		)
-		(instances
-			(project ""
-				(path "/554fcf27-dc63-4666-abbc-7481d15942c4/05acfb4b-1f70-4813-b5f6-d6a6759e8a5f"
-					(reference "J2")
-					(unit 1)
-				)
-			)
-		)
-	)
-	(symbol
 		(lib_id "power:GND")
 		(at 120.65 77.47 0)
@@
 					(unit 1)
 				)
+			)
+		)
+	)
+	(symbol
+		(lib_id "TERM_BLOCK_HDR_5POS_5.08MM:1757271")
+		(at 147.32 35.56 0)
+		(mirror y)
+		(unit 1)
+		(exclude_from_sim no)
+		(in_bom yes)
+		(on_board yes)
+		(dnp no)
+		(property "Reference" "J11"
+			(at 139.7 34.2899 0)
+			(effects
+				(font
+					(size 1.27 1.27)
+				)
+				(justify left)
+			)
+		)
+		(property "Value" "1757271"
+			(at 139.7 36.8299 0)
+			(effects
+				(font
+					(size 1.27 1.27)
+				)
+				(justify left)
+			)
+		)
+		(property "Footprint" "1757271:PHOENIX_1757271"
+			(at 147.32 35.56 0)
+			(effects
+				(font
+					(size 1.27 1.27)
+				)
+				(justify bottom)
+				(hide yes)
+			)
+		)
+		(property "Datasheet" ""
+			(at 147.32 35.56 0)
+			(effects
+				(font
+					(size 1.27 1.27)
+				)
+				(hide yes)
+			)
+		)
+		(property "Description" ""
+			(at 147.32 35.56 0)
+			(effects
+				(font
+					(size 1.27 1.27)
+				)
+				(hide yes)
+			)
+		)
+		(property "PARTREV" "28.07.2023"
+			(at 147.32 35.56 0)
+			(effects
+				(font
+					(size 1.27 1.27)
+				)
+				(justify bottom)
+				(hide yes)
+			)
+		)
+		(property "STANDARD" "Manufacturer Recommendations"
+			(at 147.32 35.56 0)
+			(effects
+				(font
+					(size 1.27 1.27)
+				)
+				(justify bottom)
+				(hide yes)
+			)
+		)
+		(property "MANUFACTURER" "Phoenix Contact"
+			(at 147.32 35.56 0)
+			(effects
+				(font
+					(size 1.27 1.27)
+				)
+				(justify bottom)
+				(hide yes)
+			)
+		)
+		(pin "03"
+		)
+		(pin "04"
+		)
+		(pin "05"
+		)
+		(pin "02"
+		)
+		(pin "01"
+		)
+		(instances
+			(project ""
+				(path "/554fcf27-dc63-4666-abbc-7481d15942c4/05acfb4b-1f70-4813-b5f6-d6a6759e8a5f"
+					(reference "J11")
+					(unit 1)
+				)

Commit message: Added test point to spindle interface for V_spin.
Parts:
- added TP98: TestPoint, symbol Connector:TestPoint
Connections:
- net SPIN_SPEED: now also TP98.1
Changed lines of the file:
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@@
+	)
+	(label "V_SPIN"
+		(at 63.5 152.4 0)
+		(effects
+			(font
+				(size 1.27 1.27)
+			)
+			(justify left bottom)
+		)
 	)
 	(label "V_SPIN"
@@
 					(unit 1)
 				)
+			)
+		)
+	)
+	(symbol
+		(lib_id "Connector:TestPoint")
+		(at 63.5 152.4 90)
+		(unit 1)
+		(exclude_from_sim no)
+		(in_bom yes)
+		(on_board yes)
+		(dnp no)
+		(fields_autoplaced yes)
+		(property "Reference" "TP98"
+			(at 60.198 147.32 90)
+			(effects
+				(font
+					(size 1.27 1.27)
+				)
+			)
+		)
+		(property "Value" "TestPoint"
+			(at 60.198 149.86 90)
+			(effects
+				(font
+					(size 1.27 1.27)
+				)
+			)
+		)
+		(property "Footprint" ""
+			(at 63.5 147.32 0)
+			(effects
+				(font
+					(size 1.27 1.27)
+				)
+				(hide yes)
+			)
+		)
+		(property "Datasheet" "~"
+			(at 63.5 147.32 0)
+			(effects
+				(font
+					(size 1.27 1.27)
+				)
+				(hide yes)
+			)
+		)
+		(property "Description" "test point"
+			(at 63.5 152.4 0)
+			(effects
+				(font
+					(size 1.27 1.27)
+				)
+				(hide yes)
+			)
+		)
+		(pin "1"
+		)
+		(instances
+			(project "mega_shield"
+				(path "/554fcf27-dc63-4666-abbc-7481d15942c4/05acfb4b-1f70-4813-b5f6-d6a6759e8a5f"
+					(reference "TP98")
+					(unit 1)
+				)

Commit message: Added the ESD protection on the PWM for the spindle interface.
Parts:
- added U31: NUP2202, Package_TO_SOT_SMD:SOT-363_SC-70-6, symbol Power_Protection:NUP2202
Connections:
- net GND: now also U31.2
- net SPIN_SPEED: now also U31.1, U31.5, U31.6
Changed lines of the file:
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@@
 	(rectangle
 		(start 25.4 63.5)
-		(end 127 127)
+		(end 137.16 127)
 		(stroke
 			(width 0)
@@
 			(justify left top)
 		)
+	)
+	(junction
+		(at 109.22 95.25)
+		(diameter 0)
+		(color 0 0 0 0)
 	)
 	(junction
@@
 	)
 	(junction
+		(at 109.22 102.87)
+		(diameter 0)
+		(color 0 0 0 0)
+	)
+	(junction
 		(at 54.61 34.29)
 		(diameter 0)
@@
 	(wire
 		(pts
+			(xy 109.22 102.87) (xy 109.22 113.03)
+		)
+		(stroke
+			(width 0)
+			(type default)
+		)
+	)
+	(wire
+		(pts
 			(xy 50.8 119.38) (xy 105.41 119.38)
 		)
@@
 	(wire
 		(pts
+			(xy 124.46 102.87) (xy 109.22 102.87)
+		)
+		(stroke
+			(width 0)
+			(type default)
+		)
+	)
+	(wire
+		(pts
 			(xy 114.3 68.58) (xy 114.3 72.39)
 		)
@@
 	(wire
 		(pts
+			(xy 109.22 95.25) (xy 111.76 95.25)
+		)
+		(stroke
+			(width 0)
+			(type default)
+		)
+	)
+	(wire
+		(pts
 			(xy 157.48 30.48) (xy 165.1 30.48)
 		)
@@
 	(wire
 		(pts
-			(xy 105.41 95.25) (xy 111.76 95.25)
+			(xy 124.46 113.03) (xy 119.38 113.03)
+		)
+		(stroke
+			(width 0)
+			(type default)
+		)
+	)
+	(wire
+		(pts
+			(xy 105.41 95.25) (xy 109.22 95.25)
 		)
 		(stroke
@@
 	(wire
 		(pts
+			(xy 109.22 95.25) (xy 109.22 102.87)
+		)
+		(stroke
+			(width 0)
+			(type default)
+		)
+	)
+	(wire
+		(pts
 			(xy 154.94 81.28) (xy 154.94 92.71)
+		)
+		(stroke
+			(width 0)
+			(type default)
+		)
+	)
+	(wire
+		(pts
+			(xy 124.46 113.03) (xy 124.46 102.87)
 		)
 		(stroke
@@
 	(label "V_SPIN"
 		(at 63.5 152.4 0)
+		(effects
+			(font
+				(size 1.27 1.27)
+			)
+			(justify left bottom)
+		)
+	)
+	(label "V_SPIN"
+		(at 114.3 107.95 0)
 		(effects
 			(font
@@
 					(unit 1)
 				)
+			)
+		)
+	)
+	(symbol
+		(lib_id "power:GND")
+		(at 114.3 118.11 0)
+		(unit 1)
+		(exclude_from_sim no)
+		(in_bom yes)
+		(on_board yes)
+		(dnp no)
+		(fields_autoplaced yes)
+		(property "Reference" "#PWR068"
+			(at 114.3 124.46 0)
+			(effects
+				(font
+					(size 1.27 1.27)
+				)
+				(hide yes)
+			)
+		)
+		(property "Value" "GND"
+			(at 114.3 123.19 0)
+			(effects
+				(font
+					(size 1.27 1.27)
+				)
+			)
+		)
+		(property "Footprint" ""
+			(at 114.3 118.11 0)
+			(effects
+				(font
+					(size 1.27 1.27)
+				)
+				(hide yes)
+			)
+		)
+		(property "Datasheet" ""
+			(at 114.3 118.11 0)
+			(effects
+				(font
+					(size 1.27 1.27)
+				)
+				(hide yes)
+			)
+		)
+		(property "Description" "Power symbol creates a global label with name \"GND\" , ground"
+			(at 114.3 118.11 0)
+			(effects
+				(font
+					(size 1.27 1.27)
+				)
+				(hide yes)
+			)
+		)
+		(pin "1"
+		)
+		(instances
+			(project "mega_shield"
+				(path "/554fcf27-dc63-4666-abbc-7481d15942c4/05acfb4b-1f70-4813-b5f6-d6a6759e8a5f"
+					(reference "#PWR068")
+					(unit 1)
+				)
+			)
+		)
+	)
+	(symbol
+		(lib_id "Power_Protection:NUP2202")
+		(at 114.3 113.03 0)
+		(unit 1)
+		(exclude_from_sim no)
+		(in_bom yes)
+		(on_board yes)
+		(dnp no)
+		(property "Reference" "U31"
+			(at 123.19 112.776 0)
+			(effects
+				(font
+					(size 1.27 1.27)
+				)
+			)
+		)
+		(property "Value" "NUP2202"
+			(at 123.19 114.808 0)
+			(effects
+				(font
+					(size 1.27 1.27)
+				)
+			)
+		)
+		(property "Footprint" "Package_TO_SOT_SMD:SOT-363_SC-70-6"
+			(at 116.332 111.125 0)
+			(effects
+				(font
+					(size 1.27 1.27)
+				)
+				(hide yes)
+			)
+		)
+		(property "Datasheet" "https://www.onsemi.com/pdf/datasheet/nup2202w1-d.pdf"
+			(at 116.332 111.125 0)
+			(effects
+				(font
+					(size 1.27 1.27)
+				)
+				(hide yes)
+			)
+		)
+		(property "Description" "Transient voltage suppressor designed to protect high speed data lines from ESD, EFT, and lightning"
+			(at 114.3 113.03 0)
+			(effects
+				(font
+					(size 1.27 1.27)
+				)
+				(hide yes)
+			)
+		)
+		(property "jlcpcb" "C4355033"
+			(at 114.3 113.03 0)
+			(effects
+				(font
+					(size 1.27 1.27)
+				)
+			)
+		)
+		(pin "2"
+		)
+		(pin "1"
+		)
+		(pin "3"
+		)
+		(pin "4"
+		)
+		(pin "5"
+		)
+		(pin "6"
+		)
+		(instances
+			(project "mega_shield"
+				(path "/554fcf27-dc63-4666-abbc-7481d15942c4/05acfb4b-1f70-4813-b5f6-d6a6759e8a5f"
+					(reference "U31")
+					(unit 1)
+				)

Commit message: Ran the annotation operation on all schematics.
Parts:
- renumbered C56 to C13, C55 to C14, C54 to C15, C53 to C16, C57 to C17, C58 to C18, J11 to J3, Q7 to Q13, Q8 to Q14, R5 to R10, R1 to R7, R3 to R8, R4 to R9, TP91 to TP27, TP92 to TP28, TP93 to TP29, TP94 to TP30, TP98 to TP31, TP95 to TP32, TP96 to TP33, TP97 to TP34, U1 to U7, U31 to U8, U4 to U9

Commit message: Assigned 0603 footprint to all 1uF caps.
Parts:
- C17, C18: footprint (none) -> Capacitor_SMD:C_0201_0603Metric
Changed lines of the file:
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@@
 			)
 		)
-		(property "Footprint" ""
+		(property "Footprint" "Capacitor_SMD:C_0201_0603Metric"
 			(at 200.66 80.3148 0)
 			(effects
@@
 			)
 		)
-		(property "Footprint" ""
+		(property "Footprint" "Capacitor_SMD:C_0201_0603Metric"
 			(at 167.64 80.3148 0)
 			(effects
