File: mega_shield/spin_interface.kicad_sch (KiCad schematic)
At the start: 25 parts, among them J3 1757271, Q10 2N7002, Q9 2N7002, U32 LMV321, U4 NUP2202, U5 ADuM1200

Commit message: mega_shield, updated the calculations for the filters.
Parts:
- R51, R52: value 10k -> 20k
Other:
- note added: "PWM signal filter(slow rise time)"
- note removed: "PWM signal filter"
Changed lines of the file:
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@@
 		)
 	)
-	(text "PWM signal filter\n"
+	(text "PWM signal filter(slow rise time)\n"
 		(exclude_from_sim no)
-		(at 34.29 62.738 0)
+		(at 41.656 62.738 0)
 		(effects
 			(font
@@
 		)
 	)
-	(text_box "LMV321: Vos = 0.8mV, Ios = 10pA, Ib = 10pA\n\nFcutoff = 1/(2*Pi*R*C)\nFcutoff = 1.5Hz = 1/(2*Pi*10k*C)\nC = 10uF\n\n2Pole RC filter, C1 = C2 = 10uF/2, accounting for extra trace len etc.\nC1 = C2 = 4.7uF"
+	(text_box "LMV321: Vos = 0.8mV, Ios = 10pA, Ib = 10pA\n\nFcutoff = 1/(2*Pi*R*C)\nFcutoff = 1.5Hz = 1/(2*Pi*20k*C)\nC = 5.3uF\n\n2Pole RC filter, C1 = C2 = 10uF/2, accounting for extra trace len etc.\nC1 = C2 = 5.3uF"
 		(exclude_from_sim no)
 		(at 26.67 105.41 0)
@@
 			)
 		)
-		(property "Value" "10k"
+		(property "Value" "20k"
 			(at 44.45 85.09 90)
 			(effects
@@
 			)
 		)
-		(property "Value" "10k"
+		(property "Value" "20k"
 			(at 57.15 85.09 90)
 			(effects

Commit message: mega_shield, calculated/simulated stabilization time and switched to unity gain active filter
+ Active filter nearly half's the time to stabablize to approximatly
250mS.
Parts:
- removed C44, C45: 4.7u, symbol Device:C
- added C44, C5, C6: 1u, symbol Device:C_Small
- R51, R52: value 20k -> 75k
Connections:
- net GND: now also C44.2
- net SPIN_SPEED: now also C5.2, C6.2; no longer C7.2, C8.2, J3.01, R5.1, R6.1, TP34.1, U32.5 (V+), U4.5
- net at R51.1, R52.2: now also C5.1, C6.1
- net at R51.2, U32.1 (+): now also C44.1
- new net V_SPIN: C7.2, C8.2, J3.01, R5.1, R6.1, TP34.1, U32.5 (V+), U4.5
Other:
- note added: "PWM signal filter(Active)"
- note removed: "PWM signal filter(slow rise time)"

Commit message: mega_shield, assigned JLCPCB numbers for new active filter caps.
Parts:
- C44, C5, C6: value 1u -> 1u/50V; footprint (none) -> Capacitor_SMD:C_0805_2012Metric_Pad1.18x1.45mm_HandSolder; jlcpcb (none) -> C28323
Changed lines of the file:
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@@
 			)
 		)
-		(property "Value" "1u"
+		(property "Value" "1u/50V"
 			(at 69.8563 83.82 90)
 			(effects
@@
 			)
 		)
-		(property "Footprint" ""
+		(property "Footprint" "Capacitor_SMD:C_0805_2012Metric_Pad1.18x1.45mm_HandSolder"
 			(at 69.85 80.01 0)
 			(effects
@@
 		(property "Description" "Unpolarized capacitor, small symbol"
 			(at 69.85 80.01 0)
+			(effects
+				(font
+					(size 1.27 1.27)
+				)
+				(hide yes)
+			)
+		)
+		(property "jlcpcb" "C28323"
+			(at 69.85 80.01 90)
 			(effects
 				(font
@@
 			)
 		)
-		(property "Value" "1u"
+		(property "Value" "1u/50V"
 			(at 69.8563 72.39 90)
 			(effects
@@
 			)
 		)
-		(property "Footprint" ""
+		(property "Footprint" "Capacitor_SMD:C_0805_2012Metric_Pad1.18x1.45mm_HandSolder"
 			(at 69.85 76.2 0)
 			(effects
@@
 		(property "Description" "Unpolarized capacitor, small symbol"
 			(at 69.85 76.2 0)
+			(effects
+				(font
+					(size 1.27 1.27)
+				)
+				(hide yes)
+			)
+		)
+		(property "jlcpcb" "C28323"
+			(at 69.85 76.2 90)
 			(effects
 				(font
@@
 			)
 		)
-		(property "Value" "1u"
+		(property "Value" "1u/50V"
 			(at 60.96 96.5262 0)
 			(effects
@@
 			)
 		)
-		(property "Footprint" ""
+		(property "Footprint" "Capacitor_SMD:C_0805_2012Metric_Pad1.18x1.45mm_HandSolder"
 			(at 63.5 95.25 0)
 			(effects
@@
 			(at 63.5 95.25 0)
 			(effects
+				(font
+					(size 1.27 1.27)
+				)
+				(hide yes)
+			)
+		)
+		(property "jlcpcb" "C28323"
+			(at 63.5 95.25 0)
+			(effects

Commit message: mega_shield, asigned active filter footprints and jlcpcb numbers.
Parts:
- R51, R52: footprint (none) -> Resistor_SMD:R_0805_2012Metric_Pad1.20x1.40mm_HandSolder; jlcpcb (none) -> C17819
Changed lines of the file:
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@@
 			)
 		)
-		(property "Footprint" ""
+		(property "Footprint" "Resistor_SMD:R_0805_2012Metric_Pad1.20x1.40mm_HandSolder"
 			(at 44.45 90.678 90)
 			(effects
@@
 		(property "Description" "Resistor"
 			(at 44.45 88.9 0)
+			(effects
+				(font
+					(size 1.27 1.27)
+				)
+				(hide yes)
+			)
+		)
+		(property "jlcpcb" "C17819"
+			(at 44.45 88.9 90)
 			(effects
 				(font
@@
 			)
 		)
-		(property "Footprint" ""
+		(property "Footprint" "Resistor_SMD:R_0805_2012Metric_Pad1.20x1.40mm_HandSolder"
 			(at 57.15 90.678 90)
 			(effects
@@
 			(effects
 				(font
+					(size 1.27 1.27)
+				)
+				(hide yes)
+			)
+		)
+		(property "jlcpcb" "C17819"
+			(at 57.15 88.9 90)
+			(effects
+				(font

Commit message: mega_shield, re-annotated schematic's components.
Parts:
- renumbered C9 to C10, C10 to C11, C44 to C5, C5 to C6, C6 to C7, C7 to C8, C8 to C9, R52 to R3, R51 to R4, U32 to U3
Changed lines of the file:
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@@
 		(on_board yes)
 		(dnp no)
-		(property "Reference" "C6"
+		(property "Reference" "C7"
 			(at 69.8563 86.36 90)
 			(effects
@@
 			(project "mega_shield"
 				(path "/554fcf27-dc63-4666-abbc-7481d15942c4/05acfb4b-1f70-4813-b5f6-d6a6759e8a5f"
-					(reference "C6")
+					(reference "C7")
 					(unit 1)
 				)
@@
 		(dnp no)
 		(fields_autoplaced yes)
-		(property "Reference" "R52"
+		(property "Reference" "R3"
 			(at 44.45 82.55 90)
 			(effects
@@
 			(project "mega_shield"
 				(path "/554fcf27-dc63-4666-abbc-7481d15942c4/05acfb4b-1f70-4813-b5f6-d6a6759e8a5f"
-					(reference "R52")
+					(reference "R3")
 					(unit 1)
 				)
@@
 		(dnp no)
 		(fields_autoplaced yes)
-		(property "Reference" "C5"
+		(property "Reference" "C6"
 			(at 69.8563 69.85 90)
 			(effects
@@
 			(project ""
 				(path "/554fcf27-dc63-4666-abbc-7481d15942c4/05acfb4b-1f70-4813-b5f6-d6a6759e8a5f"
-					(reference "C5")
+					(reference "C6")
 					(unit 1)
 				)
@@
 		(dnp no)
 		(fields_autoplaced yes)
-		(property "Reference" "R51"
+		(property "Reference" "R4"
 			(at 57.15 82.55 90)
 			(effects
@@
 			(project ""
 				(path "/554fcf27-dc63-4666-abbc-7481d15942c4/05acfb4b-1f70-4813-b5f6-d6a6759e8a5f"
-					(reference "R51")
+					(reference "R4")
 					(unit 1)
 				)
@@
 		(dnp no)
 		(fields_autoplaced yes)
-		(property "Reference" "C10"
+		(property "Reference" "C11"
 			(at 194.31 77.47 90)
 			(effects
@@
 			(project "mega_shield"
 				(path "/554fcf27-dc63-4666-abbc-7481d15942c4/05acfb4b-1f70-4813-b5f6-d6a6759e8a5f"
-					(reference "C10")
+					(reference "C11")
 					(unit 1)
 				)
@@
 		(on_board yes)
 		(dnp no)
-		(property "Reference" "C44"
+		(property "Reference" "C5"
 			(at 60.96 93.9862 0)
 			(effects
@@
 			(project ""
 				(path "/554fcf27-dc63-4666-abbc-7481d15942c4/05acfb4b-1f70-4813-b5f6-d6a6759e8a5f"
-					(reference "C44")
+					(reference "C5")
 					(unit 1)
 				)
@@
 		(dnp no)
 		(fields_autoplaced yes)
-		(property "Reference" "C9"
+		(property "Reference" "C10"
 			(at 166.37 77.47 90)
 			(effects
@@
 			(project "mega_shield"
 				(path "/554fcf27-dc63-4666-abbc-7481d15942c4/05acfb4b-1f70-4813-b5f6-d6a6759e8a5f"
-					(reference "C9")
+					(reference "C10")
 					(unit 1)
 				)
@@
 		(on_board yes)
 		(dnp no)
-		(property "Reference" "C7"
+		(property "Reference" "C8"
 			(at 109.728 65.786 90)
 			(effects
@@
 			(project "mega_shield"
 				(path "/554fcf27-dc63-4666-abbc-7481d15942c4/05acfb4b-1f70-4813-b5f6-d6a6759e8a5f"
-					(reference "C7")
+					(reference "C8")
 					(unit 1)
 				)
@@
 		(on_board yes)
 		(dnp no)
-		(property "Reference" "C8"
+		(property "Reference" "C9"
 			(at 109.982 73.406 90)
 			(effects
@@
 			(project ""
 				(path "/554fcf27-dc63-4666-abbc-7481d15942c4/05acfb4b-1f70-4813-b5f6-d6a6759e8a5f"
-					(reference "C8")
+					(reference "C9")
 					(unit 1)
 				)
@@
 		(dnp no)
 		(fields_autoplaced yes)
-		(property "Reference" "U32"
+		(property "Reference" "U3"
 			(at 93.98 82.4798 0)
 			(effects
@@
 			(project ""
 				(path "/554fcf27-dc63-4666-abbc-7481d15942c4/05acfb4b-1f70-4813-b5f6-d6a6759e8a5f"
-					(reference "U32")
+					(reference "U3")
 					(unit 1)
 				)
@@
 		(dnp no)
 		(fields_autoplaced yes)
-		(property "Reference" "#PWR0117"
+		(property "Reference" "#PWR037"
 			(at 80.01 107.95 0)
 			(effects
@@
 			(project "mega_shield"
 				(path "/554fcf27-dc63-4666-abbc-7481d15942c4/05acfb4b-1f70-4813-b5f6-d6a6759e8a5f"
-					(reference "#PWR0117")
+					(reference "#PWR037")
 					(unit 1)
 				)

Commit message: mega_shield, Added notes on 2N7002 fets. Added gate resistors.
+ Added 100Ohm gate resistors.
+ Added textbox/notes on the built-in diodes.
Parts:
- added R59, R60: 100, symbol Device:R
Connections:
- net at U5.6 (Vout_a): now also R59.2; no longer Q10.1 (G)
- net at U5.7 (Vout_b): now also R60.1; no longer Q9.1 (G)
- new net: Q9.1 (G), R60.2
- new net: Q10.1 (G), R59.1
Changed lines of the file:
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@@
+		)
+	)
+	(text_box "The 2N7002 N-Channel mosfets contain their own built in soruce drain diode.\n\nNo extra external components are needed for that particular issue."
+		(exclude_from_sim no)
+		(at 139.7 143.51 0)
+		(size 76.2 17.78)
+		(margins 0.9525 0.9525 0.9525 0.9525)
+		(stroke
+			(width 0)
+			(type solid)
+		)
+		(fill
+			(type none)
+		)
+		(effects
+			(font
+				(size 1.27 1.27)
+			)
+			(justify left top)
 		)
 	)
@@
 	(wire
 		(pts
-			(xy 222.25 88.9) (xy 219.71 88.9)
-		)
-		(stroke
-			(width 0)
-			(type default)
-		)
-	)
-	(wire
-		(pts
 			(xy 205.74 118.11) (xy 205.74 109.22)
 		)
@@
 	(wire
 		(pts
-			(xy 196.85 105.41) (xy 217.17 105.41)
-		)
-		(stroke
-			(width 0)
-			(type default)
-		)
-	)
-	(wire
-		(pts
-			(xy 217.17 120.65) (xy 217.17 105.41)
+			(xy 215.9 109.22) (xy 215.9 105.41)
 		)
 		(stroke
@@
 	(wire
 		(pts
+			(xy 215.9 99.06) (xy 215.9 100.33)
+		)
+		(stroke
+			(width 0)
+			(type default)
+		)
+	)
+	(wire
+		(pts
+			(xy 215.9 88.9) (xy 215.9 91.44)
+		)
+		(stroke
+			(width 0)
+			(type default)
+		)
+	)
+	(wire
+		(pts
 			(xy 101.6 88.9) (xy 104.14 88.9)
 		)
@@
 	(wire
 		(pts
-			(xy 222.25 120.65) (xy 217.17 120.65)
-		)
-		(stroke
-			(width 0)
-			(type default)
-		)
-	)
-	(wire
-		(pts
 			(xy 114.3 76.2) (xy 109.22 76.2)
 		)
@@
 	(wire
 		(pts
+			(xy 215.9 116.84) (xy 215.9 120.65)
+		)
+		(stroke
+			(width 0)
+			(type default)
+		)
+	)
+	(wire
+		(pts
 			(xy 74.93 88.9) (xy 63.5 88.9)
 		)
@@
 	(wire
 		(pts
+			(xy 215.9 120.65) (xy 222.25 120.65)
+		)
+		(stroke
+			(width 0)
+			(type default)
+		)
+	)
+	(wire
+		(pts
 			(xy 198.12 85.09) (xy 204.47 85.09)
 		)
@@
 	(wire
 		(pts
-			(xy 219.71 88.9) (xy 219.71 100.33)
-		)
-		(stroke
-			(width 0)
-			(type default)
-		)
-	)
-	(wire
-		(pts
 			(xy 163.83 109.22) (xy 153.67 109.22)
 		)
@@
 	(wire
 		(pts
+			(xy 215.9 100.33) (xy 196.85 100.33)
+		)
+		(stroke
+			(width 0)
+			(type default)
+		)
+	)
+	(wire
+		(pts
 			(xy 157.48 41.91) (xy 165.1 41.91)
 		)
@@
 	(wire
 		(pts
+			(xy 222.25 88.9) (xy 215.9 88.9)
+		)
+		(stroke
+			(width 0)
+			(type default)
+		)
+	)
+	(wire
+		(pts
 			(xy 157.48 85.09) (xy 157.48 96.52)
 		)
@@
 	(wire
 		(pts
-			(xy 219.71 100.33) (xy 196.85 100.33)
-		)
-		(stroke
-			(width 0)
-			(type default)
-		)
-	)
-	(wire
-		(pts
 			(xy 196.85 109.22) (xy 205.74 109.22)
 		)
@@
 		(pts
 			(xy 71.12 91.44) (xy 74.93 91.44)
+		)
+		(stroke
+			(width 0)
+			(type default)
+		)
+	)
+	(wire
+		(pts
+			(xy 215.9 105.41) (xy 196.85 105.41)
 		)
 		(stroke
@@
 			)
 			(justify left bottom)
-		)
-	)
-	(label "+5V_SPIN"
-		(at 157.48 85.09 180)
-		(effects
-			(font
-				(size 1.27 1.27)
-			)
-			(justify right bottom)
 		)
 	)
@@
 			)
 			(justify left)
+		)
+	)
+	(hierarchical_label "+5V_IN"
+		(shape input)
+		(at 157.48 85.09 180)
+		(effects
+			(font
+				(size 1.27 1.27)
+			)
+			(justify right)
 		)
 	)
@@
 	)
 	(symbol
+		(lib_id "Device:R")
+		(at 215.9 95.25 180)
+		(unit 1)
+		(exclude_from_sim no)
+		(in_bom yes)
+		(on_board yes)
+		(dnp no)
+		(fields_autoplaced yes)
+		(property "Reference" "R60"
+			(at 218.44 93.9799 0)
+			(effects
+				(font
+					(size 1.27 1.27)
+				)
+				(justify right)
+			)
+		)
+		(property "Value" "100"
+			(at 218.44 96.5199 0)
+			(effects
+				(font
+					(size 1.27 1.27)
+				)
+				(justify right)
+			)
+		)
+		(property "Footprint" ""
+			(at 217.678 95.25 90)
+			(effects
+				(font
+					(size 1.27 1.27)
+				)
+				(hide yes)
+			)
+		)
+		(property "Datasheet" "~"
+			(at 215.9 95.25 0)
+			(effects
+				(font
+					(size 1.27 1.27)
+				)
+				(hide yes)
+			)
+		)
+		(property "Description" "Resistor"
+			(at 215.9 95.25 0)
+			(effects
+				(font
+					(size 1.27 1.27)
+				)
+				(hide yes)
+			)
+		)
+		(pin "2"
+		)
+		(pin "1"
+		)
+		(instances
+			(project "mega_shield"
+				(path "/554fcf27-dc63-4666-abbc-7481d15942c4/05acfb4b-1f70-4813-b5f6-d6a6759e8a5f"
+					(reference "R60")
+					(unit 1)
+				)
+			)
+		)
+	)
+	(symbol
 		(lib_id "Connector:TestPoint")
 		(at 38.1 167.64 90)
@@
 					(unit 1)
 				)
+			)
+		)
+	)
+	(symbol
+		(lib_id "Device:R")
+		(at 215.9 113.03 180)
+		(unit 1)
+		(exclude_from_sim no)
+		(in_bom yes)
+		(on_board yes)
+		(dnp no)
+		(fields_autoplaced yes)
+		(property "Reference" "R59"
+			(at 218.44 111.7599 0)
+			(effects
+				(font
+					(size 1.27 1.27)
+				)
+				(justify right)
+			)
+		)
+		(property "Value" "100"
+			(at 218.44 114.2999 0)
+			(effects
+				(font
+					(size 1.27 1.27)
+				)
+				(justify right)
+			)
+		)
+		(property "Footprint" ""
+			(at 217.678 113.03 90)
+			(effects
+				(font
+					(size 1.27 1.27)
+				)
+				(hide yes)
+			)
+		)
+		(property "Datasheet" "~"
+			(at 215.9 113.03 0)
+			(effects
+				(font
+					(size 1.27 1.27)
+				)
+				(hide yes)
+			)
+		)
+		(property "Description" "Resistor"
+			(at 215.9 113.03 0)
+			(effects
+				(font
+					(size 1.27 1.27)
+				)
+				(hide yes)
+			)
+		)
+		(pin "2"
+		)
+		(pin "1"
+		)
+		(instances
+			(project ""
+				(path "/554fcf27-dc63-4666-abbc-7481d15942c4/05acfb4b-1f70-4813-b5f6-d6a6759e8a5f"
+					(reference "R59")
+					(unit 1)
+				)

Commit message: mega_shield, updated 3D models for servo interfaces.
Parts:
- R59, R60: footprint (none) -> Resistor_SMD:R_0805_2012Metric_Pad1.20x1.40mm_HandSolder; jlcpcb (none) -> C17408
Changed lines of the file:
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@@
 			)
 		)
-		(property "Footprint" ""
+		(property "Footprint" "Resistor_SMD:R_0805_2012Metric_Pad1.20x1.40mm_HandSolder"
 			(at 217.678 95.25 90)
 			(effects
@@
 		)
 		(property "Description" "Resistor"
+			(at 215.9 95.25 0)
+			(effects
+				(font
+					(size 1.27 1.27)
+				)
+				(hide yes)
+			)
+		)
+		(property "jlcpcb" "C17408"
 			(at 215.9 95.25 0)
 			(effects
@@
 			)
 		)
-		(property "Footprint" ""
+		(property "Footprint" "Resistor_SMD:R_0805_2012Metric_Pad1.20x1.40mm_HandSolder"
 			(at 217.678 113.03 90)
 			(effects
@@
 			(at 215.9 113.03 0)
 			(effects
+				(font
+					(size 1.27 1.27)
+				)
+				(hide yes)
+			)
+		)
+		(property "jlcpcb" "C17408"
+			(at 215.9 113.03 0)
+			(effects

Commit message: mega_shield, re-annotated all components.
Parts:
- U3: footprint (none) -> Package_TO_SOT_SMD:SOT-23-5; jlcpcb (none) -> C7972
- renumbered R3 to R11, R4 to R12, R60 to R13, R59 to R14, R5 to R15, R6 to R16
Changed lines of the file:
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@@
 		(dnp no)
 		(fields_autoplaced yes)
-		(property "Reference" "R3"
+		(property "Reference" "R11"
 			(at 44.45 82.55 90)
 			(effects
@@
 			(project "mega_shield"
 				(path "/554fcf27-dc63-4666-abbc-7481d15942c4/05acfb4b-1f70-4813-b5f6-d6a6759e8a5f"
-					(reference "R3")
+					(reference "R11")
 					(unit 1)
 				)
@@
 		(dnp no)
 		(fields_autoplaced yes)
-		(property "Reference" "R4"
+		(property "Reference" "R12"
 			(at 57.15 82.55 90)
 			(effects
@@
 			(project ""
 				(path "/554fcf27-dc63-4666-abbc-7481d15942c4/05acfb4b-1f70-4813-b5f6-d6a6759e8a5f"
-					(reference "R4")
+					(reference "R12")
 					(unit 1)
 				)
@@
 		(dnp no)
 		(fields_autoplaced yes)
-		(property "Reference" "R60"
+		(property "Reference" "R13"
 			(at 218.44 93.9799 0)
 			(effects
@@
 			(project "mega_shield"
 				(path "/554fcf27-dc63-4666-abbc-7481d15942c4/05acfb4b-1f70-4813-b5f6-d6a6759e8a5f"
-					(reference "R60")
+					(reference "R13")
 					(unit 1)
 				)
@@
 		(dnp no)
 		(fields_autoplaced yes)
-		(property "Reference" "R59"
+		(property "Reference" "R14"
 			(at 218.44 111.7599 0)
 			(effects
@@
 			(project ""
 				(path "/554fcf27-dc63-4666-abbc-7481d15942c4/05acfb4b-1f70-4813-b5f6-d6a6759e8a5f"
-					(reference "R59")
+					(reference "R14")
 					(unit 1)
 				)
@@
 		(dnp no)
 		(fields_autoplaced yes)
-		(property "Reference" "R6"
+		(property "Reference" "R16"
 			(at 231.14 111.7599 0)
 			(effects
@@
 			(project "mega_shield"
 				(path "/554fcf27-dc63-4666-abbc-7481d15942c4/05acfb4b-1f70-4813-b5f6-d6a6759e8a5f"
-					(reference "R6")
+					(reference "R16")
 					(unit 1)
 				)
@@
 			)
 		)
-		(property "Footprint" ""
+		(property "Footprint" "Package_TO_SOT_SMD:SOT-23-5"
 			(at 82.55 88.9 0)
 			(effects
@@
 			)
 		)
+		(property "jlcpcb" "C7972"
+			(at 82.55 88.9 0)
+			(effects
+				(font
+					(size 1.27 1.27)
+				)
+				(hide yes)
+			)
+		)
 		(pin "1"
 		)
@@
 		(dnp no)
 		(fields_autoplaced yes)
-		(property "Reference" "R5"
+		(property "Reference" "R15"
 			(at 231.14 80.0099 0)
 			(effects
@@
 			(project "mega_shield"
 				(path "/554fcf27-dc63-4666-abbc-7481d15942c4/05acfb4b-1f70-4813-b5f6-d6a6759e8a5f"
-					(reference "R5")
+					(reference "R15")
 					(unit 1)
 				)
