File: mega_shield/solenoid_interface.kicad_sch (KiCad schematic)
At the start: 0 parts

Commit message: Imported sheet pins for solenoid interface sheet.
Parts:
- added C41: 10u, symbol Device:C
- added J6: T4140012121-000, T4140012121-000:TE_T4140012121-000, symbol T4140012121-000:T4140012121-000
- added R31: R, symbol Device:R
- added U21: NUP2202, Package_TO_SOT_SMD:SOT-363_SC-70-6, symbol Power_Protection:NUP2202

Commit message: Added sheet labels for channels 1-10 to the solenoid interface sheet. Imported pins.
Other:
- moved on the sheet: R31
Changed lines of the file:
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@@
+		)
+	)
+	(label "SLND_2_OUT"
+		(at 88.9 66.04 0)
+		(effects
+			(font
+				(size 1.27 1.27)
+			)
+			(justify left bottom)
+		)
+	)
+	(hierarchical_label "SLND_6"
+		(shape input)
+		(at 152.4 76.2 0)
+		(effects
+			(font
+				(size 1.27 1.27)
+			)
+			(justify left)
+		)
+	)
+	(hierarchical_label "SLND_9"
+		(shape input)
+		(at 152.4 83.82 0)
+		(effects
+			(font
+				(size 1.27 1.27)
+			)
+			(justify left)
+		)
+	)
+	(hierarchical_label "SLND_2"
+		(shape input)
+		(at 152.4 66.04 0)
+		(effects
+			(font
+				(size 1.27 1.27)
+			)
+			(justify left)
+		)
+	)
+	(hierarchical_label "SLND_8"
+		(shape input)
+		(at 152.4 81.28 0)
+		(effects
+			(font
+				(size 1.27 1.27)
+			)
+			(justify left)
 		)
 	)
@@
 		)
 	)
+	(hierarchical_label "SLND_4"
+		(shape input)
+		(at 152.4 71.12 0)
+		(effects
+			(font
+				(size 1.27 1.27)
+			)
+			(justify left)
+		)
+	)
+	(hierarchical_label "SLND_3"
+		(shape input)
+		(at 152.4 68.58 0)
+		(effects
+			(font
+				(size 1.27 1.27)
+			)
+			(justify left)
+		)
+	)
 	(hierarchical_label "+5V_IN"
 		(shape input)
@@
 		(shape input)
 		(at 154.94 46.99 0)
+		(effects
+			(font
+				(size 1.27 1.27)
+			)
+			(justify left)
+		)
+	)
+	(hierarchical_label "SLND_10"
+		(shape input)
+		(at 152.4 86.36 0)
+		(effects
+			(font
+				(size 1.27 1.27)
+			)
+			(justify left)
+		)
+	)
+	(hierarchical_label "SLND_7"
+		(shape input)
+		(at 152.4 78.74 0)
+		(effects
+			(font
+				(size 1.27 1.27)
+			)
+			(justify left)
+		)
+	)
+	(hierarchical_label "SLND_5"
+		(shape input)
+		(at 152.4 73.66 0)
 		(effects
 			(font
@@
 	(symbol
 		(lib_id "Device:R")
-		(at 152.4 93.98 0)
+		(at 152.4 109.22 0)
 		(unit 1)
 		(exclude_from_sim no)
@@
 		(fields_autoplaced yes)
 		(property "Reference" "R31"
-			(at 154.94 92.7099 0)
+			(at 154.94 107.9499 0)
 			(effects
 				(font
@@
 		)
 		(property "Value" "R"
-			(at 154.94 95.2499 0)
+			(at 154.94 110.4899 0)
 			(effects
 				(font
@@
 		)
 		(property "Footprint" ""
-			(at 150.622 93.98 90)
+			(at 150.622 109.22 90)
 			(effects
 				(font
@@
 		)
 		(property "Datasheet" "~"
-			(at 152.4 93.98 0)
+			(at 152.4 109.22 0)
 			(effects
 				(font
@@
 		)
 		(property "Description" "Resistor"
-			(at 152.4 93.98 0)
-			(effects
-				(font
+			(at 152.4 109.22 0)
+			(effects
+				(font

Commit message: Added JLCPCB number for the ESD protection IC.
Parts:
- U21: jlcpcb (none) -> C4355033
Changed lines of the file:
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@@
+			)
+		)
+		(property "jlcpcb" "C4355033"
+			(at 127 105.41 0)
+			(effects
+				(font
+					(size 1.27 1.27)
+				)
 			)
 		)

Commit message: Added ESD protection circuit for all 10 channels on solenoid interface.
Parts:
- added F13: SMD1812P050TF, symbol Device:Polyfuse
- added LED13: LED_0603_Red, PCM_LED_SMD_AKL:LED_0603_1608Metric, symbol PCM_LED_AKL:LED_0603_Red
- added R33: 2k, symbol Device:R
- added R34, R36, R37, R38, R39, R40, R41, R42, R43: 4k7, symbol Device:R
- added U23, U24, U25, U26: NUP2202, Package_TO_SOT_SMD:SOT-363_SC-70-6, symbol Power_Protection:NUP2202
- R31: value R -> 4k7
Connections:
- net +5V_IN: now also F13.1, LED13.2 (A)
- net GND: now also U21.2, U23.2, U24.2, U25.2, U26.2
- net SLND_1: now also R31.2, U21.6
- net SLND_10: now also R43.2, U26.1
- net SLND_2: now also U21.1, R34.2
- net SLND_3: now also R36.2, U23.6
- net SLND_4: now also R37.2, U23.1
- net SLND_5: now also R38.2, U24.6
- net SLND_6: now also R39.2, U24.1
- net SLND_7: now also R40.2, U25.6
- net SLND_8: now also R41.2, U25.1
- net SLND_9: now also R42.2, U26.6
- net +5V_SOL: now reaches U21.5
- net +5V_SOL: now also F13.2, R33.2, U23.5, U24.5, U25.5, U26.5
- new net: LED13.1 (K), R33.1
Other:
- note added: "Fuse Indicator, turns on led when tripped"
- note added: "Polyfuse: I_Hold: 0.5A I_Trip: 1.0A V_Max: 15V"
- moved on the sheet: J6, R31, U21

Commit message: Added connections and over-current protection for 24v line. Added note on PTC configuration and JLCPCB numbers.
Parts:
- added F14, F15, F16: SMD1812P110TF/33, symbol Device:Polyfuse
- added LED14: LED_0603_Red, PCM_LED_SMD_AKL:LED_0603_1608Metric, symbol PCM_LED_AKL:LED_0603_Red
- added R44: 2k, symbol Device:R
Connections:
- net +24V_IN: now also F14.1, F15.1, F16.1, LED14.2 (A)
- net +5V_SOL: now also C41.1
- net GND: now also C41.2, J6.12
- net SLND_OUT_5: now reaches R38.1
- net SLND_OUT_5: now also J6.10
- net SLND_OUT_7: now reaches R40.1
- net SLND_OUT_7: now also J6.9
- net SLND_OUT_10: now reaches R43.1
- net SLND_OUT_10: now also J6.6
- net SLND_OUT_8: now reaches R41.1
- net SLND_OUT_8: now also J6.8
- net SLND_OUT_2: now reaches R34.1
- net SLND_OUT_2: now also J6.4
- net SLND_OUT_6: now reaches J6.1
- net SLND_OUT_6: now also R39.1
- net +24V_SOL: now reaches J6.11
- net +24V_SOL: now also F14.2, F15.2, F16.2, R44.2
- net SLND_OUT_4: now reaches J6.2
- net SLND_OUT_4: now also R37.1
- net SLND_OUT_3: now reaches J6.3
- net SLND_OUT_3: now also R36.1
- net SLND_OUT_1: now reaches J6.5
- net SLND_OUT_1: now also R31.1
- net SLND_OUT_9: now reaches J6.7
- net SLND_OUT_9: now also R42.1
- new net: LED14.1 (K), R44.1
Other:
- note added: "M12 Connector 12 Pin"
- note added: "Polyfuse: I_Hold: 2.5A I_Trip: 1.0A V_Max: 30V"
- note added: "Solenoid ESD protection"
- moved on the sheet: C41, F13, J6, LED13, R31, R33, R34, R36, R37, R38, R39, R40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

Commit message: Ran the annotation operation on all schematics.
Parts:
- renumbered C41 to C37, F14 to F6, F15 to F7, F16 to F8, F13 to F9, J6 to J7, LED14 to LED6, LED13 to LED7, R44 to R20, R33 to R21, R31 to R22, R34 to R23, R36 to R24, R37 to R25, R38 to R26, R39 to R27, R40 to R28, R41 to R29, R42 to R30, R43 to R31, U21 to U19, U23 to U20, U24 to U21, U25 to U22, U26 to U23
Changed lines of the file:
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@@
 		(dnp no)
 		(fields_autoplaced yes)
-		(property "Reference" "R38"
+		(property "Reference" "R26"
 			(at 245.11 80.01 90)
 			(effects
@@
 			(project "mega_shield"
 				(path "/554fcf27-dc63-4666-abbc-7481d15942c4/2699417b-945f-4287-8f74-1d8b0d60679f"
-					(reference "R38")
+					(reference "R26")
 					(unit 1)
 				)
@@
 		(dnp no)
 		(fields_autoplaced yes)
-		(property "Reference" "R44"
+		(property "Reference" "R20"
 			(at 62.23 67.31 90)
 			(effects
@@
 			(project "mega_shield"
 				(path "/554fcf27-dc63-4666-abbc-7481d15942c4/2699417b-945f-4287-8f74-1d8b0d60679f"
-					(reference "R44")
+					(reference "R20")
 					(unit 1)
 				)
@@
 		(dnp no)
 		(fields_autoplaced yes)
-		(property "Reference" "F14"
+		(property "Reference" "F6"
 			(at 54.61 27.94 90)
 			(effects
@@
 			(project "mega_shield"
 				(path "/554fcf27-dc63-4666-abbc-7481d15942c4/2699417b-945f-4287-8f74-1d8b0d60679f"
-					(reference "F14")
+					(reference "F6")
 					(unit 1)
 				)
@@
 		(dnp no)
 		(fields_autoplaced yes)
-		(property "Reference" "R40"
+		(property "Reference" "R28"
 			(at 245.11 105.41 90)
 			(effects
@@
 			(project "mega_shield"
 				(path "/554fcf27-dc63-4666-abbc-7481d15942c4/2699417b-945f-4287-8f74-1d8b0d60679f"
-					(reference "R40")
+					(reference "R28")
 					(unit 1)
 				)
@@
 		(dnp no)
 		(fields_autoplaced yes)
-		(property "Reference" "F16"
+		(property "Reference" "F8"
 			(at 54.61 53.34 90)
 			(effects
@@
 			(project "mega_shield"
 				(path "/554fcf27-dc63-4666-abbc-7481d15942c4/2699417b-945f-4287-8f74-1d8b0d60679f"
-					(reference "F16")
+					(reference "F8")
 					(unit 1)
 				)
@@
 		(dnp no)
 		(fields_autoplaced yes)
-		(property "Reference" "R43"
+		(property "Reference" "R31"
 			(at 245.11 146.05 90)
 			(effects
@@
 			(project "mega_shield"
 				(path "/554fcf27-dc63-4666-abbc-7481d15942c4/2699417b-945f-4287-8f74-1d8b0d60679f"
-					(reference "R43")
+					(reference "R31")
 					(unit 1)
 				)
@@
 		(dnp no)
 		(fields_autoplaced yes)
-		(property "Reference" "#PWR0143"
+		(property "Reference" "#PWR0117"
 			(at 76.2 116.84 0)
 			(effects
@@
 			(project "mega_shield"
 				(path "/554fcf27-dc63-4666-abbc-7481d15942c4/2699417b-945f-4287-8f74-1d8b0d60679f"
-					(reference "#PWR0143")
+					(reference "#PWR0117")
 					(unit 1)
 				)
@@
 		(dnp no)
 		(fields_autoplaced yes)
-		(property "Reference" "F15"
+		(property "Reference" "F7"
 			(at 54.61 40.64 90)
 			(effects
@@
 			(project "mega_shield"
 				(path "/554fcf27-dc63-4666-abbc-7481d15942c4/2699417b-945f-4287-8f74-1d8b0d60679f"
-					(reference "F15")
+					(reference "F7")
 					(unit 1)
 				)
@@
 		(dnp no)
 		(fields_autoplaced yes)
-		(property "Reference" "R41"
+		(property "Reference" "R29"
 			(at 245.11 120.65 90)
 			(effects
@@
 			(project "mega_shield"
 				(path "/554fcf27-dc63-4666-abbc-7481d15942c4/2699417b-945f-4287-8f74-1d8b0d60679f"
-					(reference "R41")
+					(reference "R29")
 					(unit 1)
 				)
@@
 		(dnp no)
 		(fields_autoplaced yes)
-		(property "Reference" "R34"
+		(property "Reference" "R23"
 			(at 245.11 43.18 90)
 			(effects
@@
 			(project "mega_shield"
 				(path "/554fcf27-dc63-4666-abbc-7481d15942c4/2699417b-945f-4287-8f74-1d8b0d60679f"
-					(reference "R34")
+					(reference "R23")
 					(unit 1)
 				)
@@
 		(on_board yes)
 		(dnp no)
-		(property "Reference" "J6"
+		(property "Reference" "J7"
 			(at 49.53 144.7799 0)
 			(effects
@@
 			(project ""
 				(path "/554fcf27-dc63-4666-abbc-7481d15942c4/2699417b-945f-4287-8f74-1d8b0d60679f"
-					(reference "J6")
+					(reference "J7")
 					(unit 1)
 				)
@@
 		(dnp no)
 		(fields_autoplaced yes)
-		(property "Reference" "R31"
+		(property "Reference" "R22"
 			(at 245.11 27.94 90)
 			(effects
@@
 			(project ""
 				(path "/554fcf27-dc63-4666-abbc-7481d15942c4/2699417b-945f-4287-8f74-1d8b0d60679f"
-					(reference "R31")
+					(reference "R22")
 					(unit 1)
 				)
@@
 		(dnp no)
 		(fields_autoplaced yes)
-		(property "Reference" "LED14"
+		(property "Reference" "LED6"
 			(at 48.26 64.77 0)
 			(effects
@@
 			(project "mega_shield"
 				(path "/554fcf27-dc63-4666-abbc-7481d15942c4/2699417b-945f-4287-8f74-1d8b0d60679f"
-					(reference "LED14")
+					(reference "LED6")
 					(unit 1)
 				)
@@
 		(dnp no)
 		(fields_autoplaced yes)
-		(property "Reference" "F13"
+		(property "Reference" "F9"
 			(at 54.61 93.98 90)
 			(effects
@@
 			(project "mega_shield"
 				(path "/554fcf27-dc63-4666-abbc-7481d15942c4/2699417b-945f-4287-8f74-1d8b0d60679f"
-					(reference "F13")
+					(reference "F9")
 					(unit 1)
 				)
@@
 		(dnp no)
 		(fields_autoplaced yes)
-		(property "Reference" "#PWR0131"
+		(property "Reference" "#PWR0116"
 			(at 63.5 166.37 0)
 			(effects
@@
 			(project "mega_shield"
 				(path "/554fcf27-dc63-4666-abbc-7481d15942c4/2699417b-945f-4287-8f74-1d8b0d60679f"
-					(reference "#PWR0131")
+					(reference "#PWR0116")
 					(unit 1)
 				)
@@
 		(dnp no)
 		(fields_autoplaced yes)
-		(property "Reference" "R42"
+		(property "Reference" "R30"
 			(at 245.11 130.81 90)
 			(effects
@@
 			(project "mega_shield"
 				(path "/554fcf27-dc63-4666-abbc-7481d15942c4/2699417b-945f-4287-8f74-1d8b0d60679f"
-					(reference "R42")
+					(reference "R30")
 					(unit 1)
 				)
@@
 		(on_board yes)
 		(dnp no)
-		(property "Reference" "U24"
+		(property "Reference" "U21"
 			(at 257.7398 85.09 0)
 			(effects
@@
 			(project "mega_shield"
 				(path "/554fcf27-dc63-4666-abbc-7481d15942c4/2699417b-945f-4287-8f74-1d8b0d60679f"
-					(reference "U24")
+					(reference "U21")
 					(unit 1)
 				)
@@
 		(on_board yes)
 		(dnp no)
-		(property "Reference" "U26"
+		(property "Reference" "U23"
 			(at 257.7398 135.89 0)
 			(effects
@@
 			(project "mega_shield"
 				(path "/554fcf27-dc63-4666-abbc-7481d15942c4/2699417b-945f-4287-8f74-1d8b0d60679f"
-					(reference "U26")
+					(reference "U23")
 					(unit 1)
 				)
@@
 		(dnp no)
 		(fields_autoplaced yes)
-		(property "Reference" "LED13"
+		(property "Reference" "LED7"
 			(at 48.26 104.14 0)
 			(effects
@@
 			(project "mega_shield"
 				(path "/554fcf27-dc63-4666-abbc-7481d15942c4/2699417b-945f-4287-8f74-1d8b0d60679f"
-					(reference "LED13")
+					(reference "LED7")
 					(unit 1)
 				)
@@
 		(dnp no)
 		(fields_autoplaced yes)
-		(property "Reference" "R39"
+		(property "Reference" "R27"
 			(at 245.11 95.25 90)
 			(effects
@@
 			(project "mega_shield"
 				(path "/554fcf27-dc63-4666-abbc-7481d15942c4/2699417b-945f-4287-8f74-1d8b0d60679f"
-					(reference "R39")
+					(reference "R27")
 					(unit 1)
 				)
@@
 		(dnp no)
 		(fields_autoplaced yes)
-		(property "Reference" "R37"
+		(property "Reference" "R25"
 			(at 245.11 69.85 90)
 			(effects
@@
 			(project "mega_shield"
 				(path "/554fcf27-dc63-4666-abbc-7481d15942c4/2699417b-945f-4287-8f74-1d8b0d60679f"
-					(reference "R37")
+					(reference "R25")
 					(unit 1)
 				)
@@
 		(dnp no)
 		(fields_autoplaced yes)
-		(property "Reference" "#FLG08"
+		(property "Reference" "#FLG010"
 			(at 69.85 34.925 0)
 			(effects
@@
 			(project "mega_shield"
 				(path "/554fcf27-dc63-4666-abbc-7481d15942c4/2699417b-945f-4287-8f74-1d8b0d60679f"
-					(reference "#FLG08")
+					(reference "#FLG010")
 					(unit 1)
 				)
@@
 		(on_board yes)
 		(dnp no)
-		(property "Reference" "U25"
+		(property "Reference" "U22"
 			(at 257.7398 110.49 0)
 			(effects
@@
 			(project "mega_shield"
 				(path "/554fcf27-dc63-4666-abbc-7481d15942c4/2699417b-945f-4287-8f74-1d8b0d60679f"
-					(reference "U25")
+					(reference "U22")
 					(unit 1)
 				)
@@
 		(dnp no)
 		(fields_autoplaced yes)
-		(property "Reference" "R33"
+		(property "Reference" "R21"
 			(at 62.23 106.68 90)
 			(effects
@@
 			(project "mega_shield"
 				(path "/554fcf27-dc63-4666-abbc-7481d15942c4/2699417b-945f-4287-8f74-1d8b0d60679f"
-					(reference "R33")
+					(reference "R21")
 					(unit 1)
 				)
@@
 		(dnp no)
 		(fields_autoplaced yes)
-		(property "Reference" "C41"
+		(property "Reference" "C37"
 			(at 80.01 105.4099 0)
 			(effects
@@
 			(project ""
 				(path "/554fcf27-dc63-4666-abbc-7481d15942c4/2699417b-945f-4287-8f74-1d8b0d60679f"
-					(reference "C41")
+					(reference "C37")
 					(unit 1)
 				)
@@
 		(on_board yes)
 		(dnp no)
-		(property "Reference" "U21"
+		(property "Reference" "U19"
 			(at 257.7398 33.02 0)
 			(effects
@@
 			(project ""
 				(path "/554fcf27-dc63-4666-abbc-7481d15942c4/2699417b-945f-4287-8f74-1d8b0d60679f"
-					(reference "U21")
+					(reference "U19")
 					(unit 1)
 				)
@@
 		(on_board yes)
 		(dnp no)
-		(property "Reference" "U23"
+		(property "Reference" "U20"
 			(at 257.7398 59.69 0)
 			(effects
@@
 			(project "mega_shield"
 				(path "/554fcf27-dc63-4666-abbc-7481d15942c4/2699417b-945f-4287-8f74-1d8b0d60679f"
-					(reference "U23")
+					(reference "U20")
 					(unit 1)
 				)
@@
 		(dnp no)
 		(fields_autoplaced yes)
-		(property "Reference" "#FLG06"
+		(property "Reference" "#FLG011"
 			(at 69.85 98.425 0)
 			(effects
@@
 			(project "mega_shield"
 				(path "/554fcf27-dc63-4666-abbc-7481d15942c4/2699417b-945f-4287-8f74-1d8b0d60679f"
-					(reference "#FLG06")
+					(reference "#FLG011")
 					(unit 1)
 				)
@@
 		(dnp no)
 		(fields_autoplaced yes)
-		(property "Reference" "R36"
+		(property "Reference" "R24"
 			(at 245.11 54.61 90)
 			(effects
@@
 			(project "mega_shield"
 				(path "/554fcf27-dc63-4666-abbc-7481d15942c4/2699417b-945f-4287-8f74-1d8b0d60679f"
-					(reference "R36")
+					(reference "R24")
 					(unit 1)
 				)
@@
 		(dnp no)
 		(fields_autoplaced yes)
-		(property "Reference" "#PWR0130"
+		(property "Reference" "#PWR0118"
 			(at 276.86 161.29 0)
 			(effects
@@
 			(project ""
 				(path "/554fcf27-dc63-4666-abbc-7481d15942c4/2699417b-945f-4287-8f74-1d8b0d60679f"
-					(reference "#PWR0130")
-					(unit 1)
-				)
+					(reference "#PWR0118")
+					(unit 1)
+				)

Commit message: Set the JLCPCB number and footprints for all components minus fuses and connectors.
Parts:
- C37: footprint (none) -> Capacitor_SMD:C_0201_0603Metric; jlcpcb (none) -> C96446
- F6, F7, F8: footprint (none) -> Fuse:Fuse_1812_4532Metric
- F9: footprint (none) -> Fuse:Fuse_1812_4532Metric; jlcpcb (none) -> C12558
- R20, R21: footprint (none) -> Resistor_SMD:R_0201_0603Metric; jlcpcb (none) -> C22975
- R22, R23, R24, R25, R26, R27, R28, R29, R30, R31: footprint (none) -> Resistor_SMD:R_0201_0603Metric; jlcpcb (none) -> C23162
Changed lines of the file:
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@@
 			)
 		)
-		(property "Footprint" ""
+		(property "Footprint" "Resistor_SMD:R_0201_0603Metric"
 			(at 245.11 88.138 90)
 			(effects
@@
 				)
 				(hide yes)
+			)
+		)
+		(property "jlcpcb" "C23162"
+			(at 245.11 86.36 0)
+			(effects
+				(font
+					(size 1.27 1.27)
+				)
 			)
 		)
@@
 			)
 		)
-		(property "Footprint" ""
+		(property "Footprint" "Resistor_SMD:R_0201_0603Metric"
 			(at 62.23 75.438 90)
 			(effects
@@
 				)
 				(hide yes)
+			)
+		)
+		(property "jlcpcb" "C22975"
+			(at 62.23 73.66 0)
+			(effects
+				(font
+					(size 1.27 1.27)
+				)
 			)
 		)
@@
 			)
 		)
-		(property "Footprint" ""
+		(property "Footprint" "Fuse:Fuse_1812_4532Metric"
 			(at 59.69 35.56 0)
 			(effects
@@
 			)
 		)
-		(property "Footprint" ""
+		(property "Footprint" "Resistor_SMD:R_0201_0603Metric"
 			(at 245.11 113.538 90)
 			(effects
@@
 				)
 				(hide yes)
+			)
+		)
+		(property "jlcpcb" "C23162"
+			(at 245.11 111.76 0)
+			(effects
+				(font
+					(size 1.27 1.27)
+				)
 			)
 		)
@@
 			)
 		)
-		(property "Footprint" ""
+		(property "Footprint" "Fuse:Fuse_1812_4532Metric"
 			(at 59.69 60.96 0)
 			(effects
@@
 			)
 		)
-		(property "Footprint" ""
+		(property "Footprint" "Resistor_SMD:R_0201_0603Metric"
 			(at 245.11 154.178 90)
 			(effects
@@
 				)
 				(hide yes)
+			)
+		)
+		(property "jlcpcb" "C23162"
+			(at 245.11 152.4 0)
+			(effects
+				(font
+					(size 1.27 1.27)
+				)
 			)
 		)
@@
 			)
 		)
-		(property "Footprint" ""
+		(property "Footprint" "Fuse:Fuse_1812_4532Metric"
 			(at 59.69 48.26 0)
 			(effects
@@
 			)
 		)
-		(property "Footprint" ""
+		(property "Footprint" "Resistor_SMD:R_0201_0603Metric"
 			(at 245.11 128.778 90)
 			(effects
@@
 				)
 				(hide yes)
+			)
+		)
+		(property "jlcpcb" "C23162"
+			(at 245.11 127 0)
+			(effects
+				(font
+					(size 1.27 1.27)
+				)
 			)
 		)
@@
 			)
 		)
-		(property "Footprint" ""
+		(property "Footprint" "Resistor_SMD:R_0201_0603Metric"
 			(at 245.11 51.308 90)
 			(effects
@@
 				)
 				(hide yes)
+			)
+		)
+		(property "jlcpcb" "C23162"
+			(at 245.11 49.53 0)
+			(effects
+				(font
+					(size 1.27 1.27)
+				)
 			)
 		)
@@
 			)
 		)
-		(property "Footprint" ""
+		(property "Footprint" "Resistor_SMD:R_0201_0603Metric"
 			(at 245.11 36.068 90)
 			(effects
@@
 				)
 				(hide yes)
+			)
+		)
+		(property "jlcpcb" "C23162"
+			(at 245.11 34.29 0)
+			(effects
+				(font
+					(size 1.27 1.27)
+				)
 			)
 		)
@@
 			)
 		)
-		(property "Footprint" ""
+		(property "Footprint" "Fuse:Fuse_1812_4532Metric"
 			(at 59.69 99.06 0)
 			(effects
@@
 				)
 				(hide yes)
+			)
+		)
+		(property "jlcpcb" "C12558"
+			(at 54.61 100.33 0)
+			(effects
+				(font
+					(size 1.27 1.27)
+				)
 			)
 		)
@@
 			)
 		)
-		(property "Footprint" ""
+		(property "Footprint" "Resistor_SMD:R_0201_0603Metric"
 			(at 245.11 138.938 90)
 			(effects
@@
 				)
 				(hide yes)
+			)
+		)
+		(property "jlcpcb" "C23162"
+			(at 245.11 137.16 0)
+			(effects
+				(font
+					(size 1.27 1.27)
+				)
 			)
 		)
@@
 			)
 		)
-		(property "Footprint" ""
+		(property "Footprint" "Resistor_SMD:R_0201_0603Metric"
 			(at 245.11 103.378 90)
 			(effects
@@
 				)
 				(hide yes)
+			)
+		)
+		(property "jlcpcb" "C23162"
+			(at 245.11 101.6 0)
+			(effects
+				(font
+					(size 1.27 1.27)
+				)
 			)
 		)
@@
 			)
 		)
-		(property "Footprint" ""
+		(property "Footprint" "Resistor_SMD:R_0201_0603Metric"
 			(at 245.11 77.978 90)
 			(effects
@@
 				)
 				(hide yes)
+			)
+		)
+		(property "jlcpcb" "C23162"
+			(at 245.11 76.2 0)
+			(effects
+				(font
+					(size 1.27 1.27)
+				)
 			)
 		)
@@
 			)
 		)
-		(property "Footprint" ""
+		(property "Footprint" "Resistor_SMD:R_0201_0603Metric"
 			(at 62.23 114.808 90)
 			(effects
@@
 				)
 				(hide yes)
+			)
+		)
+		(property "jlcpcb" "C22975"
+			(at 62.23 113.03 0)
+			(effects
+				(font
+					(size 1.27 1.27)
+				)
 			)
 		)
@@
 			)
 		)
-		(property "Footprint" ""
+		(property "Footprint" "Capacitor_SMD:C_0201_0603Metric"
 			(at 77.1652 110.49 0)
 			(effects
@@
 				)
 				(hide yes)
+			)
+		)
+		(property "jlcpcb" "C96446"
+			(at 76.2 106.68 0)
+			(effects
+				(font
+					(size 1.27 1.27)
+				)
 			)
 		)
@@
 			)
 		)
-		(property "Footprint" ""
+		(property "Footprint" "Resistor_SMD:R_0201_0603Metric"
 			(at 245.11 62.738 90)
 			(effects
@@
 			)
 		)
+		(property "jlcpcb" "C23162"
+			(at 245.11 60.96 0)
+			(effects
+				(font
+					(size 1.27 1.27)
+				)
+			)
+		)

Commit message: fixed footprint path of the T4140012121-000 connectors.
Parts:
- J7: footprint T4140012121-000:TE_T4140012121-000 -> footprints:TE_T4140012121-000
Changed lines of the file:
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@@
 			)
 		)
-		(property "Footprint" "T4140012121-000:TE_T4140012121-000"
+		(property "Footprint" "footprints:TE_T4140012121-000"
 			(at 55.88 144.78 0)
 			(effects
@@
 			)
 		)
+		(property "Purpose" ""
+			(at 55.88 144.78 0)
+			(effects
+				(font
+					(size 1.27 1.27)
+				)
+			)
+		)
