File: mega_shield/solenoid_interface.kicad_sch (KiCad schematic)
At the start: 25 parts, among them J20 T4140012121-000, U19 NUP2202, U20 NUP2202, U21 NUP2202, U22 NUP2202, U23 NUP2202

Commit message: Set the JLCPCB number for the M12P12 connector
Parts:
- J20: jlcpcb (none) -> C7423418
Changed lines of the file:
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@@
+			)
+		)
+		(property "jlcpcb" "C7423418"
+			(at 55.88 144.78 0)
+			(effects
+				(font
+					(size 1.27 1.27)
+				)
 			)
 		)

Commit message: consolidated indicator leds to use all 0603 footprint and lower cost part. Changed the jlcpcb numbers.
Parts:
- LED6, LED7: value LED_0603_Red -> KT-0603R; footprint PCM_LED_SMD_AKL:LED_0603_1608Metric -> PCM_LED_SMD_AKL:LED_0201_0603Metric; jlcpcb C94743 -> C2286
Changed lines of the file:
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@@
 			)
 		)
-		(property "Value" "LED_0603_Red"
+		(property "Value" "KT-0603R"
 			(at 48.26 67.31 0)
 			(effects
@@
 			)
 		)
-		(property "Footprint" "PCM_LED_SMD_AKL:LED_0603_1608Metric"
+		(property "Footprint" "PCM_LED_SMD_AKL:LED_0201_0603Metric"
 			(at 48.26 73.66 0)
 			(effects
@@
 			)
 		)
-		(property "jlcpcb" "C94743"
+		(property "jlcpcb" "C2286"
 			(at 48.26 73.66 0)
 			(effects
@@
 			)
 		)
-		(property "Value" "LED_0603_Red"
+		(property "Value" "KT-0603R"
 			(at 48.26 106.68 0)
 			(effects
@@
 			)
 		)
-		(property "Footprint" "PCM_LED_SMD_AKL:LED_0603_1608Metric"
+		(property "Footprint" "PCM_LED_SMD_AKL:LED_0201_0603Metric"
 			(at 48.26 113.03 0)
 			(effects
@@
 			)
 		)
-		(property "jlcpcb" "C94743"
+		(property "jlcpcb" "C2286"
 			(at 48.26 113.03 0)
 			(effects

Commit message: re-annotating for entire schematic completed.
Parts:
- renumbered C37 to C17, J20 to J7, R20 to R10, R21 to R11, R22 to R12, R23 to R13, R24 to R14, R25 to R15, R26 to R16, R27 to R17, R28 to R18, R29 to R19, R30 to R20, R31 to R21, U20 to U10, U21 to U11, U22 to U12, U23 to U13, U19 to U9
Changed lines of the file:
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@@
 		(dnp no)
 		(fields_autoplaced yes)
-		(property "Reference" "R26"
+		(property "Reference" "R16"
 			(at 245.11 80.01 90)
 			(effects
@@
 			(project "mega_shield"
 				(path "/554fcf27-dc63-4666-abbc-7481d15942c4/2699417b-945f-4287-8f74-1d8b0d60679f"
-					(reference "R26")
+					(reference "R16")
 					(unit 1)
 				)
@@
 		(dnp no)
 		(fields_autoplaced yes)
-		(property "Reference" "R20"
+		(property "Reference" "R10"
 			(at 62.23 67.31 90)
 			(effects
@@
 			(project "mega_shield"
 				(path "/554fcf27-dc63-4666-abbc-7481d15942c4/2699417b-945f-4287-8f74-1d8b0d60679f"
-					(reference "R20")
+					(reference "R10")
 					(unit 1)
 				)
@@
 		(dnp no)
 		(fields_autoplaced yes)
-		(property "Reference" "R28"
+		(property "Reference" "R18"
 			(at 245.11 105.41 90)
 			(effects
@@
 			(project "mega_shield"
 				(path "/554fcf27-dc63-4666-abbc-7481d15942c4/2699417b-945f-4287-8f74-1d8b0d60679f"
-					(reference "R28")
+					(reference "R18")
 					(unit 1)
 				)
@@
 		(on_board yes)
 		(dnp no)
-		(property "Reference" "J20"
+		(property "Reference" "J7"
 			(at 49.53 144.7799 0)
 			(effects
@@
 			(project ""
 				(path "/554fcf27-dc63-4666-abbc-7481d15942c4/2699417b-945f-4287-8f74-1d8b0d60679f"
-					(reference "J20")
+					(reference "J7")
 					(unit 1)
 				)
@@
 		(dnp no)
 		(fields_autoplaced yes)
-		(property "Reference" "R31"
+		(property "Reference" "R21"
 			(at 245.11 146.05 90)
 			(effects
@@
 			(project "mega_shield"
 				(path "/554fcf27-dc63-4666-abbc-7481d15942c4/2699417b-945f-4287-8f74-1d8b0d60679f"
-					(reference "R31")
+					(reference "R21")
 					(unit 1)
 				)
@@
 		(dnp no)
 		(fields_autoplaced yes)
-		(property "Reference" "#PWR0117"
+		(property "Reference" "#PWR078"
 			(at 76.2 116.84 0)
 			(effects
@@
 			(project "mega_shield"
 				(path "/554fcf27-dc63-4666-abbc-7481d15942c4/2699417b-945f-4287-8f74-1d8b0d60679f"
-					(reference "#PWR0117")
+					(reference "#PWR078")
 					(unit 1)
 				)
@@
 		(dnp no)
 		(fields_autoplaced yes)
-		(property "Reference" "R29"
+		(property "Reference" "R19"
 			(at 245.11 120.65 90)
 			(effects
@@
 			(project "mega_shield"
 				(path "/554fcf27-dc63-4666-abbc-7481d15942c4/2699417b-945f-4287-8f74-1d8b0d60679f"
-					(reference "R29")
+					(reference "R19")
 					(unit 1)
 				)
@@
 		(dnp no)
 		(fields_autoplaced yes)
-		(property "Reference" "R23"
+		(property "Reference" "R13"
 			(at 245.11 43.18 90)
 			(effects
@@
 			(project "mega_shield"
 				(path "/554fcf27-dc63-4666-abbc-7481d15942c4/2699417b-945f-4287-8f74-1d8b0d60679f"
-					(reference "R23")
+					(reference "R13")
 					(unit 1)
 				)
@@
 		(dnp no)
 		(fields_autoplaced yes)
-		(property "Reference" "R22"
+		(property "Reference" "R12"
 			(at 245.11 27.94 90)
 			(effects
@@
 			(project ""
 				(path "/554fcf27-dc63-4666-abbc-7481d15942c4/2699417b-945f-4287-8f74-1d8b0d60679f"
-					(reference "R22")
+					(reference "R12")
 					(unit 1)
 				)
@@
 		(dnp no)
 		(fields_autoplaced yes)
-		(property "Reference" "#PWR0116"
+		(property "Reference" "#PWR077"
 			(at 63.5 166.37 0)
 			(effects
@@
 			(project "mega_shield"
 				(path "/554fcf27-dc63-4666-abbc-7481d15942c4/2699417b-945f-4287-8f74-1d8b0d60679f"
-					(reference "#PWR0116")
+					(reference "#PWR077")
 					(unit 1)
 				)
@@
 		(dnp no)
 		(fields_autoplaced yes)
-		(property "Reference" "R30"
+		(property "Reference" "R20"
 			(at 245.11 130.81 90)
 			(effects
@@
 			(project "mega_shield"
 				(path "/554fcf27-dc63-4666-abbc-7481d15942c4/2699417b-945f-4287-8f74-1d8b0d60679f"
-					(reference "R30")
+					(reference "R20")
 					(unit 1)
 				)
@@
 		(on_board yes)
 		(dnp no)
-		(property "Reference" "U21"
+		(property "Reference" "U11"
 			(at 257.7398 85.09 0)
 			(effects
@@
 			(project "mega_shield"
 				(path "/554fcf27-dc63-4666-abbc-7481d15942c4/2699417b-945f-4287-8f74-1d8b0d60679f"
-					(reference "U21")
+					(reference "U11")
 					(unit 1)
 				)
@@
 		(on_board yes)
 		(dnp no)
-		(property "Reference" "U23"
+		(property "Reference" "U13"
 			(at 257.7398 135.89 0)
 			(effects
@@
 			(project "mega_shield"
 				(path "/554fcf27-dc63-4666-abbc-7481d15942c4/2699417b-945f-4287-8f74-1d8b0d60679f"
-					(reference "U23")
+					(reference "U13")
 					(unit 1)
 				)
@@
 		(dnp no)
 		(fields_autoplaced yes)
-		(property "Reference" "R27"
+		(property "Reference" "R17"
 			(at 245.11 95.25 90)
 			(effects
@@
 			(project "mega_shield"
 				(path "/554fcf27-dc63-4666-abbc-7481d15942c4/2699417b-945f-4287-8f74-1d8b0d60679f"
-					(reference "R27")
+					(reference "R17")
 					(unit 1)
 				)
@@
 		(dnp no)
 		(fields_autoplaced yes)
-		(property "Reference" "R25"
+		(property "Reference" "R15"
 			(at 245.11 69.85 90)
 			(effects
@@
 			(project "mega_shield"
 				(path "/554fcf27-dc63-4666-abbc-7481d15942c4/2699417b-945f-4287-8f74-1d8b0d60679f"
-					(reference "R25")
+					(reference "R15")
 					(unit 1)
 				)
@@
 		(dnp no)
 		(fields_autoplaced yes)
-		(property "Reference" "#FLG010"
+		(property "Reference" "#FLG09"
 			(at 69.85 34.925 0)
 			(effects
@@
 			(project "mega_shield"
 				(path "/554fcf27-dc63-4666-abbc-7481d15942c4/2699417b-945f-4287-8f74-1d8b0d60679f"
-					(reference "#FLG010")
+					(reference "#FLG09")
 					(unit 1)
 				)
@@
 		(on_board yes)
 		(dnp no)
-		(property "Reference" "U22"
+		(property "Reference" "U12"
 			(at 257.7398 110.49 0)
 			(effects
@@
 			(project "mega_shield"
 				(path "/554fcf27-dc63-4666-abbc-7481d15942c4/2699417b-945f-4287-8f74-1d8b0d60679f"
-					(reference "U22")
+					(reference "U12")
 					(unit 1)
 				)
@@
 		(dnp no)
 		(fields_autoplaced yes)
-		(property "Reference" "R21"
+		(property "Reference" "R11"
 			(at 62.23 106.68 90)
 			(effects
@@
 			(project "mega_shield"
 				(path "/554fcf27-dc63-4666-abbc-7481d15942c4/2699417b-945f-4287-8f74-1d8b0d60679f"
-					(reference "R21")
+					(reference "R11")
 					(unit 1)
 				)
@@
 		(dnp no)
 		(fields_autoplaced yes)
-		(property "Reference" "C37"
+		(property "Reference" "C17"
 			(at 80.01 105.4099 0)
 			(effects
@@
 			(project ""
 				(path "/554fcf27-dc63-4666-abbc-7481d15942c4/2699417b-945f-4287-8f74-1d8b0d60679f"
-					(reference "C37")
+					(reference "C17")
 					(unit 1)
 				)
@@
 		(on_board yes)
 		(dnp no)
-		(property "Reference" "U19"
+		(property "Reference" "U9"
 			(at 257.7398 33.02 0)
 			(effects
@@
 			(project ""
 				(path "/554fcf27-dc63-4666-abbc-7481d15942c4/2699417b-945f-4287-8f74-1d8b0d60679f"
-					(reference "U19")
+					(reference "U9")
 					(unit 1)
 				)
@@
 		(on_board yes)
 		(dnp no)
-		(property "Reference" "U20"
+		(property "Reference" "U10"
 			(at 257.7398 59.69 0)
 			(effects
@@
 			(project "mega_shield"
 				(path "/554fcf27-dc63-4666-abbc-7481d15942c4/2699417b-945f-4287-8f74-1d8b0d60679f"
-					(reference "U20")
+					(reference "U10")
 					(unit 1)
 				)
@@
 		(dnp no)
 		(fields_autoplaced yes)
-		(property "Reference" "#FLG011"
+		(property "Reference" "#FLG010"
 			(at 69.85 98.425 0)
 			(effects
@@
 			(project "mega_shield"
 				(path "/554fcf27-dc63-4666-abbc-7481d15942c4/2699417b-945f-4287-8f74-1d8b0d60679f"
-					(reference "#FLG011")
+					(reference "#FLG010")
 					(unit 1)
 				)
@@
 		(dnp no)
 		(fields_autoplaced yes)
-		(property "Reference" "R24"
+		(property "Reference" "R14"
 			(at 245.11 54.61 90)
 			(effects
@@
 			(project "mega_shield"
 				(path "/554fcf27-dc63-4666-abbc-7481d15942c4/2699417b-945f-4287-8f74-1d8b0d60679f"
-					(reference "R24")
+					(reference "R14")
 					(unit 1)
 				)
@@
 		(dnp no)
 		(fields_autoplaced yes)
-		(property "Reference" "#PWR0118"
+		(property "Reference" "#PWR079"
 			(at 276.86 161.29 0)
 			(effects
@@
 			(project ""
 				(path "/554fcf27-dc63-4666-abbc-7481d15942c4/2699417b-945f-4287-8f74-1d8b0d60679f"
-					(reference "#PWR0118")
-					(unit 1)
-				)
+					(reference "#PWR079")
+					(unit 1)
+				)

Commit message: mega_shield, changed footprint for the led to built in 0603(IMPRL)/1608(Metric)
Parts:
- LED6, LED7: footprint PCM_LED_SMD_AKL:LED_0201_0603Metric -> LED_SMD:LED_0603_1608Metric_Pad1.05x0.95mm_HandSolder
Changed lines of the file:
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@@
 			)
 		)
-		(property "Footprint" "PCM_LED_SMD_AKL:LED_0201_0603Metric"
+		(property "Footprint" "LED_SMD:LED_0603_1608Metric_Pad1.05x0.95mm_HandSolder"
 			(at 48.26 73.66 0)
 			(effects
@@
 			)
 		)
-		(property "Footprint" "PCM_LED_SMD_AKL:LED_0201_0603Metric"
+		(property "Footprint" "LED_SMD:LED_0603_1608Metric_Pad1.05x0.95mm_HandSolder"
 			(at 48.26 113.03 0)
 			(effects

Commit message: mega_shield, Changed out all caps where needed for in-stock and lower cost parts.
+ Changed out for parts with higher stock.
+ Changed out for 0805 sized components.
+ Changed out for higher voltage.
+ Removed 22uF SMD caps for lower cost 10uF caps in parallel.
+ Updated diode footprint to SOD-123F

BOM cost reduced, and reliability improved.
Parts:
- C17: value 10u -> 10u/50V; footprint Capacitor_SMD:C_0201_0603Metric -> Capacitor_SMD:C_0805_2012Metric_Pad1.18x1.45mm_HandSolder; jlcpcb C96446 -> C440198
Changed lines of the file:
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@@
 			)
 		)
-		(property "Value" "10u"
+		(property "Value" "10u/50V"
 			(at 80.01 107.9499 0)
 			(effects
@@
 			)
 		)
-		(property "Footprint" "Capacitor_SMD:C_0201_0603Metric"
+		(property "Footprint" "Capacitor_SMD:C_0805_2012Metric_Pad1.18x1.45mm_HandSolder"
 			(at 77.1652 110.49 0)
 			(effects
@@
 			)
 		)
-		(property "jlcpcb" "C96446"
+		(property "jlcpcb" "C440198"
 			(at 76.2 106.68 0)
 			(effects

Commit message: mega_shield, updated multiple resistors and added comments.
+ Updated optoisolator resistor value --> 15k for better protection.
+ Changed all resistors to 0805 footprints
+ Swapped out expensive values to standardized E24/E96.
+ Updated jlcpcb numbers for all resistors.
Parts:
- R10, R11: footprint Resistor_SMD:R_0201_0603Metric -> Resistor_SMD:R_0805_2012Metric_Pad1.20x1.40mm_HandSolder; jlcpcb C22975 -> C17604
- R12, R13, R14, R15, R16, R17, R18, R19, R20, R21: footprint Resistor_SMD:R_0201_0603Metric -> Resistor_SMD:R_0805_2012Metric_Pad1.20x1.40mm_HandSolder; jlcpcb C23162 -> C17673
Changed lines of the file:
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@@
 			)
 		)
-		(property "Footprint" "Resistor_SMD:R_0201_0603Metric"
+		(property "Footprint" "Resistor_SMD:R_0805_2012Metric_Pad1.20x1.40mm_HandSolder"
 			(at 245.11 88.138 90)
 			(effects
@@
 			)
 		)
-		(property "jlcpcb" "C23162"
+		(property "jlcpcb" "C17673"
 			(at 245.11 86.36 0)
 			(effects
@@
 			)
 		)
-		(property "Footprint" "Resistor_SMD:R_0201_0603Metric"
+		(property "Footprint" "Resistor_SMD:R_0805_2012Metric_Pad1.20x1.40mm_HandSolder"
 			(at 62.23 75.438 90)
 			(effects
@@
 			)
 		)
-		(property "jlcpcb" "C22975"
+		(property "jlcpcb" "C17604"
 			(at 62.23 73.66 0)
 			(effects
@@
 			)
 		)
-		(property "Footprint" "Resistor_SMD:R_0201_0603Metric"
+		(property "Footprint" "Resistor_SMD:R_0805_2012Metric_Pad1.20x1.40mm_HandSolder"
 			(at 245.11 113.538 90)
 			(effects
@@
 			)
 		)
-		(property "jlcpcb" "C23162"
+		(property "jlcpcb" "C17673"
 			(at 245.11 111.76 0)
 			(effects
@@
 			)
 		)
-		(property "Footprint" "Resistor_SMD:R_0201_0603Metric"
+		(property "Footprint" "Resistor_SMD:R_0805_2012Metric_Pad1.20x1.40mm_HandSolder"
 			(at 245.11 154.178 90)
 			(effects
@@
 			)
 		)
-		(property "jlcpcb" "C23162"
+		(property "jlcpcb" "C17673"
 			(at 245.11 152.4 0)
 			(effects
@@
 			)
 		)
-		(property "Footprint" "Resistor_SMD:R_0201_0603Metric"
+		(property "Footprint" "Resistor_SMD:R_0805_2012Metric_Pad1.20x1.40mm_HandSolder"
 			(at 245.11 128.778 90)
 			(effects
@@
 			)
 		)
-		(property "jlcpcb" "C23162"
+		(property "jlcpcb" "C17673"
 			(at 245.11 127 0)
 			(effects
@@
 			)
 		)
-		(property "Footprint" "Resistor_SMD:R_0201_0603Metric"
+		(property "Footprint" "Resistor_SMD:R_0805_2012Metric_Pad1.20x1.40mm_HandSolder"
 			(at 245.11 51.308 90)
 			(effects
@@
 			)
 		)
-		(property "jlcpcb" "C23162"
+		(property "jlcpcb" "C17673"
 			(at 245.11 49.53 0)
 			(effects
@@
 			)
 		)
-		(property "Footprint" "Resistor_SMD:R_0201_0603Metric"
+		(property "Footprint" "Resistor_SMD:R_0805_2012Metric_Pad1.20x1.40mm_HandSolder"
 			(at 245.11 36.068 90)
 			(effects
@@
 			)
 		)
-		(property "jlcpcb" "C23162"
+		(property "jlcpcb" "C17673"
 			(at 245.11 34.29 0)
 			(effects
@@
 			)
 		)
-		(property "Footprint" "Resistor_SMD:R_0201_0603Metric"
+		(property "Footprint" "Resistor_SMD:R_0805_2012Metric_Pad1.20x1.40mm_HandSolder"
 			(at 245.11 138.938 90)
 			(effects
@@
 			)
 		)
-		(property "jlcpcb" "C23162"
+		(property "jlcpcb" "C17673"
 			(at 245.11 137.16 0)
 			(effects
@@
 			)
 		)
-		(property "Footprint" "Resistor_SMD:R_0201_0603Metric"
+		(property "Footprint" "Resistor_SMD:R_0805_2012Metric_Pad1.20x1.40mm_HandSolder"
 			(at 245.11 103.378 90)
 			(effects
@@
 			)
 		)
-		(property "jlcpcb" "C23162"
+		(property "jlcpcb" "C17673"
 			(at 245.11 101.6 0)
 			(effects
@@
 			)
 		)
-		(property "Footprint" "Resistor_SMD:R_0201_0603Metric"
+		(property "Footprint" "Resistor_SMD:R_0805_2012Metric_Pad1.20x1.40mm_HandSolder"
 			(at 245.11 77.978 90)
 			(effects
@@
 			)
 		)
-		(property "jlcpcb" "C23162"
+		(property "jlcpcb" "C17673"
 			(at 245.11 76.2 0)
 			(effects
@@
 			)
 		)
-		(property "Footprint" "Resistor_SMD:R_0201_0603Metric"
+		(property "Footprint" "Resistor_SMD:R_0805_2012Metric_Pad1.20x1.40mm_HandSolder"
 			(at 62.23 114.808 90)
 			(effects
@@
 			)
 		)
-		(property "jlcpcb" "C22975"
+		(property "jlcpcb" "C17604"
 			(at 62.23 113.03 0)
 			(effects
@@
 			)
 		)
-		(property "Footprint" "Resistor_SMD:R_0201_0603Metric"
+		(property "Footprint" "Resistor_SMD:R_0805_2012Metric_Pad1.20x1.40mm_HandSolder"
 			(at 245.11 62.738 90)
 			(effects
@@
 			)
 		)
-		(property "jlcpcb" "C23162"
+		(property "jlcpcb" "C17673"
 			(at 245.11 60.96 0)
 			(effects
