File: mega_shield/solenoid_interface.kicad_sch (KiCad schematic)
At the start: 25 parts, among them J7 T4141012121-000, U10 NUP2202, U11 NUP2202, U12 NUP2202, U13 NUP2202, U9 NUP2202

Commit message: Automatic project files update
Parts:
- J7: MANUFACTURER TE Connectivity -> (none)
Changed lines of the file:
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@@
 			)
 		)
-		(property "MANUFACTURER" "TE Connectivity"
+		(property "Manufacturer" "TE Connectivity"
 			(at 53.34 144.78 0)
 			(hide yes)
