File: mega_shield/power_interface.kicad_sch (KiCad schematic)
At the start: 2 parts, among them J11 Screw_Terminal_01x02, J18 Screw_Terminal_01x02

Commit message: Added fuse and power flags to the +5V and +24v lines.
Parts:
- removed J11, J18: Screw_Terminal_01x02, symbol Connector:Screw_Terminal_01x02
- added F1, F3: Fuse, symbol Device:Fuse
- added J19, J20: 1757242, 1757242:PHOENIX_1757242, symbol TERM_BLOCK_HDR_2POS_5.08MM:1757242
Connections:
- net +24V_EXTERN: now also J20.01
- net +5V_EXTERN: now also J19.01
- net GND: now also J19.02, J20.02

Commit message: Added the basic over-voltage & over-current protection to both power lines(5v/24v)
Parts:
- added D1, D2: 5.6V, symbol Device:D_Zener
- F1, F3: value Fuse -> 2.5A
Connections:
- net +24V_EXTERN: now also F3.1
- net +24V_OUT: now also F3.2, D2.1 (K)
- net +5V_EXTERN: now also F1.1
- net +5V_OUT: now also F1.2, D1.1 (K)
- net GND: now also D1.2 (A), D2.2 (A)
Other:
- note added: "24V Over-Voltage & Over-Current Protection"
- note added: "5V Over-Voltage & Over-Current Protection"
- moved on the sheet: F1, J19

Commit message: Ran the annotation operation on all schematics.
Parts:
- renumbered F1 to F10, F3 to F11, J19 to J14, J20 to J15
Changed lines of the file:
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@@
 		(dnp no)
 		(fields_autoplaced yes)
-		(property "Reference" "#FLG010"
+		(property "Reference" "#FLG012"
 			(at 95.25 31.115 0)
 			(effects
@@
 			(project "mega_shield"
 				(path "/554fcf27-dc63-4666-abbc-7481d15942c4/79aa91ed-20a6-424f-83a6-c5f215a1df0b"
-					(reference "#FLG010")
+					(reference "#FLG012")
 					(unit 1)
 				)
@@
 		(dnp no)
 		(fields_autoplaced yes)
-		(property "Reference" "F1"
+		(property "Reference" "F10"
 			(at 83.82 27.94 90)
 			(effects
@@
 			(project ""
 				(path "/554fcf27-dc63-4666-abbc-7481d15942c4/79aa91ed-20a6-424f-83a6-c5f215a1df0b"
-					(reference "F1")
+					(reference "F10")
 					(unit 1)
 				)
@@
 		(dnp no)
 		(fields_autoplaced yes)
-		(property "Reference" "#PWR052"
+		(property "Reference" "#PWR0139"
 			(at 90.17 53.34 0)
 			(effects
@@
 			(project "mega_shield"
 				(path "/554fcf27-dc63-4666-abbc-7481d15942c4/79aa91ed-20a6-424f-83a6-c5f215a1df0b"
-					(reference "#PWR052")
+					(reference "#PWR0139")
 					(unit 1)
 				)
@@
 		(dnp no)
 		(fields_autoplaced yes)
-		(property "Reference" "#FLG012"
+		(property "Reference" "#FLG013"
 			(at 95.25 81.915 0)
 			(effects
@@
 			(project "mega_shield"
 				(path "/554fcf27-dc63-4666-abbc-7481d15942c4/79aa91ed-20a6-424f-83a6-c5f215a1df0b"
-					(reference "#FLG012")
+					(reference "#FLG013")
 					(unit 1)
 				)
@@
 		(dnp no)
 		(fields_autoplaced yes)
-		(property "Reference" "#PWR045"
+		(property "Reference" "#PWR0137"
 			(at 52.07 46.99 0)
 			(effects
@@
 			(project ""
 				(path "/554fcf27-dc63-4666-abbc-7481d15942c4/79aa91ed-20a6-424f-83a6-c5f215a1df0b"
-					(reference "#PWR045")
+					(reference "#PWR0137")
 					(unit 1)
 				)
@@
 		(dnp no)
 		(fields_autoplaced yes)
-		(property "Reference" "#PWR053"
+		(property "Reference" "#PWR0140"
 			(at 90.17 104.14 0)
 			(effects
@@
 			(project "mega_shield"
 				(path "/554fcf27-dc63-4666-abbc-7481d15942c4/79aa91ed-20a6-424f-83a6-c5f215a1df0b"
-					(reference "#PWR053")
+					(reference "#PWR0140")
 					(unit 1)
 				)
@@
 		(dnp no)
 		(fields_autoplaced yes)
-		(property "Reference" "F3"
+		(property "Reference" "F11"
 			(at 83.82 78.74 90)
 			(effects
@@
 			(project "mega_shield"
 				(path "/554fcf27-dc63-4666-abbc-7481d15942c4/79aa91ed-20a6-424f-83a6-c5f215a1df0b"
-					(reference "F3")
+					(reference "F11")
 					(unit 1)
 				)
@@
 		(on_board yes)
 		(dnp no)
-		(property "Reference" "J19"
+		(property "Reference" "J14"
 			(at 34.29 44.45 0)
 			(effects
@@
 			(project ""
 				(path "/554fcf27-dc63-4666-abbc-7481d15942c4/79aa91ed-20a6-424f-83a6-c5f215a1df0b"
-					(reference "J19")
+					(reference "J14")
 					(unit 1)
 				)
@@
 		(dnp no)
 		(fields_autoplaced yes)
-		(property "Reference" "#PWR047"
+		(property "Reference" "#PWR0138"
 			(at 52.07 97.79 0)
 			(effects
@@
 			(project "mega_shield"
 				(path "/554fcf27-dc63-4666-abbc-7481d15942c4/79aa91ed-20a6-424f-83a6-c5f215a1df0b"
-					(reference "#PWR047")
+					(reference "#PWR0138")
 					(unit 1)
 				)
@@
 		(on_board yes)
 		(dnp no)
-		(property "Reference" "J20"
+		(property "Reference" "J15"
 			(at 34.29 95.25 0)
 			(effects
@@
 			(project "mega_shield"
 				(path "/554fcf27-dc63-4666-abbc-7481d15942c4/79aa91ed-20a6-424f-83a6-c5f215a1df0b"
-					(reference "J20")
-					(unit 1)
-				)
+					(reference "J15")
+					(unit 1)
+				)

Commit message: changed fuses to resetable fuses on the power input connections.
Parts:
- removed F10, F11: 2.5A, symbol Device:Fuse
- added F11, F12: SMD1812P200TF/30, symbol Device:Polyfuse
Connections:
- net +24V_EXTERN: now also F12.1
- net +24V_OUT: now also F12.2
- net +5V_EXTERN: now also F11.1
- net +5V_OUT: now also F11.2

Commit message: Added the JLCPCB numbers and footprints for the polyfuses and input diodes.
Parts:
- D1: footprint (none) -> Diode_SMD:D_SMA; jlcpcb (none) -> C19077488
- D2: value 5.6V -> 27V; footprint (none) -> Diode_SMD:D_SOD-123F; jlcpcb (none) -> C2943770
- F11, F12: jlcpcb (none) -> C5188720
Changed lines of the file:
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@@
+	)
+	(junction
+		(at 90.17 85.09)
+		(diameter 0)
+		(color 0 0 0 0)
 	)
 	(junction
@@
 	)
 	(junction
-		(at 90.17 85.09)
-		(diameter 0)
-		(color 0 0 0 0)
-	)
-	(junction
 		(at 95.25 34.29)
 		(diameter 0)
@@
 	(wire
 		(pts
+			(xy 90.17 85.09) (xy 95.25 85.09)
+		)
+		(stroke
+			(width 0)
+			(type default)
+		)
+	)
+	(wire
+		(pts
 			(xy 44.45 85.09) (xy 80.01 85.09)
 		)
@@
 		(pts
 			(xy 95.25 85.09) (xy 101.6 85.09)
-		)
-		(stroke
-			(width 0)
-			(type default)
-		)
-	)
-	(wire
-		(pts
-			(xy 90.17 85.09) (xy 95.25 85.09)
 		)
 		(stroke
@@
 	)
 	(symbol
+		(lib_id "Device:D_Zener")
+		(at 90.17 88.9 270)
+		(unit 1)
+		(exclude_from_sim no)
+		(in_bom yes)
+		(on_board yes)
+		(dnp no)
+		(fields_autoplaced yes)
+		(property "Reference" "D2"
+			(at 92.71 87.6299 90)
+			(effects
+				(font
+					(size 1.27 1.27)
+				)
+				(justify left)
+			)
+		)
+		(property "Value" "27V"
+			(at 92.71 90.1699 90)
+			(effects
+				(font
+					(size 1.27 1.27)
+				)
+				(justify left)
+			)
+		)
+		(property "Footprint" "Diode_SMD:D_SOD-123F"
+			(at 90.17 88.9 0)
+			(effects
+				(font
+					(size 1.27 1.27)
+				)
+				(hide yes)
+			)
+		)
+		(property "Datasheet" "~"
+			(at 90.17 88.9 0)
+			(effects
+				(font
+					(size 1.27 1.27)
+				)
+				(hide yes)
+			)
+		)
+		(property "Description" "Zener diode"
+			(at 90.17 88.9 0)
+			(effects
+				(font
+					(size 1.27 1.27)
+				)
+				(hide yes)
+			)
+		)
+		(property "Purpose" ""
+			(at 90.17 88.9 0)
+			(effects
+				(font
+					(size 1.27 1.27)
+				)
+			)
+		)
+		(property "jlcpcb" "C2943770"
+			(at 90.17 88.9 0)
+			(effects
+				(font
+					(size 1.27 1.27)
+				)
+			)
+		)
+		(pin "2"
+		)
+		(pin "1"
+		)
+		(instances
+			(project "mega_shield"
+				(path "/554fcf27-dc63-4666-abbc-7481d15942c4/79aa91ed-20a6-424f-83a6-c5f215a1df0b"
+					(reference "D2")
+					(unit 1)
+				)
+			)
+		)
+	)
+	(symbol
 		(lib_id "Device:Polyfuse")
 		(at 83.82 85.09 90)
@@
 			)
 		)
+		(property "jlcpcb" "C5188720"
+			(at 83.82 85.09 0)
+			(effects
+				(font
+					(size 1.27 1.27)
+				)
+			)
+		)
 		(pin "1"
 		)
@@
 			)
 		)
+		(property "jlcpcb" "C5188720"
+			(at 83.82 34.29 0)
+			(effects
+				(font
+					(size 1.27 1.27)
+				)
+			)
+		)
 		(pin "1"
 		)
@@
 			)
 		)
-		(property "Footprint" ""
+		(property "Footprint" "Diode_SMD:D_SMA"
 			(at 90.17 38.1 0)
 			(effects
@@
 				)
 				(hide yes)
+			)
+		)
+		(property "Purpose" ""
+			(at 90.17 38.1 0)
+			(effects
+				(font
+					(size 1.27 1.27)
+				)
+			)
+		)
+		(property "jlcpcb" "C19077488"
+			(at 90.17 38.1 0)
+			(effects
+				(font
+					(size 1.27 1.27)
+				)
 			)
 		)
@@
 					(unit 1)
 				)
-			)
-		)
-	)
-	(symbol
-		(lib_id "Device:D_Zener")
-		(at 90.17 88.9 270)
-		(unit 1)
-		(exclude_from_sim no)
-		(in_bom yes)
-		(on_board yes)
-		(dnp no)
-		(fields_autoplaced yes)
-		(property "Reference" "D2"
-			(at 92.71 87.6299 90)
-			(effects
-				(font
-					(size 1.27 1.27)
-				)
-				(justify left)
-			)
-		)
-		(property "Value" "5.6V"
-			(at 92.71 90.1699 90)
-			(effects
-				(font
-					(size 1.27 1.27)
-				)
-				(justify left)
-			)
-		)
-		(property "Footprint" ""
-			(at 90.17 88.9 0)
-			(effects
-				(font
-					(size 1.27 1.27)
-				)
-				(hide yes)
-			)
-		)
-		(property "Datasheet" "~"
-			(at 90.17 88.9 0)
-			(effects
-				(font
-					(size 1.27 1.27)
-				)
-				(hide yes)
-			)
-		)
-		(property "Description" "Zener diode"
-			(at 90.17 88.9 0)
-			(effects
-				(font
-					(size 1.27 1.27)
-				)
-				(hide yes)
-			)
-		)
-		(pin "2"
-		)
-		(pin "1"
-		)
-		(instances
-			(project "mega_shield"
-				(path "/554fcf27-dc63-4666-abbc-7481d15942c4/79aa91ed-20a6-424f-83a6-c5f215a1df0b"
-					(reference "D2")
-					(unit 1)
-				)

Commit message: Ran ERC, fixed footprint path of the 1757242 connectors.
Parts:
- J14, J15: footprint 1757242:PHOENIX_1757242 -> footprints:PHOENIX_1757242
Changed lines of the file:
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@@
 			)
 		)
-		(property "Footprint" "1757242:PHOENIX_1757242"
+		(property "Footprint" "footprints:PHOENIX_1757242"
 			(at 34.29 36.83 0)
 			(effects
@@
 				(justify bottom)
 				(hide yes)
+			)
+		)
+		(property "Purpose" ""
+			(at 34.29 36.83 0)
+			(effects
+				(font
+					(size 1.27 1.27)
+				)
 			)
 		)
@@
 			)
 		)
-		(property "Footprint" "1757242:PHOENIX_1757242"
+		(property "Footprint" "footprints:PHOENIX_1757242"
 			(at 34.29 87.63 0)
 			(effects
@@
 			)
 		)
+		(property "Purpose" ""
+			(at 34.29 87.63 0)
+			(effects
+				(font
+					(size 1.27 1.27)
+				)
+			)
+		)

Commit message: set the JLCPCB number for the 2pin terminal connector.
Parts:
- J14, J15: jlcpcb (none) -> C90074
Changed lines of the file:
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@@
+			)
+		)
+		(property "jlcpcb" "C90074"
+			(at 34.29 36.83 0)
+			(effects
+				(font
+					(size 1.27 1.27)
+				)
 			)
 		)
@@
 			(at 34.29 87.63 0)
 			(effects
+				(font
+					(size 1.27 1.27)
+				)
+			)
+		)
+		(property "jlcpcb" "C90074"
+			(at 34.29 87.63 0)
+			(effects
