File: mega_shield/power_interface.kicad_sch (KiCad schematic)
At the start: 5 parts, among them J14 XT30PW-M, J15 B2B-XH-A_LF__SN_

Commit message: re-annotating for entire schematic completed.
Parts:
- renumbered F11 to F10
Changed lines of the file:
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@@
 		(dnp no)
 		(fields_autoplaced yes)
-		(property "Reference" "#FLG012"
+		(property "Reference" "#FLG011"
 			(at 95.25 31.115 0)
 			(effects
@@
 			(project "mega_shield"
 				(path "/554fcf27-dc63-4666-abbc-7481d15942c4/79aa91ed-20a6-424f-83a6-c5f215a1df0b"
-					(reference "#FLG012")
+					(reference "#FLG011")
 					(unit 1)
 				)
@@
 		(dnp no)
 		(fields_autoplaced yes)
-		(property "Reference" "#PWR0139"
+		(property "Reference" "#PWR094"
 			(at 90.17 53.34 0)
 			(effects
@@
 			(project "mega_shield"
 				(path "/554fcf27-dc63-4666-abbc-7481d15942c4/79aa91ed-20a6-424f-83a6-c5f215a1df0b"
-					(reference "#PWR0139")
+					(reference "#PWR094")
 					(unit 1)
 				)
@@
 		(dnp no)
 		(fields_autoplaced yes)
-		(property "Reference" "#FLG013"
+		(property "Reference" "#FLG012"
 			(at 95.25 81.915 0)
 			(effects
@@
 			(project "mega_shield"
 				(path "/554fcf27-dc63-4666-abbc-7481d15942c4/79aa91ed-20a6-424f-83a6-c5f215a1df0b"
-					(reference "#FLG013")
+					(reference "#FLG012")
 					(unit 1)
 				)
@@
 		(dnp no)
 		(fields_autoplaced yes)
-		(property "Reference" "#PWR0137"
+		(property "Reference" "#PWR092"
 			(at 52.07 46.99 0)
 			(effects
@@
 			(project ""
 				(path "/554fcf27-dc63-4666-abbc-7481d15942c4/79aa91ed-20a6-424f-83a6-c5f215a1df0b"
-					(reference "#PWR0137")
+					(reference "#PWR092")
 					(unit 1)
 				)
@@
 		(dnp no)
 		(fields_autoplaced yes)
-		(property "Reference" "#PWR0140"
+		(property "Reference" "#PWR095"
 			(at 90.17 104.14 0)
 			(effects
@@
 			(project "mega_shield"
 				(path "/554fcf27-dc63-4666-abbc-7481d15942c4/79aa91ed-20a6-424f-83a6-c5f215a1df0b"
-					(reference "#PWR0140")
+					(reference "#PWR095")
 					(unit 1)
 				)
@@
 		(dnp no)
 		(fields_autoplaced yes)
-		(property "Reference" "F11"
+		(property "Reference" "F10"
 			(at 83.82 27.94 90)
 			(effects
@@
 			(project ""
 				(path "/554fcf27-dc63-4666-abbc-7481d15942c4/79aa91ed-20a6-424f-83a6-c5f215a1df0b"
-					(reference "F11")
+					(reference "F10")
 					(unit 1)
 				)
@@
 		(dnp no)
 		(fields_autoplaced yes)
-		(property "Reference" "#PWR0138"
+		(property "Reference" "#PWR093"
 			(at 52.07 97.79 0)
 			(effects
@@
 			(project "mega_shield"
 				(path "/554fcf27-dc63-4666-abbc-7481d15942c4/79aa91ed-20a6-424f-83a6-c5f215a1df0b"
-					(reference "#PWR0138")
-					(unit 1)
-				)
+					(reference "#PWR093")
+					(unit 1)
+				)

Commit message: Added optional electrolytic capacitor footprints for both the +5V and +24V rails.
Parts:
- added C31, C32, C33, C34: 220u, Capacitor_THT:CP_Radial_D8.0mm_P2.50mm, symbol Device:C_Polarized
Connections:
- net +24V_EXTERN: now also C33.1, C34.1
- net +5V_EXTERN: now also C31.1, C32.1
- net GND: now also C31.2, C32.2, C33.2, C34.2

Commit message: mega_shield, Changed out all caps where needed for in-stock and lower cost parts.
+ Changed out for parts with higher stock.
+ Changed out for 0805 sized components.
+ Changed out for higher voltage.
+ Removed 22uF SMD caps for lower cost 10uF caps in parallel.
+ Updated diode footprint to SOD-123F

BOM cost reduced, and reliability improved.
Parts:
- renumbered C33 to C30, C34 to C33
Changed lines of the file:
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@@
 		(on_board yes)
 		(dnp yes)
-		(property "Reference" "C33"
+		(property "Reference" "C30"
 			(at 95.504 96.012 90)
 			(effects
@@
 			(project "mega_shield"
 				(path "/554fcf27-dc63-4666-abbc-7481d15942c4/79aa91ed-20a6-424f-83a6-c5f215a1df0b"
-					(reference "C33")
+					(reference "C30")
 					(unit 1)
 				)
@@
 		(on_board yes)
 		(dnp yes)
-		(property "Reference" "C34"
+		(property "Reference" "C33"
 			(at 115.316 96.012 90)
 			(effects
@@
 			(project "mega_shield"
 				(path "/554fcf27-dc63-4666-abbc-7481d15942c4/79aa91ed-20a6-424f-83a6-c5f215a1df0b"
-					(reference "C34")
-					(unit 1)
-				)
+					(reference "C33")
+					(unit 1)
+				)

Commit message: mega_shield, updated the external power input for the +5V DC rail
+ Added JLCPCB part number for the CH213K
+ Added the ideal diode to the power interface.
+ Added notes on input protection.
Parts:
- removed C32: 220u, Capacitor_THT:CP_Radial_D8.0mm_P2.50mm, symbol Device:C_Polarized
- removed D1: 5.6V, Diode_SMD:D_SMA, symbol Device:D_Zener
- removed F10: SMD1812P200TF/30, Fuse:Fuse_1812_4532Metric, symbol Device:Polyfuse
- added U29: CH213K, Package_TO_SOT_SMD:SOT-23-3, symbol mega_shield:CH213K
Connections:
- net +5V_EXTERN: now also U29.2 (VO-)
- net GND: now also U29.1 (GND)
- net at J15.1: now also U29.3 (VI+)
Other:
- note added: "5V@1A Reverse Polarity and over-current protection."
- note removed: "5V Over-Voltage & Over-Current Protection"
- moved on the sheet: C30, C31, C33, D2, J14

Commit message: mega_shield, re-annotated components, routed and placed new symbols for 5V external power section.
Parts:
- added R34: 0, Resistor_THT:R_Axial_DIN0207_L6.3mm_D2.5mm_P7.62mm_Horizontal, symbol Device:R
- renumbered C33 to C31, C31 to C32, D2 to D1, U29 to U20
Connections:
- net +5V_EXTERN: now also R34.2
- net at J15.1, U20.3 (VI+): now also R34.1
Other:
- moved on the sheet: U20
Changed lines of the file:
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@@
 		)
 	)
-	(text_box "The 5V DC system is what supplies the board except for the MCU itself,\nas the system operates using the +5V USB rail.\n\nThe ground is shared accross power domains and the \"ideal diode\" is here to prevent\nbackfeeding the external +5V power supply."
+	(text_box "The 5V DC system is what supplies the board except for the MCU itself,\nas the system operates using the +5V USB rail.\n\nThe ground is shared accross power domains and the \"ideal diode\" is here to prevent\nbackfeeding the external +5V power supply.\n\nThe zero ohm resistor is for bypassing the CH213K if needed."
 		(exclude_from_sim no)
 		(at 68.58 57.15 0)
-		(size 71.12 19.05)
+		(size 71.12 27.94)
 		(margins 0.9525 0.9525 0.9525 0.9525)
 		(stroke
@@
 	)
 	(junction
+		(at 101.6 33.02)
+		(diameter 0)
+		(color 0 0 0 0)
+	)
+	(junction
 		(at 90.17 110.49)
 		(diameter 0)
@@
 	)
 	(junction
+		(at 73.66 43.18)
+		(diameter 0)
+		(color 0 0 0 0)
+	)
+	(junction
 		(at 95.25 110.49)
 		(diameter 0)
@@
 	(wire
 		(pts
-			(xy 73.66 35.56) (xy 60.96 35.56)
+			(xy 73.66 43.18) (xy 60.96 43.18)
 		)
 		(stroke
@@
 	(wire
 		(pts
+			(xy 73.66 30.48) (xy 73.66 43.18)
+		)
+		(stroke
+			(width 0)
+			(type default)
+		)
+	)
+	(wire
+		(pts
 			(xy 101.6 44.45) (xy 114.3 44.45)
 		)
@@
 	(wire
 		(pts
+			(xy 82.55 30.48) (xy 73.66 30.48)
+		)
+		(stroke
+			(width 0)
+			(type default)
+		)
+	)
+	(wire
+		(pts
 			(xy 60.96 34.29) (xy 44.45 34.29)
 		)
@@
 	(wire
 		(pts
-			(xy 99.06 36.83) (xy 101.6 36.83)
+			(xy 99.06 44.45) (xy 101.6 44.45)
 		)
 		(stroke
@@
 	(wire
 		(pts
+			(xy 90.17 30.48) (xy 101.6 30.48)
+		)
+		(stroke
+			(width 0)
+			(type default)
+		)
+	)
+	(wire
+		(pts
 			(xy 101.6 110.49) (xy 109.22 110.49)
 		)
@@
 	(wire
 		(pts
-			(xy 101.6 34.29) (xy 101.6 33.02)
+			(xy 101.6 41.91) (xy 101.6 33.02)
 		)
 		(stroke
@@
 	(wire
 		(pts
-			(xy 101.6 36.83) (xy 101.6 44.45)
-		)
-		(stroke
-			(width 0)
-			(type default)
-		)
-	)
-	(wire
-		(pts
 			(xy 101.6 110.49) (xy 101.6 115.57)
 		)
@@
 	(wire
 		(pts
+			(xy 101.6 30.48) (xy 101.6 33.02)
+		)
+		(stroke
+			(width 0)
+			(type default)
+		)
+	)
+	(wire
+		(pts
 			(xy 44.45 36.83) (xy 52.07 36.83)
 		)
@@
 	(wire
 		(pts
-			(xy 99.06 34.29) (xy 101.6 34.29)
+			(xy 99.06 41.91) (xy 101.6 41.91)
 		)
 		(stroke
@@
 	(wire
 		(pts
-			(xy 60.96 35.56) (xy 60.96 34.29)
+			(xy 60.96 43.18) (xy 60.96 34.29)
 		)
 		(stroke
@@
 		(on_board yes)
 		(dnp yes)
-		(property "Reference" "C31"
+		(property "Reference" "C32"
 			(at 108.204 42.672 90)
 			(effects
@@
 			(project ""
 				(path "/554fcf27-dc63-4666-abbc-7481d15942c4/79aa91ed-20a6-424f-83a6-c5f215a1df0b"
-					(reference "C31")
+					(reference "C32")
 					(unit 1)
 				)
@@
 		(dnp no)
 		(fields_autoplaced yes)
-		(property "Reference" "#FLG011"
+		(property "Reference" "#FLG012"
 			(at 114.3 29.845 0)
 			(effects
@@
 			(project "mega_shield"
 				(path "/554fcf27-dc63-4666-abbc-7481d15942c4/79aa91ed-20a6-424f-83a6-c5f215a1df0b"
-					(reference "#FLG011")
+					(reference "#FLG012")
 					(unit 1)
 				)
@@
 		(dnp no)
 		(fields_autoplaced yes)
-		(property "Reference" "D2"
+		(property "Reference" "D1"
 			(at 92.71 113.0299 90)
 			(effects
@@
 			(project "mega_shield"
 				(path "/554fcf27-dc63-4666-abbc-7481d15942c4/79aa91ed-20a6-424f-83a6-c5f215a1df0b"
-					(reference "D2")
+					(reference "D1")
 					(unit 1)
 				)
@@
 		(dnp no)
 		(fields_autoplaced yes)
-		(property "Reference" "#PWR0100"
+		(property "Reference" "#PWR0101"
 			(at 101.6 50.8 0)
 			(effects
@@
 			(project "mega_shield"
 				(path "/554fcf27-dc63-4666-abbc-7481d15942c4/79aa91ed-20a6-424f-83a6-c5f215a1df0b"
-					(reference "#PWR0100")
+					(reference "#PWR0101")
 					(unit 1)
 				)
@@
 		(dnp no)
 		(fields_autoplaced yes)
-		(property "Reference" "#FLG012"
+		(property "Reference" "#FLG011"
 			(at 95.25 107.315 0)
 			(effects
@@
 			(project "mega_shield"
 				(path "/554fcf27-dc63-4666-abbc-7481d15942c4/79aa91ed-20a6-424f-83a6-c5f215a1df0b"
-					(reference "#FLG012")
+					(reference "#FLG011")
 					(unit 1)
 				)
@@
 		(dnp no)
 		(fields_autoplaced yes)
-		(property "Reference" "#PWR0101"
+		(property "Reference" "#PWR0100"
 			(at 90.17 129.54 0)
 			(effects
@@
 			(project "mega_shield"
 				(path "/554fcf27-dc63-4666-abbc-7481d15942c4/79aa91ed-20a6-424f-83a6-c5f215a1df0b"
-					(reference "#PWR0101")
+					(reference "#PWR0100")
 					(unit 1)
 				)
@@
 		(on_board yes)
 		(dnp yes)
-		(property "Reference" "C33"
+		(property "Reference" "C31"
 			(at 115.316 121.412 90)
 			(effects
@@
 			(project "mega_shield"
 				(path "/554fcf27-dc63-4666-abbc-7481d15942c4/79aa91ed-20a6-424f-83a6-c5f215a1df0b"
-					(reference "C33")
+					(reference "C31")
 					(unit 1)
 				)
@@
 	(symbol
 		(lib_id "mega_shield:CH213K")
-		(at 86.36 35.56 0)
+		(at 86.36 43.18 0)
 		(mirror y)
 		(unit 1)
@@
 		(on_board yes)
 		(dnp no)
-		(property "Reference" "U29"
-			(at 86.36 26.67 0)
+		(property "Reference" "U20"
+			(at 86.36 34.29 0)
 			(effects
 				(font
@@
 		)
 		(property "Value" "CH213K"
-			(at 86.36 29.21 0)
+			(at 86.36 36.83 0)
 			(effects
 				(font
@@
 		)
 		(property "Footprint" "Package_TO_SOT_SMD:SOT-23-3"
-			(at 86.36 35.56 0)
+			(at 86.36 43.18 0)
 			(effects
 				(font
@@
 		)
 		(property "Datasheet" ""
-			(at 86.36 35.56 0)
+			(at 86.36 43.18 0)
 			(effects
 				(font
@@
 		)
 		(property "Description" "WCH 5V 0.5A low voltage drop diode chip (Ideal diode w/ current limiting)"
-			(at 86.36 35.56 0)
+			(at 86.36 43.18 0)
 			(effects
 				(font
@@
 		)
 		(property "jlcpcb" "C5456874"
-			(at 86.36 35.56 0)
+			(at 86.36 43.18 0)
 			(effects
 				(font
@@
 			(project ""
 				(path "/554fcf27-dc63-4666-abbc-7481d15942c4/79aa91ed-20a6-424f-83a6-c5f215a1df0b"
-					(reference "U29")
+					(reference "U20")
 					(unit 1)
 				)
@@
 					(unit 1)
 				)
+			)
+		)
+	)
+	(symbol
+		(lib_id "Device:R")
+		(at 86.36 30.48 90)
+		(unit 1)
+		(exclude_from_sim no)
+		(in_bom no)
+		(on_board yes)
+		(dnp yes)
+		(property "Reference" "R34"
+			(at 86.36 28.448 90)
+			(effects
+				(font
+					(size 1.27 1.27)
+				)
+			)
+		)
+		(property "Value" "0"
+			(at 86.36 30.48 90)
+			(effects
+				(font
+					(size 1.27 1.27)
+				)
+			)
+		)
+		(property "Footprint" "Resistor_THT:R_Axial_DIN0207_L6.3mm_D2.5mm_P7.62mm_Horizontal"
+			(at 86.36 32.258 90)
+			(effects
+				(font
+					(size 1.27 1.27)
+				)
+				(hide yes)
+			)
+		)
+		(property "Datasheet" "~"
+			(at 86.36 30.48 0)
+			(effects
+				(font
+					(size 1.27 1.27)
+				)
+				(hide yes)
+			)
+		)
+		(property "Description" "Resistor"
+			(at 86.36 30.48 0)
+			(effects
+				(font
+					(size 1.27 1.27)
+				)
+				(hide yes)
+			)
+		)
+		(property "jlcpcb" "C119982"
+			(at 86.36 30.48 90)
+			(effects
+				(font
+					(size 1.27 1.27)
+				)
+				(hide yes)
+			)
+		)
+		(pin "2"
+		)
+		(pin "1"
+		)
+		(instances
+			(project ""
+				(path "/554fcf27-dc63-4666-abbc-7481d15942c4/79aa91ed-20a6-424f-83a6-c5f215a1df0b"
+					(reference "R34")
+					(unit 1)
+				)

Commit message: mega_shield, Updated project library table, adjusted ideal diode footprint/symbols.
Parts:
- added Q32: PMOS, symbol Simulation_SPICE:PMOS
Changed lines of the file:
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@@
+	(wire
+		(pts
+			(xy 252.73 76.2) (xy 254 76.2)
+		)
+		(stroke
+			(width 0)
+			(type default)
+		)
+	)
 	(wire
 		(pts
@@
 		(shape output)
 		(at 110.49 110.49 0)
+		(effects
+			(font
+				(size 1.27 1.27)
+			)
+			(justify left)
+		)
+	)
+	(hierarchical_label "+24V_EXTERN"
+		(shape output)
+		(at 254 76.2 0)
 		(effects
 			(font
@@
 					(unit 1)
 				)
+			)
+		)
+	)
+	(symbol
+		(lib_id "Simulation_SPICE:PMOS")
+		(at 161.29 104.14 90)
+		(unit 1)
+		(exclude_from_sim no)
+		(in_bom yes)
+		(on_board yes)
+		(dnp no)
+		(property "Reference" "Q32"
+			(at 161.29 95.25 90)
+			(effects
+				(font
+					(size 1.27 1.27)
+				)
+			)
+		)
+		(property "Value" "PMOS"
+			(at 161.29 97.79 90)
+			(effects
+				(font
+					(size 1.27 1.27)
+				)
+			)
+		)
+		(property "Footprint" ""
+			(at 158.75 99.06 0)
+			(effects
+				(font
+					(size 1.27 1.27)
+				)
+				(hide yes)
+			)
+		)
+		(property "Datasheet" "https://ngspice.sourceforge.io/docs/ngspice-html-manual/manual.xhtml#cha_MOSFETs"
+			(at 173.99 104.14 0)
+			(effects
+				(font
+					(size 1.27 1.27)
+				)
+				(hide yes)
+			)
+		)
+		(property "Description" "P-MOSFET transistor, drain/source/gate"
+			(at 161.29 104.14 0)
+			(effects
+				(font
+					(size 1.27 1.27)
+				)
+				(hide yes)
+			)
+		)
+		(property "Sim.Device" "PMOS"
+			(at 178.435 104.14 0)
+			(effects
+				(font
+					(size 1.27 1.27)
+				)
+				(hide yes)
+			)
+		)
+		(property "Sim.Type" "VDMOS"
+			(at 180.34 104.14 0)
+			(effects
+				(font
+					(size 1.27 1.27)
+				)
+				(hide yes)
+			)
+		)
+		(property "Sim.Pins" "1=D 2=G 3=S"
+			(at 176.53 104.14 0)
+			(effects
+				(font
+					(size 1.27 1.27)
+				)
+				(hide yes)
+			)
+		)
+		(pin "2"
+		)
+		(pin "3"
+		)
+		(pin "1"
+		)
+		(instances
+			(project "mega_shield"
+				(path "/554fcf27-dc63-4666-abbc-7481d15942c4/79aa91ed-20a6-424f-83a6-c5f215a1df0b"
+					(reference "Q32")
+					(unit 1)
+				)

Commit message: mega_shield, placed ideal diode and added jlcpcb number for it.
Parts:
- removed Q32: PMOS, symbol Simulation_SPICE:PMOS
- added U21: DZDH0401DW-7, footprints:SOIC6_DZDH0401DW-7_DIO, symbol DZDH0401DW-7:DZDH0401DW-7
