File: mega_shield/mega_shield.kicad_pcb (KiCad board)
At the start: 2 copper layers, 296 parts, among them J11 T4040014031-000, J13 T4040014031-000, J14 1757242, J15 1757242, J17 T4040014031-000, J19 T4040014031-000, J20 T4140012121-000, J3 1757271, J9 T4040014031-000, Q1 2SK3018, Q10 2SK3018, Q11 2SK3018, Q12 2SK3018, Q13 2SK3018, Q14 2SK3018, Q15 2SK3018, Q16 2SK3018, Q17 2SK3018, Q18 2SK3018, Q19 2SK3018, Q2 2SK3018, Q20 2SK3018, Q21 2SK3018, Q22 2SK3018, Q23 2SK3018, Q24 2SK3018, Q25 2SK3018, Q26 2SK3018, Q27 2SK3018, Q28 2SK3018, Q29 2SK3018, Q3 2SK3018, Q30 2SK3018, Q31 2SK3018, Q32 2SK3018, Q33 2SK3018, Q34 2SK3018, Q35 2SK3018, Q36 2SK3018, Q37 2SK3018, Q38 2SK3018, Q39 2SK3018, Q4 2SK3018, Q40 2SK3018, Q41 2SK3018, Q42 2SK3018, Q5 2SK3018, Q6 2SK3018, Q7 2SK3018, Q8 2SK3018, Q9 2SK3018, U1 CS817x22HS, U10 CS817x22HS, U11 CS817x22HS, U12 CS817x22HS, U13 CS817x22HS, U14 CS817x22HS, U15 CS817x22HS, U16 CS817x22HS, U17 CS817x22HS, U18 CS817x22HS, U19 NUP2202, U2 CS817x22HS, U20 NUP2202, U21 NUP2202, U22 NUP2202, U23 NUP2202, U24 CS817x22HS, U25 CS817x22HS, U26 CS817x22HS, U27 CS817x22HS, U28 CS817x22HS, U3 CS817x22HS, U4 CS817x22HS, U5 CS817x22HS, U6 CS817x22HS, U7 MCP6241RT-I-OT, U8 NUP2202, U9 CS817x22HS

Commit message: moved mega shield to x:75, y:150
Parts:
- moved A1 52.5 mm to (75.0, 150.0)
Changed lines of the file:
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@@
 		(legacy_teardrops no)
 	)
-	(paper "A4")
+	(paper "A3")
 	(layers
 		(0 "F.Cu" signal)
@@
 	(footprint "PCM_arduino-library:Arduino_Mega2560_R3_Shield"
 		(layer "F.Cu")
-		(at 112.4 113.2)
+		(at 75 150)
 		(descr "https://docs.arduino.cc/hardware/mega-2560")
 		(property "Reference" "A1"

Commit message: fixed DNP mark on M12P8 connectors.
Parts:
- added J1: T4140012081-000, footprints:TE_T4140012081-000, F.Cu at (-201.3, 65.2)
- added J2: T4140012081-000, footprints:TE_T4140012081-000, F.Cu at (-224.8, 65.2)
- added J4: T4140012081-000, footprints:TE_T4140012081-000, F.Cu at (-201.3, 41.3)
- added J5: T4140012081-000, footprints:TE_T4140012081-000, F.Cu at (-132.2, 9.30)
- added J6: T4140012081-000, footprints:TE_T4140012081-000, F.Cu at (-224.8, 41.3)
- moved J15 154.5 mm to (68.0, 155.6), turned to -90 degrees
- moved J14 152.3 mm to (68.7, 79.6), turned to -90 degrees
- moved TP48 93.3 mm to (-134.5, 27.1)
- moved TP49 93.3 mm to (-134.5, 30.1)
- moved TP50 93.3 mm to (-134.5, 33.2)
- moved TP51 93.3 mm to (-134.5, 36.2)
- moved TP52 93.3 mm to (-134.5, 39.3)
- moved TP53 93.3 mm to (-131.4, 27.1)
- moved TP54 93.3 mm to (-131.4, 30.1)
- moved TP55 93.3 mm to (-131.4, 33.2)
- moved TP56 93.3 mm to (-131.4, 36.2)
- moved TP57 93.3 mm to (-131.4, 39.3)
- moved TP58 93.3 mm to (-128.4, 27.1)
- moved TP59 93.3 mm to (-128.4, 30.1)
- moved TP60 93.3 mm to (-128.4, 33.2)
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
Commit message: organized the digital isolators
Parts:
- moved C27 53.3 mm to (-72.2, -3.92), turned to -90 degrees
- moved C25 50.5 mm to (-77.2, -3.92), turned to 90 degrees
- moved R15 36.9 mm to (-78.5, 37.8)
- moved C30 34.1 mm to (-71.9, 27.0), turned to -90 degrees
- moved C26 33.0 mm to (-76.8, 12.1), turned to 90 degrees
- moved R14 27.1 mm to (-105.5, 7.30), turned to 180 degrees
- moved R16 22.8 mm to (-72.0, 37.6)
- moved C28 22.8 mm to (-71.8, 12.1), turned to -90 degrees
- moved C29 18.4 mm to (-76.9, 27.0), turned to 90 degrees
- moved Q26 10.9 mm to (-66.8, 33.3)
- moved Q25 10.9 mm to (-66.8, 28.3)
- moved U15 10.8 mm to (-74.4, 30.6)
- moved U14 5.97 mm to (-74.3, 15.7)
- moved Q23 5.97 mm to (-66.7, 13.3)
- moved Q24 5.97 mm to (-66.7, 18.4)

Commit message: Set the test points values.
Parts:
- TP48: value TestPoint -> +5V_Servo
- TP49: value TestPoint -> STEP
- TP50: value TestPoint -> DIR
- TP51: value TestPoint -> EN
- TP52: value TestPoint -> AUX_IN
- TP53: value TestPoint -> PED_IN
- TP54: value TestPoint -> ALARM_IN
- TP55: value TestPoint -> DIR_OUT
- TP56: value TestPoint -> STEP_OUT
- TP58: value TestPoint -> AUX_OUT
- TP59: value TestPoint -> PED
- TP60: value TestPoint -> ALARM
- moved J5 85.5 mm to (-46.8, 11.6)
- moved TP54 72.6 mm to (-58.8, 31.0)
- moved TP58 70.6 mm to (-61.7, 3.95)
- moved TP53 65.5 mm to (-66.0, 30.9)
- moved TP59 55.3 mm to (-73.0, 30.9)
- moved TP48 53.7 mm to (-85.2, 5.70)
- moved TP49 40.7 mm to (-101.8, 5.88)
- moved TP52 40.4 mm to (-101.8, 15.5)
- moved TP56 38.9 mm to (-92.7, 33.0)
- moved TP60 35.0 mm to (-101.8, 10.3)
- moved TP51 33.2 mm to (-103.6, 24.1)
- moved TP50 32.8 mm to (-104.4, 20.0)
- moved TP55 32.6 mm to (-98.8, 32.9)
- moved TP57 25.7 mm to (-106.5, 32.9)
- moved R14 22.3 mm to (-85.9, 18.1), turned to 0 degrees
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
Commit message: replicated servo interface layout.
Parts:
- TP57: value TestPoint -> EN_OUT
- moved J6 231.6 mm to (-4.87, 113.7)
- moved J4 221.1 mm to (-4.92, 142.8)
- moved J2 210.4 mm to (-29.2, 142.8)
- moved J1 199.6 mm to (-2.41, 82.1)
- moved TP57 56.6 mm to (-61.6, -1.68)
- moved TP55 43.9 mm to (-61.7, 9.43)
- moved TP19 38.7 mm to (-43.5, 153.8)
- moved TP40 38.7 mm to (-19.2, 153.8)
- moved TP6 38.7 mm to (-16.7, 93.1)
- moved TP66 38.7 mm to (-19.1, 124.7)
- moved TP56 36.0 mm to (-61.8, 14.6)
- moved Q10 33.7 mm to (-48.9, 145.2)
- moved Q18 33.7 mm to (-24.6, 145.2)
- moved Q30 33.7 mm to (-24.5, 116.1)
- moved Q4 33.7 mm to (-22.1, 84.5)
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
Commit message: Re-applied replication operation after adding seperation of sheets components.
Parts:
- moved C10 260.3 mm to (-297.4, 46.5)
- moved C9 260.3 mm to (-297.3, 35.4)
- moved J2 260.3 mm to (-272.6, 50.4)
- moved Q11 260.3 mm to (-301.7, 61.2)
- moved Q12 260.3 mm to (-301.7, 56.2)
- moved Q8 260.3 mm to (-292.2, 41.7)
- moved R4 260.3 mm to (-316.7, 56.4)
- moved R5 260.3 mm to (-305.9, 61.2)
- moved R6 260.3 mm to (-305.9, 56.2)
- moved TP14 260.3 mm to (-316.0, 43.8)
- moved TP15 260.3 mm to (-310.1, 47.8)
- moved TP16 260.3 mm to (-310.1, 52.1)
- moved TP17 260.3 mm to (-310.1, 37.1)
- moved TP18 260.3 mm to (-310.1, 41.3)
- moved TP19 260.3 mm to (-286.9, 61.4)
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
Commit message: setup all the servo interfaces in order X, Y, Z, A, B
Parts:
- moved C10 542.0 mm to (243.5, 82.6)
- moved Q11 542.0 mm to (239.1, 97.2)
- moved Q12 542.0 mm to (239.1, 92.2)
- moved TP14 542.0 mm to (224.8, 79.8)
- moved TP15 542.0 mm to (230.7, 83.8)
- moved C11 542.0 mm to (249.1, 98.6)
- moved C12 542.0 mm to (244.2, 98.6)
- moved C7 542.0 mm to (238.5, 71.5)
- moved C8 542.0 mm to (238.5, 82.6)
- moved C9 542.0 mm to (243.5, 71.5)
- moved F2 542.0 mm to (222.6, 86.2)
- moved J2 542.0 mm to (268.2, 86.5)
- moved LED2 542.0 mm to (221.2, 92.5)
- moved Q10 542.0 mm to (248.5, 88.9)
- moved Q7 542.0 mm to (248.6, 72.8)
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
Commit message: organized the power interface compoenents.
Parts:
- moved D2 174.0 mm to (99.7, 160.5), turned to -90 degrees
- moved D1 166.9 mm to (101.2, 85.1), turned to -90 degrees
- moved F12 165.8 mm to (89.1, 159.1)
- moved F11 156.0 mm to (90.3, 83.1)
Changed lines of the file:
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@@
 	(footprint "Diode_SMD:D_SMA"
 		(layer "F.Cu")
-		(at -64.685 103.35)
+		(at 101.25 85.125 -90)
 		(descr "Diode SMA (DO-214AC)")
 		(tags "Diode SMA (DO-214AC)")
 		(property "Reference" "D1"
-			(at 0 -2.5 0)
+			(at 0 -2.5 90)
 			(layer "F.SilkS")
 			(effects
@@
 		)
 		(property "Value" "5.6V"
-			(at 0 2.6 0)
+			(at 0 2.6 90)
 			(layer "F.Fab")
 			(effects
@@
 		)
 		(property "Datasheet" ""
-			(at 0 0 0)
+			(at 0 0 270)
 			(unlocked yes)
 			(layer "F.Fab")
@@
 		)
 		(property "Description" "Zener diode"
-			(at 0 0 0)
+			(at 0 0 270)
 			(unlocked yes)
 			(layer "F.Fab")
@@
 		)
 		(property "Purpose" ""
-			(at 0 0 0)
+			(at 0 0 270)
 			(unlocked yes)
 			(layer "F.Fab")
@@
 		)
 		(property "jlcpcb" "C19077488"
-			(at 0 0 0)
+			(at 0 0 270)
 			(unlocked yes)
 			(layer "F.Fab")
@@
 		(attr smd)
 		(fp_line
-			(start -3.51 -1.65)
-			(end -3.51 1.65)
+			(start -3.51 1.65)
+			(end 2 1.65)
 			(stroke
 				(width 0.12)
@@
 		(fp_line
 			(start -3.51 -1.65)
-			(end 2 -1.65)
+			(end -3.51 1.65)
 			(stroke
 				(width 0.12)
@@
 		)
 		(fp_line
-			(start -3.51 1.65)
-			(end 2 1.65)
+			(start -3.51 -1.65)
+			(end 2 -1.65)
 			(stroke
 				(width 0.12)
@@
 		)
 		(fp_line
-			(start -3.5 -1.75)
-			(end 3.5 -1.75)
+			(start -3.5 1.75)
+			(end -3.5 -1.75)
 			(stroke
 				(width 0.05)
@@
 		)
 		(fp_line
-			(start -3.5 1.75)
-			(end -3.5 -1.75)
+			(start 3.5 1.75)
+			(end -3.5 1.75)
 			(stroke
 				(width 0.05)
@@
 		)
 		(fp_line
-			(start 3.5 -1.75)
-			(end 3.5 1.75)
+			(start -3.5 -1.75)
+			(end 3.5 -1.75)
 			(stroke
 				(width 0.05)
@@
 		)
 		(fp_line
-			(start 3.5 1.75)
-			(end -3.5 1.75)
+			(start 3.5 -1.75)
+			(end 3.5 1.75)
 			(stroke
 				(width 0.05)
@@
 		)
 		(fp_line
-			(start -0.64944 -0.79908)
-			(end -0.64944 0.80112)
+			(start 2.3 1.5)
+			(end -2.3 1.5)
 			(stroke
 				(width 0.1)
@@
 		)
 		(fp_line
-			(start -0.64944 0.00102)
-			(end -1.55114 0.00102)
+			(start 0.50118 0.75032)
+			(end 0.50118 -0.79908)
 			(stroke
 				(width 0.1)
@@
 		(fp_line
 			(start -0.64944 0.00102)
-			(end 0.50118 -0.79908)
+			(end 0.50118 0.75032)
 			(stroke
 				(width 0.1)
@@
 		(fp_line
 			(start -0.64944 0.00102)
-			(end 0.50118 0.75032)
+			(end -1.55114 0.00102)
 			(stroke
 				(width 0.1)
@@
 		)
 		(fp_line
-			(start 0.50118 0.00102)
-			(end 1.4994 0.00102)
+			(start -0.64944 0.00102)
+			(end 0.50118 -0.79908)
 			(stroke
 				(width 0.1)
@@
 		)
 		(fp_line
-			(start 0.50118 0.75032)
-			(end 0.50118 -0.79908)
+			(start 0.50118 0.00102)
+			(end 1.4994 0.00102)
 			(stroke
 				(width 0.1)
@@
 		)
 		(fp_line
-			(start 2.3 -1.5)
-			(end -2.3 -1.5)
+			(start -0.64944 -0.79908)
+			(end -0.64944 0.80112)
 			(stroke
 				(width 0.1)
@@
 		)
 		(fp_line
-			(start 2.3 1.5)
-			(end -2.3 1.5)
+			(start 2.3 -1.5)
+			(end -2.3 -1.5)
 			(stroke
 				(width 0.1)
@@
 		)
 		(fp_text user "${REFERENCE}"
-			(at 0 -2.5 0)
+			(at 0 -2.5 90)
 			(layer "F.Fab")
 			(effects
@@
 		)
 		(pad "1" smd roundrect
-			(at -2 0)
+			(at -2 0 270)
 			(size 2.5 1.8)
 			(layers "F.Cu" "F.Mask" "F.Paste")
@@
 		)
 		(pad "2" smd roundrect
-			(at 2 0)
+			(at 2 0 270)
 			(size 2.5 1.8)
 			(layers "F.Cu" "F.Mask" "F.Paste")
@@
 	(footprint "Fuse:Fuse_1812_4532Metric"
 		(layer "F.Cu")
-		(at -65.28 98.6)
+		(at 89.125 159.075)
 		(descr "Fuse SMD 1812 (4532 Metric), square (rectangular) end terminal, IPC_7351 nominal, (Body size source: https://www.nikhef.nl/pub/departments/mt/projects/detectorR_D/dtddice/ERJ2G.pdf), generated with kicad-footprint-generator")
 		(tags "fuse")
@@
 	(footprint "Fuse:Fuse_1812_4532Metric"
 		(layer "F.Cu")
-		(at -65.28 93.65)
+		(at 90.325 83.125)
 		(descr "Fuse SMD 1812 (4532 Metric), square (rectangular) end terminal, IPC_7351 nominal, (Body size source: https://www.nikhef.nl/pub/departments/mt/projects/detectorR_D/dtddice/ERJ2G.pdf), generated with kicad-footprint-generator")
 		(tags "fuse")
@@
 	(footprint "Diode_SMD:D_SOD-123F"
 		(layer "F.Cu")
-		(at -65.985 107.3)
+		(at 99.725 160.475 -90)
 		(descr "D_SOD-123F")
 		(tags "D_SOD-123F")
 		(property "Reference" "D2"
-			(at -0.127 -1.905 0)
+			(at -0.127 -1.905 90)
 			(layer "F.SilkS")
 			(effects
@@
 		)
 		(property "Value" "27V"
-			(at 0 2.1 0)
+			(at 0 2.1 90)
 			(layer "F.Fab")
 			(effects
@@
 		)
 		(property "Datasheet" ""
-			(at 0 0 0)
+			(at 0 0 270)
 			(unlocked yes)
 			(layer "F.Fab")
@@
 		)
 		(property "Description" "Zener diode"
-			(at 0 0 0)
+			(at 0 0 270)
 			(unlocked yes)
 			(layer "F.Fab")
@@
 		)
 		(property "Purpose" ""
-			(at 0 0 0)
+			(at 0 0 270)
 			(unlocked yes)
 			(layer "F.Fab")
@@
 		)
 		(property "jlcpcb" "C2943770"
-			(at 0 0 0)
+			(at 0 0 270)
 			(unlocked yes)
 			(layer "F.Fab")
@@
 		(attr smd)
 		(fp_line
-			(start -2.21 -1)
-			(end -2.21 1)
+			(start -2.21 1)
+			(end 1.65 1)
 			(stroke
 				(width 0.12)
@@
 		(fp_line
 			(start -2.21 -1)
-			(end 1.65 -1)
+			(end -2.21 1)
 			(stroke
 				(width 0.12)
@@
 		)
 		(fp_line
-			(start -2.21 1)
-			(end 1.65 1)
+			(start -2.21 -1)
+			(end 1.65 -1)
 			(stroke
 				(width 0.12)
@@
 		)
 		(fp_line
-			(start -2.2 -1.15)
+			(start 2.2 1.15)
 			(end -2.2 1.15)
 			(stroke
@@
 		(fp_line
 			(start -2.2 -1.15)
-			(end 2.2 -1.15)
+			(end -2.2 1.15)
 			(stroke
 				(width 0.05)
@@
 		)
 		(fp_line
-			(start 2.2 -1.15)
-			(end 2.2 1.15)
+			(start -2.2 -1.15)
+			(end 2.2 -1.15)
 			(stroke
 				(width 0.05)
@@
 		)
 		(fp_line
-			(start 2.2 1.15)
-			(end -2.2 1.15)
+			(start 2.2 -1.15)
+			(end 2.2 1.15)
 			(stroke
 				(width 0.05)
@@
 		)
 		(fp_line
-			(start -1.4 -0.9)
-			(end 1.4 -0.9)
+			(start -1.4 0.9)
+			(end -1.4 -0.9)
 			(stroke
 				(width 0.1)
@@
 		)
 		(fp_line
-			(start -1.4 0.9)
-			(end -1.4 -0.9)
+			(start 1.4 0.9)
+			(end -1.4 0.9)
 			(stroke
 				(width 0.1)
@@
 		)
 		(fp_line
-			(start -0.75 0)
+			(start 0.25 0.4)
 			(end -0.35 0)
 			(stroke
@@
 		)
 		(fp_line
-			(start -0.35 0)
-			(end -0.35 -0.55)
+			(start -0.75 0)
+			(end -0.35 0)
 			(stroke
 				(width 0.1)
@@
 		)
 		(fp_line
-			(start 0.25 -0.4)
-			(end 0.25 0.4)
+			(start -0.35 0)
+			(end -0.35 -0.55)
 			(stroke
 				(width 0.1)
@@
 		)
 		(fp_line
-			(start 0.25 0.4)
-			(end -0.35 0)
+			(start 0.25 -0.4)
+			(end 0.25 0.4)
 			(stroke
 				(width 0.1)
@@
 		)
 		(fp_line
-			(start 1.4 -0.9)
-			(end 1.4 0.9)
+			(start -1.4 -0.9)
+			(end 1.4 -0.9)
 			(stroke
 				(width 0.1)
@@
 		)
 		(fp_line
-			(start 1.4 0.9)
-			(end -1.4 0.9)
+			(start 1.4 -0.9)
+			(end 1.4 0.9)
 			(stroke
 				(width 0.1)
@@
 		)
 		(fp_text user "${REFERENCE}"
-			(at -0.127 -1.905 0)
+			(at -0.127 -1.905 90)
 			(layer "F.Fab")
 			(effects
@@
 		)
 		(pad "1" smd roundrect
-			(at -1.4 0)
+			(at -1.4 0 270)
 			(size 1.1 1.1)
 			(layers "F.Cu" "F.Mask" "F.Paste")
@@
 		)
 		(pad "2" smd roundrect
-			(at 1.4 0)
+			(at 1.4 0 270)
 			(size 1.1 1.1)
 			(layers "F.Cu" "F.Mask" "F.Paste")
