File: mega_shield/mega_shield.kicad_pcb (KiCad board)
At the start: 2 copper layers, 301 parts, among them J1 T4140012081-000, J11 T4040014031-000, J13 T4040014031-000, J14 1757242, J15 1757242, J17 T4040014031-000, J19 T4040014031-000, J2 T4140012081-000, J20 T4140012121-000, J3 1757271, J4 T4140012081-000, J5 T4140012081-000, J6 T4140012081-000, J9 T4040014031-000, Q1 2SK3018, Q10 2SK3018, Q11 2SK3018, Q12 2SK3018, Q13 2SK3018, Q14 2SK3018, Q15 2SK3018, Q16 2SK3018, Q17 2SK3018, Q18 2SK3018, Q19 2SK3018, Q2 2SK3018, Q20 2SK3018, Q21 2SK3018, Q22 2SK3018, Q23 2SK3018, Q24 2SK3018, Q25 2SK3018, Q26 2SK3018, Q27 2SK3018, Q28 2SK3018, Q29 2SK3018, Q3 2SK3018, Q30 2SK3018, Q31 2SK3018, Q32 2SK3018, Q33 2SK3018, Q34 2SK3018, Q35 2SK3018, Q36 2SK3018, Q37 2SK3018, Q38 2SK3018, Q39 2SK3018, Q4 2SK3018, Q40 2SK3018, Q41 2SK3018, Q42 2SK3018, Q5 2SK3018, Q6 2SK3018, Q7 2SK3018, Q8 2SK3018, Q9 2SK3018, U1 CS817x22HS, U10 CS817x22HS, U11 CS817x22HS, U12 CS817x22HS, U13 CS817x22HS, U14 CS817x22HS, U15 CS817x22HS, U16 CS817x22HS, U17 CS817x22HS, U18 CS817x22HS, U19 NUP2202, U2 CS817x22HS, U20 NUP2202, U21 NUP2202, U22 NUP2202, U23 NUP2202, U24 CS817x22HS, U25 CS817x22HS, U26 CS817x22HS, U27 CS817x22HS, U28 CS817x22HS, U3 CS817x22HS, U4 CS817x22HS, U5 CS817x22HS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

Commit message: marked the secondary 3pin connectors as included in bom.
Parts:
- moved C52 84.0 mm to (-47.8, 190.4)
- moved C53 84.0 mm to (-47.8, 192.2)
- moved R38 84.0 mm to (-47.8, 193.9)
- moved R39 84.0 mm to (-47.8, 195.7)
- moved TP89 84.0 mm to (-55.2, 176.8)
- moved TP91 84.0 mm to (-55.2, 182.9)
- moved J17 84.0 mm to (-47.3, 182.4)
- moved Q39 84.0 mm to (-51.3, 191.5)
- moved TP90 84.0 mm to (-55.2, 179.8)
- moved TP92 84.0 mm to (-55.2, 185.9)
- moved TP93 84.0 mm to (-55.2, 189.0)
- moved U27 84.0 mm to (-42.3, 192.9)
- moved C50 84.0 mm to (-36.2, 176.8)
- moved C51 84.0 mm to (-36.2, 179.8)
- moved Q40 84.0 mm to (-51.3, 195.4)
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
Commit message: seperated the multiple proximity sensor interfaces.
Parts:
- added J10: T4040014031-000, footprints:CONN3_T4040014031-000_TEC, F.Cu at (-217.6, 25.1)
- added J12: T4040014031-000, footprints:CONN3_T4040014031-000_TEC, F.Cu at (-178.1, 24.8)
- added J16: T4040014031-000, footprints:CONN3_T4040014031-000_TEC, F.Cu at (-133.4, 21.6)
- added J18: T4040014031-000, footprints:CONN3_T4040014031-000_TEC, F.Cu at (-84.4, 19.1)
- added J8: T4040014031-000, footprints:CONN3_T4040014031-000_TEC, F.Cu at (-273.6, 26.4)
- TP48: value +5V_Servo -> TestPoint
- TP49: value STEP -> TestPoint
- TP50: value DIR -> TestPoint
- TP51: value EN -> TestPoint
- TP52: value AUX_IN -> TestPoint
- TP53: value PED_IN -> TestPoint
- TP54: value ALARM_IN -> TestPoint
- TP55: value DIR_OUT -> TestPoint
- TP56: value STEP_OUT -> TestPoint
- TP57: value EN_OUT -> TestPoint
- TP58: value AUX_OUT -> TestPoint
- TP59: value PED -> TestPoint
- TP60: value ALARM -> TestPoint
- moved C40 208.4 mm to (-273.8, 51.0)
- moved C41 208.4 mm to (-273.8, 52.8)
- moved J9 208.4 mm to (-273.3, 43.0)
- moved R32 208.4 mm to (-273.8, 54.5)
- moved R33 208.4 mm to (-273.8, 56.3)
- moved TP74 208.4 mm to (-281.3, 37.4)
- moved TP75 208.4 mm to (-281.3, 40.5)
- moved TP76 208.4 mm to (-281.3, 43.5)
- moved TP77 208.4 mm to (-281.3, 46.6)
- moved TP78 208.4 mm to (-281.3, 49.6)
- moved U24 208.4 mm to (-268.4, 53.5)
- moved C38 208.4 mm to (-262.2, 37.4)
- moved C39 208.4 mm to (-262.2, 40.4)
- moved Q33 208.4 mm to (-277.4, 52.1)
- moved Q34 208.4 mm to (-277.4, 56.0)
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
Commit message: Applied replicate on proximity sensor sheets.
Parts:
- moved TP97 117.3 mm to (24.9, 29.6)
- moved TP96 109.7 mm to (17.6, 29.5)
- moved C42 109.4 mm to (-206.4, 26.4), turned to 90 degrees
- moved TP92 105.7 mm to (-35.2, 35.9)
- moved C55 101.1 mm to (27.1, 19.6), turned to 90 degrees
- moved J19 101.0 mm to (15.2, 18.8)
- moved TP94 100.2 mm to (8.59, 29.5)
- moved Q41 98.9 mm to (11.2, 46.5), turned to 180 degrees
- moved TP91 98.2 mm to (-42.5, 35.8)
- moved C56 97.6 mm to (12.7, 35.3)
- moved C57 97.2 mm to (12.7, 40.2)
- moved R40 96.6 mm to (12.2, 43.3), turned to -90 degrees
- moved Q42 93.7 mm to (5.79, 46.5), turned to 180 degrees
- moved TP95 91.4 mm to (-0.46, 29.5)
- moved R41 91.3 mm to (6.76, 43.4), turned to -90 degrees
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
Commit message: finished basic layout of proximity sensors.
Parts:
- moved C40 471.1 mm to (194.0, 54.5)
- moved C41 471.1 mm to (194.0, 59.4)
- moved R33 471.1 mm to (188.0, 62.6)
- moved TP76 471.1 mm to (198.9, 48.7)
- moved U24 471.1 mm to (189.8, 56.9)
- moved C38 471.1 mm to (171.6, 38.9)
- moved C39 471.1 mm to (208.4, 38.8)
- moved J8 471.1 mm to (180.1, 37.9)
- moved J9 471.1 mm to (196.5, 38.0)
- moved Q34 471.1 mm to (187.1, 65.7)
- moved TP74 471.1 mm to (189.9, 48.7)
- moved TP75 471.1 mm to (180.8, 48.7)
- moved TP77 471.1 mm to (206.2, 48.8)
- moved TP78 471.1 mm to (172.9, 48.7)
- moved Q33 471.1 mm to (192.5, 65.7)
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
Commit message: set the values for test points and finished initial layout of op-amp circuit and isolator
Parts:
- TP27: value TestPoint -> +5V_SPIN
- TP28: value TestPoint -> SPIN_PWM
- TP29: value TestPoint -> SPIN_DIR
- TP30: value TestPoint -> SPIN_EN
- TP31: value TestPoint -> V_SPIN
- TP32: value TestPoint -> SPIN_SPEED
- TP33: value TestPoint -> SPIN_DIR_OC
- TP34: value TestPoint -> SPIN_EN_OC
- moved J3 89.3 mm to (-117.9, 209.4)
- moved TP34 84.4 mm to (-81.1, 176.4)
- moved TP32 77.8 mm to (-90.6, 174.6)
- moved TP30 77.8 mm to (-98.2, 182.5)
- moved TP33 77.5 mm to (-86.2, 168.0)
- moved TP31 74.1 mm to (-90.5, 162.2)
- moved TP28 72.6 mm to (-102.2, 173.9)
- moved TP29 70.0 mm to (-98.4, 163.2)
- moved TP27 66.2 mm to (-106.5, 165.4)
- moved U7 61.5 mm to (-91.6, 139.8), turned to -90 degrees
- moved U8 58.5 mm to (-85.2, 139.8), turned to 90 degrees
- moved C15 58.4 mm to (-91.0, 143.4), turned to 90 degrees
- moved C16 57.0 mm to (-92.3, 143.4), turned to 90 degrees
- moved C14 53.5 mm to (-95.8, 138.5), turned to -90 degrees
- moved C13 49.1 mm to (-100.5, 141.5), turned to 90 degrees
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
Commit message: placed the spindle interface components.
Parts:
- moved C18 244.6 mm to (109.9, 182.0)
- moved Q14 244.6 mm to (115.9, 188.4)
- moved U9 244.6 mm to (107.4, 185.8)
- moved C17 244.6 mm to (104.9, 182.0)
- moved Q13 244.6 mm to (115.9, 183.1)
- moved R10 244.6 mm to (119.3, 187.7)
- moved R9 244.6 mm to (119.0, 182.5)
- moved J3 209.1 mm to (91.2, 213.2)
- moved TP30 207.6 mm to (109.3, 174.6), turned to 90 degrees
- moved TP29 203.3 mm to (104.7, 174.6), turned to 90 degrees
- moved TP28 202.2 mm to (100.0, 174.6), turned to 90 degrees
- moved TP27 202.1 mm to (95.4, 174.5), turned to 90 degrees
- moved TP33 193.2 mm to (104.9, 196.2), turned to 90 degrees
- moved TP34 192.1 mm to (110.0, 196.2), turned to 90 degrees
- moved TP32 191.6 mm to (99.8, 196.1), turned to 90 degrees
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
Commit message: organized ESD protection chips.
Parts:
- moved J20 187.0 mm to (20.1, 42.2)
- moved R22 38.5 mm to (-122.8, 85.3)
- moved R23 37.0 mm to (-128.8, 85.3)
- moved R24 29.3 mm to (-119.9, 92.8)
- moved R20 29.1 mm to (-172.4, 122.5)
- moved R28 27.4 mm to (-117.3, 107.4)
- moved R25 26.2 mm to (-126.2, 92.8)
- moved R21 23.1 mm to (-165.8, 124.8)
- moved R26 23.1 mm to (-125.2, 99.7)
- moved R27 20.6 mm to (-131.3, 99.6)
- moved R29 17.0 mm to (-123.3, 107.4)
- moved U22 16.7 mm to (-120.3, 108.0)
- moved R30 16.4 mm to (-123.4, 114.0)
- moved F8 15.0 mm to (-149.5, 90.3)
- moved F7 14.1 mm to (-149.5, 86.3)
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Changed lines of the file:
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@@
 	(footprint "Fuse:Fuse_1812_4532Metric"
 		(layer "F.Cu")
-		(at -142.4 108.5)
+		(at -149.475 98.725)
 		(descr "Fuse SMD 1812 (4532 Metric), square (rectangular) end terminal, IPC_7351 nominal, (Body size source: https://www.nikhef.nl/pub/departments/mt/projects/detectorR_D/dtddice/ERJ2G.pdf), generated with kicad-footprint-generator")
 		(tags "fuse")
@@
 	(footprint "footprints:TE_T4140012121-000"
 		(layer "F.Cu")
-		(at -157.07 101.9)
+		(at 20.139 42.158)
 		(property "Reference" "J20"
 			(at -0.325 -10.885 0)
@@
 	(footprint "Resistor_SMD:R_0201_0603Metric"
 		(layer "F.Cu")
-		(at -142.2 111.85)
+		(at -119.855 92.825)
 		(descr "Resistor SMD 0201 (0603 Metric), square (rectangular) end terminal, IPC_7351 nominal, (Body size source: https://www.vishay.com/docs/20052/crcw0201e3.pdf), generated with kicad-footprint-generator")
 		(tags "resistor")
@@
 	(footprint "Resistor_SMD:R_0201_0603Metric"
 		(layer "F.Cu")
-		(at -142.2 115.35)
+		(at -125.25 99.65)
 		(descr "Resistor SMD 0201 (0603 Metric), square (rectangular) end terminal, IPC_7351 nominal, (Body size source: https://www.vishay.com/docs/20052/crcw0201e3.pdf), generated with kicad-footprint-generator")
 		(tags "resistor")
@@
 	(footprint "Package_TO_SOT_SMD:SOT-363_SC-70-6"
 		(layer "F.Cu")
-		(at -136.8 93.175)
+		(at -125.825 86)
 		(descr "SOT-363, SC-70-6, SC-88")
 		(tags "SOT-363 SC-70-6 SC-88")
@@
 	(footprint "Resistor_SMD:R_0201_0603Metric"
 		(layer "F.Cu")
-		(at -144.65 113.6)
+		(at -172.355 122.525)
 		(descr "Resistor SMD 0201 (0603 Metric), square (rectangular) end terminal, IPC_7351 nominal, (Body size source: https://www.vishay.com/docs/20052/crcw0201e3.pdf), generated with kicad-footprint-generator")
 		(tags "resistor")
@@
 	(footprint "Resistor_SMD:R_0201_0603Metric"
 		(layer "F.Cu")
-		(at -142.2 117.1)
+		(at -131.275 99.625)
 		(descr "Resistor SMD 0201 (0603 Metric), square (rectangular) end terminal, IPC_7351 nominal, (Body size source: https://www.vishay.com/docs/20052/crcw0201e3.pdf), generated with kicad-footprint-generator")
 		(tags "resistor")
@@
 	(footprint "Resistor_SMD:R_0201_0603Metric"
 		(layer "F.Cu")
-		(at -142.2 113.6)
+		(at -126.23 92.825)
 		(descr "Resistor SMD 0201 (0603 Metric), square (rectangular) end terminal, IPC_7351 nominal, (Body size source: https://www.vishay.com/docs/20052/crcw0201e3.pdf), generated with kicad-footprint-generator")
 		(tags "resistor")
@@
 	(footprint "Package_TO_SOT_SMD:SOT-363_SC-70-6"
 		(layer "F.Cu")
-		(at -136.8 97.1)
+		(at -123.15 93.475)
 		(descr "SOT-363, SC-70-6, SC-88")
 		(tags "SOT-363 SC-70-6 SC-88")
@@
 	(footprint "Resistor_SMD:R_0201_0603Metric"
 		(layer "F.Cu")
-		(at -139.75 113.6)
+		(at -123.355 113.95)
 		(descr "Resistor SMD 0201 (0603 Metric), square (rectangular) end terminal, IPC_7351 nominal, (Body size source: https://www.vishay.com/docs/20052/crcw0201e3.pdf), generated with kicad-footprint-generator")
 		(tags "resistor")
@@
 	(footprint "Package_TO_SOT_SMD:SOT-363_SC-70-6"
 		(layer "F.Cu")
-		(at -136.8 101.025)
+		(at -128.25 100.275)
 		(descr "SOT-363, SC-70-6, SC-88")
 		(tags "SOT-363 SC-70-6 SC-88")
@@
 	(footprint "Fuse:Fuse_1812_4532Metric"
 		(layer "F.Cu")
-		(at -142.4 93.65)
+		(at -149.45 82.4)
 		(descr "Fuse SMD 1812 (4532 Metric), square (rectangular) end terminal, IPC_7351 nominal, (Body size source: https://www.nikhef.nl/pub/departments/mt/projects/detectorR_D/dtddice/ERJ2G.pdf), generated with kicad-footprint-generator")
 		(tags "fuse")
@@
 	(footprint "Fuse:Fuse_1812_4532Metric"
 		(layer "F.Cu")
-		(at -142.4 98.6)
+		(at -149.475 86.35)
 		(descr "Fuse SMD 1812 (4532 Metric), square (rectangular) end terminal, IPC_7351 nominal, (Body size source: https://www.nikhef.nl/pub/departments/mt/projects/detectorR_D/dtddice/ERJ2G.pdf), generated with kicad-footprint-generator")
 		(tags "fuse")
@@
 	(footprint "Capacitor_SMD:C_0201_0603Metric"
 		(layer "F.Cu")
-		(at -144.65 111.85)
+		(at -147.325 102.2 -90)
 		(descr "Capacitor SMD 0201 (0603 Metric), square (rectangular) end terminal, IPC_7351 nominal, (Body size source: https://www.vishay.com/docs/20052/crcw0201e3.pdf), generated with kicad-footprint-generator")
 		(tags "capacitor")
 		(property "Reference" "C37"
-			(at 0 -1.05 0)
+			(at 0 -1.05 90)
 			(layer "F.SilkS")
 			(effects
@@
 		)
 		(property "Value" "10u"
-			(at 0 1.05 0)
+			(at 0 1.05 90)
 			(layer "F.Fab")
 			(effects
@@
 		)
 		(property "Datasheet" ""
-			(at 0 0 0)
+			(at 0 0 270)
 			(unlocked yes)
 			(layer "F.Fab")
@@
 		)
 		(property "Description" "Unpolarized capacitor"
-			(at 0 0 0)
+			(at 0 0 270)
 			(unlocked yes)
 			(layer "F.Fab")
@@
 		)
 		(property "jlcpcb" "C96446"
-			(at 0 0 0)
+			(at 0 0 270)
 			(unlocked yes)
 			(layer "F.Fab")
@@
 		(attr smd)
 		(fp_line
-			(start -0.7 -0.35)
-			(end 0.7 -0.35)
+			(start -0.7 0.35)
+			(end -0.7 -0.35)
 			(stroke
 				(width 0.05)
@@
 		)
 		(fp_line
-			(start -0.7 0.35)
-			(end -0.7 -0.35)
+			(start 0.7 0.35)
+			(end -0.7 0.35)
 			(stroke
 				(width 0.05)
@@
 		)
 		(fp_line
-			(start 0.7 -0.35)
-			(end 0.7 0.35)
+			(start -0.7 -0.35)
+			(end 0.7 -0.35)
 			(stroke
 				(width 0.05)
@@
 		)
 		(fp_line
-			(start 0.7 0.35)
-			(end -0.7 0.35)
+			(start 0.7 -0.35)
+			(end 0.7 0.35)
 			(stroke
 				(width 0.05)
@@
 		)
 		(fp_line
-			(start -0.3 -0.15)
-			(end 0.3 -0.15)
+			(start -0.3 0.15)
+			(end -0.3 -0.15)
 			(stroke
 				(width 0.1)
@@
 		)
 		(fp_line
-			(start -0.3 0.15)
-			(end -0.3 -0.15)
+			(start 0.3 0.15)
+			(end -0.3 0.15)
 			(stroke
 				(width 0.1)
@@
 		)
 		(fp_line
-			(start 0.3 -0.15)
-			(end 0.3 0.15)
+			(start -0.3 -0.15)
+			(end 0.3 -0.15)
 			(stroke
 				(width 0.1)
@@
 		)
 		(fp_line
-			(start 0.3 0.15)
-			(end -0.3 0.15)
+			(start 0.3 -0.15)
+			(end 0.3 0.15)
 			(stroke
 				(width 0.1)
@@
 		)
 		(fp_text user "${REFERENCE}"
-			(at 0 -0.68 0)
+			(at 0 -0.68 90)
 			(layer "F.Fab")
 			(effects
@@
 		)
 		(pad "" smd roundrect
-			(at -0.345 0)
+			(at -0.345 0 270)
 			(size 0.318 0.36)
 			(layers "F.Paste")
@@
 		)
 		(pad "" smd roundrect
-			(at 0.345 0)
+			(at 0.345 0 270)
 			(size 0.318 0.36)
 			(layers "F.Paste")
@@
 		)
 		(pad "1" smd roundrect
-			(at -0.32 0)
+			(at -0.32 0 270)
 			(size 0.46 0.4)
 			(layers "F.Cu" "F.Mask")
@@
 		)
 		(pad "2" smd roundrect
-			(at 0.32 0)
+			(at 0.32 0 270)
 			(size 0.46 0.4)
 			(layers "F.Cu" "F.Mask")
@@
 	(footprint "Package_TO_SOT_SMD:SOT-363_SC-70-6"
 		(layer "F.Cu")
-		(at -136.8 104.95)
+		(at -120.35 108.05)
 		(descr "SOT-363, SC-70-6, SC-88")
 		(tags "SOT-363 SC-70-6 SC-88")
@@
 	(footprint "Package_TO_SOT_SMD:SOT-363_SC-70-6"
 		(layer "F.Cu")
-		(at -136.8 108.875)
+		(at -126.275 114.6)
 		(descr "SOT-363, SC-70-6, SC-88")
 		(tags "SOT-363 SC-70-6 SC-88")
@@
 	(footprint "Resistor_SMD:R_0201_0603Metric"
 		(layer "F.Cu")
-		(at -142.2 118.85)
+		(at -117.275 107.425)
 		(descr "Resistor SMD 0201 (0603 Metric), square (rectangular) end terminal, IPC_7351 nominal, (Body size source: https://www.vishay.com/docs/20052/crcw0201e3.pdf), generated with kicad-footprint-generator")
 		(tags "resistor")
@@
 	(footprint "Resistor_SMD:R_0201_0603Metric"
 		(layer "F.Cu")
-		(at -144.65 118.85)
+		(at -128.825 85.35)
 		(descr "Resistor SMD 0201 (0603 Metric), square (rectangular) end terminal, IPC_7351 nominal, (Body size source: https://www.vishay.com/docs/20052/crcw0201e3.pdf), generated with kicad-footprint-generator")
 		(tags "resistor")
@@
 	(footprint "Resistor_SMD:R_0201_0603Metric"
 		(layer "F.Cu")
-		(at -139.75 111.85)
+		(at -123.325 107.4)
 		(descr "Resistor SMD 0201 (0603 Metric), square (rectangular) end terminal, IPC_7351 nominal, (Body size source: https://www.vishay.com/docs/20052/crcw0201e3.pdf), generated with kicad-footprint-generator")
 		(tags "resistor")
@@
 	(footprint "Resistor_SMD:R_0201_0603Metric"
 		(layer "F.Cu")
-		(at -144.65 115.35)
+		(at -165.755 124.825)
 		(descr "Resistor SMD 0201 (0603 Metric), square (rectangular) end terminal, IPC_7351 nominal, (Body size source: https://www.vishay.com/docs/20052/crcw0201e3.pdf), generated with kicad-footprint-generator")
 		(tags "resistor")
@@
 	(footprint "Resistor_SMD:R_0201_0603Metric"
 		(layer "F.Cu")
-		(at -144.65 117.1)
+		(at -122.825 85.35)
 		(descr "Resistor SMD 0201 (0603 Metric), square (rectangular) end terminal, IPC_7351 nominal, (Body size source: https://www.vishay.com/docs/20052/crcw0201e3.pdf), generated with kicad-footprint-generator")
 		(tags "resistor")
@@
 	(footprint "Resistor_SMD:R_0201_0603Metric"
 		(layer "F.Cu")
-		(at -139.75 115.35)
+		(at -129.425 113.95)
 		(descr "Resistor SMD 0201 (0603 Metric), square (rectangular) end terminal, IPC_7351 nominal, (Body size source: https://www.vishay.com/docs/20052/crcw0201e3.pdf), generated with kicad-footprint-generator")
 		(tags "resistor")
@@
 	(footprint "Fuse:Fuse_1812_4532Metric"
 		(layer "F.Cu")
-		(at -142.4 103.55)
+		(at -149.525 90.325)
 		(descr "Fuse SMD 1812 (4532 Metric), square (rectangular) end terminal, IPC_7351 nominal, (Body size source: https://www.nikhef.nl/pub/departments/mt/projects/detectorR_D/dtddice/ERJ2G.pdf), generated with kicad-footprint-generator")
 		(tags "fuse")

Commit message: finished placing M12P12 connector and components from solenoid interface sheet.
Parts:
- moved R21 295.0 mm to (116.9, 209.3)
- moved LED7 294.9 mm to (114.6, 209.2), turned to 180 degrees
- moved R20 294.9 mm to (117.0, 179.5)
- moved LED6 287.9 mm to (114.6, 179.5), turned to 180 degrees
- moved C37 284.7 mm to (118.1, 205.3)
- moved F6 284.7 mm to (116.0, 185.5)
- moved F7 284.7 mm to (116.0, 189.4)
- moved F8 284.7 mm to (115.9, 193.4)
- moved F9 284.7 mm to (116.0, 201.8)
- moved R23 247.8 mm to (87.1, 207.0), turned to 90 degrees
- moved U19 244.0 mm to (87.8, 204.0), turned to 90 degrees
- moved R31 240.1 mm to (95.1, 199.1), turned to 90 degrees
- moved R22 239.7 mm to (87.1, 201.0), turned to 90 degrees
- moved U23 236.5 mm to (95.7, 196.0), turned to 90 degrees
- moved R29 233.0 mm to (95.0, 188.9), turned to 90 degrees
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