File: mega_shield/mega_shield.kicad_pcb (KiCad board)
At the start: 2 copper layers, 306 parts, among them J1 T4140012081-000, J10 T4040014031-000, J11 T4040014031-000, J12 T4040014031-000, J13 T4040014031-000, J14 1757242, J15 1757242, J16 T4040014031-000, J17 T4040014031-000, J18 T4040014031-000, J19 T4040014031-000, J2 T4140012081-000, J20 T4140012121-000, J3 1757271, J4 T4140012081-000, J5 T4140012081-000, J6 T4140012081-000, J8 T4040014031-000, J9 T4040014031-000, Q1 2SK3018, Q10 2SK3018, Q11 2SK3018, Q12 2SK3018, Q13 2SK3018, Q14 2SK3018, Q15 2SK3018, Q16 2SK3018, Q17 2SK3018, Q18 2SK3018, Q19 2SK3018, Q2 2SK3018, Q20 2SK3018, Q21 2SK3018, Q22 2SK3018, Q23 2SK3018, Q24 2SK3018, Q25 2SK3018, Q26 2SK3018, Q27 2SK3018, Q28 2SK3018, Q29 2SK3018, Q3 2SK3018, Q30 2SK3018, Q31 2SK3018, Q32 2SK3018, Q33 2SK3018, Q34 2SK3018, Q35 2SK3018, Q36 2SK3018, Q37 2SK3018, Q38 2SK3018, Q39 2SK3018, Q4 2SK3018, Q40 2SK3018, Q41 2SK3018, Q42 2SK3018, Q5 2SK3018, Q6 2SK3018, Q7 2SK3018, Q8 2SK3018, Q9 2SK3018, U1 CS817x22HS, U10 CS817x22HS, U11 CS817x22HS, U12 CS817x22HS, U13 CS817x22HS, U14 CS817x22HS, U15 CS817x22HS, U16 CS817x22HS, U17 CS817x22HS, U18 CS817x22HS, U19 NUP2202, U2 CS817x22HS, U20 NUP2202, U21 NUP2202, U22 NUP2202, U23 NUP2202, U24 CS817x22HS, U25 CS817x22HS, U26 CS817x22HS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

Commit message: ungrouped layout of all proxy connections groups. Adjusted group X for smaller footprint.
Parts:
- moved D1 165.3 mm to (31.4, 239.8)
- moved F11 165.3 mm to (20.4, 237.8)
- moved J14 165.3 mm to (-1.25, 234.3)
- moved F12 115.2 mm to (19.7, 254.6)
- moved J15 115.2 mm to (-1.35, 251.0)
- moved D2 115.2 mm to (30.3, 255.9)
- moved C52 56.1 mm to (201.2, 244.5)
- moved C53 56.1 mm to (201.2, 239.5)
- moved R38 56.1 mm to (201.7, 236.4)
- moved R39 56.1 mm to (207.2, 236.4)
- moved TP90 56.1 mm to (214.4, 250.2)
- moved TP91 56.1 mm to (196.3, 250.2)
- moved TP93 56.1 mm to (222.3, 250.2)
- moved U27 56.1 mm to (205.4, 242.0)
- moved C50 56.1 mm to (223.6, 260.1)
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
Commit message: Tightened spacing of the X axis sensor group.
Parts:
- moved C48 2.97 mm to (109.2, 51.5)
- moved C49 2.97 mm to (109.2, 56.5)
- moved Q37 2.97 mm to (115.6, 52.0)
- moved R36 2.97 mm to (118.7, 53.0)
- moved R37 2.97 mm to (99.2, 52.9)
- moved U26 2.97 mm to (105.0, 54.0)
- moved Q38 2.97 mm to (96.1, 52.0)
- moved TP84 1.67 mm to (105.1, 47.0)
- moved TP85 1.67 mm to (96.0, 47.1)
- moved TP86 1.67 mm to (114.1, 47.1)
- moved TP87 1.67 mm to (121.4, 47.1)
- moved TP88 1.67 mm to (88.1, 47.1)
Changed lines of the file:
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@@
 	(footprint "TestPoint:TestPoint_Pad_1.0x1.0mm"
 		(layer "F.Cu")
-		(at 121.4 48.790575)
+		(at 121.4 47.125)
 		(descr "SMD rectangular pad as test Point, square 1.0mm side length")
 		(tags "test point SMD pad rectangle square")
@@
 	(footprint "Capacitor_SMD:C_0201_0603Metric"
 		(layer "F.Cu")
-		(at 109.17 59.440575)
+		(at 109.17 56.475)
 		(descr "Capacitor SMD 0201 (0603 Metric), square (rectangular) end terminal, IPC_7351 nominal, (Body size source: https://www.vishay.com/docs/20052/crcw0201e3.pdf), generated with kicad-footprint-generator")
 		(tags "capacitor")
@@
 	(footprint "Capacitor_SMD:C_0201_0603Metric"
 		(layer "F.Cu")
-		(at 109.17 54.465575)
+		(at 109.17 51.5)
 		(descr "Capacitor SMD 0201 (0603 Metric), square (rectangular) end terminal, IPC_7351 nominal, (Body size source: https://www.vishay.com/docs/20052/crcw0201e3.pdf), generated with kicad-footprint-generator")
 		(tags "capacitor")
@@
 	(footprint "TestPoint:TestPoint_Pad_1.0x1.0mm"
 		(layer "F.Cu")
-		(at 114.125 48.740575)
+		(at 114.125 47.075)
 		(descr "SMD rectangular pad as test Point, square 1.0mm side length")
 		(tags "test point SMD pad rectangle square")
@@
 	(footprint "Resistor_SMD:R_0201_0603Metric"
 		(layer "F.Cu")
-		(at 118.695 55.975 180)
+		(at 118.695 53.009425 180)
 		(descr "Resistor SMD 0201 (0603 Metric), square (rectangular) end terminal, IPC_7351 nominal, (Body size source: https://www.vishay.com/docs/20052/crcw0201e3.pdf), generated with kicad-footprint-generator")
 		(tags "resistor")
@@
 	(footprint "TestPoint:TestPoint_Pad_1.0x1.0mm"
 		(layer "F.Cu")
-		(at 96.025 48.740575)
+		(at 96.025 47.075)
 		(descr "SMD rectangular pad as test Point, square 1.0mm side length")
 		(tags "test point SMD pad rectangle square")
@@
 	(footprint "Resistor_SMD:R_0201_0603Metric"
 		(layer "F.Cu")
-		(at 99.175 55.9 180)
+		(at 99.175 52.934425 180)
 		(descr "Resistor SMD 0201 (0603 Metric), square (rectangular) end terminal, IPC_7351 nominal, (Body size source: https://www.vishay.com/docs/20052/crcw0201e3.pdf), generated with kicad-footprint-generator")
 		(tags "resistor")
@@
 	(footprint "Package_SO:SOIC-8_3.9x4.9mm_P1.27mm"
 		(layer "F.Cu")
-		(at 105 56.940575 -90)
+		(at 105 53.975 -90)
 		(descr "SOIC, 8 Pin (JEDEC MS-012AA, https://www.analog.com/media/en/package-pcb-resources/package/pkg_pdf/soic_narrow-r/r_8.pdf), generated with kicad-footprint-generator ipc_gullwing_generator.py")
 		(tags "SOIC SO")
@@
 	(footprint "PCM_Package_TO_SOT_SMD_AKL:SOT-323_SC-70"
 		(layer "F.Cu")
-		(at 115.575 54.975 90)
+		(at 115.575 52.009425 90)
 		(descr "SOT-323, SC-70, Alternate KiCad Library")
 		(tags "SOT-323 SC-70")
@@
 	(footprint "TestPoint:TestPoint_Pad_1.0x1.0mm"
 		(layer "F.Cu")
-		(at 88.1 48.740575)
+		(at 88.1 47.075)
 		(descr "SMD rectangular pad as test Point, square 1.0mm side length")
 		(tags "test point SMD pad rectangle square")
@@
 	(footprint "PCM_Package_TO_SOT_SMD_AKL:SOT-323_SC-70"
 		(layer "F.Cu")
-		(at 96.075 54.925 90)
+		(at 96.075 51.959425 90)
 		(descr "SOT-323, SC-70, Alternate KiCad Library")
 		(tags "SOT-323 SC-70")
@@
 	(footprint "TestPoint:TestPoint_Pad_1.0x1.0mm"
 		(layer "F.Cu")
-		(at 105.075 48.665575)
+		(at 105.075 47)
 		(descr "SMD rectangular pad as test Point, square 1.0mm side length")
 		(tags "test point SMD pad rectangle square")

Commit message: replicated layout accross all axis sensor groups.
Parts:
- moved Q35 15.8 mm to (158.3, -0.91), turned to 90 degrees
- moved Q33 15.8 mm to (210.1, 10.1), turned to 90 degrees
- moved Q39 15.8 mm to (194.8, 247.0), turned to -90 degrees
- moved Q41 15.8 mm to (132.8, 229.5), turned to -90 degrees
- moved Q40 15.0 mm to (214.3, 247.0), turned to -90 degrees
- moved Q42 15.0 mm to (152.3, 229.5), turned to -90 degrees
- moved Q34 15.0 mm to (190.6, 10.0), turned to 90 degrees
- moved Q36 15.0 mm to (138.8, -0.96), turned to 90 degrees
- moved R32 13.8 mm to (213.2, 11.1), turned to 180 degrees
- moved R34 13.8 mm to (161.4, 0.09), turned to 180 degrees
- moved R38 13.8 mm to (191.7, 246.0), turned to 0 degrees
- moved R40 13.8 mm to (129.7, 228.5), turned to 0 degrees
- moved R39 10.5 mm to (211.2, 246.1), turned to 0 degrees
- moved R41 10.5 mm to (149.2, 228.6), turned to 0 degrees
- moved R35 10.5 mm to (141.9, 0.02), turned to 180 degrees
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
Commit message: Imported mounting holes.
Parts:
- added H1: MountingHole_Pad, MountingHole:MountingHole_3.2mm_M3_DIN965_Pad, F.Cu at (-40.4, 46.5)
- added H2: MountingHole_Pad, MountingHole:MountingHole_3.2mm_M3_DIN965_Pad, F.Cu at (-40.4, 53.6)
- added H3: MountingHole_Pad, MountingHole:MountingHole_3.2mm_M3_DIN965_Pad, F.Cu at (-40.4, 60.8)
- added H4: MountingHole_Pad, MountingHole:MountingHole_3.2mm_M3_DIN965_Pad, F.Cu at (-40.4, 68.0)
- TP27: value +5V_SPIN -> TestPoint
- TP28: value SPIN_PWM -> TestPoint
- TP29: value SPIN_DIR -> TestPoint
- TP30: value SPIN_EN -> TestPoint
- TP31: value V_SPIN -> TestPoint
- TP32: value SPIN_SPEED -> TestPoint
- TP33: value SPIN_DIR_OC -> TestPoint
- TP34: value SPIN_EN_OC -> TestPoint

Commit message: updated schematic and PCB to use the mounting hole pads as ground connections.
Connections:
- H1 pad 1: unconnected-(H1-Pad1) -> GND
- H2 pad 1: unconnected-(H2-Pad1) -> GND
- H3 pad 1: unconnected-(H3-Pad1) -> GND
- H4 pad 1: unconnected-(H4-Pad1) -> GND
Changed lines of the file:
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@@
 	(net 227 "unconnected-(U23-Pad3)")
 	(net 228 "unconnected-(U23-Pad4)")
-	(net 229 "unconnected-(H1-Pad1)")
-	(net 230 "unconnected-(H2-Pad1)")
-	(net 231 "unconnected-(H3-Pad1)")
-	(net 232 "unconnected-(H4-Pad1)")
 	(footprint "TestPoint:TestPoint_Pad_1.0x1.0mm"
 		(layer "F.Cu")
@@
 			(layers "*.Cu" "*.Mask")
 			(remove_unused_layers no)
-			(net 230 "unconnected-(H2-Pad1)")
+			(net 2 "GND")
 			(pinfunction "1")
 			(pintype "input")
@@
 			(layers "*.Cu" "*.Mask")
 			(remove_unused_layers no)
-			(net 229 "unconnected-(H1-Pad1)")
+			(net 2 "GND")
 			(pinfunction "1")
 			(pintype "input")
@@
 			(layers "*.Cu" "*.Mask")
 			(remove_unused_layers no)
-			(net 231 "unconnected-(H3-Pad1)")
+			(net 2 "GND")
 			(pinfunction "1")
 			(pintype "input")
@@
 			(layers "*.Cu" "*.Mask")
 			(remove_unused_layers no)
-			(net 232 "unconnected-(H4-Pad1)")
+			(net 2 "GND")
 			(pinfunction "1")
 			(pintype "input")

Commit message: rotated the X-axis sensor group to position populated sensor connector on outter edge.
Parts:
- moved C47 28.1 mm to (97.9, 27.5), turned to 180 degrees
- moved C46 27.7 mm to (97.9, 64.2), turned to 180 degrees
- moved TP88 24.1 mm to (106.2, 63.0), turned to 90 degrees
- moved TP87 23.1 mm to (106.2, 29.7), turned to 90 degrees
- moved R36 21.7 mm to (112.1, 32.4), turned to -90 degrees
- moved J12 18.0 mm to (97.0, 55.8), turned to 90 degrees
- moved Q37 17.1 mm to (111.1, 35.5), turned to 180 degrees
- moved C49 15.9 mm to (115.5, 41.9), turned to 90 degrees
- moved Q38 15.3 mm to (111.0, 55.0), turned to 180 degrees
- moved J13 14.7 mm to (97.1, 39.4), turned to 90 degrees
- moved TP85 12.9 mm to (106.2, 55.0), turned to 90 degrees
- moved TP86 12.9 mm to (106.2, 37.0), turned to 90 degrees
- moved R37 12.9 mm to (112.0, 51.9), turned to -90 degrees
- moved U26 11.3 mm to (113.0, 46.1), turned to 0 degrees
- moved C48 9.70 mm to (110.6, 41.9), turned to 90 degrees
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
Commit message: flipped the mega interface
Parts:
- A1: moved to B.Cu
- moved J3 206.1 mm to (-40.6, 200.3), turned to 0 degrees
- moved TP31 172.8 mm to (-37.1, 183.2), turned to 90 degrees
- moved C13 172.7 mm to (-48.1, 175.3), turned to 90 degrees
- moved R7 169.8 mm to (-49.7, 172.0), turned to 0 degrees
- moved TP32 167.9 mm to (-32.0, 183.2), turned to 90 degrees
- moved C16 165.8 mm to (-40.0, 177.2), turned to 90 degrees
- moved R8 165.7 mm to (-46.6, 172.0), turned to 0 degrees
- moved C15 164.4 mm to (-38.7, 177.2), turned to 90 degrees
- moved TP33 163.4 mm to (-26.9, 183.3), turned to 90 degrees
- moved C14 162.2 mm to (-43.5, 172.3), turned to -90 degrees
- moved TP34 159.4 mm to (-21.9, 183.2), turned to 90 degrees
- moved U7 159.0 mm to (-39.3, 173.5), turned to -90 degrees
- moved U8 151.9 mm to (-32.9, 173.5), turned to 90 degrees
- moved U9 143.5 mm to (-24.3, 173.5), turned to 0 degrees
- moved Q14 141.7 mm to (-15.8, 176.0), turned to 180 degrees
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
Commit message: setup new revision of board layout.
Parts:
- moved H3 351.4 mm to (280.0, 205.0)
- moved H2 320.9 mm to (280.0, 35.0)
- moved C51 224.1 mm to (170.7, 36.6), turned to 180 degrees
- moved C55 218.9 mm to (198.7, 36.6), turned to 180 degrees
- moved J17 214.4 mm to (169.9, 48.5), turned to 90 degrees
- moved TP92 213.3 mm to (179.1, 38.8), turned to 90 degrees
- moved TP97 211.3 mm to (207.1, 38.8), turned to 90 degrees
- moved TP91 206.6 mm to (179.0, 46.1), turned to 90 degrees
- moved R40 204.6 mm to (212.9, 41.5), turned to -90 degrees
- moved R38 204.6 mm to (184.9, 41.5), turned to -90 degrees
- moved J19 204.4 mm to (197.9, 48.5), turned to 90 degrees
- moved C13 204.2 mm to (156.0, 180.3)
- moved C17 204.2 mm to (177.4, 174.7)
- moved C18 204.2 mm to (182.3, 174.7)
- moved Q14 204.2 mm to (188.3, 181.1)
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