File: mega_shield/digital_gpio.kicad_sch (KiCad schematic)
At the start: 2 parts, among them J23 1803277, Q46 AO4486

Commit message: Added design for discrete mosfet gate driver into the gpio sheet.
Parts:
- removed J23: 1803277, footprints:PHOENIX_1803277, symbol TERM_BLOCK_HDR_2POS_3.81MM:1803277
- removed Q46: AO4486, PCM_Package_SO_AKL:SO-8_3.9x4.9mm_P1.27mm, symbol PCM_Transistor_MOSFET_AKL:AO4486
- added C59, C62: 1u, Capacitor_SMD:C_0201_0603Metric, symbol Device:C
- added D5, D6: SM4007PL, PCM_Diode_SMD_AKL:D_SOD-123F, symbol PCM_Diode_AKL:SM4007PL
- added F14, F15: SMD1812P030TF, Fuse:Fuse_1812_4532Metric_Pad1.30x3.40mm_HandSolder, symbol Device:Polyfuse
- added J24, J25: 1803277, footprints:PHOENIX_1803277, symbol TERM_BLOCK_HDR_2POS_3.81MM:1803277
- added Q46, Q47: MMBT3904, PCM_Package_TO_SOT_SMD_AKL:SOT-23, symbol PCM_Transistor_BJT_AKL:MMBT3904
- added Q49, Q52: AO4486, PCM_Package_SO_AKL:SO-8_3.9x4.9mm_P1.27mm, symbol PCM_Transistor_MOSFET_AKL:AO4486
- added Q50, Q51: MMBT3906, PCM_Package_TO_SOT_SMD_AKL:SOT-23, symbol PCM_Transistor_BJT_AKL:MMBT3906
- added R49, R51: 10k, symbol Device:R
- added R50, R52: 100, symbol Device:R
- added U31: CS817x22HS, Package_SO:SOIC-8_3.9x4.9mm_P1.27mm, symbol mega_shield:CS817x20HS
Connections:
- net +24V_IN: now also C62.2, F14.1, F15.1, Q46.3 (C), Q47.3 (C), U31.8 (VDD2)
- net +5V_IN: now also C59.1, U31.1 (VDD1)
- net GND: now also C59.2, C62.1, Q49.1 (S), Q49.2 (S), Q49.3 (S), Q50.3 (C), Q51.3 (C), Q52.1 (S), Q52.2 (S), Q52.3 (S), R49.2, R51.2, U31.4 (GND1), U31.5 (GND2)
- net digital_out1: now also U31.2 (INA)
- net digital_out2: now also U31.3 (INB)
- new net: D6.1 (K), F15.2, J25.01
- new net: D6.2 (A), J25.02, Q52.5 (D), Q52.6 (D), Q52.7 (D), Q52.8 (D)
- new net: Q46.2 (E), Q50.2 (E), R50.1
- new net: D5.1 (K), F14.2, J24.01
- new net: D5.2 (A), J24.02, Q49.5 (D), Q49.6 (D), Q49.7 (D), Q49.8 (D)
- new net: Q47.2 (E), Q51.2 (E), R52.1
- new net driver_input_A: Q46.1 (B), Q50.1 (B), R49.1, U31.7 (OUTA)
- new net driver_input_B: Q47.1 (B), Q51.1 (B), R51.1, U31.6 (OUTB)
- new net vgate_A: Q49.4 (G), R50.2
- new net vgate_B: Q52.4 (G), R52.2
Other:
- note added: "Digital Isolator(Channels A/B)"
- note added: "MOSFET Channel A"
- note added: "Mosfet Gate Drivers(Channels A/B)"

Commit message: Added PNP and NPN transistor jlcpcb numbers.
Parts:
- Q46, Q47: jlcpcb (none) -> C20526
- Q50, Q51: jlcpcb (none) -> C2891809
Changed lines of the file:
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@@
+			)
+		)
+		(property "jlcpcb" "C2891809"
+			(at 129.54 74.93 0)
+			(effects
+				(font
+					(size 1.27 1.27)
+				)
 			)
 		)
@@
 			)
 		)
+		(property "jlcpcb" "C20526"
+			(at 129.54 102.87 0)
+			(effects
+				(font
+					(size 1.27 1.27)
+				)
+			)
+		)
 		(pin "3"
 		)
@@
 			)
 		)
+		(property "jlcpcb" "C20526"
+			(at 129.54 62.23 0)
+			(effects
+				(font
+					(size 1.27 1.27)
+				)
+			)
+		)
 		(pin "3"
 		)
@@
 			)
 		)
+		(property "jlcpcb" "C2891809"
+			(at 129.54 115.57 0)
+			(effects
+				(font
+					(size 1.27 1.27)
+				)
+			)
+		)

Commit message: Added footprints and jlcpcb numbers for the resistors in the gate driver circuits.
Parts:
- R49, R51: footprint (none) -> Resistor_SMD:R_0201_0603Metric; jlcpcb (none) -> C25804
- R50, R52: footprint (none) -> Resistor_SMD:R_0201_0603Metric; jlcpcb (none) -> C22775
Changed lines of the file:
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@@
 			)
 		)
-		(property "Footprint" ""
+		(property "Footprint" "Resistor_SMD:R_0201_0603Metric"
 			(at 140.97 70.358 90)
 			(effects
@@
 			)
 		)
+		(property "jlcpcb" "C22775"
+			(at 140.97 68.58 0)
+			(effects
+				(font
+					(size 1.27 1.27)
+				)
+			)
+		)
 		(pin "2"
 		)
@@
 			)
 		)
-		(property "Footprint" ""
+		(property "Footprint" "Resistor_SMD:R_0201_0603Metric"
 			(at 115.062 115.57 90)
 			(effects
@@
 				)
 				(hide yes)
+			)
+		)
+		(property "jlcpcb" "C25804"
+			(at 116.84 115.57 0)
+			(effects
+				(font
+					(size 1.27 1.27)
+				)
 			)
 		)
@@
 			)
 		)
-		(property "Footprint" ""
+		(property "Footprint" "Resistor_SMD:R_0201_0603Metric"
 			(at 115.062 74.93 90)
 			(effects
@@
 			)
 		)
+		(property "jlcpcb" "C25804"
+			(at 116.84 74.93 0)
+			(effects
+				(font
+					(size 1.27 1.27)
+				)
+			)
+		)
 		(pin "2"
 		)
@@
 			)
 		)
-		(property "Footprint" ""
+		(property "Footprint" "Resistor_SMD:R_0201_0603Metric"
 			(at 140.97 110.998 90)
 			(effects
@@
 			)
 		)
+		(property "jlcpcb" "C22775"
+			(at 140.97 109.22 0)
+			(effects
+				(font
+					(size 1.27 1.27)
+				)
+			)
+		)

Commit message: Added jlcpcb number to the snubber diodes used in the solenoid drivers and gpio output.
Parts:
- D5, D6: jlcpcb (none) -> C64898
Changed lines of the file:
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@@
+			)
+		)
+		(property "jlcpcb" "C64898"
+			(at 217.17 49.53 0)
+			(effects
+				(font
+					(size 1.27 1.27)
+				)
 			)
 		)
@@
 			(at 217.17 116.84 0)
 			(effects
+				(font
+					(size 1.27 1.27)
+				)
+			)
+		)
+		(property "jlcpcb" "C64898"
+			(at 217.17 116.84 0)
+			(effects

Commit message: changed the single polyfuse for a dual polyfuse setup for higher holding current. Added jlcpcb numbers for them as well.
Parts:
- added F16, F17: SMD1812P200TF/30, symbol Device:Polyfuse
- F14, F15: value SMD1812P030TF -> SMD1812P200TF/30; footprint Fuse:Fuse_1812_4532Metric_Pad1.30x3.40mm_HandSolder -> (none); JLCPCB C20995 -> (none); jlcpcb (none) -> C5188720
Connections:
- net +24V_IN: now also F16.1, F17.1
- net at D6.1 (K), J25.01: now also F16.2, F17.2; no longer F15.2
- net at D5.1 (K), F14.2, J24.01: now also F15.2
Changed lines of the file:
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@@
 		)
 	)
-	(text_box "Selected N-Channel MOSFET: AO4486\nContinuous Drain Current(T_ambiant = 25C): 4.2A\nContinuous Drain Current(T_ambiant = 70C): 3.4A"
+	(text_box "Selected N-Channel MOSFET: AO4486\nContinuous Drain Current(T_ambiant = 25C): 4.2A\nContinuous Drain Current(T_ambiant = 70C): 3.4A\n\nFor safety the current is limited through the polyfuses approximatly 4A\nunder ideal conditions."
 		(exclude_from_sim no)
-		(at 198.12 12.7 0)
-		(size 50.8 10.16)
+		(at 101.6 152.4 0)
+		(size 50.8 25.4)
 		(margins 0.9525 0.9525 0.9525 0.9525)
 		(stroke
@@
 	)
 	(junction
+		(at 195.58 49.53)
+		(diameter 0)
+		(color 0 0 0 0)
+	)
+	(junction
 		(at 223.52 62.23)
+		(diameter 0)
+		(color 0 0 0 0)
+	)
+	(junction
+		(at 195.58 116.84)
 		(diameter 0)
 		(color 0 0 0 0)
@@
 	)
 	(junction
+		(at 203.2 49.53)
+		(diameter 0)
+		(color 0 0 0 0)
+	)
+	(junction
 		(at 116.84 68.58)
 		(diameter 0)
@@
 	)
 	(junction
+		(at 203.2 116.84)
+		(diameter 0)
+		(color 0 0 0 0)
+	)
+	(junction
 		(at 132.08 68.58)
 		(diameter 0)
@@
 	(wire
 		(pts
+			(xy 195.58 45.72) (xy 195.58 49.53)
+		)
+		(stroke
+			(width 0)
+			(type default)
+		)
+	)
+	(wire
+		(pts
 			(xy 102.87 68.58) (xy 116.84 68.58)
 		)
@@
 	(wire
 		(pts
+			(xy 193.04 116.84) (xy 195.58 116.84)
+		)
+		(stroke
+			(width 0)
+			(type default)
+		)
+	)
+	(wire
+		(pts
 			(xy 220.98 49.53) (xy 223.52 49.53)
 		)
@@
 	(wire
 		(pts
+			(xy 203.2 113.03) (xy 203.2 116.84)
+		)
+		(stroke
+			(width 0)
+			(type default)
+		)
+	)
+	(wire
+		(pts
 			(xy 132.08 95.25) (xy 132.08 97.79)
 		)
@@
 	(wire
 		(pts
+			(xy 203.2 45.72) (xy 203.2 49.53)
+		)
+		(stroke
+			(width 0)
+			(type default)
+		)
+	)
+	(wire
+		(pts
 			(xy 132.08 67.31) (xy 132.08 68.58)
 		)
@@
 	(wire
 		(pts
-			(xy 193.04 116.84) (xy 195.58 116.84)
-		)
-		(stroke
-			(width 0)
-			(type default)
-		)
-	)
-	(wire
-		(pts
 			(xy 215.9 62.23) (xy 218.44 62.23)
 		)
@@
 		(pts
 			(xy 144.78 109.22) (xy 149.86 109.22)
+		)
+		(stroke
+			(width 0)
+			(type default)
+		)
+	)
+	(wire
+		(pts
+			(xy 195.58 113.03) (xy 195.58 116.84)
 		)
 		(stroke
@@
 		)
 	)
+	(hierarchical_label "+24V_IN"
+		(shape input)
+		(at 193.04 116.84 180)
+		(effects
+			(font
+				(size 1.27 1.27)
+			)
+			(justify right)
+		)
+	)
 	(hierarchical_label "digital_out1"
 		(shape input)
@@
 		(shape input)
 		(at 43.18 92.71 180)
-		(effects
-			(font
-				(size 1.27 1.27)
-			)
-			(justify right)
-		)
-	)
-	(hierarchical_label "+24V_IN"
-		(shape input)
-		(at 193.04 116.84 180)
 		(effects
 			(font
@@
 		(on_board yes)
 		(dnp no)
-		(fields_autoplaced yes)
-		(property "Reference" "F15"
+		(property "Reference" "F17"
 			(at 199.39 123.19 90)
 			(effects
@@
 			)
 		)
-		(property "Value" "SMD1812P030TF"
+		(property "Value" "SMD1812P200TF/30"
 			(at 199.39 120.65 90)
 			(effects
@@
 			)
 		)
-		(property "Footprint" "Fuse:Fuse_1812_4532Metric_Pad1.30x3.40mm_HandSolder"
+		(property "Footprint" ""
 			(at 204.47 118.11 0)
 			(effects
@@
 			)
 		)
-		(property "JLCPCB" "C20995"
-			(at 199.39 116.84 0)
+		(property "jlcpcb" "C5188720"
+			(at 199.39 118.872 90)
 			(effects
 				(font
@@
 			(project "mega_shield"
 				(path "/554fcf27-dc63-4666-abbc-7481d15942c4/32d6b15b-5472-4f1d-a1b7-d12adc0e25c3"
-					(reference "F15")
+					(reference "F17")
 					(unit 1)
 				)
@@
 		(on_board yes)
 		(dnp no)
-		(fields_autoplaced yes)
-		(property "Reference" "F14"
+		(property "Reference" "F15"
 			(at 199.39 55.88 90)
 			(effects
@@
 			)
 		)
-		(property "Value" "SMD1812P030TF"
+		(property "Value" "SMD1812P200TF/30"
 			(at 199.39 53.34 90)
 			(effects
@@
 			)
 		)
-		(property "Footprint" "Fuse:Fuse_1812_4532Metric_Pad1.30x3.40mm_HandSolder"
+		(property "Footprint" ""
 			(at 204.47 50.8 0)
 			(effects
@@
 			)
 		)
-		(property "JLCPCB" "C20995"
-			(at 199.39 49.53 0)
+		(property "jlcpcb" "C5188720"
+			(at 199.39 51.816 90)
 			(effects
 				(font
@@
 			(project "mega_shield"
 				(path "/554fcf27-dc63-4666-abbc-7481d15942c4/32d6b15b-5472-4f1d-a1b7-d12adc0e25c3"
-					(reference "F14")
+					(reference "F15")
 					(unit 1)
 				)
@@
 	)
 	(symbol
+		(lib_id "Device:Polyfuse")
+		(at 199.39 45.72 90)
+		(unit 1)
+		(exclude_from_sim no)
+		(in_bom yes)
+		(on_board yes)
+		(dnp no)
+		(property "Reference" "F14"
+			(at 199.39 39.37 90)
+			(effects
+				(font
+					(size 1.27 1.27)
+				)
+			)
+		)
+		(property "Value" "SMD1812P200TF/30"
+			(at 199.39 41.91 90)
+			(effects
+				(font
+					(size 1.27 1.27)
+				)
+			)
+		)
+		(property "Footprint" ""
+			(at 204.47 44.45 0)
+			(effects
+				(font
+					(size 1.27 1.27)
+				)
+				(justify left)
+				(hide yes)
+			)
+		)
+		(property "Datasheet" "~"
+			(at 199.39 45.72 0)
+			(effects
+				(font
+					(size 1.27 1.27)
+				)
+				(hide yes)
+			)
+		)
+		(property "Description" "Resettable fuse, polymeric positive temperature coefficient"
+			(at 199.39 45.72 0)
+			(effects
+				(font
+					(size 1.27 1.27)
+				)
+				(hide yes)
+			)
+		)
+		(property "jlcpcb" "C5188720"
+			(at 199.39 43.688 90)
+			(effects
+				(font
+					(size 1.27 1.27)
+				)
+			)
+		)
+		(pin "2"
+		)
+		(pin "1"
+		)
+		(instances
+			(project ""
+				(path "/554fcf27-dc63-4666-abbc-7481d15942c4/32d6b15b-5472-4f1d-a1b7-d12adc0e25c3"
+					(reference "F14")
+					(unit 1)
+				)
+			)
+		)
+	)
+	(symbol
 		(lib_id "PCM_Transistor_BJT_AKL:MMBT3906")
 		(at 129.54 115.57 0)
@@
 					(unit 1)
 				)
+			)
+		)
+	)
+	(symbol
+		(lib_id "Device:Polyfuse")
+		(at 199.39 113.03 90)
+		(unit 1)
+		(exclude_from_sim no)
+		(in_bom yes)
+		(on_board yes)
+		(dnp no)
+		(property "Reference" "F16"
+			(at 199.39 106.68 90)
+			(effects
+				(font
+					(size 1.27 1.27)
+				)
+			)
+		)
+		(property "Value" "SMD1812P200TF/30"
+			(at 199.39 109.22 90)
+			(effects
+				(font
+					(size 1.27 1.27)
+				)
+			)
+		)
+		(property "Footprint" ""
+			(at 204.47 111.76 0)
+			(effects
+				(font
+					(size 1.27 1.27)
+				)
+				(justify left)
+				(hide yes)
+			)
+		)
+		(property "Datasheet" "~"
+			(at 199.39 113.03 0)
+			(effects
+				(font
+					(size 1.27 1.27)
+				)
+				(hide yes)
+			)
+		)
+		(property "Description" "Resettable fuse, polymeric positive temperature coefficient"
+			(at 199.39 113.03 0)
+			(effects
+				(font
+					(size 1.27 1.27)
+				)
+				(hide yes)
+			)
+		)
+		(property "jlcpcb" "C5188720"
+			(at 199.39 111.252 90)
+			(effects
+				(font
+					(size 1.27 1.27)
+				)
+			)
+		)
+		(pin "2"
+		)
+		(pin "1"
+		)
+		(instances
+			(project "mega_shield"
+				(path "/554fcf27-dc63-4666-abbc-7481d15942c4/32d6b15b-5472-4f1d-a1b7-d12adc0e25c3"
+					(reference "F16")
+					(unit 1)
+				)
