File: mega_shield/digital_gpio.kicad_sch (KiCad schematic)
At the start: 21 parts, among them J24 1803277, J25 1803277, Q46 MMBT3904, Q47 MMBT3904, Q49 AO4486, Q50 MMBT3906, Q51 MMBT3906, Q52 AO4486, U31 CS817x22HS

Commit message: set the AO4486 N-Channel mosfet jlcpcb number.
Parts:
- Q49, Q52: jlcpcb (none) -> C5125950
Changed lines of the file:
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@@
+			)
+		)
+		(property "jlcpcb" "C5125950"
+			(at 213.36 135.89 0)
+			(effects
+				(font
+					(size 1.27 1.27)
+				)
 			)
 		)
@@
 			(at 213.36 68.58 0)
 			(effects
+				(font
+					(size 1.27 1.27)
+				)
+			)
+		)
+		(property "jlcpcb" "C5125950"
+			(at 213.36 68.58 0)
+			(effects

Commit message: set the footprint for all the polyfuses for more compact spacing.
Parts:
- F14, F15, F16, F17: footprint (none) -> Fuse:Fuse_1812_4532Metric
Changed lines of the file:
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@@
 			)
 		)
-		(property "Footprint" ""
+		(property "Footprint" "Fuse:Fuse_1812_4532Metric"
 			(at 204.47 118.11 0)
 			(effects
@@
 			)
 		)
-		(property "Footprint" ""
+		(property "Footprint" "Fuse:Fuse_1812_4532Metric"
 			(at 204.47 50.8 0)
 			(effects
@@
 			)
 		)
-		(property "Footprint" ""
+		(property "Footprint" "Fuse:Fuse_1812_4532Metric"
 			(at 204.47 44.45 0)
 			(effects
@@
 			)
 		)
-		(property "Footprint" ""
+		(property "Footprint" "Fuse:Fuse_1812_4532Metric"
 			(at 204.47 111.76 0)
 			(effects

Commit message: changed name of sheet to be exclusivly digital outputs. Re-arranged schematic to make room for digital inputs sheet.
Parts:
- removed C59, C62: 1u, Capacitor_SMD:C_0201_0603Metric, symbol Device:C
- removed D5, D6: SM4007PL, PCM_Diode_SMD_AKL:D_SOD-123F, symbol PCM_Diode_AKL:SM4007PL
- removed F14, F15, F16, F17: SMD1812P200TF/30, Fuse:Fuse_1812_4532Metric, symbol Device:Polyfuse
- removed J24, J25: 1803277, footprints:PHOENIX_1803277, symbol TERM_BLOCK_HDR_2POS_3.81MM:1803277
- removed Q46, Q47: MMBT3904, PCM_Package_TO_SOT_SMD_AKL:SOT-23, symbol PCM_Transistor_BJT_AKL:MMBT3904
- removed Q49, Q52: AO4486, PCM_Package_SO_AKL:SO-8_3.9x4.9mm_P1.27mm, symbol PCM_Transistor_MOSFET_AKL:AO4486
- removed Q50, Q51: MMBT3906, PCM_Package_TO_SOT_SMD_AKL:SOT-23, symbol PCM_Transistor_BJT_AKL:MMBT3906
- removed R49, R51: 10k, Resistor_SMD:R_0201_0603Metric, symbol Device:R
- removed R50, R52: 100, Resistor_SMD:R_0201_0603Metric, symbol Device:R
- removed U31: CS817x22HS, Package_SO:SOIC-8_3.9x4.9mm_P1.27mm, symbol mega_shield:CS817x20HS
Other:
- note removed: "Digital Isolator(Channels A/B)"
- note removed: "MOSFET Channel A"
- note removed: "Mosfet Gate Drivers(Channels A/B)"
