File: mega_shield/local_solenoid_drivers.kicad_sch (KiCad schematic)
At the start: 0 parts

Commit message: Added solenoid N-channel mosfet, led indicator, snubber diode and polyfuse.
Parts:
- added D3: SM4007PL, PCM_Diode_SMD_AKL:D_SOD-123F, symbol PCM_Diode_AKL:SM4007PL
- added F10: SMD1812P030TF, Fuse:Fuse_1812_4532Metric_Pad1.30x3.40mm_HandSolder, symbol Device:Polyfuse
- added LED8: KT-0603R, PCM_LED_SMD_AKL:LED_0201_0603Metric, symbol PCM_LED_AKL:LED_1.8mm_SMD
- added Q43: AO4486, PCM_Package_SO_AKL:SO-8_3.9x4.9mm_P1.27mm, symbol PCM_Transistor_MOSFET_AKL:AO4486
- added R42: 4k7, Resistor_SMD:R_0805_2012Metric_Pad1.20x1.40mm_HandSolder, symbol PCM_Elektuur:R
- added R43: 1k2, Resistor_SMD:R_0805_2012Metric_Pad1.20x1.40mm_HandSolder, symbol PCM_Elektuur:R
Connections:
- new net: Q43.4 (G), R42.2 (-)
- new net: LED8.1 (K), R43.2 (-)
- new net 24V: F10.1
- new net GND: Q43.1 (S), Q43.2 (S), Q43.3 (S)
- new net solenoid_N: D3.2 (A), Q43.5 (D), Q43.6 (D), Q43.7 (D), Q43.8 (D), R43.1 (+)
- new net solenoid_P: D3.1 (K), F10.2, LED8.2 (A)

Commit message: Added 2pos term block header to first solenoid driver output.
Parts:
- added J7: 1803277, footprints:PHOENIX_1803277, symbol TERM_BLOCK_HDR_2POS_3.81MM:1803277
Connections:
- net solenoid_N: now also J7.02
- net solenoid_P: now also J7.01
Changed lines of the file:
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@@
 	)
 	(junction
-		(at 152.4 64.77)
+		(at 139.7 50.8)
 		(diameter 0)
 		(color 0 0 0 0)
@@
 		(color 0 0 0 0)
 	)
+	(junction
+		(at 139.7 76.2)
+		(diameter 0)
+		(color 0 0 0 0)
+	)
 	(wire
 		(pts
@@
 	(wire
 		(pts
-			(xy 152.4 71.12) (xy 152.4 64.77)
-		)
-		(stroke
-			(width 0)
-			(type default)
-		)
-	)
-	(wire
-		(pts
 			(xy 144.78 90.17) (xy 144.78 88.9)
 		)
@@
 	(wire
 		(pts
+			(xy 128.27 60.96) (xy 128.27 50.8)
+		)
+		(stroke
+			(width 0)
+			(type default)
+		)
+	)
+	(wire
+		(pts
 			(xy 144.78 88.9) (xy 147.32 88.9)
 		)
@@
 	(wire
 		(pts
-			(xy 139.7 38.1) (xy 152.4 38.1)
+			(xy 128.27 38.1) (xy 152.4 38.1)
 		)
 		(stroke
@@
 	(wire
 		(pts
+			(xy 128.27 76.2) (xy 139.7 76.2)
+		)
+		(stroke
+			(width 0)
+			(type default)
+		)
+	)
+	(wire
+		(pts
 			(xy 147.32 88.9) (xy 149.86 88.9)
 		)
@@
 	(wire
 		(pts
+			(xy 128.27 63.5) (xy 128.27 76.2)
+		)
+		(stroke
+			(width 0)
+			(type default)
+		)
+	)
+	(wire
+		(pts
 			(xy 144.78 100.33) (xy 144.78 102.87)
 		)
@@
 		(pts
 			(xy 152.4 48.26) (xy 152.4 50.8)
+		)
+		(stroke
+			(width 0)
+			(type default)
+		)
+	)
+	(wire
+		(pts
+			(xy 128.27 50.8) (xy 139.7 50.8)
 		)
 		(stroke
@@
 	(hierarchical_label "24V"
 		(shape input)
-		(at 139.7 38.1 180)
+		(at 128.27 38.1 180)
 		(effects
 			(font
@@
 					(unit 1)
 				)
+			)
+		)
+	)
+	(symbol
+		(lib_id "TERM_BLOCK_HDR_2POS_3.81MM:1803277")
+		(at 118.11 63.5 0)
+		(mirror y)
+		(unit 1)
+		(exclude_from_sim no)
+		(in_bom yes)
+		(on_board yes)
+		(dnp no)
+		(property "Reference" "J7"
+			(at 118.11 71.12 0)
+			(effects
+				(font
+					(size 1.27 1.27)
+				)
+			)
+		)
+		(property "Value" "1803277"
+			(at 118.11 68.58 0)
+			(effects
+				(font
+					(size 1.27 1.27)
+				)
+			)
+		)
+		(property "Footprint" "footprints:PHOENIX_1803277"
+			(at 118.11 63.5 0)
+			(effects
+				(font
+					(size 1.27 1.27)
+				)
+				(justify bottom)
+				(hide yes)
+			)
+		)
+		(property "Datasheet" ""
+			(at 118.11 63.5 0)
+			(effects
+				(font
+					(size 1.27 1.27)
+				)
+				(hide yes)
+			)
+		)
+		(property "Description" ""
+			(at 118.11 63.5 0)
+			(effects
+				(font
+					(size 1.27 1.27)
+				)
+				(hide yes)
+			)
+		)
+		(property "SnapEDA_Link" "https://www.snapeda.com/parts/1803277/Phoenix+Contact/view-part/?ref=snap"
+			(at 118.11 63.5 0)
+			(effects
+				(font
+					(size 1.27 1.27)
+				)
+				(justify bottom)
+				(hide yes)
+			)
+		)
+		(property "Description_1" "Pluggable Header 3.81mm 16AWG 160V 8A 2 Position COMBICON MC Series | Phoenix Contact 1803277"
+			(at 118.11 63.5 0)
+			(effects
+				(font
+					(size 1.27 1.27)
+				)
+				(justify bottom)
+				(hide yes)
+			)
+		)
+		(property "Package" "None"
+			(at 118.11 63.5 0)
+			(effects
+				(font
+					(size 1.27 1.27)
+				)
+				(justify bottom)
+				(hide yes)
+			)
+		)
+		(property "Price" "None"
+			(at 118.11 63.5 0)
+			(effects
+				(font
+					(size 1.27 1.27)
+				)
+				(justify bottom)
+				(hide yes)
+			)
+		)
+		(property "MF" "Phoenix Contact"
+			(at 118.11 63.5 0)
+			(effects
+				(font
+					(size 1.27 1.27)
+				)
+				(justify bottom)
+				(hide yes)
+			)
+		)
+		(property "MP" "1803277"
+			(at 118.11 63.5 0)
+			(effects
+				(font
+					(size 1.27 1.27)
+				)
+				(justify bottom)
+				(hide yes)
+			)
+		)
+		(property "Availability" "In Stock"
+			(at 118.11 63.5 0)
+			(effects
+				(font
+					(size 1.27 1.27)
+				)
+				(justify bottom)
+				(hide yes)
+			)
+		)
+		(property "Check_prices" "https://www.snapeda.com/parts/1803277/Phoenix+Contact/view-part/?ref=eda"
+			(at 118.11 63.5 0)
+			(effects
+				(font
+					(size 1.27 1.27)
+				)
+				(justify bottom)
+				(hide yes)
+			)
+		)
+		(pin "01"
+		)
+		(pin "02"
+		)
+		(instances
+			(project ""
+				(path "/554fcf27-dc63-4666-abbc-7481d15942c4/b5800b9f-f464-4485-8ad8-035cc7cf2bac"
+					(reference "J7")
+					(unit 1)
+				)

Commit message: Added ESD protection to the local solenoid driver sheet.
Parts:
- added R44, R45: 4k7, Resistor_SMD:R_0201_0603Metric, symbol Device:R
- added U29: NUP2202, Package_TO_SOT_SMD:SOT-363_SC-70-6, symbol Power_Protection:NUP2202
Connections:
- net +5V_IN: now also U29.5
- net GND: now also U29.2
- new net SLND_11: R44.2, U29.6
- new net SLND_12: R45.2, U29.1
- new net SLND_OUT_11: R44.1
- new net SLND_OUT_12: R45.1
Other:
- note added: "Solenoid ESD protection"

Commit message: finished adding the local solenoid dirver's
Parts:
- removed R42: 4k7, Resistor_SMD:R_0805_2012Metric_Pad1.20x1.40mm_HandSolder, symbol PCM_Elektuur:R
- added D4: SM4007PL, PCM_Diode_SMD_AKL:D_SOD-123F, symbol PCM_Diode_AKL:SM4007PL
- added F13: SMD1812P030TF, Fuse:Fuse_1812_4532Metric_Pad1.30x3.40mm_HandSolder, symbol Device:Polyfuse
- added J21: 1803277, footprints:PHOENIX_1803277, symbol TERM_BLOCK_HDR_2POS_3.81MM:1803277
- added LED9: KT-0603R, PCM_LED_SMD_AKL:LED_0201_0603Metric, symbol PCM_LED_AKL:LED_1.8mm_SMD
- added Q44: AO4486, PCM_Package_SO_AKL:SO-8_3.9x4.9mm_P1.27mm, symbol PCM_Transistor_MOSFET_AKL:AO4486
- added R46: 1k2, Resistor_SMD:R_0805_2012Metric_Pad1.20x1.40mm_HandSolder, symbol PCM_Elektuur:R
Connections:
- net 24V is gone; now on net +24V_IN: F10.1
- net +24V_IN: now also F13.1
- net GND: now also Q44.1 (S), Q44.2 (S), Q44.3 (S)
- net SLND_OUT_11: now also Q43.4 (G)
- net SLND_OUT_12: now also Q44.4 (G)
- net solenoid_N: now also D4.2 (A), J21.02, Q44.5 (D), Q44.6 (D), Q44.7 (D), Q44.8 (D), R46.1 (+)
- net solenoid_P: now also D4.1 (K), F13.2, J21.01, LED9.2 (A)
- new net: LED9.1 (K), R46.2 (-)
Other:
- note added: "SLND_11 Driver"
- note added: "SLND_12 Driver"
- moved on the sheet: R44, R45, U29

Commit message: fixed labeling issue with solenoid P/N
Connections:
- net solenoid_N renamed solenoid11_N
- net solenoid11_N: no longer D4.2 (A), J21.02, Q44.5 (D), Q44.6 (D), Q44.7 (D), Q44.8 (D), R46.1 (+)
- net solenoid_P renamed solenoid11_P
- net solenoid11_P: no longer D4.1 (K), F13.2, J21.01, LED9.2 (A)
- new net solenoid12_N: D4.2 (A), J21.02, Q44.5 (D), Q44.6 (D), Q44.7 (D), Q44.8 (D), R46.1 (+)
- new net solenoid12_P: D4.1 (K), F13.2, J21.01, LED9.2 (A)
Changed lines of the file:
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@@
 		)
 	)
-	(label "solenoid_N"
+	(label "solenoid11_N"
 		(at 139.7 76.2 180)
 		(effects
@@
 		)
 	)
-	(label "solenoid_P"
+	(label "solenoid12_P"
 		(at 198.12 50.8 180)
 		(effects
@@
 		)
 	)
-	(label "solenoid_P"
+	(label "solenoid11_P"
 		(at 139.7 50.8 180)
 		(effects
@@
 		)
 	)
-	(label "solenoid_N"
+	(label "solenoid12_N"
 		(at 198.12 76.2 180)
 		(effects

Commit message: updated jlcpcb number for the 1k2 resistors. Changed footprint from 0805 --> 0603.
Parts:
- R43, R46: footprint Resistor_SMD:R_0805_2012Metric_Pad1.20x1.40mm_HandSolder -> Resistor_SMD:R_0201_0603Metric; jlcpcb (none) -> C22765
Changed lines of the file:
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@@
 			)
 		)
-		(property "Footprint" "Resistor_SMD:R_0805_2012Metric_Pad1.20x1.40mm_HandSolder"
+		(property "Footprint" "Resistor_SMD:R_0201_0603Metric"
 			(at 152.4 69.85 0)
 			(effects
@@
 		)
 		(property "JLCPCB" "C17379"
+			(at 152.4 69.85 0)
+			(effects
+				(font
+					(size 1.27 1.27)
+				)
+			)
+		)
+		(property "jlcpcb" "C22765"
 			(at 152.4 69.85 0)
 			(effects
@@
 			)
 		)
-		(property "Footprint" "Resistor_SMD:R_0805_2012Metric_Pad1.20x1.40mm_HandSolder"
+		(property "Footprint" "Resistor_SMD:R_0201_0603Metric"
 			(at 210.82 69.85 0)
 			(effects
@@
 			(at 210.82 69.85 0)
 			(effects
+				(font
+					(size 1.27 1.27)
+				)
+			)
+		)
+		(property "jlcpcb" "C22765"
+			(at 210.82 69.85 0)
+			(effects

Commit message: Added jlcpcb number to the snubber diodes used in the solenoid drivers and gpio output.
Parts:
- D3, D4: jlcpcb (none) -> C64898
Changed lines of the file:
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@@
+			)
+		)
+		(property "jlcpcb" "C64898"
+			(at 198.12 57.15 0)
+			(effects
+				(font
+					(size 1.27 1.27)
+				)
 			)
 		)
@@
 			(at 139.7 57.15 0)
 			(effects
+				(font
+					(size 1.27 1.27)
+				)
+			)
+		)
+		(property "jlcpcb" "C64898"
+			(at 139.7 57.15 0)
+			(effects

Commit message: consolidated indicator leds to use all 0603 footprint and lower cost part. Changed the jlcpcb numbers.
Parts:
- F10, F13: jlcpcb (none) -> C20995
- LED8, LED9: jlcpcb (none) -> C2286
Changed lines of the file:
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@@
+			)
+		)
+		(property "jlcpcb" "C2286"
+			(at 152.4 57.15 0)
+			(effects
+				(font
+					(size 1.27 1.27)
+				)
 			)
 		)
@@
 			)
 		)
+		(property "jlcpcb" "C2286"
+			(at 210.82 57.15 0)
+			(effects
+				(font
+					(size 1.27 1.27)
+				)
+			)
+		)
 		(pin "1"
 		)
@@
 			)
 		)
+		(property "jlcpcb" "C20995"
+			(at 152.4 44.45 0)
+			(effects
+				(font
+					(size 1.27 1.27)
+				)
+			)
+		)
 		(pin "2"
 		)
@@
 			(at 210.82 44.45 0)
 			(effects
+				(font
+					(size 1.27 1.27)
+				)
+			)
+		)
+		(property "jlcpcb" "C20995"
+			(at 210.82 44.45 0)
+			(effects
