File: mega_shield/local_solenoid_drivers.kicad_sch (KiCad schematic)
At the start: 15 parts, among them J18 1803277, J19 1803277, Q23 AO4486, Q24 AO4486, U22 NUP2202

Commit message: mega_shield, re-annotated components, routed and placed new symbols for 5V external power section.
Parts:
- renumbered D3 to D2, D4 to D3, F11 to F10, F12 to F11, R38 to R39, R39 to R40, R40 to R41, R41 to R42, U22 to U23
Changed lines of the file:
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@@
 		(dnp no)
 		(fields_autoplaced yes)
-		(property "Reference" "R38"
+		(property "Reference" "R39"
 			(at 69.85 59.69 90)
 			(effects
@@
 			(project "mega_shield"
 				(path "/554fcf27-dc63-4666-abbc-7481d15942c4/b5800b9f-f464-4485-8ad8-035cc7cf2bac"
-					(reference "R38")
+					(reference "R39")
 					(unit 1)
 				)
@@
 		(dnp no)
 		(fields_autoplaced yes)
-		(property "Reference" "R40"
+		(property "Reference" "R41"
 			(at 158.75 69.85 90)
 			(effects
@@
 			(project "mega_shield"
 				(path "/554fcf27-dc63-4666-abbc-7481d15942c4/b5800b9f-f464-4485-8ad8-035cc7cf2bac"
-					(reference "R40")
+					(reference "R41")
 					(unit 1)
 				)
@@
 		(on_board yes)
 		(dnp no)
-		(property "Reference" "U22"
+		(property "Reference" "U23"
 			(at 57.2202 64.77 0)
 			(effects
@@
 			(project "mega_shield"
 				(path "/554fcf27-dc63-4666-abbc-7481d15942c4/b5800b9f-f464-4485-8ad8-035cc7cf2bac"
-					(reference "U22")
+					(reference "U23")
 					(unit 1)
 				)
@@
 		(dnp no)
 		(fields_autoplaced yes)
-		(property "Reference" "D4"
+		(property "Reference" "D3"
 			(at 204.47 57.15 0)
 			(effects
@@
 			(project "mega_shield"
 				(path "/554fcf27-dc63-4666-abbc-7481d15942c4/b5800b9f-f464-4485-8ad8-035cc7cf2bac"
-					(reference "D4")
+					(reference "D3")
 					(unit 1)
 				)
@@
 		(dnp no)
 		(fields_autoplaced yes)
-		(property "Reference" "R39"
+		(property "Reference" "R40"
 			(at 69.85 74.93 90)
 			(effects
@@
 			(project "mega_shield"
 				(path "/554fcf27-dc63-4666-abbc-7481d15942c4/b5800b9f-f464-4485-8ad8-035cc7cf2bac"
-					(reference "R39")
+					(reference "R40")
 					(unit 1)
 				)
@@
 		(dnp no)
 		(fields_autoplaced yes)
-		(property "Reference" "F11"
+		(property "Reference" "F10"
 			(at 158.75 44.45 90)
 			(effects
@@
 			(project "mega_shield"
 				(path "/554fcf27-dc63-4666-abbc-7481d15942c4/b5800b9f-f464-4485-8ad8-035cc7cf2bac"
-					(reference "F11")
+					(reference "F10")
 					(unit 1)
 				)
@@
 		(dnp no)
 		(fields_autoplaced yes)
-		(property "Reference" "R41"
+		(property "Reference" "R42"
 			(at 217.17 69.85 90)
 			(effects
@@
 			(project "mega_shield"
 				(path "/554fcf27-dc63-4666-abbc-7481d15942c4/b5800b9f-f464-4485-8ad8-035cc7cf2bac"
-					(reference "R41")
+					(reference "R42")
 					(unit 1)
 				)
@@
 		(dnp no)
 		(fields_autoplaced yes)
-		(property "Reference" "D3"
+		(property "Reference" "D2"
 			(at 146.05 57.15 0)
 			(effects
@@
 			(project "mega_shield"
 				(path "/554fcf27-dc63-4666-abbc-7481d15942c4/b5800b9f-f464-4485-8ad8-035cc7cf2bac"
-					(reference "D3")
+					(reference "D2")
 					(unit 1)
 				)
@@
 		(dnp no)
 		(fields_autoplaced yes)
-		(property "Reference" "F12"
+		(property "Reference" "F11"
 			(at 217.17 44.45 90)
 			(effects
@@
 			(project "mega_shield"
 				(path "/554fcf27-dc63-4666-abbc-7481d15942c4/b5800b9f-f464-4485-8ad8-035cc7cf2bac"
-					(reference "F12")
-					(unit 1)
-				)
+					(reference "F11")
+					(unit 1)
+				)

Commit message: mega_shield, placed ideal diode and added jlcpcb number for it.
Parts:
- renumbered U23 to U24

Commit message: mega_shield, re-ran annotation of entire project.
Parts:
- renumbered Q23 to Q24, Q24 to Q25, R39 to R41, R40 to R42, R41 to R43, R42 to R44
Changed lines of the file:
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@@
 		(dnp no)
 		(fields_autoplaced yes)
-		(property "Reference" "R39"
+		(property "Reference" "R41"
 			(at 69.85 59.69 90)
 			(effects
@@
 			(project "mega_shield"
 				(path "/554fcf27-dc63-4666-abbc-7481d15942c4/b5800b9f-f464-4485-8ad8-035cc7cf2bac"
-					(reference "R39")
+					(reference "R41")
 					(unit 1)
 				)
@@
 		(dnp no)
 		(fields_autoplaced yes)
-		(property "Reference" "R41"
+		(property "Reference" "R43"
 			(at 158.75 69.85 90)
 			(effects
@@
 			(project "mega_shield"
 				(path "/554fcf27-dc63-4666-abbc-7481d15942c4/b5800b9f-f464-4485-8ad8-035cc7cf2bac"
-					(reference "R41")
+					(reference "R43")
 					(unit 1)
 				)
@@
 		(dnp no)
 		(fields_autoplaced yes)
-		(property "Reference" "Q23"
+		(property "Reference" "Q24"
 			(at 153.67 93.9799 0)
 			(effects
@@
 			(project "mega_shield"
 				(path "/554fcf27-dc63-4666-abbc-7481d15942c4/b5800b9f-f464-4485-8ad8-035cc7cf2bac"
-					(reference "Q23")
+					(reference "Q24")
 					(unit 1)
 				)
@@
 		(dnp no)
 		(fields_autoplaced yes)
-		(property "Reference" "R40"
+		(property "Reference" "R42"
 			(at 69.85 74.93 90)
 			(effects
@@
 			(project "mega_shield"
 				(path "/554fcf27-dc63-4666-abbc-7481d15942c4/b5800b9f-f464-4485-8ad8-035cc7cf2bac"
-					(reference "R40")
+					(reference "R42")
 					(unit 1)
 				)
@@
 		(dnp no)
 		(fields_autoplaced yes)
-		(property "Reference" "R42"
+		(property "Reference" "R44"
 			(at 217.17 69.85 90)
 			(effects
@@
 			(project "mega_shield"
 				(path "/554fcf27-dc63-4666-abbc-7481d15942c4/b5800b9f-f464-4485-8ad8-035cc7cf2bac"
-					(reference "R42")
+					(reference "R44")
 					(unit 1)
 				)
@@
 		(dnp no)
 		(fields_autoplaced yes)
-		(property "Reference" "Q24"
+		(property "Reference" "Q25"
 			(at 212.09 93.9799 0)
 			(effects
@@
 			(project "mega_shield"
 				(path "/554fcf27-dc63-4666-abbc-7481d15942c4/b5800b9f-f464-4485-8ad8-035cc7cf2bac"
-					(reference "Q24")
+					(reference "Q25")
 					(unit 1)
 				)

Commit message: mega_shield, marked circular components as DNP, added jlcpcb numbers to 90degree terminal blocks.
Parts:
- J18, J19: jlcpcb (none) -> C480537
Changed lines of the file:
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@@
+			)
+		)
+		(property "jlcpcb" "C480537"
+			(at 118.11 63.5 0)
+			(effects
+				(font
+					(size 1.27 1.27)
+				)
+				(hide yes)
 			)
 		)
@@
 			(at 176.53 63.5 0)
 			(effects
+				(font
+					(size 1.27 1.27)
+				)
+				(hide yes)
+			)
+		)
+		(property "jlcpcb" "C480537"
+			(at 176.53 63.5 0)
+			(effects

Commit message: mega_shield, re-annotated all components.
Parts:
- renumbered R41 to R63, R42 to R64, R43 to R65, R44 to R66
Changed lines of the file:
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@@
 		(dnp no)
 		(fields_autoplaced yes)
-		(property "Reference" "R41"
+		(property "Reference" "R63"
 			(at 69.85 59.69 90)
 			(effects
@@
 			(project "mega_shield"
 				(path "/554fcf27-dc63-4666-abbc-7481d15942c4/b5800b9f-f464-4485-8ad8-035cc7cf2bac"
-					(reference "R41")
+					(reference "R63")
 					(unit 1)
 				)
@@
 		(dnp no)
 		(fields_autoplaced yes)
-		(property "Reference" "R43"
+		(property "Reference" "R65"
 			(at 158.75 69.85 90)
 			(effects
@@
 			(project "mega_shield"
 				(path "/554fcf27-dc63-4666-abbc-7481d15942c4/b5800b9f-f464-4485-8ad8-035cc7cf2bac"
-					(reference "R43")
+					(reference "R65")
 					(unit 1)
 				)
@@
 		(dnp no)
 		(fields_autoplaced yes)
-		(property "Reference" "R42"
+		(property "Reference" "R64"
 			(at 69.85 74.93 90)
 			(effects
@@
 			(project "mega_shield"
 				(path "/554fcf27-dc63-4666-abbc-7481d15942c4/b5800b9f-f464-4485-8ad8-035cc7cf2bac"
-					(reference "R42")
+					(reference "R64")
 					(unit 1)
 				)
@@
 		(dnp no)
 		(fields_autoplaced yes)
-		(property "Reference" "R44"
+		(property "Reference" "R66"
 			(at 217.17 69.85 90)
 			(effects
@@
 			(project "mega_shield"
 				(path "/554fcf27-dc63-4666-abbc-7481d15942c4/b5800b9f-f464-4485-8ad8-035cc7cf2bac"
-					(reference "R44")
+					(reference "R66")
 					(unit 1)
 				)

Commit message: mega_shield, passing all ERC(electrical rules check). Zero errors
+ Fixed missing symbols from defunct digikey lib.
+ Fixed created custom symbol for AO4486 NMOS.
+ Fixed all Power flag and pin conflicts.
+ Excluded passive/unspecified warnings/errors.
Parts:
- removed D2, D3: SM4007PL, Diode_SMD:D_SOD-123F, symbol PCM_Diode_AKL:SM4007PL
- removed LED9: KT-0603R, LED_SMD:LED_0603_1608Metric_Pad1.05x0.95mm_HandSolder, symbol PCM_LED_AKL:LED_1.8mm_SMD
- removed Q24: AO4486, Package_SO:SOP-8_3.76x4.96mm_P1.27mm, symbol PCM_Transistor_MOSFET_AKL:AO4486
- removed R66: 1k2, Resistor_SMD:R_0805_2012Metric_Pad1.20x1.40mm_HandSolder, symbol PCM_Elektuur:R
- added D2, D3: SM4007PL, symbol Device:D_Filled
- added LED9: KT-0603R, LED_SMD:LED_0603_1608Metric_Pad1.05x0.95mm_HandSolder, symbol Device:LED
- added Q24: AO4486, Package_SO:SOP-8_3.76x4.96mm_P1.27mm, symbol mega_shield:UMW_AO4486
- added R66: 1k2, Resistor_SMD:R_0805_2012Metric_Pad1.20x1.40mm_HandSolder, symbol Device:R
- LED8: symbol PCM_LED_AKL:LED_1.8mm_SMD -> Device:LED; jlcpcb C2286 -> (none)
- Q25: symbol PCM_Transistor_MOSFET_AKL:AO4486 -> mega_shield:UMW_AO4486
- R65: symbol PCM_Elektuur:R -> Device:R; jlcpcb C17379 -> (none)
Connections:
- net GND: now also Q24.1, Q24.2, Q24.3
- net SLND_OUT_11: now also Q24.4
- net solenoid11_N: now also D2.2 (A), Q24.5, Q24.6, Q24.7, Q24.8
- net solenoid11_P: now also D2.1 (K)
- net solenoid12_N: now also D3.2 (A), R66.1
- net solenoid12_P: now also D3.1 (K), LED9.2 (A)
- new net: LED9.1 (K), R66.2

Commit message: mega_shield, rerouted and place components for spindle interface
Parts:
- D2, D3: footprint (none) -> Diode_SMD:D_SOD-123F; jlcpcb (none) -> C64898
- LED8, LED9: jlcpcb (none) -> C2286
- R65, R66: jlcpcb (none) -> C17379
Changed lines of the file:
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@@
 			)
 		)
-		(property "Footprint" ""
+		(property "Footprint" "Diode_SMD:D_SOD-123F"
 			(at 198.12 62.23 0)
 			(effects
@@
 		)
 		(property "JLCPCB" "C64898"
+			(at 198.12 62.23 90)
+			(effects
+				(font
+					(size 1.27 1.27)
+				)
+				(hide yes)
+			)
+		)
+		(property "jlcpcb" "C64898"
 			(at 198.12 62.23 90)
 			(effects
@@
 			)
 		)
+		(property "jlcpcb" "C17379"
+			(at 152.4 69.85 0)
+			(effects
+				(font
+					(size 1.27 1.27)
+				)
+				(hide yes)
+			)
+		)
 		(pin "2"
 		)
@@
 			)
 		)
-		(property "Footprint" ""
+		(property "Footprint" "Diode_SMD:D_SOD-123F"
 			(at 139.7 63.5 0)
 			(effects
@@
 		)
 		(property "JLCPCB" "C64898"
+			(at 139.7 63.5 90)
+			(effects
+				(font
+					(size 1.27 1.27)
+				)
+				(hide yes)
+			)
+		)
+		(property "jlcpcb" "C64898"
 			(at 139.7 63.5 90)
 			(effects
@@
 		(property "Status" ""
 			(at 152.4 57.15 0)
+			(effects
+				(font
+					(size 1.27 1.27)
+				)
+				(hide yes)
+			)
+		)
+		(property "jlcpcb" "C2286"
+			(at 152.4 57.15 90)
 			(effects
 				(font
@@
 			)
 		)
+		(property "jlcpcb" "C2286"
+			(at 210.82 57.15 90)
+			(effects
+				(font
+					(size 1.27 1.27)
+				)
+				(hide yes)
+			)
+		)
 		(pin "1"
 		)
@@
 			(effects
 				(font
+					(size 1.27 1.27)
+				)
+				(hide yes)
+			)
+		)
+		(property "jlcpcb" "C17379"
+			(at 210.82 69.85 0)
+			(effects
+				(font
