File: mega_shield/servo_interface_.kicad_sch (KiCad schematic)
At the start: 34 parts, among them J1 T4140012081-000, Q1 2SK3018, Q2 2SK3018, Q3 2SK3018, Q4 2SK3018, Q5 2SK3018, Q6 2SK3018, U1 CS817x22HS, U2 CS817x22HS, U3 CS817x22HS

Commit message: Set the JLCPCB number for the M12P8 connector.
Parts:
- J1: jlcpcb (none) -> C7423412
Changed lines of the file:
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@@
+			)
+		)
+		(property "jlcpcb" "C7423412"
+			(at 55.88 86.36 0)
+			(effects
+				(font
+					(size 1.27 1.27)
+				)
 			)
 		)

Commit message: Added mounting holes to each sevo interface.
Parts:
- added H5, H6: MountingHole_Pad, MountingHole:MountingHole_3.2mm_M3_DIN965_Pad, symbol Mechanical:MountingHole_Pad
Connections:
- net GND: now also H5.1, H6.1

Commit message: consolidated indicator leds to use all 0603 footprint and lower cost part. Changed the jlcpcb numbers.
Parts:
- LED1: value LED_0603_Red -> KT-0603R; footprint PCM_LED_SMD_AKL:LED_0603_1608Metric -> PCM_LED_SMD_AKL:LED_0201_0603Metric; jlcpcb C94743 -> C2286
Changed lines of the file:
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@@
 			)
 		)
-		(property "Value" "LED_0603_Red"
+		(property "Value" "KT-0603R"
 			(at 48.26 43.18 0)
 			(effects
@@
 			)
 		)
-		(property "Footprint" "PCM_LED_SMD_AKL:LED_0603_1608Metric"
+		(property "Footprint" "PCM_LED_SMD_AKL:LED_0201_0603Metric"
 			(at 48.26 49.53 0)
 			(effects
@@
 			)
 		)
-		(property "jlcpcb" "C94743"
+		(property "jlcpcb" "C2286"
 			(at 48.26 49.53 0)
 			(effects

Commit message: simplified servo interfaces input sections.
Parts:
- removed Q5, Q6: 2SK3018, PCM_Package_TO_SOT_SMD_AKL:SOT-323_SC-70, symbol PCM_Transistor_MOSFET_AKL:2SK3018
- removed R2, R3: 1k, Resistor_SMD:R_0201_0603Metric, symbol Device:R
Connections:
- net ALARM: now also U3.6 (OUTB)
- net PED: now also U3.7 (OUTA)

Commit message: redesigned servo interface, reduced number of isolator ICs need from 3 to a single IC.
Parts:
- removed C2, C3, C4, C5: 1u, Capacitor_SMD:C_0201_0603Metric, symbol Device:C
- removed U1, U2, U3: CS817x22HS, Package_SO:SOIC-8_3.9x4.9mm_P1.27mm, symbol mega_shield:CS817x20HS
- added U33: ~, Package_SO:SOIC-16_3.9x9.9mm_P1.27mm, symbol mega_shield:π162M
- C1, C6: value 1u -> 0.1uF; footprint Capacitor_SMD:C_0201_0603Metric -> (none); jlcpcb C15849 -> (none)
Connections:
- net +5V_Servo: now also C1.2, C6.1, U33.1 (VDD1), U33.16 (VDD2); no longer C1.1, C6.2
- net ALARM: now also U33.7 (vout_f)
- net ALARM_IN: now also U33.10 (vin_f)
- net AUX_IN: now also U33.5 (vin_d)
- net DIR: now also U33.3 (vin_b)
- net EN: now also U33.4 (vin_c)
- net GND: now also C1.1, C6.2, U33.8 (GND1), U33.9 (GND1); no longer C1.2, C6.1
- net PED: now also U33.6 (vout_e)
- net PED_IN: now also U33.11 (vin_e)
- net STEP: now also U33.2 (vin_a)
- net at Q2.1 (G): now also U33.12 (vout_d)
- net at Q1.1 (G): now also U33.13 (vout_c)
- net at Q4.1 (G): now also U33.15 (vout_a)
- net at Q3.1 (G): now also U33.14 (vout_b)
Other:
- note removed: "Digitally Isolated Inputs"
- moved on the sheet: Q1, Q2, Q3, Q4

Commit message: Updated symbols value/name
Parts:
- U33: value ~ -> Pi_162M
Changed lines of the file:
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@@
 			)
 		)
-		(property "Value" "~"
+		(property "Value" "Pi_162M"
 			(at 165.1 100.33 0)
 			(effects
@@
 			)
 		)
+		(property "Purpose" ""
+			(at 165.1 115.57 0)
+			(effects
+				(font
+					(size 1.27 1.27)
+				)
+			)
+		)

Commit message: updated JLCPCB numbers and added new ones.
Parts:
- C1, C6: footprint (none) -> Capacitor_SMD:C_0201_0603Metric; jlcpcb (none) -> C1591
- U33: jlcpcb (none) -> C471610
Changed lines of the file:
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@@
 			)
 		)
-		(property "Footprint" ""
+		(property "Footprint" "Capacitor_SMD:C_0201_0603Metric"
 			(at 152.4 90.4748 0)
 			(effects
@@
 				)
 				(hide yes)
+			)
+		)
+		(property "jlcpcb" "C1591"
+			(at 148.59 91.44 0)
+			(effects
+				(font
+					(size 1.27 1.27)
+				)
 			)
 		)
@@
 			)
 		)
+		(property "jlcpcb" "C471610"
+			(at 165.1 115.57 0)
+			(effects
+				(font
+					(size 1.27 1.27)
+				)
+			)
+		)
 		(pin "13"
 		)
@@
 			)
 		)
-		(property "Footprint" ""
+		(property "Footprint" "Capacitor_SMD:C_0201_0603Metric"
 			(at 185.42 90.4748 0)
 			(effects
@@
 			)
 		)
+		(property "jlcpcb" "C1591"
+			(at 181.61 91.44 0)
+			(effects
+				(font
+					(size 1.27 1.27)
+				)
+			)
+		)
