File: mega_shield/servo_interface_.kicad_sch (KiCad schematic)
At the start: 26 parts, among them J1 T4140012081-000, Q1 2SK3018, Q2 2SK3018, Q3 2SK3018, Q4 2SK3018, U33 Pi_162M

Commit message: re-annotating for entire schematic completed.
Parts:
- renumbered C6 to C1, C1 to C2, Q4 to Q1, Q3 to Q2, Q1 to Q3, Q2 to Q4, U33 to U1

Commit message: updated the value of all tests points in the servo interfaces.
Parts:
- TP1: value TestPoint -> +5V_Servo
- TP10: value TestPoint -> EN_OUT
- TP11: value TestPoint -> AUX_OUT
- TP12: value TestPoint -> PED
- TP13: value TestPoint -> ALARM
- TP2: value TestPoint -> STEP
- TP3: value TestPoint -> DIR
- TP4: value TestPoint -> EN
- TP5: value TestPoint -> AUX_IN
- TP6: value TestPoint -> PED_IN
- TP7: value TestPoint -> ALARM_IN
- TP8: value TestPoint -> DIR_OUT
- TP9: value TestPoint -> STEP_OUT
Changed lines of the file:
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@@
 			)
 		)
-		(property "Value" "TestPoint"
+		(property "Value" "EN_OUT"
 			(at 55.118 160.02 90)
 			(effects
@@
 			)
 		)
-		(property "Value" "TestPoint"
+		(property "Value" "STEP_OUT"
 			(at 53.848 152.4 90)
 			(effects
@@
 			)
 		)
-		(property "Value" "TestPoint"
+		(property "Value" "PED"
 			(at 55.118 175.26 90)
 			(effects
@@
 			)
 		)
-		(property "Value" "TestPoint"
+		(property "Value" "DIR"
 			(at 34.798 152.4 90)
 			(effects
@@
 			)
 		)
-		(property "Value" "TestPoint"
+		(property "Value" "AUX_OUT"
 			(at 55.118 167.64 90)
 			(effects
@@
 			)
 		)
-		(property "Value" "TestPoint"
+		(property "Value" "+5V_Servo"
 			(at 34.798 137.16 90)
 			(effects
@@
 			)
 		)
-		(property "Value" "TestPoint"
+		(property "Value" "STEP"
 			(at 34.798 144.78 90)
 			(effects
@@
 			)
 		)
-		(property "Value" "TestPoint"
+		(property "Value" "EN"
 			(at 34.798 160.02 90)
 			(effects
@@
 			)
 		)
-		(property "Value" "TestPoint"
+		(property "Value" "ALARM_IN"
 			(at 34.798 182.88 90)
 			(effects
@@
 			)
 		)
-		(property "Value" "TestPoint"
+		(property "Value" "AUX_IN"
 			(at 34.798 167.64 90)
 			(effects
@@
 			)
 		)
-		(property "Value" "TestPoint"
+		(property "Value" "ALARM"
 			(at 55.118 182.88 90)
 			(effects
@@
 			)
 		)
-		(property "Value" "TestPoint"
+		(property "Value" "DIR_OUT"
 			(at 53.848 144.78 90)
 			(effects
@@
 			)
 		)
-		(property "Value" "TestPoint"
+		(property "Value" "PED_IN"
 			(at 34.798 175.26 90)
 			(effects

Commit message: mega_shield, changed footprint for the led to built in 0603(IMPRL)/1608(Metric)
Parts:
- LED1: footprint PCM_LED_SMD_AKL:LED_0201_0603Metric -> LED_SMD:LED_0603_1608Metric_Pad1.05x0.95mm_HandSolder
Changed lines of the file:
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@@
 			)
 		)
-		(property "Footprint" "PCM_LED_SMD_AKL:LED_0201_0603Metric"
+		(property "Footprint" "LED_SMD:LED_0603_1608Metric_Pad1.05x0.95mm_HandSolder"
 			(at 48.26 49.53 0)
 			(effects

Commit message: mega_shield, changed out 2SK3018(extended) for 2N7002(basic) part that's in stock in large qty.
Parts:
- Q1, Q2, Q3, Q4: value 2SK3018 -> 2N7002; footprint PCM_Package_TO_SOT_SMD_AKL:SOT-323_SC-70 -> Package_TO_SOT_SMD:SOT-23; jlcpcb C20069149 -> C8545
Changed lines of the file:
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@@
 			)
 		)
-		(property "Value" "2SK3018"
+		(property "Value" "2N7002"
 			(at 245.11 146.0499 0)
 			(effects
@@
 			)
 		)
-		(property "Footprint" "PCM_Package_TO_SOT_SMD_AKL:SOT-323_SC-70"
+		(property "Footprint" "Package_TO_SOT_SMD:SOT-23"
 			(at 243.84 147.32 0)
 			(effects
@@
 			)
 		)
-		(property "jlcpcb" "C20069149"
+		(property "jlcpcb" "C8545"
 			(at 238.76 144.78 0)
 			(effects
@@
 			)
 		)
-		(property "Value" "2SK3018"
+		(property "Value" "2N7002"
 			(at 245.11 120.6499 0)
 			(effects
@@
 			)
 		)
-		(property "Footprint" "PCM_Package_TO_SOT_SMD_AKL:SOT-323_SC-70"
+		(property "Footprint" "Package_TO_SOT_SMD:SOT-23"
 			(at 243.84 121.92 0)
 			(effects
@@
 			)
 		)
-		(property "jlcpcb" "C20069149"
+		(property "jlcpcb" "C8545"
 			(at 238.76 119.38 0)
 			(effects
@@
 			)
 		)
-		(property "Value" "2SK3018"
+		(property "Value" "2N7002"
 			(at 245.11 69.8499 0)
 			(effects
@@
 			)
 		)
-		(property "Footprint" "PCM_Package_TO_SOT_SMD_AKL:SOT-323_SC-70"
+		(property "Footprint" "Package_TO_SOT_SMD:SOT-23"
 			(at 243.84 71.12 0)
 			(effects
@@
 			)
 		)
-		(property "jlcpcb" "C20069149"
+		(property "jlcpcb" "C8545"
 			(at 238.76 68.58 0)
 			(effects
@@
 			)
 		)
-		(property "Value" "2SK3018"
+		(property "Value" "2N7002"
 			(at 245.11 95.2499 0)
 			(effects
@@
 			)
 		)
-		(property "Footprint" "PCM_Package_TO_SOT_SMD_AKL:SOT-323_SC-70"
+		(property "Footprint" "Package_TO_SOT_SMD:SOT-23"
 			(at 243.84 96.52 0)
 			(effects
@@
 			)
 		)
-		(property "jlcpcb" "C20069149"
+		(property "jlcpcb" "C8545"
 			(at 238.76 93.98 0)
 			(effects

Commit message: mega_shield, Changed out all caps where needed for in-stock and lower cost parts.
+ Changed out for parts with higher stock.
+ Changed out for 0805 sized components.
+ Changed out for higher voltage.
+ Removed 22uF SMD caps for lower cost 10uF caps in parallel.
+ Updated diode footprint to SOD-123F

BOM cost reduced, and reliability improved.
Parts:
- C1, C2: value 0.1uF -> 100n/50V; footprint Capacitor_SMD:C_0201_0603Metric -> Capacitor_SMD:C_0805_2012Metric_Pad1.18x1.45mm_HandSolder; jlcpcb C1591 -> C49678
Changed lines of the file:
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@@
 			)
 		)
-		(property "Value" "0.1uF"
+		(property "Value" "100n/50V"
 			(at 148.59 86.36 90)
 			(effects
@@
 			)
 		)
-		(property "Footprint" "Capacitor_SMD:C_0201_0603Metric"
+		(property "Footprint" "Capacitor_SMD:C_0805_2012Metric_Pad1.18x1.45mm_HandSolder"
 			(at 152.4 90.4748 0)
 			(effects
@@
 			)
 		)
-		(property "jlcpcb" "C1591"
+		(property "jlcpcb" "C49678"
 			(at 148.59 91.44 0)
 			(effects
@@
 			)
 		)
-		(property "Value" "0.1uF"
+		(property "Value" "100n/50V"
 			(at 181.61 86.36 90)
 			(effects
@@
 			)
 		)
-		(property "Footprint" "Capacitor_SMD:C_0201_0603Metric"
+		(property "Footprint" "Capacitor_SMD:C_0805_2012Metric_Pad1.18x1.45mm_HandSolder"
 			(at 185.42 90.4748 0)
 			(effects
@@
 			)
 		)
-		(property "jlcpcb" "C1591"
+		(property "jlcpcb" "C49678"
 			(at 181.61 91.44 0)
 			(effects

Commit message: mega_shield, updated multiple resistors and added comments.
+ Updated optoisolator resistor value --> 15k for better protection.
+ Changed all resistors to 0805 footprints
+ Swapped out expensive values to standardized E24/E96.
+ Updated jlcpcb numbers for all resistors.
Parts:
- R1: footprint Resistor_SMD:R_0201_0603Metric -> Resistor_SMD:R_0805_2012Metric_Pad1.20x1.40mm_HandSolder; jlcpcb C22975 -> C17604
Changed lines of the file:
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@@
 			)
 		)
-		(property "Footprint" "Resistor_SMD:R_0201_0603Metric"
+		(property "Footprint" "Resistor_SMD:R_0805_2012Metric_Pad1.20x1.40mm_HandSolder"
 			(at 62.23 51.308 90)
 			(effects
@@
 			)
 		)
-		(property "jlcpcb" "C22975"
+		(property "jlcpcb" "C17604"
 			(at 62.23 49.53 0)
 			(effects

Commit message: mega_shield, Set all test points to use the keystone 5000-5004 footprints.
Parts:
- TP1, TP10, TP11, TP12, TP13, TP2, TP3, TP4, TP5, TP6, TP7, TP8, TP9: footprint TestPoint:TestPoint_Pad_1.0x1.0mm -> TestPoint:TestPoint_Keystone_5000-5004_Miniature
Changed lines of the file:
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@@
 			)
 		)
-		(property "Footprint" "TestPoint:TestPoint_Pad_1.0x1.0mm"
+		(property "Footprint" "TestPoint:TestPoint_Keystone_5000-5004_Miniature"
 			(at 58.42 157.48 0)
 			(effects
@@
 			)
 		)
-		(property "Footprint" "TestPoint:TestPoint_Pad_1.0x1.0mm"
+		(property "Footprint" "TestPoint:TestPoint_Keystone_5000-5004_Miniature"
 			(at 57.15 149.86 0)
 			(effects
@@
 			)
 		)
-		(property "Footprint" "TestPoint:TestPoint_Pad_1.0x1.0mm"
+		(property "Footprint" "TestPoint:TestPoint_Keystone_5000-5004_Miniature"
 			(at 58.42 172.72 0)
 			(effects
@@
 			)
 		)
-		(property "Footprint" "TestPoint:TestPoint_Pad_1.0x1.0mm"
+		(property "Footprint" "TestPoint:TestPoint_Keystone_5000-5004_Miniature"
 			(at 38.1 149.86 0)
 			(effects
@@
 			)
 		)
-		(property "Footprint" "TestPoint:TestPoint_Pad_1.0x1.0mm"
+		(property "Footprint" "TestPoint:TestPoint_Keystone_5000-5004_Miniature"
 			(at 58.42 165.1 0)
 			(effects
@@
 			)
 		)
-		(property "Footprint" "TestPoint:TestPoint_Pad_1.0x1.0mm"
+		(property "Footprint" "TestPoint:TestPoint_Keystone_5000-5004_Miniature"
 			(at 38.1 134.62 0)
 			(effects
@@
 			)
 		)
-		(property "Footprint" "TestPoint:TestPoint_Pad_1.0x1.0mm"
+		(property "Footprint" "TestPoint:TestPoint_Keystone_5000-5004_Miniature"
 			(at 38.1 142.24 0)
 			(effects
@@
 			)
 		)
-		(property "Footprint" "TestPoint:TestPoint_Pad_1.0x1.0mm"
+		(property "Footprint" "TestPoint:TestPoint_Keystone_5000-5004_Miniature"
 			(at 38.1 157.48 0)
 			(effects
@@
 			)
 		)
-		(property "Footprint" "TestPoint:TestPoint_Pad_1.0x1.0mm"
+		(property "Footprint" "TestPoint:TestPoint_Keystone_5000-5004_Miniature"
 			(at 38.1 180.34 0)
 			(effects
@@
 			)
 		)
-		(property "Footprint" "TestPoint:TestPoint_Pad_1.0x1.0mm"
+		(property "Footprint" "TestPoint:TestPoint_Keystone_5000-5004_Miniature"
 			(at 38.1 165.1 0)
 			(effects
@@
 			)
 		)
-		(property "Footprint" "TestPoint:TestPoint_Pad_1.0x1.0mm"
+		(property "Footprint" "TestPoint:TestPoint_Keystone_5000-5004_Miniature"
 			(at 58.42 180.34 0)
 			(effects
@@
 			)
 		)
-		(property "Footprint" "TestPoint:TestPoint_Pad_1.0x1.0mm"
+		(property "Footprint" "TestPoint:TestPoint_Keystone_5000-5004_Miniature"
 			(at 57.15 142.24 0)
 			(effects
@@
 			)
 		)
-		(property "Footprint" "TestPoint:TestPoint_Pad_1.0x1.0mm"
+		(property "Footprint" "TestPoint:TestPoint_Keystone_5000-5004_Miniature"
 			(at 38.1 172.72 0)
 			(effects

Commit message: mega_shield, updated all 116 test points, changed values based on color code, added jlcpcb numbers and set footprints.
Parts:
- added TP109: RH-5001, TestPoint:TestPoint_Keystone_5000-5004_Miniature, symbol Connector:TestPoint
- TP1: value +5V_Servo -> RH-5000; jlcpcb (none) -> C5277086; now in the parts list
- TP10: value EN_OUT -> RH-5117; jlcpcb (none) -> C5199807; now in the parts list
- TP11: value AUX_OUT -> RH-5117; jlcpcb (none) -> C5199807; now in the parts list
- TP12: value PED -> RH-5000; jlcpcb (none) -> C5277086; now in the parts list
- TP13: value ALARM -> RH-5000; jlcpcb (none) -> C5277086; now in the parts list
- TP2: value STEP -> RH-5000; jlcpcb (none) -> C5277086; now in the parts list
- TP3: value DIR -> RH-5000; jlcpcb (none) -> C5277086; now in the parts list
- TP4: value EN -> RH-5000; jlcpcb (none) -> C5277086; now in the parts list
- TP5: value AUX_IN -> RH-5000; jlcpcb (none) -> C5277086; now in the parts list
- TP6: value PED_IN -> RH-5002; jlcpcb (none) -> C5199802; now in the parts list
- TP7: value ALARM_IN -> RH-5002; jlcpcb (none) -> C5199802; now in the parts list
- TP8: value DIR_OUT -> RH-5117; jlcpcb (none) -> C5199807; now in the parts list
- TP9: value STEP_OUT -> RH-5117; jlcpcb (none) -> C5199807; now in the parts list
Connections:
- net GND: now also TP109.1
