File: mega_shield/servo_interface_.kicad_sch (KiCad schematic)
At the start: 27 parts, among them J1 T4141012081-000, Q1 2N7002, Q2 2N7002, Q3 2N7002, Q4 2N7002, U1 Pi_162M

Commit message: mega_shield, marked circular components as DNP, added jlcpcb numbers to 90degree terminal blocks.
Parts:
- J1: now not fitted
Changed lines of the file:
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@@
 		(in_bom yes)
 		(on_board yes)
-		(dnp no)
+		(dnp yes)
 		(fields_autoplaced yes)
 		(property "Reference" "J1"

Commit message: mega_shield, re-annotated all components.
Parts:
- added R2, R3, R4, R5: 100, Resistor_SMD:R_0805_2012Metric_Pad1.20x1.40mm_HandSolder, symbol Device:R
Connections:
- net +5V_Servo: now also J1.7; no longer J1.2
- net ALARM_IN: now also J1.5; no longer J1.4
- net AUX_OUT: now also J1.6; no longer J1.3
- net DIR_OUT: now also J1.2; no longer J1.7
- net EN_OUT: now also J1.3; no longer J1.6
- net PED_IN: now also J1.4; no longer J1.5
- net at Q4.1 (G): now also R5.1; no longer U1.12 (vout_d)
- net at Q3.1 (G): now also R4.1; no longer U1.13 (vout_c)
- net at Q2.1 (G): now also R3.1; no longer U1.14 (vout_b)
- net at Q1.1 (G): now also R2.1; no longer U1.15 (vout_a)
- new net: R5.2, U1.12 (vout_d)
- new net: R3.2, U1.14 (vout_b)
- new net: R2.2, U1.15 (vout_a)
- new net: R4.2, U1.13 (vout_c)

Commit message: mega_shield, swapped out hex channel digital isolator for all servo interfaces.
Parts:
- U1: value Pi_162M -> PI162U31; symbol mega_shield:π162M -> mega_shield:π162U; jlcpcb C471610 -> C471609
Changed lines of the file:
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@@
 	)
 	(symbol
-		(lib_id "mega_shield:π162M")
+		(lib_id "mega_shield:π162U")
 		(at 165.1 115.57 0)
 		(unit 1)
@@
 		(fields_autoplaced yes)
 		(property "Reference" "U1"
-			(at 165.1 97.79 0)
+			(at 165.1 93.98 0)
 			(effects
 				(font
@@
 			)
 		)
-		(property "Value" "Pi_162M"
-			(at 165.1 100.33 0)
+		(property "Value" "PI162U31"
+			(at 165.1 96.52 0)
 			(effects
 				(font
@@
 			)
 		)
-		(property "Description" ""
+		(property "Description" "Digital Isolator, 150kbps 3kV RMS Hex/Six channel"
 			(at 165.1 115.57 0)
 			(effects
@@
 			)
 		)
-		(property "jlcpcb" "C471610"
-			(at 165.1 115.57 0)
+		(property "jlcpcb" "C471609"
+			(at 165.1 99.06 0)
 			(effects
 				(font

Commit message: mega_shield, passing all ERC(electrical rules check). Zero errors
+ Fixed missing symbols from defunct digikey lib.
+ Fixed created custom symbol for AO4486 NMOS.
+ Fixed all Power flag and pin conflicts.
+ Excluded passive/unspecified warnings/errors.
Parts:
- Q1, Q2, Q3, Q4: symbol PCM_Transistor_MOSFET_AKL:2SK3018 -> Transistor_FET:2N7002
