File: mega_shield/servo_interface_.kicad_sch (KiCad schematic)
At the start: 31 parts, among them J1 T4141012081-000, Q1 2N7002, Q2 2N7002, Q3 2N7002, Q4 2N7002, U1 PI162U31

Commit message: Automatic project files update
Parts:
- J1: MANUFACTURER TE Connectivity -> (none)
- TP1, TP13, TP14, TP2, TP3, TP4, TP5: MANUFACTURER Keystone Electronics -> (none)
- TP10, TP11, TP12, TP6, TP7, TP8, TP9: MANUFACTURER Keystone -> (none)
Changed lines of the file:
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@@
 			)
 		)
-		(property "MANUFACTURER" "Keystone Electronics"
+		(property "Manufacturer" "Keystone Electronics"
 			(at 50.8 171.45 0)
 			(hide yes)
@@
 			)
 		)
-		(property "MANUFACTURER" "Keystone"
+		(property "Manufacturer" "Keystone"
 			(at 50.8 135.89 0)
 			(hide yes)
@@
 			)
 		)
-		(property "MANUFACTURER" "Keystone Electronics"
+		(property "Manufacturer" "Keystone Electronics"
 			(at 50.8 180.34 0)
 			(hide yes)
@@
 			)
 		)
-		(property "MANUFACTURER" "TE Connectivity"
+		(property "Manufacturer" "TE Connectivity"
 			(at 43.18 86.36 0)
 			(hide yes)
@@
 			)
 		)
-		(property "MANUFACTURER" "Keystone Electronics"
+		(property "Manufacturer" "Keystone Electronics"
 			(at 33.02 153.67 0)
 			(hide yes)
@@
 			)
 		)
-		(property "MANUFACTURER" "Keystone Electronics"
+		(property "Manufacturer" "Keystone Electronics"
 			(at 33.02 171.45 0)
 			(hide yes)
@@
 			)
 		)
-		(property "MANUFACTURER" "Keystone"
+		(property "Manufacturer" "Keystone"
 			(at 33.02 180.34 0)
 			(hide yes)
@@
 			)
 		)
-		(property "MANUFACTURER" "Keystone Electronics"
+		(property "Manufacturer" "Keystone Electronics"
 			(at 33.02 135.89 0)
 			(hide yes)
@@
 			)
 		)
-		(property "MANUFACTURER" "Keystone"
+		(property "Manufacturer" "Keystone"
 			(at 33.02 199.39 0)
 			(hide yes)
@@
 			)
 		)
-		(property "MANUFACTURER" "Keystone"
+		(property "Manufacturer" "Keystone"
 			(at 50.8 153.67 0)
 			(hide yes)
@@
 			)
 		)
-		(property "MANUFACTURER" "Keystone"
+		(property "Manufacturer" "Keystone"
 			(at 50.8 162.56 0)
 			(hide yes)
@@
 			)
 		)
-		(property "MANUFACTURER" "Keystone"
+		(property "Manufacturer" "Keystone"
 			(at 33.02 189.23 0)
 			(hide yes)
@@
 			)
 		)
-		(property "MANUFACTURER" "Keystone Electronics"
+		(property "Manufacturer" "Keystone Electronics"
 			(at 33.02 162.56 0)
 			(hide yes)
@@
 			)
 		)
-		(property "MANUFACTURER" "Keystone Electronics"
+		(property "Manufacturer" "Keystone Electronics"
 			(at 33.02 144.78 0)
 			(hide yes)
@@
 			)
 		)
-		(property "MANUFACTURER" "Keystone"
+		(property "Manufacturer" "Keystone"
 			(at 50.8 144.78 0)
 			(hide yes)

Commit message: Re-Annotated megashield, added the new totem pole driver JLCPCB numbers and imported into PCB.
Parts:
- renumbered J1 to J9
Changed lines of the file:
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@@
 		(dnp yes)
 		(fields_autoplaced yes)
-		(property "Reference" "J1"
+		(property "Reference" "J9"
 			(at 42.545 71.12 0)
 			(show_name no)
@@
 			(project "mega_shield"
 				(path "/554fcf27-dc63-4666-abbc-7481d15942c4/48beda80-76ca-4f49-9215-034afc6013b0"
-					(reference "J6")
+					(reference "J14")
 					(unit 1)
 				)
 				(path "/554fcf27-dc63-4666-abbc-7481d15942c4/60dac8cc-38c4-4167-a27d-cdec6a027d6c"
-					(reference "J2")
+					(reference "J10")
 					(unit 1)
 				)
 				(path "/554fcf27-dc63-4666-abbc-7481d15942c4/8af2ab12-86f3-4750-9b6f-9fe6810fd117"
-					(reference "J4")
+					(reference "J12")
 					(unit 1)
 				)
 				(path "/554fcf27-dc63-4666-abbc-7481d15942c4/eda7baa6-daec-4ca4-afdf-9fae7ddc238a"
-					(reference "J5")
+					(reference "J13")
 					(unit 1)
 				)
 				(path "/554fcf27-dc63-4666-abbc-7481d15942c4/fa2aff00-6b7c-4012-8bde-20724615a437"
-					(reference "J1")
-					(unit 1)
-				)
+					(reference "J9")
+					(unit 1)
+				)
