File: mega_shield/digital_gpo.kicad_sch (KiCad schematic)
At the start: 21 parts, among them J24 1803277, J25 1803277, Q46 MMBT3904, Q47 MMBT3904, Q49 AO4486, Q50 MMBT3906, Q51 MMBT3906, Q52 AO4486, U10 ADuM1200

Commit message: swapped all homing interfaces into using opto-isolators.
Parts:
- added R62: 3k8, symbol Device:R
- added R63: 1k, symbol Device:R
Connections:
- net +24V_IN: now also R62.1; no longer C62.2, U10.8 (VDD2)
- net GND: now also R63.2
- new net +5V_DIV: C62.2, R62.2, R63.1, U10.8 (VDD2)
Other:
- note added: "Voltage Divider"

Commit message: Added power flag to the voltage divider in the gpo sheet.
Changed lines of the file:
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@@
 	(rectangle
 		(start 29.21 119.38)
-		(end 50.8 160.02)
+		(end 62.23 160.02)
 		(stroke
 			(width 0)
@@
 	)
 	(junction
+		(at 38.1 139.7)
+		(diameter 0)
+		(color 0 0 0 0)
+	)
+	(junction
 		(at 195.58 49.53)
 		(diameter 0)
@@
 	)
 	(junction
+		(at 52.07 139.7)
+		(diameter 0)
+		(color 0 0 0 0)
+	)
+	(junction
 		(at 203.2 116.84)
 		(diameter 0)
@@
 	(wire
 		(pts
+			(xy 53.34 139.7) (xy 52.07 139.7)
+		)
+		(stroke
+			(width 0)
+			(type default)
+		)
+	)
+	(wire
+		(pts
 			(xy 78.74 87.63) (xy 100.33 87.63)
 		)
@@
 	(wire
 		(pts
-			(xy 38.1 137.16) (xy 38.1 142.24)
+			(xy 38.1 137.16) (xy 38.1 139.7)
 		)
 		(stroke
@@
 	(wire
 		(pts
+			(xy 38.1 139.7) (xy 38.1 142.24)
+		)
+		(stroke
+			(width 0)
+			(type default)
+		)
+	)
+	(wire
+		(pts
 			(xy 220.98 49.53) (xy 223.52 49.53)
 		)
@@
 		(pts
 			(xy 220.98 76.2) (xy 218.44 76.2)
+		)
+		(stroke
+			(width 0)
+			(type default)
+		)
+	)
+	(wire
+		(pts
+			(xy 38.1 139.7) (xy 52.07 139.7)
 		)
 		(stroke
@@
 	)
 	(label "+5V_DIV"
-		(at 38.1 139.7 0)
+		(at 53.34 139.7 0)
 		(effects
 			(font
@@
 		)
 	)
+	(symbol
+		(lib_id "power:PWR_FLAG")
+		(at 52.07 139.7 0)
+		(unit 1)
+		(exclude_from_sim no)
+		(in_bom yes)
+		(on_board yes)
+		(dnp no)
+		(fields_autoplaced yes)
+		(property "Reference" "#FLG03"
+			(at 52.07 137.795 0)
+			(effects
+				(font
+					(size 1.27 1.27)
+				)
+				(hide yes)
+			)
+		)
+		(property "Value" "PWR_FLAG"
+			(at 52.07 134.62 0)
+			(effects
+				(font
+					(size 1.27 1.27)
+				)
+			)
+		)
+		(property "Footprint" ""
+			(at 52.07 139.7 0)
+			(effects
+				(font
+					(size 1.27 1.27)
+				)
+				(hide yes)
+			)
+		)
+		(property "Datasheet" "~"
+			(at 52.07 139.7 0)
+			(effects
+				(font
+					(size 1.27 1.27)
+				)
+				(hide yes)
+			)
+		)
+		(property "Description" "Special symbol for telling ERC where power comes from"
+			(at 52.07 139.7 0)
+			(effects
+				(font
+					(size 1.27 1.27)
+				)
+				(hide yes)
+			)
+		)
+		(pin "1"
+		)
+		(instances
+			(project ""
+				(path "/554fcf27-dc63-4666-abbc-7481d15942c4/4360f303-59e6-4d3f-8a36-4d5595cafc98"
+					(reference "#FLG03")
+					(unit 1)
+				)
+			)
+		)
+	)

Commit message: Finished adding test points to the GPO sheet.
Parts:
- added TP101: +5V_DIV, TestPoint:TestPoint_Pad_1.0x1.0mm, symbol Connector:TestPoint
- added TP103: vgate_A, TestPoint:TestPoint_Pad_1.0x1.0mm, symbol Connector:TestPoint
- added TP104: vgate_B, TestPoint:TestPoint_Pad_1.0x1.0mm, symbol Connector:TestPoint
Connections:
- net +5V_DIV: now also TP101.1
- net vgate_A: now also TP103.1
- net vgate_B: now also TP104.1
Other:
- note added: "GPO Test Points"
Changed lines of the file:
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@@
 	)
 	(rectangle
+		(start 30.48 170.18)
+		(end 63.5 187.96)
+		(stroke
+			(width 0)
+			(type default)
+		)
+		(fill
+			(type none)
+		)
+	)
+	(rectangle
 		(start 177.8 25.4)
 		(end 233.68 88.9)
@@
 		)
 	)
+	(text "GPO Test Points"
+		(exclude_from_sim no)
+		(at 39.116 168.656 0)
+		(effects
+			(font
+				(size 1.27 1.27)
+			)
+		)
+	)
 	(text "MOSFET Channel A"
 		(exclude_from_sim no)
@@
 		)
 	)
+	(label "vgate_A"
+		(at 38.1 185.42 0)
+		(effects
+			(font
+				(size 1.27 1.27)
+			)
+			(justify left bottom)
+		)
+	)
 	(label "vgate_B"
 		(at 149.86 109.22 0)
@@
 		)
 	)
+	(label "vgate_B"
+		(at 54.61 185.42 0)
+		(effects
+			(font
+				(size 1.27 1.27)
+			)
+			(justify left bottom)
+		)
+	)
 	(label "+5V_DIV"
 		(at 53.34 139.7 0)
@@
 		)
 	)
+	(label "+5V_DIV"
+		(at 38.1 177.8 0)
+		(effects
+			(font
+				(size 1.27 1.27)
+			)
+			(justify left bottom)
+		)
+	)
 	(hierarchical_label "+24V_IN"
 		(shape input)
@@
 	)
 	(symbol
+		(lib_id "Connector:TestPoint")
+		(at 54.61 185.42 90)
+		(unit 1)
+		(exclude_from_sim no)
+		(in_bom no)
+		(on_board yes)
+		(dnp no)
+		(fields_autoplaced yes)
+		(property "Reference" "TP104"
+			(at 51.308 180.34 90)
+			(effects
+				(font
+					(size 1.27 1.27)
+				)
+			)
+		)
+		(property "Value" "vgate_B"
+			(at 51.308 182.88 90)
+			(effects
+				(font
+					(size 1.27 1.27)
+				)
+			)
+		)
+		(property "Footprint" "TestPoint:TestPoint_Pad_1.0x1.0mm"
+			(at 54.61 180.34 0)
+			(effects
+				(font
+					(size 1.27 1.27)
+				)
+				(hide yes)
+			)
+		)
+		(property "Datasheet" "~"
+			(at 54.61 180.34 0)
+			(effects
+				(font
+					(size 1.27 1.27)
+				)
+				(hide yes)
+			)
+		)
+		(property "Description" "test point"
+			(at 54.61 185.42 0)
+			(effects
+				(font
+					(size 1.27 1.27)
+				)
+				(hide yes)
+			)
+		)
+		(pin "1"
+		)
+		(instances
+			(project "mega_shield"
+				(path "/554fcf27-dc63-4666-abbc-7481d15942c4/4360f303-59e6-4d3f-8a36-4d5595cafc98"
+					(reference "TP104")
+					(unit 1)
+				)
+			)
+		)
+	)
+	(symbol
 		(lib_id "PCM_Transistor_BJT_AKL:MMBT3906")
 		(at 129.54 74.93 0)
@@
 	)
 	(symbol
+		(lib_id "Connector:TestPoint")
+		(at 38.1 177.8 90)
+		(unit 1)
+		(exclude_from_sim no)
+		(in_bom no)
+		(on_board yes)
+		(dnp no)
+		(fields_autoplaced yes)
+		(property "Reference" "TP101"
+			(at 34.798 172.72 90)
+			(effects
+				(font
+					(size 1.27 1.27)
+				)
+			)
+		)
+		(property "Value" "+5V_DIV"
+			(at 34.798 175.26 90)
+			(effects
+				(font
+					(size 1.27 1.27)
+				)
+			)
+		)
+		(property "Footprint" "TestPoint:TestPoint_Pad_1.0x1.0mm"
+			(at 38.1 172.72 0)
+			(effects
+				(font
+					(size 1.27 1.27)
+				)
+				(hide yes)
+			)
+		)
+		(property "Datasheet" "~"
+			(at 38.1 172.72 0)
+			(effects
+				(font
+					(size 1.27 1.27)
+				)
+				(hide yes)
+			)
+		)
+		(property "Description" "test point"
+			(at 38.1 177.8 0)
+			(effects
+				(font
+					(size 1.27 1.27)
+				)
+				(hide yes)
+			)
+		)
+		(pin "1"
+		)
+		(instances
+			(project "mega_shield"
+				(path "/554fcf27-dc63-4666-abbc-7481d15942c4/4360f303-59e6-4d3f-8a36-4d5595cafc98"
+					(reference "TP101")
+					(unit 1)
+				)
+			)
+		)
+	)
+	(symbol
 		(lib_id "PCM_Transistor_MOSFET_AKL:AO4486")
 		(at 213.36 68.58 0)
@@
 					(unit 1)
 				)
+			)
+		)
+	)
+	(symbol
+		(lib_id "Connector:TestPoint")
+		(at 38.1 185.42 90)
+		(unit 1)
+		(exclude_from_sim no)
+		(in_bom no)
+		(on_board yes)
+		(dnp no)
+		(fields_autoplaced yes)
+		(property "Reference" "TP103"
+			(at 34.798 180.34 90)
+			(effects
+				(font
+					(size 1.27 1.27)
+				)
+			)
+		)
+		(property "Value" "vgate_A"
+			(at 34.798 182.88 90)
+			(effects
+				(font
+					(size 1.27 1.27)
+				)
+			)
+		)
+		(property "Footprint" "TestPoint:TestPoint_Pad_1.0x1.0mm"
+			(at 38.1 180.34 0)
+			(effects
+				(font
+					(size 1.27 1.27)
+				)
+				(hide yes)
+			)
+		)
+		(property "Datasheet" "~"
+			(at 38.1 180.34 0)
+			(effects
+				(font
+					(size 1.27 1.27)
+				)
+				(hide yes)
+			)
+		)
+		(property "Description" "test point"
+			(at 38.1 185.42 0)
+			(effects
+				(font
+					(size 1.27 1.27)
+				)
+				(hide yes)
+			)
+		)
+		(pin "1"
+		)
+		(instances
+			(project "mega_shield"
+				(path "/554fcf27-dc63-4666-abbc-7481d15942c4/4360f303-59e6-4d3f-8a36-4d5595cafc98"
+					(reference "TP103")
+					(unit 1)
+				)

Commit message: updated JLCPCB numbers and added new ones.
Parts:
- R62: value 3k8 -> 3k9; footprint (none) -> Resistor_SMD:R_0201_0603Metric; jlcpcb (none) -> C23018
- R63: footprint (none) -> Resistor_SMD:R_0201_0603Metric; jlcpcb (none) -> C21190
- U10: jlcpcb (none) -> C30230
Changed lines of the file:
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@@
+			)
+		)
+		(property "jlcpcb" "C30230"
+			(at 62.23 85.09 0)
+			(effects
+				(font
+					(size 1.27 1.27)
+				)
 			)
 		)
@@
 			)
 		)
-		(property "Footprint" ""
+		(property "Footprint" "Resistor_SMD:R_0201_0603Metric"
 			(at 36.322 146.05 90)
 			(effects
@@
 			)
 		)
+		(property "jlcpcb" "C21190"
+			(at 38.1 146.05 0)
+			(effects
+				(font
+					(size 1.27 1.27)
+				)
+			)
+		)
 		(pin "2"
 		)
@@
 			)
 		)
-		(property "Value" "3k8"
+		(property "Value" "3k9"
 			(at 40.64 134.6199 0)
 			(effects
@@
 			)
 		)
-		(property "Footprint" ""
+		(property "Footprint" "Resistor_SMD:R_0201_0603Metric"
 			(at 36.322 133.35 90)
 			(effects
@@
 			)
 		)
+		(property "jlcpcb" "C23018"
+			(at 38.1 133.35 0)
+			(effects
+				(font
+					(size 1.27 1.27)
+				)
+			)
+		)

Commit message: re-annotating for entire schematic completed.
Parts:
- renumbered C59 to C29, C62 to C30, F14 to F13, F15 to F14, F16 to F15, F17 to F16, J24 to J23, J25 to J24, Q46 to Q25, Q50 to Q26, Q47 to Q27, Q51 to Q28, Q49 to Q29, Q52 to Q30, R62 to R48, R63 to R49, R49 to R50, R50 to R52, R52 to R53, TP101 to TP102, U10 to U26

Commit message: mega_shield, changed footprint for AO4486 to use the built in SO-8-8_3.9mmx4.9mm_P1.27mm
Parts:
- Q29, Q30: footprint PCM_Package_SO_AKL:SO-8_3.9x4.9mm_P1.27mm -> Package_SO:SOP-8_3.76x4.96mm_P1.27mm
Changed lines of the file:
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@@
 			)
 		)
-		(property "Footprint" "PCM_Package_SO_AKL:SO-8_3.9x4.9mm_P1.27mm"
+		(property "Footprint" "Package_SO:SOP-8_3.76x4.96mm_P1.27mm"
 			(at 218.44 133.35 0)
 			(effects
@@
 			)
 		)
-		(property "Footprint" "PCM_Package_SO_AKL:SO-8_3.9x4.9mm_P1.27mm"
+		(property "Footprint" "Package_SO:SOP-8_3.76x4.96mm_P1.27mm"
 			(at 218.44 66.04 0)
 			(effects

Commit message: mega_shield, changed the footprints of the NPN adn PNP bjts to builtin sot-23
Parts:
- Q25, Q26, Q27, Q28: footprint PCM_Package_TO_SOT_SMD_AKL:SOT-23 -> Package_TO_SOT_SMD:SOT-23
Changed lines of the file:
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@@
 			)
 		)
-		(property "Footprint" "PCM_Package_TO_SOT_SMD_AKL:SOT-23"
+		(property "Footprint" "Package_TO_SOT_SMD:SOT-23"
 			(at 134.62 72.39 0)
 			(effects
@@
 			)
 		)
-		(property "Footprint" "PCM_Package_TO_SOT_SMD_AKL:SOT-23"
+		(property "Footprint" "Package_TO_SOT_SMD:SOT-23"
 			(at 134.62 100.33 0)
 			(effects
@@
 			)
 		)
-		(property "Footprint" "PCM_Package_TO_SOT_SMD_AKL:SOT-23"
+		(property "Footprint" "Package_TO_SOT_SMD:SOT-23"
 			(at 134.62 59.69 0)
 			(effects
@@
 			)
 		)
-		(property "Footprint" "PCM_Package_TO_SOT_SMD_AKL:SOT-23"
+		(property "Footprint" "Package_TO_SOT_SMD:SOT-23"
 			(at 134.62 113.03 0)
 			(effects

Commit message: mega_shield, Changed out all caps where needed for in-stock and lower cost parts.
+ Changed out for parts with higher stock.
+ Changed out for 0805 sized components.
+ Changed out for higher voltage.
+ Removed 22uF SMD caps for lower cost 10uF caps in parallel.
+ Updated diode footprint to SOD-123F

BOM cost reduced, and reliability improved.
Parts:
- C43: renamed from C29; value 1u -> 1u/50V; footprint Capacitor_SMD:C_0201_0603Metric -> Capacitor_SMD:C_0805_2012Metric_Pad1.18x1.45mm_HandSolder; jlcpcb C15849 -> C28323
- C44: renamed from C30; value 1u -> 1u/50V; footprint Capacitor_SMD:C_0201_0603Metric -> Capacitor_SMD:C_0805_2012Metric_Pad1.18x1.45mm_HandSolder; jlcpcb C15849 -> C28323
- D5, D6: footprint PCM_Diode_SMD_AKL:D_SOD-123F -> Diode_SMD:D_SOD-123F
Changed lines of the file:
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@@
 			)
 		)
-		(property "Footprint" "PCM_Diode_SMD_AKL:D_SOD-123F"
+		(property "Footprint" "Diode_SMD:D_SOD-123F"
 			(at 217.17 49.53 0)
 			(effects
@@
 		(dnp no)
 		(fields_autoplaced yes)
-		(property "Reference" "C29"
+		(property "Reference" "C43"
 			(at 45.72 60.96 90)
 			(effects
@@
 			)
 		)
-		(property "Value" "1u"
+		(property "Value" "1u/50V"
 			(at 45.72 63.5 90)
 			(effects
@@
 			)
 		)
-		(property "Footprint" "Capacitor_SMD:C_0201_0603Metric"
+		(property "Footprint" "Capacitor_SMD:C_0805_2012Metric_Pad1.18x1.45mm_HandSolder"
 			(at 49.53 67.6148 0)
 			(effects
@@
 			)
 		)
-		(property "jlcpcb" "C15849"
+		(property "jlcpcb" "C28323"
 			(at 45.72 68.58 0)
 			(effects
@@
 			(project "mega_shield"
 				(path "/554fcf27-dc63-4666-abbc-7481d15942c4/4360f303-59e6-4d3f-8a36-4d5595cafc98"
-					(reference "C29")
+					(reference "C43")
 					(unit 1)
 				)
@@
 		(dnp no)
 		(fields_autoplaced yes)
-		(property "Reference" "C30"
+		(property "Reference" "C44"
 			(at 78.74 60.96 90)
 			(effects
@@
 			)
 		)
-		(property "Value" "1u"
+		(property "Value" "1u/50V"
 			(at 78.74 63.5 90)
 			(effects
@@
 			)
 		)
-		(property "Footprint" "Capacitor_SMD:C_0201_0603Metric"
+		(property "Footprint" "Capacitor_SMD:C_0805_2012Metric_Pad1.18x1.45mm_HandSolder"
 			(at 82.55 67.6148 0)
 			(effects
@@
 			)
 		)
-		(property "jlcpcb" "C15849"
+		(property "jlcpcb" "C28323"
 			(at 78.74 68.58 0)
 			(effects
@@
 			(project "mega_shield"
 				(path "/554fcf27-dc63-4666-abbc-7481d15942c4/4360f303-59e6-4d3f-8a36-4d5595cafc98"
-					(reference "C30")
+					(reference "C44")
 					(unit 1)
 				)
@@
 			)
 		)
-		(property "Footprint" "PCM_Diode_SMD_AKL:D_SOD-123F"
+		(property "Footprint" "Diode_SMD:D_SOD-123F"
 			(at 217.17 116.84 0)
 			(effects
