File: mega_shield/digital_gpo.kicad_sch (KiCad schematic)
At the start: 26 parts, among them J23 1803277, J24 1803277, Q26 MMBT3904, Q27 MMBT3906, Q28 MMBT3904, Q29 MMBT3906, Q30 AO4486, Q31 AO4486, U28 L78L05_SOT89, U29 ADuM1200

Commit message: mega_shield, marked circular components as DNP, added jlcpcb numbers to 90degree terminal blocks.
Parts:
- J23, J24: jlcpcb (none) -> C480537
Changed lines of the file:
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@@
+			)
+		)
+		(property "jlcpcb" "C480537"
+			(at 219.71 102.87 0)
+			(effects
+				(font
+					(size 1.27 1.27)
+				)
+				(hide yes)
 			)
 		)
@@
 			(at 219.71 35.56 0)
 			(effects
+				(font
+					(size 1.27 1.27)
+				)
+				(hide yes)
+			)
+		)
+		(property "jlcpcb" "C480537"
+			(at 219.71 35.56 0)
+			(effects

Commit message: mega_shield, re-annotated all components.
Parts:
- renumbered R51 to R73, R52 to R74, R53 to R75, R54 to R76
Changed lines of the file:
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@@
 		(on_board yes)
 		(dnp no)
-		(property "Reference" "R53"
+		(property "Reference" "R75"
 			(at 136.144 66.548 90)
 			(effects
@@
 			(project "mega_shield"
 				(path "/554fcf27-dc63-4666-abbc-7481d15942c4/4360f303-59e6-4d3f-8a36-4d5595cafc98"
-					(reference "R53")
+					(reference "R75")
 					(unit 1)
 				)
@@
 		(dnp no)
 		(fields_autoplaced yes)
-		(property "Reference" "R52"
+		(property "Reference" "R74"
 			(at 119.38 114.2999 0)
 			(effects
@@
 			(project "mega_shield"
 				(path "/554fcf27-dc63-4666-abbc-7481d15942c4/4360f303-59e6-4d3f-8a36-4d5595cafc98"
-					(reference "R52")
+					(reference "R74")
 					(unit 1)
 				)
@@
 		(dnp no)
 		(fields_autoplaced yes)
-		(property "Reference" "R51"
+		(property "Reference" "R73"
 			(at 119.38 73.6599 0)
 			(effects
@@
 			(project ""
 				(path "/554fcf27-dc63-4666-abbc-7481d15942c4/4360f303-59e6-4d3f-8a36-4d5595cafc98"
-					(reference "R51")
+					(reference "R73")
 					(unit 1)
 				)
@@
 		(on_board yes)
 		(dnp no)
-		(property "Reference" "R54"
+		(property "Reference" "R76"
 			(at 136.144 107.188 90)
 			(effects
@@
 			(project "mega_shield"
 				(path "/554fcf27-dc63-4666-abbc-7481d15942c4/4360f303-59e6-4d3f-8a36-4d5595cafc98"
-					(reference "R54")
-					(unit 1)
-				)
+					(reference "R76")
+					(unit 1)
+				)

Commit message: mega_shield, fixed issue with admum1200 footprint.
Parts:
- U29: footprint Package_SO:SOIC-8-1EP_3.9x4.9mm_P1.27mm_EP2.29x3mm -> Package_SO:SOIC-8_3.9x4.9mm_P1.27mm
Changed lines of the file:
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@@
 			)
 		)
-		(property "Footprint" "Package_SO:SOIC-8-1EP_3.9x4.9mm_P1.27mm_EP2.29x3mm"
+		(property "Footprint" "Package_SO:SOIC-8_3.9x4.9mm_P1.27mm"
 			(at 62.23 85.09 0)
 			(effects

Commit message: mega_shield, passing all ERC(electrical rules check). Zero errors
+ Fixed missing symbols from defunct digikey lib.
+ Fixed created custom symbol for AO4486 NMOS.
+ Fixed all Power flag and pin conflicts.
+ Excluded passive/unspecified warnings/errors.
Parts:
- removed D4, D5: SM4007PL, Diode_SMD:D_SOD-123F, symbol PCM_Diode_AKL:SM4007PL
- added D4, D5: SM4007PL, symbol Device:D_Filled
- Q26, Q28: symbol PCM_Transistor_BJT_AKL:MMBT3904 -> Transistor_BJT:MMBT3904
- Q27, Q29: symbol PCM_Transistor_BJT_AKL:MMBT3906 -> Transistor_BJT:MMBT3906
- Q30, Q31: symbol PCM_Transistor_MOSFET_AKL:AO4486 -> mega_shield:UMW_AO4486
Connections:
- net GND: now also Q27.2 (E), Q29.2 (E); no longer Q27.3 (C), Q29.3 (C)
- net at F14.2, F15.2, J24.01: now also D5.1 (K)
- net at J24.02, Q31.5, Q31.6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: now also D5.2 (A)
- net at Q26.2 (E), R75.1: now also Q27.3 (C); no longer Q27.2 (E)
- net at F12.2, F13.2, J23.01: now also D4.1 (K)
- net at J23.02, Q30.5, Q30.6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: now also D4.2 (A)
- net at Q28.2 (E), R76.1: now also Q29.3 (C); no longer Q29.2 (E)

Commit message: mega_shield, rerouted and place components for spindle interface
Parts:
- D4, D5: footprint (none) -> Diode_SMD:D_SOD-123F; jlcpcb (none) -> C64898
Changed lines of the file:
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@@
 			)
 		)
-		(property "Footprint" ""
+		(property "Footprint" "Diode_SMD:D_SOD-123F"
 			(at 217.17 49.53 0)
 			(effects
@@
 		(property "JLCPCB" "C64898"
 			(at 217.17 49.53 90)
+			(effects
+				(font
+					(size 1.27 1.27)
+				)
+				(hide yes)
+			)
+		)
+		(property "jlcpcb" "C64898"
+			(at 217.17 49.53 0)
 			(effects
 				(font
@@
 			)
 		)
-		(property "Footprint" ""
+		(property "Footprint" "Diode_SMD:D_SOD-123F"
 			(at 217.17 116.84 0)
 			(effects
@@
 			(effects
 				(font
+					(size 1.27 1.27)
+				)
+				(hide yes)
+			)
+		)
+		(property "jlcpcb" "C64898"
+			(at 217.17 116.84 0)
+			(effects
+				(font

Commit message: mega_shield, fixed up discrepencies in comments for test points. Added Axis names to silkscreen.
Parts:
- TP109: value RH-5000 -> 5000
- TP110: value RH-5001 -> 5001
- TP111, TP112: value RH-5002 -> 5002
Changed lines of the file:
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@@
 			)
 		)
-		(property "Value" "RH-5002"
+		(property "Value" "5002"
 			(at 51.308 182.88 90)
 			(effects
@@
 			)
 		)
-		(property "Value" "RH-5001"
+		(property "Value" "5001"
 			(at 34.798 182.88 90)
 			(effects
@@
 			)
 		)
-		(property "Value" "RH-5000"
+		(property "Value" "5000"
 			(at 34.798 175.26 90)
 			(effects
@@
 			)
 		)
-		(property "Value" "RH-5002"
+		(property "Value" "5002"
 			(at 51.308 175.26 90)
 			(effects
