File: mega_shield/digital_gpo.kicad_sch (KiCad schematic)
At the start: 26 parts, among them J23 1803277, J24 1803277, Q26 MMBT3904, Q27 MMBT3906, Q28 MMBT3904, Q29 MMBT3906, Q30 AO4486, Q31 AO4486, U28 L78L05_SOT89, U29 ADuM1200

Commit message: Automatic project files update
Parts:
- D4, D5: JLCPCB C64898 -> (none)
- Q30, Q31: JLCPCB C5125950 -> (none)
Changed lines of the file:
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@@
 			)
 		)
-		(property "JLCPCB" "C5125950"
+		(property "jlcpcb" "C5125950"
 			(at 224.79 137.1599 0)
 			(show_name no)
@@
 			)
 		)
-		(property "JLCPCB" "C64898"
+		(property "jlcpcb" "C64898"
 			(at 217.17 49.53 90)
 			(hide yes)
@@
 			)
 		)
-		(property "JLCPCB" "C5125950"
+		(property "jlcpcb" "C5125950"
 			(at 224.79 69.8499 0)
 			(show_name no)
@@
 			)
 		)
-		(property "JLCPCB" "C64898"
+		(property "jlcpcb" "C64898"
 			(at 217.17 116.84 90)
 			(hide yes)
