File: mega_shield/probe_interface.kicad_sch (KiCad schematic)
At the start: 10 parts, among them J22 T4040014031-000, Q45 2SK3018, U30 CS817x22HS

Commit message: removed old isolator IC from other sheets.
Parts:
- removed U30: CS817x22HS, Package_SO:SOIC-8_3.9x4.9mm_P1.27mm, symbol mega_shield:CS817x20HS
Changed lines of the file:
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@@
-	)
-	(symbol
-		(lib_id "mega_shield:CS817x20HS")
-		(at 167.64 85.09 0)
-		(unit 1)
-		(exclude_from_sim no)
-		(in_bom yes)
-		(on_board yes)
-		(dnp no)
-		(fields_autoplaced yes)
-		(property "Reference" "U30"
-			(at 167.64 67.31 0)
-			(effects
-				(font
-					(size 1.27 1.27)
-				)
-			)
-		)
-		(property "Value" "CS817x22HS"
-			(at 167.64 69.85 0)
-			(effects
-				(font
-					(size 1.27 1.27)
-				)
-			)
-		)
-		(property "Footprint" "Package_SO:SOIC-8_3.9x4.9mm_P1.27mm"
-			(at 167.64 85.09 0)
-			(effects
-				(font
-					(size 1.27 1.27)
-				)
-				(hide yes)
-			)
-		)
-		(property "Datasheet" ""
-			(at 167.64 85.09 0)
-			(effects
-				(font
-					(size 1.27 1.27)
-				)
-				(hide yes)
-			)
-		)
-		(property "Description" "Low-Power Dual-Channel Digital Isolator"
-			(at 167.64 85.09 0)
-			(effects
-				(font
-					(size 1.27 1.27)
-				)
-				(hide yes)
-			)
-		)
-		(property "jlcpcb" "C7422523"
-			(at 167.64 85.09 0)
-			(effects
-				(font
-					(size 1.27 1.27)
-				)
-			)
-		)
-		(pin "5"
-		)
-		(pin "2"
-		)
-		(pin "1"
-		)
-		(pin "3"
-		)
-		(pin "4"
-		)
-		(pin "6"
-		)
-		(pin "7"
-		)
-		(pin "8"
-		)
-		(instances
-			(project "mega_shield"
-				(path "/554fcf27-dc63-4666-abbc-7481d15942c4/e56aebf0-16bd-4ef0-8607-05648fa38946"
-					(reference "U30")
-					(unit 1)
-				)
-			)
-		)
 	)
 	(symbol

Commit message: filled the digital isolator for the probe_interface with the analog devices varient.
Parts:
- added U6: ADuM1200, Package_SO:SOIC-8-1EP_3.9x4.9mm_P1.27mm_EP2.29x3mm, symbol mega_shield:ADUM1200ARZ-RL7
Connections:
- net +24V_IN: now also U6.1 (VDD1)
- net +5V_IN: now also U6.8 (VDD2)
- net GND: now also U6.4 (GND1), U6.5 (GND2)
- net PROBE_IN: now also U6.2 (Vin_a)
- net at Q45.1 (G): now also U6.7 (Vout_b)
Changed lines of the file:
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@@
 	(rectangle
 		(start 127 45.72)
-		(end 242.57 121.92)
+		(end 242.57 114.3)
 		(stroke
 			(width 0)
@@
 	)
 	(no_connect
-		(at 186.69 88.9)
+		(at 184.15 86.36)
 	)
 	(no_connect
-		(at 148.59 88.9)
+		(at 151.13 86.36)
 	)
 	(wire
@@
 	(wire
 		(pts
-			(xy 142.24 63.5) (xy 142.24 74.93)
+			(xy 144.78 63.5) (xy 144.78 77.47)
 		)
 		(stroke
@@
 	(wire
 		(pts
-			(xy 194.31 63.5) (xy 194.31 74.93)
-		)
-		(stroke
-			(width 0)
-			(type default)
-		)
-	)
-	(wire
-		(pts
-			(xy 194.31 74.93) (xy 186.69 74.93)
+			(xy 191.77 63.5) (xy 191.77 77.47)
+		)
+		(stroke
+			(width 0)
+			(type default)
+		)
+	)
+	(wire
+		(pts
+			(xy 191.77 77.47) (xy 184.15 77.47)
 		)
 		(stroke
@@
 	(wire
 		(pts
-			(xy 142.24 74.93) (xy 148.59 74.93)
+			(xy 144.78 77.47) (xy 151.13 77.47)
 		)
 		(stroke
@@
 	(wire
 		(pts
-			(xy 186.69 95.25) (xy 195.58 95.25)
+			(xy 184.15 81.28) (xy 207.01 81.28)
+		)
+		(stroke
+			(width 0)
+			(type default)
+		)
+	)
+	(wire
+		(pts
+			(xy 184.15 90.17) (xy 193.04 90.17)
 		)
 		(stroke
@@
 	(wire
 		(pts
-			(xy 147.32 63.5) (xy 142.24 63.5)
-		)
-		(stroke
-			(width 0)
-			(type default)
-		)
-	)
-	(wire
-		(pts
-			(xy 187.96 63.5) (xy 194.31 63.5)
-		)
-		(stroke
-			(width 0)
-			(type default)
-		)
-	)
-	(wire
-		(pts
-			(xy 195.58 104.14) (xy 195.58 95.25)
-		)
-		(stroke
-			(width 0)
-			(type default)
-		)
-	)
-	(wire
-		(pts
-			(xy 148.59 95.25) (xy 138.43 95.25)
+			(xy 147.32 63.5) (xy 144.78 63.5)
+		)
+		(stroke
+			(width 0)
+			(type default)
+		)
+	)
+	(wire
+		(pts
+			(xy 187.96 63.5) (xy 191.77 63.5)
+		)
+		(stroke
+			(width 0)
+			(type default)
+		)
+	)
+	(wire
+		(pts
+			(xy 193.04 99.06) (xy 193.04 90.17)
+		)
+		(stroke
+			(width 0)
+			(type default)
+		)
+	)
+	(wire
+		(pts
+			(xy 151.13 90.17) (xy 140.97 90.17)
 		)
 		(stroke
@@
 	(wire
 		(pts
-			(xy 207.01 81.28) (xy 186.69 81.28)
-		)
-		(stroke
-			(width 0)
-			(type default)
-		)
-	)
-	(wire
-		(pts
 			(xy 207.01 71.12) (xy 207.01 81.28)
 		)
@@
 	(wire
 		(pts
-			(xy 138.43 95.25) (xy 138.43 104.14)
+			(xy 140.97 90.17) (xy 140.97 99.06)
 		)
 		(stroke
@@
 	)
 	(label "V_Proxy"
-		(at 142.24 63.5 180)
+		(at 144.78 63.5 180)
 		(effects
 			(font
@@
 	)
 	(label "PROBE_IN"
-		(at 148.59 81.28 180)
+		(at 151.13 81.28 180)
 		(effects
 			(font
@@
 	(hierarchical_label "+5V_IN"
 		(shape output)
-		(at 194.31 63.5 0)
+		(at 191.77 63.5 0)
 		(effects
 			(font
@@
 	(symbol
 		(lib_id "power:GND")
-		(at 138.43 104.14 0)
+		(at 140.97 99.06 0)
 		(unit 1)
 		(exclude_from_sim no)
@@
 		(fields_autoplaced yes)
 		(property "Reference" "#PWR0170"
-			(at 138.43 110.49 0)
+			(at 140.97 105.41 0)
 			(effects
 				(font
@@
 		)
 		(property "Value" "GND"
-			(at 138.43 109.22 0)
+			(at 140.97 104.14 0)
 			(effects
 				(font
@@
 		)
 		(property "Footprint" ""
-			(at 138.43 104.14 0)
+			(at 140.97 99.06 0)
 			(effects
 				(font
@@
 		)
 		(property "Datasheet" ""
-			(at 138.43 104.14 0)
+			(at 140.97 99.06 0)
 			(effects
 				(font
@@
 		)
 		(property "Description" "Power symbol creates a global label with name \"GND\" , ground"
-			(at 138.43 104.14 0)
+			(at 140.97 99.06 0)
 			(effects
 				(font
@@
 	)
 	(symbol
+		(lib_id "mega_shield:ADUM1200ARZ-RL7")
+		(at 167.64 83.82 0)
+		(unit 1)
+		(exclude_from_sim no)
+		(in_bom yes)
+		(on_board yes)
+		(dnp no)
+		(fields_autoplaced yes)
+		(property "Reference" "U6"
+			(at 167.64 71.12 0)
+			(effects
+				(font
+					(size 1.27 1.27)
+				)
+			)
+		)
+		(property "Value" "ADuM1200"
+			(at 167.64 73.66 0)
+			(effects
+				(font
+					(size 1.27 1.27)
+				)
+			)
+		)
+		(property "Footprint" "Package_SO:SOIC-8-1EP_3.9x4.9mm_P1.27mm_EP2.29x3mm"
+			(at 167.64 83.82 0)
+			(effects
+				(font
+					(size 1.27 1.27)
+				)
+				(hide yes)
+			)
+		)
+		(property "Datasheet" ""
+			(at 167.64 83.82 0)
+			(effects
+				(font
+					(size 1.27 1.27)
+				)
+				(hide yes)
+			)
+		)
+		(property "Description" ""
+			(at 167.64 83.82 0)
+			(effects
+				(font
+					(size 1.27 1.27)
+				)
+				(hide yes)
+			)
+		)
+		(pin "5"
+		)
+		(pin "7"
+		)
+		(pin "1"
+		)
+		(pin "2"
+		)
+		(pin "8"
+		)
+		(pin "4"
+		)
+		(pin "3"
+		)
+		(pin "6"
+		)
+		(instances
+			(project ""
+				(path "/554fcf27-dc63-4666-abbc-7481d15942c4/e56aebf0-16bd-4ef0-8607-05648fa38946"
+					(reference "U6")
+					(unit 1)
+				)
+			)
+		)
+	)
+	(symbol
 		(lib_id "power:GND")
-		(at 195.58 104.14 0)
+		(at 193.04 99.06 0)
 		(unit 1)
 		(exclude_from_sim no)
@@
 		(fields_autoplaced yes)
 		(property "Reference" "#PWR0173"
-			(at 195.58 110.49 0)
+			(at 193.04 105.41 0)
 			(effects
 				(font
@@
 		)
 		(property "Value" "GND"
-			(at 195.58 109.22 0)
+			(at 193.04 104.14 0)
 			(effects
 				(font
@@
 		)
 		(property "Footprint" ""
-			(at 195.58 104.14 0)
+			(at 193.04 99.06 0)
 			(effects
 				(font
@@
 		)
 		(property "Datasheet" ""
-			(at 195.58 104.14 0)
+			(at 193.04 99.06 0)
 			(effects
 				(font
@@
 		)
 		(property "Description" "Power symbol creates a global label with name \"GND\" , ground"
-			(at 195.58 104.14 0)
-			(effects
-				(font
+			(at 193.04 99.06 0)
+			(effects
+				(font

Commit message: propigated changes to the probe interface.
Parts:
- removed C60, C61: 1u, Capacitor_SMD:C_0201_0603Metric, symbol Device:C
- removed Q45: 2SK3018, PCM_Package_TO_SOT_SMD_AKL:SOT-323_SC-70, symbol PCM_Transistor_MOSFET_AKL:2SK3018
- removed R42: 1k, Resistor_SMD:R_0201_0603Metric, symbol Device:R
- removed U6: ADuM1200, Package_SO:SOIC-8-1EP_3.9x4.9mm_P1.27mm_EP2.29x3mm, symbol mega_shield:ADUM1200ARZ-RL7
- added R87: 2k5, symbol Device:R
- added R88: 200, symbol Device:R
- added U30: 4N35, Package_DIP:DIP-6_W7.62mm, symbol Isolator:4N35
Connections:
- net +5V_IN: now also R88.1
- net GND: now also U30.2, U30.4
- net PROBE_IN: now also R87.2
- net PROBE_OUT: now also R88.2, U30.5
- new net: R87.1, U30.1
- no-connect marks 2 -> 1
Other:
- note added: "Opto-Isolated Input"
- note removed: "Digitally Isolated Proximity sensors"

Commit message: Added net-tie to avoid testing error with labeling.
Parts:
- added NT1: NetTie_2, symbol Device:NetTie_2
Connections:
- net +24V_IN: now also NT1.1; no longer C58.1, J22.1, TP99.1
- new net V_Proxy: C58.1, J22.1, NT1.2, TP99.1
Changed lines of the file:
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@@
-	(wire
-		(pts
-			(xy 38.1 33.02) (xy 63.5 33.02)
-		)
-		(stroke
-			(width 0)
-			(type default)
-		)
-	)
 	(wire
 		(pts
@@
 	(wire
 		(pts
+			(xy 38.1 33.02) (xy 48.26 33.02)
+		)
+		(stroke
+			(width 0)
+			(type default)
+		)
+	)
+	(wire
+		(pts
 			(xy 187.96 57.15) (xy 194.31 57.15)
 		)
@@
 		(pts
 			(xy 107.95 59.69) (xy 67.31 59.69)
+		)
+		(stroke
+			(width 0)
+			(type default)
+		)
+	)
+	(wire
+		(pts
+			(xy 53.34 33.02) (xy 63.5 33.02)
 		)
 		(stroke
@@
 					(unit 1)
 				)
+			)
+		)
+	)
+	(symbol
+		(lib_id "Device:NetTie_2")
+		(at 50.8 33.02 0)
+		(mirror x)
+		(unit 1)
+		(exclude_from_sim no)
+		(in_bom no)
+		(on_board yes)
+		(dnp no)
+		(property "Reference" "NT1"
+			(at 50.8 38.1 0)
+			(effects
+				(font
+					(size 1.27 1.27)
+				)
+			)
+		)
+		(property "Value" "NetTie_2"
+			(at 50.8 35.56 0)
+			(effects
+				(font
+					(size 1.27 1.27)
+				)
+			)
+		)
+		(property "Footprint" ""
+			(at 50.8 33.02 0)
+			(effects
+				(font
+					(size 1.27 1.27)
+				)
+				(hide yes)
+			)
+		)
+		(property "Datasheet" "~"
+			(at 50.8 33.02 0)
+			(effects
+				(font
+					(size 1.27 1.27)
+				)
+				(hide yes)
+			)
+		)
+		(property "Description" "Net tie, 2 pins"
+			(at 50.8 33.02 0)
+			(effects
+				(font
+					(size 1.27 1.27)
+				)
+				(hide yes)
+			)
+		)
+		(pin "1"
+		)
+		(pin "2"
+		)
+		(instances
+			(project ""
+				(path "/554fcf27-dc63-4666-abbc-7481d15942c4/e56aebf0-16bd-4ef0-8607-05648fa38946"
+					(reference "NT1")
+					(unit 1)
+				)

Commit message: updated JLCPCB numbers and added new ones.
Parts:
- R87: footprint (none) -> Resistor_SMD:R_0201_0603Metric; jlcpcb (none) -> C25804
- R88: value 200 -> 220; footprint (none) -> Resistor_SMD:R_0201_0603Metric; jlcpcb (none) -> C1226
- U30: jlcpcb (none) -> C3014310
Changed lines of the file:
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@@
 			)
 		)
-		(property "Footprint" ""
+		(property "Footprint" "Resistor_SMD:R_0201_0603Metric"
 			(at 162.56 52.832 90)
 			(effects
@@
 				)
 				(hide yes)
+			)
+		)
+		(property "jlcpcb" "C25804"
+			(at 162.56 54.61 0)
+			(effects
+				(font
+					(size 1.27 1.27)
+				)
 			)
 		)
@@
 			)
 		)
-		(property "Value" "200"
+		(property "Value" "220"
 			(at 190.5 53.3399 0)
 			(effects
@@
 			)
 		)
-		(property "Footprint" ""
+		(property "Footprint" "Resistor_SMD:R_0201_0603Metric"
 			(at 186.182 52.07 90)
 			(effects
@@
 				)
 				(hide yes)
+			)
+		)
+		(property "jlcpcb" "C1226"
+			(at 187.96 52.07 0)
+			(effects
+				(font
+					(size 1.27 1.27)
+				)
 			)
 		)
@@
 			)
 		)
+		(property "jlcpcb" "C3014310"
+			(at 173.99 57.15 0)
+			(effects
+				(font
+					(size 1.27 1.27)
+				)
+			)
+		)

Commit message: re-annotating for entire schematic completed.
Parts:
- renumbered C58 to C28, R87 to R46, R88 to R47, TP102 to TP101, U30 to U25
Changed lines of the file:
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@@
 		(dnp no)
 		(fields_autoplaced yes)
-		(property "Reference" "C58"
+		(property "Reference" "C28"
 			(at 88.9 52.0699 0)
 			(effects
@@
 			(project "mega_shield"
 				(path "/554fcf27-dc63-4666-abbc-7481d15942c4/e56aebf0-16bd-4ef0-8607-05648fa38946"
-					(reference "C58")
+					(reference "C28")
 					(unit 1)
 				)
@@
 		(dnp no)
 		(fields_autoplaced yes)
-		(property "Reference" "TP102"
+		(property "Reference" "TP101"
 			(at 60.198 110.49 90)
 			(effects
@@
 			(project "mega_shield"
 				(path "/554fcf27-dc63-4666-abbc-7481d15942c4/e56aebf0-16bd-4ef0-8607-05648fa38946"
-					(reference "TP102")
+					(reference "TP101")
 					(unit 1)
 				)
@@
 		(dnp no)
 		(fields_autoplaced yes)
-		(property "Reference" "#PWR0229"
+		(property "Reference" "#PWR0108"
 			(at 182.88 69.85 0)
 			(effects
@@
 			(project "mega_shield"
 				(path "/554fcf27-dc63-4666-abbc-7481d15942c4/e56aebf0-16bd-4ef0-8607-05648fa38946"
-					(reference "#PWR0229")
+					(reference "#PWR0108")
 					(unit 1)
 				)
@@
 		(dnp no)
 		(fields_autoplaced yes)
-		(property "Reference" "R87"
+		(property "Reference" "R46"
 			(at 162.56 48.26 90)
 			(effects
@@
 			(project "mega_shield"
 				(path "/554fcf27-dc63-4666-abbc-7481d15942c4/e56aebf0-16bd-4ef0-8607-05648fa38946"
-					(reference "R87")
+					(reference "R46")
 					(unit 1)
 				)
@@
 		(dnp no)
 		(fields_autoplaced yes)
-		(property "Reference" "R88"
+		(property "Reference" "R47"
 			(at 190.5 50.7999 0)
 			(effects
@@
 			(project "mega_shield"
 				(path "/554fcf27-dc63-4666-abbc-7481d15942c4/e56aebf0-16bd-4ef0-8607-05648fa38946"
-					(reference "R88")
+					(reference "R47")
 					(unit 1)
 				)
@@
 		(dnp no)
 		(fields_autoplaced yes)
-		(property "Reference" "#PWR0228"
+		(property "Reference" "#PWR0107"
 			(at 165.1 69.85 0)
 			(effects
@@
 			(project "mega_shield"
 				(path "/554fcf27-dc63-4666-abbc-7481d15942c4/e56aebf0-16bd-4ef0-8607-05648fa38946"
-					(reference "#PWR0228")
+					(reference "#PWR0107")
 					(unit 1)
 				)
@@
 		(dnp no)
 		(fields_autoplaced yes)
-		(property "Reference" "U30"
+		(property "Reference" "U25"
 			(at 173.99 48.26 0)
 			(effects
@@
 			(project "mega_shield"
 				(path "/554fcf27-dc63-4666-abbc-7481d15942c4/e56aebf0-16bd-4ef0-8607-05648fa38946"
-					(reference "U30")
-					(unit 1)
-				)
+					(reference "U25")
+					(unit 1)
+				)

Commit message: mega_shield, Changed out all caps where needed for in-stock and lower cost parts.
+ Changed out for parts with higher stock.
+ Changed out for 0805 sized components.
+ Changed out for higher voltage.
+ Removed 22uF SMD caps for lower cost 10uF caps in parallel.
+ Updated diode footprint to SOD-123F

BOM cost reduced, and reliability improved.
Parts:
- removed C28: 22u, Capacitor_SMD:C_0805_2012Metric, symbol Device:C
- added C42, C45: 10u/50V, Capacitor_SMD:C_0805_2012Metric_Pad1.18x1.45mm_HandSolder, symbol Device:C
Connections:
- net V_Proxy: now also C42.1, C45.1
- net at J22.4: now also C42.2, C45.2
Changed lines of the file:
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@@
+	)
+	(junction
+		(at 83.82 49.53)
+		(diameter 0)
+		(color 0 0 0 0)
+	)
+	(junction
+		(at 83.82 57.15)
+		(diameter 0)
+		(color 0 0 0 0)
 	)
 	(junction
@@
 	(wire
 		(pts
+			(xy 83.82 57.15) (xy 67.31 57.15)
+		)
+		(stroke
+			(width 0)
+			(type default)
+		)
+	)
+	(wire
+		(pts
 			(xy 67.31 54.61) (xy 78.74 54.61)
 		)
@@
 	(wire
 		(pts
-			(xy 92.71 57.15) (xy 67.31 57.15)
-		)
-		(stroke
-			(width 0)
-			(type default)
-		)
-	)
-	(wire
-		(pts
-			(xy 78.74 49.53) (xy 92.71 49.53)
+			(xy 92.71 57.15) (xy 83.82 57.15)
+		)
+		(stroke
+			(width 0)
+			(type default)
+		)
+	)
+	(wire
+		(pts
+			(xy 83.82 49.53) (xy 92.71 49.53)
+		)
+		(stroke
+			(width 0)
+			(type default)
+		)
+	)
+	(wire
+		(pts
+			(xy 78.74 49.53) (xy 83.82 49.53)
 		)
 		(stroke
@@
 		(on_board yes)
 		(dnp no)
-		(fields_autoplaced yes)
-		(property "Reference" "C28"
-			(at 88.9 52.0699 0)
-			(effects
-				(font
-					(size 1.27 1.27)
-				)
-				(justify left)
-			)
-		)
-		(property "Value" "22u"
-			(at 88.9 54.6099 0)
-			(effects
-				(font
-					(size 1.27 1.27)
-				)
-				(justify left)
-			)
-		)
-		(property "Footprint" "Capacitor_SMD:C_0805_2012Metric"
+		(property "Reference" "C45"
+			(at 89.916 49.022 90)
+			(effects
+				(font
+					(size 1.27 1.27)
+				)
+			)
+		)
+		(property "Value" "10u/50V"
+			(at 89.916 57.15 90)
+			(effects
+				(font
+					(size 1.27 1.27)
+				)
+			)
+		)
+		(property "Footprint" "Capacitor_SMD:C_0805_2012Metric_Pad1.18x1.45mm_HandSolder"
 			(at 91.7448 57.15 0)
 			(effects
@@
 			)
 		)
-		(property "jlcpcb" "C6119901"
+		(property "jlcpcb" "C440198"
 			(at 92.71 53.34 0)
 			(effects
@@
 			)
 		)
+		(pin "1"
+		)
 		(pin "2"
-		)
-		(pin "1"
 		)
 		(instances
 			(project "mega_shield"
 				(path "/554fcf27-dc63-4666-abbc-7481d15942c4/e56aebf0-16bd-4ef0-8607-05648fa38946"
-					(reference "C28")
+					(reference "C45")
 					(unit 1)
 				)
@@
 					(unit 1)
 				)
+			)
+		)
+	)
+	(symbol
+		(lib_id "Device:C")
+		(at 83.82 53.34 0)
+		(mirror y)
+		(unit 1)
+		(exclude_from_sim no)
+		(in_bom yes)
+		(on_board yes)
+		(dnp no)
+		(property "Reference" "C42"
+			(at 81.026 49.022 90)
+			(effects
+				(font
+					(size 1.27 1.27)
+				)
+			)
+		)
+		(property "Value" "10u/50V"
+			(at 81.026 57.15 90)
+			(effects
+				(font
+					(size 1.27 1.27)
+				)
+			)
+		)
+		(property "Footprint" "Capacitor_SMD:C_0805_2012Metric_Pad1.18x1.45mm_HandSolder"
+			(at 82.8548 57.15 0)
+			(effects
+				(font
+					(size 1.27 1.27)
+				)
+				(hide yes)
+			)
+		)
+		(property "Datasheet" "~"
+			(at 83.82 53.34 0)
+			(effects
+				(font
+					(size 1.27 1.27)
+				)
+				(hide yes)
+			)
+		)
+		(property "Description" "Unpolarized capacitor"
+			(at 83.82 53.34 0)
+			(effects
+				(font
+					(size 1.27 1.27)
+				)
+				(hide yes)
+			)
+		)
+		(property "jlcpcb" "C440198"
+			(at 83.82 53.34 0)
+			(effects
+				(font
+					(size 1.27 1.27)
+				)
+			)
+		)
+		(pin "1"
+		)
+		(pin "2"
+		)
+		(instances
+			(project "mega_shield"
+				(path "/554fcf27-dc63-4666-abbc-7481d15942c4/e56aebf0-16bd-4ef0-8607-05648fa38946"
+					(reference "C42")
+					(unit 1)
+				)
