File: mega_shield/probe_interface.kicad_sch (KiCad schematic)
At the start: 10 parts, among them J22 T4040014031-000, U25 4N35

Commit message: mega_shield, Added footprint for net tie.
Parts:
- NT1: footprint (none) -> NetTie:NetTie-2_SMD_Pad0.5mm
Changed lines of the file:
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@@
 			)
 		)
-		(property "Footprint" ""
+		(property "Footprint" "NetTie:NetTie-2_SMD_Pad0.5mm"
 			(at 50.8 33.02 0)
 			(effects

Commit message: mega_shield, updated multiple resistors and added comments.
+ Updated optoisolator resistor value --> 15k for better protection.
+ Changed all resistors to 0805 footprints
+ Swapped out expensive values to standardized E24/E96.
+ Updated jlcpcb numbers for all resistors.
Parts:
- R46: value 2k5 -> 15k; footprint Resistor_SMD:R_0201_0603Metric -> Resistor_SMD:R_0805_2012Metric_Pad1.20x1.40mm_HandSolder; jlcpcb C25804 -> C17475
- R47: footprint Resistor_SMD:R_0201_0603Metric -> Resistor_SMD:R_0805_2012Metric_Pad1.20x1.40mm_HandSolder; jlcpcb C1226 -> C17557
Changed lines of the file:
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@@
 			)
 		)
-		(property "Value" "2k5"
+		(property "Value" "15k"
 			(at 162.56 50.8 90)
 			(effects
@@
 			)
 		)
-		(property "Footprint" "Resistor_SMD:R_0201_0603Metric"
+		(property "Footprint" "Resistor_SMD:R_0805_2012Metric_Pad1.20x1.40mm_HandSolder"
 			(at 162.56 52.832 90)
 			(effects
@@
 			)
 		)
-		(property "jlcpcb" "C25804"
+		(property "jlcpcb" "C17475"
 			(at 162.56 54.61 0)
 			(effects
@@
 			)
 		)
-		(property "Footprint" "Resistor_SMD:R_0201_0603Metric"
+		(property "Footprint" "Resistor_SMD:R_0805_2012Metric_Pad1.20x1.40mm_HandSolder"
 			(at 186.182 52.07 90)
 			(effects
@@
 			)
 		)
-		(property "jlcpcb" "C1226"
+		(property "jlcpcb" "C17557"
 			(at 187.96 52.07 0)
 			(effects

Commit message: mega_shield, Set all test points to use the keystone 5000-5004 footprints.
Parts:
- TP100, TP101, TP99: footprint TestPoint:TestPoint_Pad_1.0x1.0mm -> TestPoint:TestPoint_Keystone_5000-5004_Miniature
Changed lines of the file:
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@@
 			)
 		)
-		(property "Footprint" "TestPoint:TestPoint_Pad_1.0x1.0mm"
+		(property "Footprint" "TestPoint:TestPoint_Keystone_5000-5004_Miniature"
 			(at 63.5 110.49 0)
 			(effects
@@
 			)
 		)
-		(property "Footprint" "TestPoint:TestPoint_Pad_1.0x1.0mm"
+		(property "Footprint" "TestPoint:TestPoint_Keystone_5000-5004_Miniature"
 			(at 36.83 110.49 0)
 			(effects
@@
 			)
 		)
-		(property "Footprint" "TestPoint:TestPoint_Pad_1.0x1.0mm"
+		(property "Footprint" "TestPoint:TestPoint_Keystone_5000-5004_Miniature"
 			(at 36.83 102.87 0)
 			(effects

Commit message: mega_shield, updated all 116 test points, changed values based on color code, added jlcpcb numbers and set footprints.
Parts:
- added TP116: RH-5001, TestPoint:TestPoint_Keystone_5000-5004_Miniature, symbol Connector:TestPoint
- TP100, TP99: value TestPoint -> RH-5002; jlcpcb (none) -> C5199802; now in the parts list
- TP101: value TestPoint -> RH-5000; jlcpcb (none) -> C5277086; now in the parts list
Connections:
- net GND: now also TP116.1
Other:
- moved on the sheet: TP100
Changed lines of the file:
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@@
 	)
 	(label "PROBE_IN"
-		(at 36.83 115.57 0)
+		(at 63.5 106.68 0)
 		(effects
 			(font
@@
 		(unit 1)
 		(exclude_from_sim no)
-		(in_bom no)
+		(in_bom yes)
 		(on_board yes)
 		(dnp no)
@@
 			)
 		)
-		(property "Value" "TestPoint"
+		(property "Value" "RH-5000"
 			(at 60.198 113.03 90)
 			(effects
@@
 		(property "Description" "test point"
 			(at 63.5 115.57 0)
+			(effects
+				(font
+					(size 1.27 1.27)
+				)
+				(hide yes)
+			)
+		)
+		(property "jlcpcb" "C5277086"
+			(at 63.5 115.57 90)
 			(effects
 				(font
@@
 	)
 	(symbol
+		(lib_id "power:GND")
+		(at 36.83 115.57 90)
+		(unit 1)
+		(exclude_from_sim no)
+		(in_bom yes)
+		(on_board yes)
+		(dnp no)
+		(fields_autoplaced yes)
+		(property "Reference" "#PWR0130"
+			(at 43.18 115.57 0)
+			(effects
+				(font
+					(size 1.27 1.27)
+				)
+				(hide yes)
+			)
+		)
+		(property "Value" "GND"
+			(at 40.64 115.5699 90)
+			(effects
+				(font
+					(size 1.27 1.27)
+				)
+				(justify right)
+			)
+		)
+		(property "Footprint" ""
+			(at 36.83 115.57 0)
+			(effects
+				(font
+					(size 1.27 1.27)
+				)
+				(hide yes)
+			)
+		)
+		(property "Datasheet" ""
+			(at 36.83 115.57 0)
+			(effects
+				(font
+					(size 1.27 1.27)
+				)
+				(hide yes)
+			)
+		)
+		(property "Description" "Power symbol creates a global label with name \"GND\" , ground"
+			(at 36.83 115.57 0)
+			(effects
+				(font
+					(size 1.27 1.27)
+				)
+				(hide yes)
+			)
+		)
+		(pin "1"
+		)
+		(instances
+			(project "mega_shield"
+				(path "/554fcf27-dc63-4666-abbc-7481d15942c4/e56aebf0-16bd-4ef0-8607-05648fa38946"
+					(reference "#PWR0130")
+					(unit 1)
+				)
+			)
+		)
+	)
+	(symbol
 		(lib_id "Device:NetTie_2")
 		(at 50.8 33.02 0)
@@
 		(unit 1)
 		(exclude_from_sim no)
-		(in_bom no)
+		(in_bom yes)
+		(on_board yes)
+		(dnp no)
+		(property "Reference" "TP116"
+			(at 33.528 110.49 90)
+			(effects
+				(font
+					(size 1.27 1.27)
+				)
+			)
+		)
+		(property "Value" "RH-5001"
+			(at 33.528 113.03 90)
+			(effects
+				(font
+					(size 1.27 1.27)
+				)
+			)
+		)
+		(property "Footprint" "TestPoint:TestPoint_Keystone_5000-5004_Miniature"
+			(at 36.83 110.49 0)
+			(effects
+				(font
+					(size 1.27 1.27)
+				)
+				(hide yes)
+			)
+		)
+		(property "Datasheet" "~"
+			(at 36.83 110.49 0)
+			(effects
+				(font
+					(size 1.27 1.27)
+				)
+				(hide yes)
+			)
+		)
+		(property "Description" "test point"
+			(at 36.83 115.57 0)
+			(effects
+				(font
+					(size 1.27 1.27)
+				)
+				(hide yes)
+			)
+		)
+		(property "jlcpcb" "C5199801"
+			(at 36.83 115.57 90)
+			(effects
+				(font
+					(size 1.27 1.27)
+				)
+				(hide yes)
+			)
+		)
+		(pin "1"
+		)
+		(instances
+			(project "mega_shield"
+				(path "/554fcf27-dc63-4666-abbc-7481d15942c4/e56aebf0-16bd-4ef0-8607-05648fa38946"
+					(reference "TP116")
+					(unit 1)
+				)
+			)
+		)
+	)
+	(symbol
+		(lib_id "Connector:TestPoint")
+		(at 63.5 106.68 90)
+		(unit 1)
+		(exclude_from_sim no)
+		(in_bom yes)
 		(on_board yes)
 		(dnp no)
 		(fields_autoplaced yes)
 		(property "Reference" "TP100"
-			(at 33.528 110.49 90)
-			(effects
-				(font
-					(size 1.27 1.27)
-				)
-			)
-		)
-		(property "Value" "TestPoint"
-			(at 33.528 113.03 90)
+			(at 60.198 101.6 90)
+			(effects
+				(font
+					(size 1.27 1.27)
+				)
+			)
+		)
+		(property "Value" "RH-5002"
+			(at 60.198 104.14 90)
 			(effects
 				(font
@@
 		)
 		(property "Footprint" "TestPoint:TestPoint_Keystone_5000-5004_Miniature"
-			(at 36.83 110.49 0)
+			(at 63.5 101.6 0)
 			(effects
 				(font
@@
 		)
 		(property "Datasheet" "~"
-			(at 36.83 110.49 0)
+			(at 63.5 101.6 0)
 			(effects
 				(font
@@
 		)
 		(property "Description" "test point"
-			(at 36.83 115.57 0)
+			(at 63.5 106.68 0)
+			(effects
+				(font
+					(size 1.27 1.27)
+				)
+				(hide yes)
+			)
+		)
+		(property "jlcpcb" "C5199802"
+			(at 63.5 106.68 90)
 			(effects
 				(font
@@
 		(unit 1)
 		(exclude_from_sim no)
-		(in_bom no)
+		(in_bom yes)
 		(on_board yes)
 		(dnp no)
@@
 			)
 		)
-		(property "Value" "TestPoint"
+		(property "Value" "RH-5002"
 			(at 33.528 105.41 90)
 			(effects
@@
 			(effects
 				(font
+					(size 1.27 1.27)
+				)
+				(hide yes)
+			)
+		)
+		(property "jlcpcb" "C5199802"
+			(at 36.83 107.95 90)
+			(effects
+				(font

Commit message: mega_shield, Added all test point symbols and updated association of 3D models.
Parts:
- renumbered C45 to C43, TP99 to TP105, TP116 to TP106, TP100 to TP107, TP101 to TP108
Changed lines of the file:
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@@
 		(on_board yes)
 		(dnp no)
-		(property "Reference" "C45"
+		(property "Reference" "C43"
 			(at 89.916 49.022 90)
 			(effects
@@
 			(project "mega_shield"
 				(path "/554fcf27-dc63-4666-abbc-7481d15942c4/e56aebf0-16bd-4ef0-8607-05648fa38946"
-					(reference "C45")
+					(reference "C43")
 					(unit 1)
 				)
@@
 		(dnp no)
 		(fields_autoplaced yes)
-		(property "Reference" "TP101"
+		(property "Reference" "TP108"
 			(at 60.198 110.49 90)
 			(effects
@@
 			(project "mega_shield"
 				(path "/554fcf27-dc63-4666-abbc-7481d15942c4/e56aebf0-16bd-4ef0-8607-05648fa38946"
-					(reference "TP101")
+					(reference "TP108")
 					(unit 1)
 				)
@@
 		(dnp no)
 		(fields_autoplaced yes)
-		(property "Reference" "#PWR0108"
+		(property "Reference" "#PWR0115"
 			(at 182.88 69.85 0)
 			(effects
@@
 			(project "mega_shield"
 				(path "/554fcf27-dc63-4666-abbc-7481d15942c4/e56aebf0-16bd-4ef0-8607-05648fa38946"
-					(reference "#PWR0108")
+					(reference "#PWR0115")
 					(unit 1)
 				)
@@
 		(dnp no)
 		(fields_autoplaced yes)
-		(property "Reference" "#PWR0130"
+		(property "Reference" "#PWR0113"
 			(at 43.18 115.57 0)
 			(effects
@@
 			(project "mega_shield"
 				(path "/554fcf27-dc63-4666-abbc-7481d15942c4/e56aebf0-16bd-4ef0-8607-05648fa38946"
-					(reference "#PWR0130")
+					(reference "#PWR0113")
 					(unit 1)
 				)
@@
 		(on_board yes)
 		(dnp no)
-		(property "Reference" "TP116"
+		(property "Reference" "TP106"
 			(at 33.528 110.49 90)
 			(effects
@@
 			(project "mega_shield"
 				(path "/554fcf27-dc63-4666-abbc-7481d15942c4/e56aebf0-16bd-4ef0-8607-05648fa38946"
-					(reference "TP116")
+					(reference "TP106")
 					(unit 1)
 				)
@@
 		(dnp no)
 		(fields_autoplaced yes)
-		(property "Reference" "TP100"
+		(property "Reference" "TP107"
 			(at 60.198 101.6 90)
 			(effects
@@
 			(project "mega_shield"
 				(path "/554fcf27-dc63-4666-abbc-7481d15942c4/e56aebf0-16bd-4ef0-8607-05648fa38946"
-					(reference "TP100")
+					(reference "TP107")
 					(unit 1)
 				)
@@
 		(dnp no)
 		(fields_autoplaced yes)
-		(property "Reference" "TP99"
+		(property "Reference" "TP105"
 			(at 33.528 102.87 90)
 			(effects
@@
 			(project "mega_shield"
 				(path "/554fcf27-dc63-4666-abbc-7481d15942c4/e56aebf0-16bd-4ef0-8607-05648fa38946"
-					(reference "TP99")
+					(reference "TP105")
 					(unit 1)
 				)
@@
 		(dnp no)
 		(fields_autoplaced yes)
-		(property "Reference" "#PWR0107"
+		(property "Reference" "#PWR0114"
 			(at 165.1 69.85 0)
 			(effects
@@
 			(project "mega_shield"
 				(path "/554fcf27-dc63-4666-abbc-7481d15942c4/e56aebf0-16bd-4ef0-8607-05648fa38946"
-					(reference "#PWR0107")
-					(unit 1)
-				)
+					(reference "#PWR0114")
+					(unit 1)
+				)

Commit message: mega_shield, working on rebuilding homoing interface layout.
Parts:
- TP105, TP107: footprint TestPoint:TestPoint_Keystone_5000-5004_Miniature -> footprints:KEYSTONE_5002
- TP106: footprint TestPoint:TestPoint_Keystone_5000-5004_Miniature -> footprints:KEYSTONE_5001
- TP108: footprint TestPoint:TestPoint_Keystone_5000-5004_Miniature -> footprints:KEYSTONE_5000
Changed lines of the file:
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@@
 			)
 		)
-		(property "Footprint" "TestPoint:TestPoint_Keystone_5000-5004_Miniature"
+		(property "Footprint" "footprints:KEYSTONE_5000"
 			(at 63.5 110.49 0)
 			(effects
@@
 			)
 		)
-		(property "Footprint" "TestPoint:TestPoint_Keystone_5000-5004_Miniature"
+		(property "Footprint" "footprints:KEYSTONE_5001"
 			(at 36.83 110.49 0)
 			(effects
@@
 			)
 		)
-		(property "Footprint" "TestPoint:TestPoint_Keystone_5000-5004_Miniature"
+		(property "Footprint" "footprints:KEYSTONE_5002"
 			(at 63.5 101.6 0)
 			(effects
@@
 			)
 		)
-		(property "Footprint" "TestPoint:TestPoint_Keystone_5000-5004_Miniature"
+		(property "Footprint" "footprints:KEYSTONE_5002"
 			(at 36.83 102.87 0)
 			(effects

Commit message: mega_shield, changed text info in probe interface(schematic).
Other:
- note added: "Probe Interface Test Points"
- note removed: "Homing Interface Test Points"
Changed lines of the file:
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@@
 		)
 	)
-	(text "Homing Interface Test Points"
+	(text "Probe Interface Test Points"
 		(exclude_from_sim no)
 		(at 39.624 94.234 0)

Commit message: mega_shield, layout of probe interface finished, setup 1mm net-tie and routed traces.
Parts:
- NT1: footprint NetTie:NetTie-2_SMD_Pad0.5mm -> NetTie:NetTie-2_THT_Pad1.0mm
Changed lines of the file:
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@@
 			)
 		)
-		(property "Footprint" "NetTie:NetTie-2_SMD_Pad0.5mm"
+		(property "Footprint" "NetTie:NetTie-2_THT_Pad1.0mm"
 			(at 50.8 33.02 0)
 			(effects
