File: mega_shield/digital_gpi.kicad_sch (KiCad schematic)
At the start: 5 parts, among them J26 1803277, J27 1803277, U11 ADuM1200

Commit message: swapped gpi sheet to optical input, currently availble isolators pricing is not ideal.
Parts:
- removed C63, C64: 1u, Capacitor_SMD:C_0201_0603Metric, symbol Device:C
- removed U11: ADuM1200, Package_SO:SOIC-8-1EP_3.9x4.9mm_P1.27mm_EP2.29x3mm, symbol mega_shield:ADUM1200ARZ-RL7
- added R61, R65: 2k5, symbol Device:R
- added R64, R66: 200, symbol Device:R
- added U12, U13: 4N35, Package_DIP:DIP-6_W7.62mm, symbol Isolator:4N35
Connections:
- net +5V_IN: now also R64.1, R66.1
- net 24V_digital_input2: now also R65.2
- net GND: now also U12.2, U12.4, U13.2, U13.4; no longer J26.01
- net digital_input1: now also R64.2, U12.5
- net digital_input2: now also R66.2, U13.5
- new net: R61.1, U12.1
- new net: R65.1, U13.1
- new net 24V_digital_input1: J26.01, R61.2
- no-connect marks 0 -> 2
Other:
- note added: "Opto-Isolated Input"
- note removed: "Digitally Isolated Proximity sensors"
- moved on the sheet: J26

Commit message: Finished adding test points to the GPI sheet.
Parts:
- added TP105: +5V_DIV, TestPoint:TestPoint_Pad_1.0x1.0mm, symbol Connector:TestPoint
- added TP106: vgate_A, TestPoint:TestPoint_Pad_1.0x1.0mm, symbol Connector:TestPoint
- added TP107, TP108: vgate_B, TestPoint:TestPoint_Pad_1.0x1.0mm, symbol Connector:TestPoint
Connections:
- net 24V_digital_input1: now also TP105.1
- net 24V_digital_input2: now also TP106.1
- net digital_input1: now also TP108.1
- net digital_input2: now also TP107.1
Other:
- note added: "GPI Test Points"

Commit message: updated JLCPCB numbers and added new ones.
Parts:
- R61, R65: footprint (none) -> Resistor_SMD:R_0201_0603Metric; jlcpcb (none) -> C25804
- R64, R66: value 200 -> 220; footprint (none) -> Resistor_SMD:R_0201_0603Metric; jlcpcb (none) -> C1226
- U12, U13: jlcpcb (none) -> C3014310
Changed lines of the file:
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@@
 			)
 		)
-		(property "Value" "200"
+		(property "Value" "220"
 			(at 167.64 104.1399 0)
 			(effects
@@
 			)
 		)
-		(property "Footprint" ""
+		(property "Footprint" "Resistor_SMD:R_0201_0603Metric"
 			(at 163.322 102.87 90)
 			(effects
@@
 			)
 		)
+		(property "jlcpcb" "C1226"
+			(at 165.1 102.87 0)
+			(effects
+				(font
+					(size 1.27 1.27)
+				)
+			)
+		)
 		(pin "1"
 		)
@@
 			)
 		)
-		(property "Footprint" ""
+		(property "Footprint" "Resistor_SMD:R_0201_0603Metric"
 			(at 139.7 65.532 90)
 			(effects
@@
 			)
 		)
+		(property "jlcpcb" "C25804"
+			(at 139.7 67.31 0)
+			(effects
+				(font
+					(size 1.27 1.27)
+				)
+			)
+		)
 		(pin "1"
 		)
@@
 			)
 		)
+		(property "jlcpcb" "C3014310"
+			(at 151.13 69.85 0)
+			(effects
+				(font
+					(size 1.27 1.27)
+				)
+			)
+		)
 		(pin "1"
 		)
@@
 			)
 		)
-		(property "Value" "200"
+		(property "Value" "220"
 			(at 167.64 66.0399 0)
 			(effects
@@
 			)
 		)
-		(property "Footprint" ""
+		(property "Footprint" "Resistor_SMD:R_0201_0603Metric"
 			(at 163.322 64.77 90)
 			(effects
@@
 			)
 		)
+		(property "jlcpcb" "C1226"
+			(at 165.1 64.77 0)
+			(effects
+				(font
+					(size 1.27 1.27)
+				)
+			)
+		)
 		(pin "1"
 		)
@@
 			)
 		)
-		(property "Footprint" ""
+		(property "Footprint" "Resistor_SMD:R_0201_0603Metric"
 			(at 139.7 103.632 90)
 			(effects
@@
 			)
 		)
+		(property "jlcpcb" "C25804"
+			(at 139.7 105.41 0)
+			(effects
+				(font
+					(size 1.27 1.27)
+				)
+			)
+		)
 		(pin "1"
 		)
@@
 			)
 		)
+		(property "jlcpcb" "C3014310"
+			(at 151.13 107.95 0)
+			(effects
+				(font
+					(size 1.27 1.27)
+				)
+			)
+		)

Commit message: re-annotating for entire schematic completed.
Parts:
- renumbered J26 to J25, J27 to J26, R61 to R54, R65 to R55, R64 to R56, R66 to R57, TP108 to TP107, TP107 to TP108, U12 to U27, U13 to U28
Changed lines of the file:
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@@
 		(dnp no)
 		(fields_autoplaced yes)
-		(property "Reference" "R66"
+		(property "Reference" "R57"
 			(at 167.64 101.5999 0)
 			(effects
@@
 			(project "mega_shield"
 				(path "/554fcf27-dc63-4666-abbc-7481d15942c4/4443c59e-c01d-4253-ab50-7467fe3f72ca"
-					(reference "R66")
+					(reference "R57")
 					(unit 1)
 				)
@@
 		(dnp no)
 		(fields_autoplaced yes)
-		(property "Reference" "R61"
+		(property "Reference" "R54"
 			(at 139.7 60.96 90)
 			(effects
@@
 			(project ""
 				(path "/554fcf27-dc63-4666-abbc-7481d15942c4/4443c59e-c01d-4253-ab50-7467fe3f72ca"
-					(reference "R61")
+					(reference "R54")
 					(unit 1)
 				)
@@
 		(dnp no)
 		(fields_autoplaced yes)
-		(property "Reference" "#PWR0206"
+		(property "Reference" "#PWR0120"
 			(at 142.24 120.65 0)
 			(effects
@@
 			(project "mega_shield"
 				(path "/554fcf27-dc63-4666-abbc-7481d15942c4/4443c59e-c01d-4253-ab50-7467fe3f72ca"
-					(reference "#PWR0206")
+					(reference "#PWR0120")
 					(unit 1)
 				)
@@
 		(dnp no)
 		(fields_autoplaced yes)
-		(property "Reference" "TP107"
+		(property "Reference" "TP108"
 			(at 55.118 149.86 90)
 			(effects
@@
 			(project "mega_shield"
 				(path "/554fcf27-dc63-4666-abbc-7481d15942c4/4443c59e-c01d-4253-ab50-7467fe3f72ca"
-					(reference "TP107")
+					(reference "TP108")
 					(unit 1)
 				)
@@
 		(dnp no)
 		(fields_autoplaced yes)
-		(property "Reference" "#PWR0203"
+		(property "Reference" "#PWR0119"
 			(at 142.24 82.55 0)
 			(effects
@@
 			(project "mega_shield"
 				(path "/554fcf27-dc63-4666-abbc-7481d15942c4/4443c59e-c01d-4253-ab50-7467fe3f72ca"
-					(reference "#PWR0203")
+					(reference "#PWR0119")
 					(unit 1)
 				)
@@
 		(dnp no)
 		(fields_autoplaced yes)
-		(property "Reference" "#PWR0207"
+		(property "Reference" "#PWR0122"
 			(at 160.02 120.65 0)
 			(effects
@@
 			(project "mega_shield"
 				(path "/554fcf27-dc63-4666-abbc-7481d15942c4/4443c59e-c01d-4253-ab50-7467fe3f72ca"
-					(reference "#PWR0207")
+					(reference "#PWR0122")
 					(unit 1)
 				)
@@
 		(dnp no)
 		(fields_autoplaced yes)
-		(property "Reference" "#PWR0205"
+		(property "Reference" "#PWR0121"
 			(at 160.02 82.55 0)
 			(effects
@@
 			(project "mega_shield"
 				(path "/554fcf27-dc63-4666-abbc-7481d15942c4/4443c59e-c01d-4253-ab50-7467fe3f72ca"
-					(reference "#PWR0205")
+					(reference "#PWR0121")
 					(unit 1)
 				)
@@
 		(dnp no)
 		(fields_autoplaced yes)
-		(property "Reference" "U12"
+		(property "Reference" "U27"
 			(at 151.13 60.96 0)
 			(effects
@@
 			(project ""
 				(path "/554fcf27-dc63-4666-abbc-7481d15942c4/4443c59e-c01d-4253-ab50-7467fe3f72ca"
-					(reference "U12")
+					(reference "U27")
 					(unit 1)
 				)
@@
 		(dnp no)
 		(fields_autoplaced yes)
-		(property "Reference" "#PWR0189"
+		(property "Reference" "#PWR0118"
 			(at 90.17 111.76 0)
 			(effects
@@
 			(project "mega_shield"
 				(path "/554fcf27-dc63-4666-abbc-7481d15942c4/4443c59e-c01d-4253-ab50-7467fe3f72ca"
-					(reference "#PWR0189")
+					(reference "#PWR0118")
 					(unit 1)
 				)
@@
 		(dnp no)
 		(fields_autoplaced yes)
-		(property "Reference" "R64"
+		(property "Reference" "R56"
 			(at 167.64 63.4999 0)
 			(effects
@@
 			(project "mega_shield"
 				(path "/554fcf27-dc63-4666-abbc-7481d15942c4/4443c59e-c01d-4253-ab50-7467fe3f72ca"
-					(reference "R64")
+					(reference "R56")
 					(unit 1)
 				)
@@
 		(dnp no)
 		(fields_autoplaced yes)
-		(property "Reference" "R65"
+		(property "Reference" "R55"
 			(at 139.7 99.06 90)
 			(effects
@@
 			(project "mega_shield"
 				(path "/554fcf27-dc63-4666-abbc-7481d15942c4/4443c59e-c01d-4253-ab50-7467fe3f72ca"
-					(reference "R65")
+					(reference "R55")
 					(unit 1)
 				)
@@
 		(dnp no)
 		(fields_autoplaced yes)
-		(property "Reference" "U13"
+		(property "Reference" "U28"
 			(at 151.13 99.06 0)
 			(effects
@@
 			(project "mega_shield"
 				(path "/554fcf27-dc63-4666-abbc-7481d15942c4/4443c59e-c01d-4253-ab50-7467fe3f72ca"
-					(reference "U13")
+					(reference "U28")
 					(unit 1)
 				)
@@
 		(dnp no)
 		(fields_autoplaced yes)
-		(property "Reference" "TP108"
+		(property "Reference" "TP107"
 			(at 55.118 142.24 90)
 			(effects
@@
 			(project "mega_shield"
 				(path "/554fcf27-dc63-4666-abbc-7481d15942c4/4443c59e-c01d-4253-ab50-7467fe3f72ca"
-					(reference "TP108")
+					(reference "TP107")
 					(unit 1)
 				)
@@
 		(on_board yes)
 		(dnp no)
-		(property "Reference" "J26"
+		(property "Reference" "J25"
 			(at 76.2 90.17 0)
 			(effects
@@
 			(project "mega_shield"
 				(path "/554fcf27-dc63-4666-abbc-7481d15942c4/4443c59e-c01d-4253-ab50-7467fe3f72ca"
-					(reference "J26")
+					(reference "J25")
 					(unit 1)
 				)
@@
 		(on_board yes)
 		(dnp no)
-		(property "Reference" "J27"
+		(property "Reference" "J26"
 			(at 76.2 104.14 0)
 			(effects
@@
 			(project "mega_shield"
 				(path "/554fcf27-dc63-4666-abbc-7481d15942c4/4443c59e-c01d-4253-ab50-7467fe3f72ca"
-					(reference "J27")
-					(unit 1)
-				)
+					(reference "J26")
+					(unit 1)
+				)

Commit message: created layout for the gpi sheet.
Parts:
- TP107: value vgate_B -> digital_input1
- TP108: value vgate_B -> digital_input2
Changed lines of the file:
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@@
 			)
 		)
-		(property "Value" "vgate_B"
+		(property "Value" "digital_input2"
 			(at 55.118 152.4 90)
 			(effects
@@
 			)
 		)
-		(property "Value" "vgate_B"
+		(property "Value" "digital_input1"
 			(at 55.118 144.78 90)
 			(effects

Commit message: mega_shield, updated multiple resistors and added comments.
+ Updated optoisolator resistor value --> 15k for better protection.
+ Changed all resistors to 0805 footprints
+ Swapped out expensive values to standardized E24/E96.
+ Updated jlcpcb numbers for all resistors.
Parts:
- R54, R55: value 2k5 -> 15k; footprint Resistor_SMD:R_0201_0603Metric -> Resistor_SMD:R_0805_2012Metric_Pad1.20x1.40mm_HandSolder; jlcpcb C25804 -> C17475
- R56, R57: footprint Resistor_SMD:R_0201_0603Metric -> Resistor_SMD:R_0805_2012Metric_Pad1.20x1.40mm_HandSolder; jlcpcb C1226 -> C17557
Changed lines of the file:
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@@
 			)
 		)
-		(property "Footprint" "Resistor_SMD:R_0201_0603Metric"
+		(property "Footprint" "Resistor_SMD:R_0805_2012Metric_Pad1.20x1.40mm_HandSolder"
 			(at 163.322 102.87 90)
 			(effects
@@
 			)
 		)
-		(property "jlcpcb" "C1226"
+		(property "jlcpcb" "C17557"
 			(at 165.1 102.87 0)
 			(effects
@@
 			)
 		)
-		(property "Value" "2k5"
+		(property "Value" "15k"
 			(at 139.7 63.5 90)
 			(effects
@@
 			)
 		)
-		(property "Footprint" "Resistor_SMD:R_0201_0603Metric"
+		(property "Footprint" "Resistor_SMD:R_0805_2012Metric_Pad1.20x1.40mm_HandSolder"
 			(at 139.7 65.532 90)
 			(effects
@@
 			)
 		)
-		(property "jlcpcb" "C25804"
+		(property "jlcpcb" "C17475"
 			(at 139.7 67.31 0)
 			(effects
@@
 			)
 		)
-		(property "Footprint" "Resistor_SMD:R_0201_0603Metric"
+		(property "Footprint" "Resistor_SMD:R_0805_2012Metric_Pad1.20x1.40mm_HandSolder"
 			(at 163.322 64.77 90)
 			(effects
@@
 			)
 		)
-		(property "jlcpcb" "C1226"
+		(property "jlcpcb" "C17557"
 			(at 165.1 64.77 0)
 			(effects
@@
 			)
 		)
-		(property "Value" "2k5"
+		(property "Value" "15k"
 			(at 139.7 101.6 90)
 			(effects
@@
 			)
 		)
-		(property "Footprint" "Resistor_SMD:R_0201_0603Metric"
+		(property "Footprint" "Resistor_SMD:R_0805_2012Metric_Pad1.20x1.40mm_HandSolder"
 			(at 139.7 103.632 90)
 			(effects
@@
 			)
 		)
-		(property "jlcpcb" "C25804"
+		(property "jlcpcb" "C17475"
 			(at 139.7 105.41 0)
 			(effects

Commit message: mega_shield, Set all test points to use the keystone 5000-5004 footprints.
Parts:
- TP105, TP106, TP107, TP108: footprint TestPoint:TestPoint_Pad_1.0x1.0mm -> TestPoint:TestPoint_Keystone_5000-5004_Miniature
Changed lines of the file:
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@@
 			)
 		)
-		(property "Footprint" "TestPoint:TestPoint_Pad_1.0x1.0mm"
+		(property "Footprint" "TestPoint:TestPoint_Keystone_5000-5004_Miniature"
 			(at 31.75 142.24 0)
 			(effects
@@
 			)
 		)
-		(property "Footprint" "TestPoint:TestPoint_Pad_1.0x1.0mm"
+		(property "Footprint" "TestPoint:TestPoint_Keystone_5000-5004_Miniature"
 			(at 31.75 149.86 0)
 			(effects
@@
 			)
 		)
-		(property "Footprint" "TestPoint:TestPoint_Pad_1.0x1.0mm"
+		(property "Footprint" "TestPoint:TestPoint_Keystone_5000-5004_Miniature"
 			(at 58.42 149.86 0)
 			(effects
@@
 			)
 		)
-		(property "Footprint" "TestPoint:TestPoint_Pad_1.0x1.0mm"
+		(property "Footprint" "TestPoint:TestPoint_Keystone_5000-5004_Miniature"
 			(at 58.42 142.24 0)
 			(effects

Commit message: mega_shield, updated all 116 test points, changed values based on color code, added jlcpcb numbers and set footprints.
Parts:
- TP105: value +5V_DIV -> RH-5002; jlcpcb (none) -> C5199802; now in the parts list
- TP106: value vgate_A -> RH-5002; jlcpcb (none) -> C5199802; now in the parts list
- TP107: value digital_input1 -> RH-5000; jlcpcb (none) -> C5277086; now in the parts list
- TP108: value digital_input2 -> RH-5000; jlcpcb (none) -> C5277086; now in the parts list
Changed lines of the file:
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@@
 		(unit 1)
 		(exclude_from_sim no)
-		(in_bom no)
+		(in_bom yes)
 		(on_board yes)
 		(dnp no)
@@
 			)
 		)
-		(property "Value" "+5V_DIV"
+		(property "Value" "RH-5002"
 			(at 28.448 144.78 90)
 			(effects
@@
 			)
 		)
+		(property "jlcpcb" "C5199802"
+			(at 31.75 147.32 90)
+			(effects
+				(font
+					(size 1.27 1.27)
+				)
+				(hide yes)
+			)
+		)
 		(pin "1"
 		)
@@
 		(unit 1)
 		(exclude_from_sim no)
-		(in_bom no)
+		(in_bom yes)
 		(on_board yes)
 		(dnp no)
@@
 			)
 		)
-		(property "Value" "vgate_A"
+		(property "Value" "RH-5002"
 			(at 28.448 152.4 90)
 			(effects
@@
 			)
 		)
+		(property "jlcpcb" "C5199802"
+			(at 31.75 154.94 90)
+			(effects
+				(font
+					(size 1.27 1.27)
+				)
+				(hide yes)
+			)
+		)
 		(pin "1"
 		)
@@
 		(unit 1)
 		(exclude_from_sim no)
-		(in_bom no)
+		(in_bom yes)
 		(on_board yes)
 		(dnp no)
@@
 			)
 		)
-		(property "Value" "digital_input2"
+		(property "Value" "RH-5000"
 			(at 55.118 152.4 90)
 			(effects
@@
 			)
 		)
+		(property "jlcpcb" "C5277086"
+			(at 58.42 154.94 90)
+			(effects
+				(font
+					(size 1.27 1.27)
+				)
+				(hide yes)
+			)
+		)
 		(pin "1"
 		)
@@
 		(unit 1)
 		(exclude_from_sim no)
-		(in_bom no)
+		(in_bom yes)
 		(on_board yes)
 		(dnp no)
@@
 			)
 		)
-		(property "Value" "digital_input1"
+		(property "Value" "RH-5000"
 			(at 55.118 144.78 90)
 			(effects
@@
 			(effects
 				(font
+					(size 1.27 1.27)
+				)
+				(hide yes)
+			)
+		)
+		(property "jlcpcb" "C5277086"
+			(at 58.42 147.32 90)
+			(effects
+				(font
