File: mega_shield/digital_gpi.kicad_sch (KiCad schematic)
At the start: 12 parts, among them J25 1803277, J26 1803277, U30 4N35, U31 4N35

Commit message: mega_shield, updated the digital inputs section.
Parts:
- R77, R78: value 15k -> 2k7; jlcpcb C17475 -> C1854836
- R79, R80: value 220 -> 4k7; jlcpcb C17557 -> C17673
Other:
- note added: "Opto-Isolated Input(Active Low)"
- note removed: "Opto-Isolated Input"
Changed lines of the file:
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@@
 		)
 	)
-	(text "Opto-Isolated Input"
-		(exclude_from_sim no)
-		(at 127 49.53 0)
+	(text "Opto-Isolated Input(Active Low)"
+		(exclude_from_sim no)
+		(at 132.842 87.884 0)
 		(effects
 			(font
@@
 		)
 	)
-	(text "GPI Test Points"
-		(exclude_from_sim no)
-		(at 32.766 138.176 0)
+	(text "Opto-Isolated Input(Active Low)"
+		(exclude_from_sim no)
+		(at 132.334 49.53 0)
 		(effects
 			(font
@@
 		)
 	)
-	(text "Opto-Isolated Input"
-		(exclude_from_sim no)
-		(at 127.254 87.63 0)
+	(text "GPI Test Points"
+		(exclude_from_sim no)
+		(at 32.766 138.176 0)
 		(effects
 			(font
@@
 		(fields_autoplaced yes)
 		(property "Reference" "R80"
-			(at 167.64 101.5999 0)
+			(at 167.64 100.3299 0)
 			(effects
 				(font
@@
 			)
 		)
-		(property "Value" "220"
-			(at 167.64 104.1399 0)
+		(property "Value" "4k7"
+			(at 167.64 102.8699 0)
 			(effects
 				(font
@@
 			)
 		)
-		(property "jlcpcb" "C17557"
-			(at 165.1 102.87 0)
-			(effects
-				(font
-					(size 1.27 1.27)
-				)
+		(property "jlcpcb" "C17673"
+			(at 167.64 105.4099 0)
+			(effects
+				(font
+					(size 1.27 1.27)
+				)
+				(justify left)
 			)
 		)
@@
 		(fields_autoplaced yes)
 		(property "Reference" "R77"
+			(at 139.7 58.42 90)
+			(effects
+				(font
+					(size 1.27 1.27)
+				)
+			)
+		)
+		(property "Value" "2k7"
 			(at 139.7 60.96 90)
-			(effects
-				(font
-					(size 1.27 1.27)
-				)
-			)
-		)
-		(property "Value" "15k"
-			(at 139.7 63.5 90)
 			(effects
 				(font
@@
 			)
 		)
-		(property "jlcpcb" "C17475"
-			(at 139.7 67.31 0)
+		(property "jlcpcb" "C1854836"
+			(at 139.7 63.5 90)
 			(effects
 				(font
@@
 		(fields_autoplaced yes)
 		(property "Reference" "R79"
-			(at 167.64 63.4999 0)
+			(at 167.64 62.2299 0)
 			(effects
 				(font
@@
 			)
 		)
-		(property "Value" "220"
-			(at 167.64 66.0399 0)
+		(property "Value" "4k7"
+			(at 167.64 64.7699 0)
 			(effects
 				(font
@@
 			)
 		)
-		(property "jlcpcb" "C17557"
-			(at 165.1 64.77 0)
-			(effects
-				(font
-					(size 1.27 1.27)
-				)
+		(property "jlcpcb" "C17673"
+			(at 167.64 67.3099 0)
+			(effects
+				(font
+					(size 1.27 1.27)
+				)
+				(justify left)
 			)
 		)
@@
 		(fields_autoplaced yes)
 		(property "Reference" "R78"
+			(at 139.7 96.52 90)
+			(effects
+				(font
+					(size 1.27 1.27)
+				)
+			)
+		)
+		(property "Value" "2k7"
 			(at 139.7 99.06 90)
-			(effects
-				(font
-					(size 1.27 1.27)
-				)
-			)
-		)
-		(property "Value" "15k"
-			(at 139.7 101.6 90)
 			(effects
 				(font
@@
 			)
 		)
-		(property "jlcpcb" "C17475"
-			(at 139.7 105.41 0)
-			(effects
-				(font
+		(property "jlcpcb" "C1854836"
+			(at 139.7 101.6 90)
+			(effects
+				(font

Commit message: mega_shield, updated test points on spindle interface to new symbol/fp
Parts:
- removed TP113, TP114: RH-5002, footprints:KEYSTONE_5002, symbol Connector:TestPoint
- removed TP115: RH-5000, footprints:KEYSTONE_5000, symbol Connector:TestPoint
- added TP113, TP114: RH-5002, footprints:KEYSTONE_5002, symbol 5002:5002
- added TP115: RH-5000, footprints:KEYSTONE_5000, symbol 5000:5000
- TP116: symbol Connector:TestPoint -> 5000:5000; Availability (none) -> In Stock; Check_prices (none) -> https://www.snapeda.com/parts/5000/Keystone/view-part/?ref=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; Description_1 (none) -> Test Point Miniature THM H .300 Nylon 46 Insulated Red Phos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; MANUFACTURER (none) -> Keystone Electronics; MAXIMUM_PACKAGE_HEIGHT (none) -> 4.57 mm; MF (none) -> Keystone Electronics; MP (none) -> 5000; PARTREV (none) -> H; Package (none) -> Test Point Keystone Electronics; Price (none) -> None; SNAPEDA_PN (none) -> 5000; STANDARD (none) -> Manufacturer Recommendations; SnapEDA_Link (none) -> https://www.snapeda.com/parts/5000/Keystone/view-part/?ref=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
Connections:
- net 24V_digital_input1: now also TP113.1
- net 24V_digital_input2: now also TP114.1
- net digital_input1: now also TP115.1

Commit message: mega_shield, switched from 4N35 --> PC817, higher stock and 1/3 price. Started on M8P3 offset.
Parts:
- removed U30, U31: 4N35, Package_DIP:DIP-6_W7.62mm, symbol Isolator:4N35
- added U30, U31: PC817, Package_DIP:DIP-4_W7.62mm, symbol Isolator:PC817
Connections:
- net GND: now also U30.2, U30.3, U31.2, U31.3
- net digital_input1: now also U30.4
- net digital_input2: now also U31.4
- net at R77.1: now also U30.1
- net at R78.1: now also U31.1
- no-connect marks 2 -> 0
Other:
- moved on the sheet: R79, R80

Commit message: mega_shield, added missing PC817 jlcpcb numbers to u30/31
Parts:
- U30, U31: jlcpcb (none) -> C5350
Changed lines of the file:
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@@
+			)
+		)
+		(property "jlcpcb" "C5350"
+			(at 151.13 107.95 0)
+			(effects
+				(font
+					(size 1.27 1.27)
+				)
+				(hide yes)
 			)
 		)
@@
 			(at 151.13 69.85 0)
 			(effects
+				(font
+					(size 1.27 1.27)
+				)
+				(hide yes)
+			)
+		)
+		(property "jlcpcb" "C5350"
+			(at 151.13 69.85 0)
+			(effects

Commit message: mega_shield, fixed up discrepencies in comments for test points. Added Axis names to silkscreen.
Parts:
- TP113, TP114: value RH-5002 -> 5002
- TP115, TP116: value RH-5000 -> 5000
Changed lines of the file:
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@@
 			)
 		)
-		(property "Value" "RH-5000"
+		(property "Value" "5000"
 			(at 54.61 152.4 0)
 			(effects
@@
 			)
 		)
-		(property "Value" "RH-5002"
+		(property "Value" "5002"
 			(at 26.67 153.67 0)
 			(effects
@@
 			)
 		)
-		(property "Value" "RH-5000"
+		(property "Value" "5000"
 			(at 53.34 143.51 0)
 			(effects
@@
 			)
 		)
-		(property "Value" "RH-5002"
+		(property "Value" "5002"
 			(at 26.67 143.51 0)
 			(effects
