File: mega_shield/digital_gpi.kicad_sch (KiCad schematic)
At the start: 12 parts, among them J25 1803277, J26 1803277, U30 PC817, U31 PC817

Commit message: Automatic project files update
Parts:
- TP113, TP114: MANUFACTURER Keystone -> (none)
- TP115, TP116: MANUFACTURER Keystone Electronics -> (none)
Changed lines of the file:
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@@
 			)
 		)
-		(property "MANUFACTURER" "Keystone Electronics"
+		(property "Manufacturer" "Keystone Electronics"
 			(at 54.61 156.21 0)
 			(hide yes)
@@
 			)
 		)
-		(property "MANUFACTURER" "Keystone"
+		(property "Manufacturer" "Keystone"
 			(at 26.67 157.48 0)
 			(hide yes)
@@
 			)
 		)
-		(property "MANUFACTURER" "Keystone Electronics"
+		(property "Manufacturer" "Keystone Electronics"
 			(at 53.34 147.32 0)
 			(hide yes)
@@
 			)
 		)
-		(property "MANUFACTURER" "Keystone"
+		(property "Manufacturer" "Keystone"
 			(at 26.67 147.32 0)
 			(hide yes)
