File: servo_adapter/servo_adapter.kicad_sch (KiCad schematic)
At the start: 4 parts, among them Q1 MUN5233, Q2 MUN5233, Q3 MUN5233, Q4 MUN5233

Commit message: Added unspeced bypass caps and resistors.
Parts:
- added C1: C, symbol Device:C
- added H1: MountingHole_Pad, symbol Mechanical:MountingHole_Pad
- added R1, R2: 3.48k, symbol Device:R
- added TP1: TestPoint, symbol Connector:TestPoint

Commit message: Added the M12 8 pin signal connector and labels for all signal pins.
Parts:
- added J1: T4140012081-000, servo_adapter_fp:TE_T4140012081-000, symbol T4140012081-000:T4140012081-000
Connections:
- net GND: now also J1.8
- new net +5V_Servo: J1.7
- new net ALARM_OUT: J1.5
- new net AUX_IN: J1.6
- new net DIR_IN: J1.2
- new net EN_IN: J1.3
- new net PED_OUT: J1.4
- new net STEP_IN: J1.1
Other:
- note added: "M12 8Pin Signal Connector(From Mega Shield)"

Commit message: updated the labels on the servo transistors.
Parts:
- added TP2: TestPoint, symbol Connector:TestPoint
Connections:
- net AUX is gone; now on net AUX_IN: Q4.1 (B)
- net DIR is gone; now on net DIR_IN: Q2.1 (B)
- net ENA is gone; now on net EN_IN: Q1.1 (B)
- net PUL is gone; now on net STEP_IN: Q3.1 (B)
- net +5V_Servo: now also TP1.1
Other:
- moved on the sheet: TP1
Changed lines of the file:
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@@
 		)
 	)
-	(label "PUL"
+	(label "STEP_IN"
 		(at 26.67 137.16 180)
 		(effects
@@
 		)
 	)
-	(label "DIR"
+	(label "DIR_IN"
 		(at 26.67 111.76 180)
 		(effects
@@
 			)
 			(justify right bottom)
+		)
+	)
+	(label "+5V_Servo"
+		(at 123.19 76.2 0)
+		(effects
+			(font
+				(size 1.27 1.27)
+			)
+			(justify left bottom)
 		)
 	)
@@
 		)
 	)
-	(label "ENA"
-		(at 26.67 86.36 180)
-		(effects
-			(font
-				(size 1.27 1.27)
-			)
-			(justify right bottom)
-		)
-	)
-	(label "AUX"
+	(label "AUX_IN"
 		(at 26.67 162.56 180)
 		(effects
@@
 			)
 			(justify left bottom)
+		)
+	)
+	(label "EN_IN"
+		(at 26.67 86.36 180)
+		(effects
+			(font
+				(size 1.27 1.27)
+			)
+			(justify right bottom)
 		)
 	)
@@
 	(symbol
 		(lib_id "Connector:TestPoint")
-		(at 177.8 151.13 0)
+		(at 123.19 76.2 90)
 		(unit 1)
 		(exclude_from_sim no)
@@
 		(fields_autoplaced yes)
 		(property "Reference" "TP1"
-			(at 180.34 146.5579 0)
-			(effects
-				(font
-					(size 1.27 1.27)
-				)
-				(justify left)
+			(at 119.888 71.12 90)
+			(effects
+				(font
+					(size 1.27 1.27)
+				)
 			)
 		)
 		(property "Value" "TestPoint"
-			(at 180.34 149.0979 0)
-			(effects
-				(font
-					(size 1.27 1.27)
-				)
-				(justify left)
+			(at 119.888 73.66 90)
+			(effects
+				(font
+					(size 1.27 1.27)
+				)
 			)
 		)
 		(property "Footprint" ""
-			(at 182.88 151.13 0)
+			(at 123.19 71.12 0)
 			(effects
 				(font
@@
 		)
 		(property "Datasheet" "~"
-			(at 182.88 151.13 0)
+			(at 123.19 71.12 0)
 			(effects
 				(font
@@
 		)
 		(property "Description" "test point"
-			(at 177.8 151.13 0)
+			(at 123.19 76.2 0)
 			(effects
 				(font
@@
 					(unit 1)
 				)
+			)
+		)
+	)
+	(symbol
+		(lib_id "Connector:TestPoint")
+		(at 123.19 88.9 90)
+		(unit 1)
+		(exclude_from_sim no)
+		(in_bom yes)
+		(on_board yes)
+		(dnp no)
+		(fields_autoplaced yes)
+		(property "Reference" "TP2"
+			(at 119.888 83.82 90)
+			(effects
+				(font
+					(size 1.27 1.27)
+				)
+			)
+		)
+		(property "Value" "TestPoint"
+			(at 119.888 86.36 90)
+			(effects
+				(font
+					(size 1.27 1.27)
+				)
+			)
+		)
+		(property "Footprint" ""
+			(at 123.19 83.82 0)
+			(effects
+				(font
+					(size 1.27 1.27)
+				)
+				(hide yes)
+			)
+		)
+		(property "Datasheet" "~"
+			(at 123.19 83.82 0)
+			(effects
+				(font
+					(size 1.27 1.27)
+				)
+				(hide yes)
+			)
+		)
+		(property "Description" "test point"
+			(at 123.19 88.9 0)
+			(effects
+				(font
+					(size 1.27 1.27)
+				)
+				(hide yes)
+			)
+		)
+		(pin "1"
+		)
+		(instances
+			(project "servo_adapter"
+				(path "/d2a6932a-1682-4170-bbbb-2fb2c0f935d7"
+					(reference "TP2")
+					(unit 1)
+				)

Commit message: updated test point for +5V servo supply.
Parts:
- removed TP2: TestPoint, symbol Connector:TestPoint
- TP1: value TestPoint -> +5V_Servo
Changed lines of the file:
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@@
 			)
 		)
-		(property "Value" "TestPoint"
+		(property "Value" "+5V_Servo"
 			(at 119.888 73.66 90)
 			(effects
@@
 					(unit 1)
 				)
-			)
-		)
-	)
-	(symbol
-		(lib_id "Connector:TestPoint")
-		(at 123.19 88.9 90)
-		(unit 1)
-		(exclude_from_sim no)
-		(in_bom yes)
-		(on_board yes)
-		(dnp no)
-		(fields_autoplaced yes)
-		(property "Reference" "TP2"
-			(at 119.888 83.82 90)
-			(effects
-				(font
-					(size 1.27 1.27)
-				)
-			)
-		)
-		(property "Value" "TestPoint"
-			(at 119.888 86.36 90)
-			(effects
-				(font
-					(size 1.27 1.27)
-				)
-			)
-		)
-		(property "Footprint" ""
-			(at 123.19 83.82 0)
-			(effects
-				(font
-					(size 1.27 1.27)
-				)
-				(hide yes)
-			)
-		)
-		(property "Datasheet" "~"
-			(at 123.19 83.82 0)
-			(effects
-				(font
-					(size 1.27 1.27)
-				)
-				(hide yes)
-			)
-		)
-		(property "Description" "test point"
-			(at 123.19 88.9 0)
-			(effects
-				(font
-					(size 1.27 1.27)
-				)
-				(hide yes)
-			)
-		)
-		(pin "1"
-		)
-		(instances
-			(project "servo_adapter"
-				(path "/d2a6932a-1682-4170-bbbb-2fb2c0f935d7"
-					(reference "TP2")
-					(unit 1)
-				)

Commit message: Added the 10pin female socket (adapter --> servo motor) and labels for each of the pins along with passive components.
Parts:
- added J2: Conn_01x10_Socket, symbol Connector:Conn_01x10_Socket
- C1: value C -> 22uF
Connections:
- net +5V_Servo: now also C1.1, J2.1 (Pin_1), J2.3 (Pin_3), J2.5 (Pin_5), J2.7 (Pin_7), J2.9 (Pin_9)
- net ALARM_OUT: now also R2.1, J2.10 (Pin_10)
- net DIR-: now also J2.4 (Pin_4)
- net ENA-: now also J2.6 (Pin_6)
- net GND: now also C1.2, R1.2, R2.2
- net PUL-: now also J2.2 (Pin_2)
- net PED-: now reaches R1.1
- net PED-: now also J2.8 (Pin_8)
Other:
- note added: "Servo Driver Signals(Adapter --> Servo Motor)"
- moved on the sheet: C1, R1, R2

Commit message: Added power flag to the +5v line from the mega.
Changed lines of the file:
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@@
+	(wire
+		(pts
+			(xy 55.88 38.1) (xy 48.26 38.1)
+		)
+		(stroke
+			(width 0)
+			(type default)
+		)
+	)
 	(wire
 		(pts
@@
 	)
 	(label "+5V_Servo"
-		(at 48.26 38.1 0)
+		(at 55.88 38.1 0)
 		(effects
 			(font
@@
 					(unit 1)
 				)
+			)
+		)
+	)
+	(symbol
+		(lib_id "power:PWR_FLAG")
+		(at 55.88 38.1 180)
+		(unit 1)
+		(exclude_from_sim no)
+		(in_bom yes)
+		(on_board yes)
+		(dnp no)
+		(fields_autoplaced yes)
+		(property "Reference" "#FLG01"
+			(at 55.88 40.005 0)
+			(effects
+				(font
+					(size 1.27 1.27)
+				)
+				(hide yes)
+			)
+		)
+		(property "Value" "PWR_FLAG"
+			(at 55.88 43.18 0)
+			(effects
+				(font
+					(size 1.27 1.27)
+				)
+			)
+		)
+		(property "Footprint" ""
+			(at 55.88 38.1 0)
+			(effects
+				(font
+					(size 1.27 1.27)
+				)
+				(hide yes)
+			)
+		)
+		(property "Datasheet" "~"
+			(at 55.88 38.1 0)
+			(effects
+				(font
+					(size 1.27 1.27)
+				)
+				(hide yes)
+			)
+		)
+		(property "Description" "Special symbol for telling ERC where power comes from"
+			(at 55.88 38.1 0)
+			(effects
+				(font
+					(size 1.27 1.27)
+				)
+				(hide yes)
+			)
+		)
+		(pin "1"
+		)
+		(instances
+			(project ""
+				(path "/d2a6932a-1682-4170-bbbb-2fb2c0f935d7"
+					(reference "#FLG01")
+					(unit 1)
+				)

Commit message: Updated with generic 2pin symbol and labels used for the servo motor power connection.
Parts:
- added J3: Conn_01x02_Socket, symbol Connector:Conn_01x02_Socket
Connections:
- net GND: now also J3.2 (Pin_2)
- new net +48V: J3.1 (Pin_1)
Other:
- note added: "Servo Power(Adapter --> Servo Motor)"
Changed lines of the file:
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@@
+	)
+	(rectangle
+		(start 165.1 40.64)
+		(end 203.2 54.61)
+		(stroke
+			(width 0)
+			(type default)
+		)
+		(fill
+			(type none)
+		)
 	)
 	(rectangle
@@
 		(exclude_from_sim no)
 		(at 25.654 67.564 0)
+		(effects
+			(font
+				(size 1.27 1.27)
+			)
+		)
+	)
+	(text "Servo Power(Adapter --> Servo Motor)"
+		(exclude_from_sim no)
+		(at 184.658 39.624 0)
 		(effects
 			(font
@@
 			)
 			(justify left bottom)
+		)
+	)
+	(label "+48V"
+		(at 175.26 44.45 180)
+		(effects
+			(font
+				(size 1.27 1.27)
+			)
+			(justify right bottom)
 		)
 	)
@@
 	)
 	(symbol
+		(lib_id "Connector:Conn_01x02_Socket")
+		(at 180.34 44.45 0)
+		(unit 1)
+		(exclude_from_sim no)
+		(in_bom yes)
+		(on_board yes)
+		(dnp no)
+		(fields_autoplaced yes)
+		(property "Reference" "J3"
+			(at 181.61 44.4499 0)
+			(effects
+				(font
+					(size 1.27 1.27)
+				)
+				(justify left)
+			)
+		)
+		(property "Value" "Conn_01x02_Socket"
+			(at 181.61 46.9899 0)
+			(effects
+				(font
+					(size 1.27 1.27)
+				)
+				(justify left)
+			)
+		)
+		(property "Footprint" ""
+			(at 180.34 44.45 0)
+			(effects
+				(font
+					(size 1.27 1.27)
+				)
+				(hide yes)
+			)
+		)
+		(property "Datasheet" "~"
+			(at 180.34 44.45 0)
+			(effects
+				(font
+					(size 1.27 1.27)
+				)
+				(hide yes)
+			)
+		)
+		(property "Description" "Generic connector, single row, 01x02, script generated"
+			(at 180.34 44.45 0)
+			(effects
+				(font
+					(size 1.27 1.27)
+				)
+				(hide yes)
+			)
+		)
+		(pin "2"
+		)
+		(pin "1"
+		)
+		(instances
+			(project ""
+				(path "/d2a6932a-1682-4170-bbbb-2fb2c0f935d7"
+					(reference "J3")
+					(unit 1)
+				)
+			)
+		)
+	)
+	(symbol
 		(lib_id "T4140012081-000:T4140012081-000")
 		(at 40.64 30.48 0)
@@
 					(unit 1)
 				)
+			)
+		)
+	)
+	(symbol
+		(lib_id "power:GND")
+		(at 175.26 46.99 0)
+		(unit 1)
+		(exclude_from_sim no)
+		(in_bom yes)
+		(on_board yes)
+		(dnp no)
+		(fields_autoplaced yes)
+		(property "Reference" "#PWR04"
+			(at 175.26 53.34 0)
+			(effects
+				(font
+					(size 1.27 1.27)
+				)
+				(hide yes)
+			)
+		)
+		(property "Value" "GND"
+			(at 175.26 52.07 0)
+			(effects
+				(font
+					(size 1.27 1.27)
+				)
+			)
+		)
+		(property "Footprint" ""
+			(at 175.26 46.99 0)
+			(effects
+				(font
+					(size 1.27 1.27)
+				)
+				(hide yes)
+			)
+		)
+		(property "Datasheet" ""
+			(at 175.26 46.99 0)
+			(effects
+				(font
+					(size 1.27 1.27)
+				)
+				(hide yes)
+			)
+		)
+		(property "Description" "Power symbol creates a global label with name \"GND\" , ground"
+			(at 175.26 46.99 0)
+			(effects
+				(font
+					(size 1.27 1.27)
+				)
+				(hide yes)
+			)
+		)
+		(pin "1"
+		)
+		(instances
+			(project "servo_adapter"
+				(path "/d2a6932a-1682-4170-bbbb-2fb2c0f935d7"
+					(reference "#PWR04")
+					(unit 1)
+				)

Commit message: Added mounting holes and Test Points.
Added a second mounting hole. Added test points for +48VDC, +5VDC and
GND.
Parts:
- added H2: MountingHole_Pad, symbol Mechanical:MountingHole_Pad
- added TP2: +48V, symbol Connector:TestPoint
- added TP3: GND, symbol Connector:TestPoint
Connections:
- net +48V: now also TP2.1
- net GND: now also H1.1, H2.1, TP3.1
Other:
- note added: "Hardware"
- note added: "Test Points"
- moved on the sheet: C1, H1, J2, J3, R1, R2, TP1
