File: servo_adapter/servo_adapter.kicad_sch (KiCad schematic)
At the start: 15 parts, among them J1 T4140012081-000, J2 Conn_01x10_Socket, J3 Conn_01x02_Socket, Q1 MUN5233, Q2 MUN5233, Q3 MUN5233, Q4 MUN5233

Commit message: Added footprints for servo driver transistors and test points.
Parts:
- added NT1: NetTie_2, symbol Device:NetTie_2
- Q1, Q2, Q3, Q4: footprint PCM_Package_TO_SOT_SMD_AKL:SOT-323_SC-70 -> Package_TO_SOT_SMD:SOT-323_SC-70
- TP1, TP2, TP3: footprint (none) -> TestPoint:TestPoint_Pad_1.0x1.0mm
Connections:
- net PED-: now also NT1.2
- net PED_OUT: now also NT1.1
Changed lines of the file:
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@@
+		)
+	)
+	(label "PED_OUT"
+		(at 92.71 25.4 180)
+		(effects
+			(font
+				(size 1.27 1.27)
+			)
+			(justify right bottom)
 		)
 	)
@@
 		)
 	)
+	(label "PED-"
+		(at 97.79 25.4 0)
+		(effects
+			(font
+				(size 1.27 1.27)
+			)
+			(justify left bottom)
+		)
+	)
 	(label "AUX_IN"
 		(at 26.67 162.56 180)
@@
 			)
 		)
-		(property "Footprint" "PCM_Package_TO_SOT_SMD_AKL:SOT-323_SC-70"
+		(property "Footprint" "Package_TO_SOT_SMD:SOT-323_SC-70"
 			(at 35.56 163.83 0)
 			(effects
@@
 			)
 		)
-		(property "Footprint" "PCM_Package_TO_SOT_SMD_AKL:SOT-323_SC-70"
+		(property "Footprint" "Package_TO_SOT_SMD:SOT-323_SC-70"
 			(at 35.56 113.03 0)
 			(effects
@@
 			)
 		)
-		(property "Footprint" ""
+		(property "Footprint" "TestPoint:TestPoint_Pad_1.0x1.0mm"
 			(at 265.43 113.03 0)
 			(effects
@@
 			)
 		)
-		(property "Footprint" ""
+		(property "Footprint" "TestPoint:TestPoint_Pad_1.0x1.0mm"
 			(at 265.43 120.65 0)
 			(effects
@@
 	)
 	(symbol
+		(lib_id "Device:NetTie_2")
+		(at 95.25 25.4 0)
+		(unit 1)
+		(exclude_from_sim no)
+		(in_bom no)
+		(on_board yes)
+		(dnp no)
+		(fields_autoplaced yes)
+		(property "Reference" "NT1"
+			(at 95.25 20.32 0)
+			(effects
+				(font
+					(size 1.27 1.27)
+				)
+			)
+		)
+		(property "Value" "NetTie_2"
+			(at 95.25 22.86 0)
+			(effects
+				(font
+					(size 1.27 1.27)
+				)
+			)
+		)
+		(property "Footprint" ""
+			(at 95.25 25.4 0)
+			(effects
+				(font
+					(size 1.27 1.27)
+				)
+				(hide yes)
+			)
+		)
+		(property "Datasheet" "~"
+			(at 95.25 25.4 0)
+			(effects
+				(font
+					(size 1.27 1.27)
+				)
+				(hide yes)
+			)
+		)
+		(property "Description" "Net tie, 2 pins"
+			(at 95.25 25.4 0)
+			(effects
+				(font
+					(size 1.27 1.27)
+				)
+				(hide yes)
+			)
+		)
+		(pin "1"
+		)
+		(pin "2"
+		)
+		(instances
+			(project ""
+				(path "/d2a6932a-1682-4170-bbbb-2fb2c0f935d7"
+					(reference "NT1")
+					(unit 1)
+				)
+			)
+		)
+	)
+	(symbol
 		(lib_id "Connector:Conn_01x10_Socket")
 		(at 266.7 60.96 0)
@@
 			)
 		)
-		(property "Footprint" ""
+		(property "Footprint" "TestPoint:TestPoint_Pad_1.0x1.0mm"
 			(at 265.43 105.41 0)
 			(effects
@@
 			)
 		)
-		(property "Footprint" "PCM_Package_TO_SOT_SMD_AKL:SOT-323_SC-70"
+		(property "Footprint" "Package_TO_SOT_SMD:SOT-323_SC-70"
 			(at 35.56 138.43 0)
 			(effects
@@
 			)
 		)
-		(property "Footprint" "PCM_Package_TO_SOT_SMD_AKL:SOT-323_SC-70"
+		(property "Footprint" "Package_TO_SOT_SMD:SOT-323_SC-70"
 			(at 35.56 87.63 0)
 			(effects

Commit message: Added footprints for Caps, mounting holes and 2.54mm servo connector.
Parts:
- C1: footprint (none) -> Capacitor_SMD:C_0805_2012Metric
- H1, H2: footprint (none) -> MountingHole:MountingHole_2.7mm_M2.5
- J2: footprint (none) -> Connector_PinSocket_2.54mm:PinSocket_1x10_P2.54mm_Vertical
Changed lines of the file:
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@@
 			)
 		)
-		(property "Footprint" ""
+		(property "Footprint" "Capacitor_SMD:C_0805_2012Metric"
 			(at 229.5652 78.74 0)
 			(effects
@@
 			)
 		)
-		(property "Footprint" ""
+		(property "Footprint" "MountingHole:MountingHole_2.7mm_M2.5"
 			(at 228.6 110.49 0)
 			(effects
@@
 			)
 		)
-		(property "Footprint" ""
+		(property "Footprint" "Connector_PinSocket_2.54mm:PinSocket_1x10_P2.54mm_Vertical"
 			(at 266.7 60.96 0)
 			(effects
@@
 			)
 		)
-		(property "Footprint" ""
+		(property "Footprint" "MountingHole:MountingHole_2.7mm_M2.5"
 			(at 228.6 125.73 0)
 			(effects

Commit message: Removed old placeholder connector for the TL4141012051-000.
Parts:
- removed J3: Conn_01x02_Socket, symbol Connector:Conn_01x02_Socket
- added J4: T4141012051-000, servo_adapter_fp:CONN5_T4141012051, symbol T4141L12051-000:T4141012051-000
Connections:
- net +48V: now also J4.1, J4.2
- net GND: now also J4.3, J4.4
- no-connect marks 0 -> 1
Changed lines of the file:
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@@
 	)
 	(rectangle
-		(start 215.9 25.4)
+		(start 215.9 16.51)
 		(end 279.4 39.37)
 		(stroke
@@
 	(text "Servo Power(Adapter --> Servo Motor)"
 		(exclude_from_sim no)
-		(at 235.458 24.384 0)
+		(at 235.458 15.24 0)
 		(effects
 			(font
@@
 	)
 	(junction
+		(at 236.22 29.21)
+		(diameter 0)
+		(color 0 0 0 0)
+	)
+	(junction
 		(at 228.6 55.88)
 		(diameter 0)
@@
 		(color 0 0 0 0)
 	)
+	(no_connect
+		(at 241.3 31.75)
+	)
 	(wire
 		(pts
@@
 	(wire
 		(pts
+			(xy 236.22 26.67) (xy 236.22 29.21)
+		)
+		(stroke
+			(width 0)
+			(type default)
+		)
+	)
+	(wire
+		(pts
 			(xy 228.6 78.74) (xy 228.6 86.36)
 		)
@@
 	(wire
 		(pts
-			(xy 252.73 29.21) (xy 226.06 29.21)
+			(xy 241.3 26.67) (xy 236.22 26.67)
 		)
 		(stroke
@@
 	(wire
 		(pts
-			(xy 252.73 31.75) (xy 252.73 33.02)
+			(xy 241.3 29.21) (xy 236.22 29.21)
 		)
 		(stroke
@@
 	(wire
 		(pts
+			(xy 241.3 21.59) (xy 241.3 24.13)
+		)
+		(stroke
+			(width 0)
+			(type default)
+		)
+	)
+	(wire
+		(pts
 			(xy 228.6 60.96) (xy 228.6 55.88)
 		)
@@
 		(pts
 			(xy 228.6 71.12) (xy 228.6 66.04)
+		)
+		(stroke
+			(width 0)
+			(type default)
+		)
+	)
+	(wire
+		(pts
+			(xy 236.22 29.21) (xy 236.22 31.75)
 		)
 		(stroke
@@
 		)
 	)
-	(label "+48V"
-		(at 226.06 29.21 180)
-		(effects
-			(font
-				(size 1.27 1.27)
-			)
-			(justify right bottom)
-		)
-	)
 	(label "PED-"
 		(at 261.62 68.58 180)
@@
 	(label "PED_OUT"
 		(at 92.71 25.4 180)
+		(effects
+			(font
+				(size 1.27 1.27)
+			)
+			(justify right bottom)
+		)
+	)
+	(label "+48V"
+		(at 241.3 21.59 180)
 		(effects
 			(font
@@
 	)
 	(symbol
-		(lib_id "Connector:Conn_01x02_Socket")
-		(at 257.81 29.21 0)
+		(lib_id "T4141L12051-000:T4141012051-000")
+		(at 241.3 21.59 0)
 		(unit 1)
 		(exclude_from_sim no)
@@
 		(dnp no)
 		(fields_autoplaced yes)
-		(property "Reference" "J3"
-			(at 259.08 29.2099 0)
-			(effects
-				(font
-					(size 1.27 1.27)
+		(property "Reference" "J4"
+			(at 255.27 25.3999 0)
+			(effects
+				(font
+					(size 1.524 1.524)
 				)
 				(justify left)
 			)
 		)
-		(property "Value" "Conn_01x02_Socket"
-			(at 259.08 31.7499 0)
-			(effects
-				(font
-					(size 1.27 1.27)
+		(property "Value" "T4141012051-000"
+			(at 255.27 27.9399 0)
+			(effects
+				(font
+					(size 1.524 1.524)
 				)
 				(justify left)
 			)
 		)
-		(property "Footprint" ""
-			(at 257.81 29.21 0)
-			(effects
-				(font
-					(size 1.27 1.27)
-				)
-				(hide yes)
-			)
-		)
-		(property "Datasheet" "~"
-			(at 257.81 29.21 0)
-			(effects
-				(font
-					(size 1.27 1.27)
-				)
-				(hide yes)
-			)
-		)
-		(property "Description" "Generic connector, single row, 01x02, script generated"
-			(at 257.81 29.21 0)
-			(effects
-				(font
-					(size 1.27 1.27)
-				)
-				(hide yes)
-			)
+		(property "Footprint" "servo_adapter_fp:CONN5_T4141012051"
+			(at 241.3 21.59 0)
+			(effects
+				(font
+					(size 1.27 1.27)
+					(italic yes)
+				)
+				(hide yes)
+			)
+		)
+		(property "Datasheet" "T4141012051-000"
+			(at 241.3 21.59 0)
+			(effects
+				(font
+					(size 1.27 1.27)
+					(italic yes)
+				)
+				(hide yes)
+			)
+		)
+		(property "Description" ""
+			(at 241.3 21.59 0)
+			(effects
+				(font
+					(size 1.27 1.27)
+				)
+				(hide yes)
+			)
+		)
+		(pin "3"
+		)
+		(pin "4"
 		)
 		(pin "2"
 		)
 		(pin "1"
+		)
+		(pin "5"
 		)
 		(instances
 			(project ""
 				(path "/d2a6932a-1682-4170-bbbb-2fb2c0f935d7"
-					(reference "J3")
+					(reference "J4")
 					(unit 1)
 				)
@@
 	)
 	(symbol
-		(lib_id "power:GND")
-		(at 252.73 33.02 0)
-		(unit 1)
-		(exclude_from_sim no)
-		(in_bom yes)
-		(on_board yes)
-		(dnp no)
-		(fields_autoplaced yes)
-		(property "Reference" "#PWR04"
-			(at 252.73 39.37 0)
-			(effects
-				(font
-					(size 1.27 1.27)
-				)
-				(hide yes)
-			)
-		)
-		(property "Value" "GND"
-			(at 252.73 38.1 0)
-			(effects
-				(font
-					(size 1.27 1.27)
-				)
-			)
-		)
-		(property "Footprint" ""
-			(at 252.73 33.02 0)
-			(effects
-				(font
-					(size 1.27 1.27)
-				)
-				(hide yes)
-			)
-		)
-		(property "Datasheet" ""
-			(at 252.73 33.02 0)
-			(effects
-				(font
-					(size 1.27 1.27)
-				)
-				(hide yes)
-			)
-		)
-		(property "Description" "Power symbol creates a global label with name \"GND\" , ground"
-			(at 252.73 33.02 0)
-			(effects
-				(font
-					(size 1.27 1.27)
-				)
-				(hide yes)
-			)
-		)
-		(pin "1"
-		)
-		(instances
-			(project "servo_adapter"
-				(path "/d2a6932a-1682-4170-bbbb-2fb2c0f935d7"
-					(reference "#PWR04")
-					(unit 1)
-				)
-			)
-		)
-	)
-	(symbol
 		(lib_id "PCM_Transistor_BJT_Pre-Biased_AKL:MUN5233")
 		(at 35.56 138.43 0)
@@
 					(unit 1)
 				)
+			)
+		)
+	)
+	(symbol
+		(lib_id "power:GND")
+		(at 236.22 31.75 0)
+		(unit 1)
+		(exclude_from_sim no)
+		(in_bom yes)
+		(on_board yes)
+		(dnp no)
+		(fields_autoplaced yes)
+		(property "Reference" "#PWR08"
+			(at 236.22 38.1 0)
+			(effects
+				(font
+					(size 1.27 1.27)
+				)
+				(hide yes)
+			)
+		)
+		(property "Value" "GND"
+			(at 236.22 36.83 0)
+			(effects
+				(font
+					(size 1.27 1.27)
+				)
+			)
+		)
+		(property "Footprint" ""
+			(at 236.22 31.75 0)
+			(effects
+				(font
+					(size 1.27 1.27)
+				)
+				(hide yes)
+			)
+		)
+		(property "Datasheet" ""
+			(at 236.22 31.75 0)
+			(effects
+				(font
+					(size 1.27 1.27)
+				)
+				(hide yes)
+			)
+		)
+		(property "Description" "Power symbol creates a global label with name \"GND\" , ground"
+			(at 236.22 31.75 0)
+			(effects
+				(font
+					(size 1.27 1.27)
+				)
+				(hide yes)
+			)
+		)
+		(pin "1"
+		)
+		(instances
+			(project "servo_adapter"
+				(path "/d2a6932a-1682-4170-bbbb-2fb2c0f935d7"
+					(reference "#PWR08")
+					(unit 1)
+				)

Commit message: changed R1, R2 value from 3.48k --> 3.5k and set the 0603 footprint.
Parts:
- R1, R2: value 3.48k -> 3.5k; footprint (none) -> Resistor_SMD:R_0603_1608Metric
Changed lines of the file:
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@@
 			)
 		)
-		(property "Value" "3.48k"
+		(property "Value" "3.5k"
 			(at 243.84 80.0099 0)
 			(effects
@@
 			)
 		)
-		(property "Footprint" ""
+		(property "Footprint" "Resistor_SMD:R_0603_1608Metric"
 			(at 239.522 78.74 90)
 			(effects
@@
 			)
 		)
-		(property "Value" "3.48k"
+		(property "Value" "3.5k"
 			(at 256.54 80.0099 0)
 			(effects
@@
 			)
 		)
-		(property "Footprint" ""
+		(property "Footprint" "Resistor_SMD:R_0603_1608Metric"
 			(at 252.222 78.74 90)
 			(effects

Commit message: Changed PCM library symbol for project specific symbol.
Parts:
- removed Q1, Q2, Q3, Q4: MUN5233, Package_TO_SOT_SMD:SOT-323_SC-70, symbol PCM_Transistor_BJT_Pre-Biased_AKL:MUN5233
- added U1, U2, U3, U4: MUN5233T1G, SOT-323-3_2P2X1P35_ONS, symbol MUN5233T1G:MUN5233T1G
Connections:
- net AUX-: now also U4.3 (COLLECTOR)
- net AUX_IN: now also U4.1 (BASE)
- net DIR-: now also U2.3 (COLLECTOR)
- net DIR_IN: now also U2.1 (BASE)
- net ENA-: now also U1.3 (COLLECTOR)
- net EN_IN: now also U1.1 (BASE)
- net GND: now also U1.2 (EMITTER), U2.2 (EMITTER), U3.2 (EMITTER), U4.2 (EMITTER)
- net PUL-: now also U3.3 (COLLECTOR)
- net STEP_IN: now also U3.1 (BASE)

Commit message: Assigned the new footprint sot-323
Parts:
- U1, U2, U3, U4: footprint SOT-323-3_2P2X1P35_ONS -> Package_TO_SOT_SMD:SOT-323_SC-70
Changed lines of the file:
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@@
 			)
 		)
-		(property "Footprint" "SOT-323-3_2P2X1P35_ONS"
+		(property "Footprint" "Package_TO_SOT_SMD:SOT-323_SC-70"
 			(at 21.59 107.95 0)
 			(effects
@@
 			)
 		)
-		(property "Footprint" "SOT-323-3_2P2X1P35_ONS"
+		(property "Footprint" "Package_TO_SOT_SMD:SOT-323_SC-70"
 			(at 21.59 67.31 0)
 			(effects
@@
 			)
 		)
-		(property "Footprint" "SOT-323-3_2P2X1P35_ONS"
+		(property "Footprint" "Package_TO_SOT_SMD:SOT-323_SC-70"
 			(at 21.59 128.27 0)
 			(effects
@@
 			)
 		)
-		(property "Footprint" "SOT-323-3_2P2X1P35_ONS"
+		(property "Footprint" "Package_TO_SOT_SMD:SOT-323_SC-70"
 			(at 21.59 87.63 0)
 			(effects

Commit message: Ran electrical rules check and added power flags for input voltage and ground.
Changed lines of the file:
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@@
 	(rectangle
 		(start 13.97 16.51)
-		(end 66.04 49.53)
+		(end 66.04 50.8)
 		(stroke
 			(width 0)
@@
 	)
 	(junction
+		(at 241.3 21.59)
+		(diameter 0)
+		(color 0 0 0 0)
+	)
+	(junction
 		(at 82.55 90.17)
+		(diameter 0)
+		(color 0 0 0 0)
+	)
+	(junction
+		(at 48.26 44.45)
+		(diameter 0)
+		(color 0 0 0 0)
+	)
+	(junction
+		(at 228.6 21.59)
 		(diameter 0)
 		(color 0 0 0 0)
@@
 	(wire
 		(pts
+			(xy 228.6 21.59) (xy 241.3 21.59)
+		)
+		(stroke
+			(width 0)
+			(type default)
+		)
+	)
+	(wire
+		(pts
 			(xy 82.55 110.49) (xy 82.55 130.81)
 		)
@@
 	(wire
 		(pts
+			(xy 31.75 44.45) (xy 48.26 44.45)
+		)
+		(stroke
+			(width 0)
+			(type default)
+		)
+	)
+	(wire
+		(pts
+			(xy 48.26 44.45) (xy 48.26 40.64)
+		)
+		(stroke
+			(width 0)
+			(type default)
+		)
+	)
+	(wire
+		(pts
 			(xy 261.62 55.88) (xy 228.6 55.88)
 		)
@@
 	(wire
 		(pts
+			(xy 228.6 60.96) (xy 228.6 55.88)
+		)
+		(stroke
+			(width 0)
+			(type default)
+		)
+	)
+	(wire
+		(pts
+			(xy 82.55 69.85) (xy 82.55 90.17)
+		)
+		(stroke
+			(width 0)
+			(type default)
+		)
+	)
+	(wire
+		(pts
+			(xy 228.6 66.04) (xy 261.62 66.04)
+		)
+		(stroke
+			(width 0)
+			(type default)
+		)
+	)
+	(wire
+		(pts
+			(xy 228.6 71.12) (xy 228.6 66.04)
+		)
+		(stroke
+			(width 0)
+			(type default)
+		)
+	)
+	(wire
+		(pts
+			(xy 236.22 29.21) (xy 236.22 31.75)
+		)
+		(stroke
+			(width 0)
+			(type default)
+		)
+	)
+	(wire
+		(pts
+			(xy 223.52 21.59) (xy 228.6 21.59)
+		)
+		(stroke
+			(width 0)
+			(type default)
+		)
+	)
+	(wire
+		(pts
+			(xy 241.3 68.58) (xy 261.62 68.58)
+		)
+		(stroke
+			(width 0)
+			(type default)
+		)
+	)
+	(wire
+		(pts
+			(xy 228.6 66.04) (xy 228.6 60.96)
+		)
+		(stroke
+			(width 0)
+			(type default)
+		)
+	)
+	(wire
+		(pts
 			(xy 241.3 21.59) (xy 241.3 24.13)
-		)
-		(stroke
-			(width 0)
-			(type default)
-		)
-	)
-	(wire
-		(pts
-			(xy 228.6 60.96) (xy 228.6 55.88)
-		)
-		(stroke
-			(width 0)
-			(type default)
-		)
-	)
-	(wire
-		(pts
-			(xy 82.55 69.85) (xy 82.55 90.17)
-		)
-		(stroke
-			(width 0)
-			(type default)
-		)
-	)
-	(wire
-		(pts
-			(xy 228.6 66.04) (xy 261.62 66.04)
-		)
-		(stroke
-			(width 0)
-			(type default)
-		)
-	)
-	(wire
-		(pts
-			(xy 228.6 71.12) (xy 228.6 66.04)
-		)
-		(stroke
-			(width 0)
-			(type default)
-		)
-	)
-	(wire
-		(pts
-			(xy 236.22 29.21) (xy 236.22 31.75)
-		)
-		(stroke
-			(width 0)
-			(type default)
-		)
-	)
-	(wire
-		(pts
-			(xy 241.3 68.58) (xy 261.62 68.58)
-		)
-		(stroke
-			(width 0)
-			(type default)
-		)
-	)
-	(wire
-		(pts
-			(xy 228.6 66.04) (xy 228.6 60.96)
 		)
 		(stroke
@@
 	)
 	(label "+48V"
-		(at 241.3 21.59 180)
+		(at 223.52 21.59 180)
 		(effects
 			(font
@@
 			)
 			(justify right bottom)
+		)
+	)
+	(symbol
+		(lib_id "power:PWR_FLAG")
+		(at 228.6 21.59 180)
+		(unit 1)
+		(exclude_from_sim no)
+		(in_bom yes)
+		(on_board yes)
+		(dnp no)
+		(fields_autoplaced yes)
+		(property "Reference" "#FLG02"
+			(at 228.6 23.495 0)
+			(effects
+				(font
+					(size 1.27 1.27)
+				)
+				(hide yes)
+			)
+		)
+		(property "Value" "PWR_FLAG"
+			(at 228.6 26.67 0)
+			(effects
+				(font
+					(size 1.27 1.27)
+				)
+			)
+		)
+		(property "Footprint" ""
+			(at 228.6 21.59 0)
+			(effects
+				(font
+					(size 1.27 1.27)
+				)
+				(hide yes)
+			)
+		)
+		(property "Datasheet" "~"
+			(at 228.6 21.59 0)
+			(effects
+				(font
+					(size 1.27 1.27)
+				)
+				(hide yes)
+			)
+		)
+		(property "Description" "Special symbol for telling ERC where power comes from"
+			(at 228.6 21.59 0)
+			(effects
+				(font
+					(size 1.27 1.27)
+				)
+				(hide yes)
+			)
+		)
+		(pin "1"
+		)
+		(instances
+			(project "servo_adapter"
+				(path "/d2a6932a-1682-4170-bbbb-2fb2c0f935d7"
+					(reference "#FLG02")
+					(unit 1)
+				)
+			)
 		)
 	)
@@
 	(symbol
 		(lib_id "power:GND")
-		(at 48.26 40.64 0)
+		(at 48.26 44.45 0)
 		(unit 1)
 		(exclude_from_sim no)
@@
 		(fields_autoplaced yes)
 		(property "Reference" "#PWR02"
-			(at 48.26 46.99 0)
+			(at 48.26 50.8 0)
 			(effects
 				(font
@@
 		)
 		(property "Value" "GND"
-			(at 48.26 45.72 0)
+			(at 48.26 49.53 0)
 			(effects
 				(font
@@
 		)
 		(property "Footprint" ""
-			(at 48.26 40.64 0)
+			(at 48.26 44.45 0)
 			(effects
 				(font
@@
 		)
 		(property "Datasheet" ""
-			(at 48.26 40.64 0)
+			(at 48.26 44.45 0)
 			(effects
 				(font
@@
 		)
 		(property "Description" "Power symbol creates a global label with name \"GND\" , ground"
-			(at 48.26 40.64 0)
+			(at 48.26 44.45 0)
 			(effects
 				(font
@@
 					(unit 1)
 				)
+			)
+		)
+	)
+	(symbol
+		(lib_id "power:PWR_FLAG")
+		(at 31.75 44.45 90)
+		(unit 1)
+		(exclude_from_sim no)
+		(in_bom yes)
+		(on_board yes)
+		(dnp no)
+		(fields_autoplaced yes)
+		(property "Reference" "#FLG03"
+			(at 29.845 44.45 0)
+			(effects
+				(font
+					(size 1.27 1.27)
+				)
+				(hide yes)
+			)
+		)
+		(property "Value" "PWR_FLAG"
+			(at 27.94 44.4499 90)
+			(effects
+				(font
+					(size 1.27 1.27)
+				)
+				(justify left)
+			)
+		)
+		(property "Footprint" ""
+			(at 31.75 44.45 0)
+			(effects
+				(font
+					(size 1.27 1.27)
+				)
+				(hide yes)
+			)
+		)
+		(property "Datasheet" "~"
+			(at 31.75 44.45 0)
+			(effects
+				(font
+					(size 1.27 1.27)
+				)
+				(hide yes)
+			)
+		)
+		(property "Description" "Special symbol for telling ERC where power comes from"
+			(at 31.75 44.45 0)
+			(effects
+				(font
+					(size 1.27 1.27)
+				)
+				(hide yes)
+			)
+		)
+		(pin "1"
+		)
+		(instances
+			(project "servo_adapter"
+				(path "/d2a6932a-1682-4170-bbbb-2fb2c0f935d7"
+					(reference "#FLG03")
+					(unit 1)
+				)

Commit message: Added JLCPCB numbers to for the caps, resistors and driver transistors.
Parts:
- C1: JLCPCB (none) -> C5674
- R1, R2: JLCPCB (none) -> C1203
- U1, U2, U3, U4: JLCPCB (none) -> C417307
Changed lines of the file:
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@@
+			)
+		)
+		(property "JLCPCB" "C417307"
+			(at 21.59 107.95 0)
+			(effects
+				(font
+					(size 1.27 1.27)
+				)
+				(hide yes)
 			)
 		)
@@
 			)
 		)
+		(property "JLCPCB" "C5674"
+			(at 228.6 74.93 0)
+			(effects
+				(font
+					(size 1.27 1.27)
+				)
+				(hide yes)
+			)
+		)
 		(pin "2"
 		)
@@
 			)
 		)
+		(property "JLCPCB" "C417307"
+			(at 21.59 67.31 0)
+			(effects
+				(font
+					(size 1.27 1.27)
+				)
+				(hide yes)
+			)
+		)
 		(pin "3"
 		)
@@
 			)
 		)
+		(property "JLCPCB" "C417307"
+			(at 21.59 128.27 0)
+			(effects
+				(font
+					(size 1.27 1.27)
+				)
+				(hide yes)
+			)
+		)
 		(pin "3"
 		)
@@
 		)
 		(property "Description" "Resistor"
+			(at 241.3 78.74 0)
+			(effects
+				(font
+					(size 1.27 1.27)
+				)
+				(hide yes)
+			)
+		)
+		(property "JLCPCB" "C1203"
 			(at 241.3 78.74 0)
 			(effects
@@
 			)
 		)
+		(property "JLCPCB" "C1203"
+			(at 254 78.74 0)
+			(effects
+				(font
+					(size 1.27 1.27)
+				)
+				(hide yes)
+			)
+		)
 		(pin "2"
 		)
@@
 			(at 21.59 87.63 0)
 			(effects
+				(font
+					(size 1.27 1.27)
+				)
+				(hide yes)
+			)
+		)
+		(property "JLCPCB" "C417307"
+			(at 21.59 87.63 0)
+			(effects
