File: servo_adapter/servo_adapter.kicad_sch (KiCad schematic)
At the start: 16 parts, among them J1 T4140012081-000, J2 Conn_01x10_Socket, J4 T4141012051-000, U1 MUN5233T1G, U2 MUN5233T1G, U3 MUN5233T1G, U4 MUN5233T1G

Commit message: Added extra mounting holes using 3.5mm diameter.
Parts:
- added H3, H4: MountingHole_Pad, MountingHole:MountingHole_3.5mm, symbol Mechanical:MountingHole_Pad
- H1, H2: footprint MountingHole:MountingHole_2.7mm_M2.5 -> MountingHole:MountingHole_3.5mm
Connections:
- net GND: now also H3.1, H4.1

Commit message: Refactored the dimensions and footprints
+ Re-dimensioned the step file.
+ Relocated the 2.54mm du-pont connector/socket.
+ Changed the MH3 and MH4 to use 2.2mm holes.(closest to 2.0mm).
+ Relocated MH1 and MH2
Parts:
- H3, H4: footprint MountingHole:MountingHole_3.5mm -> MountingHole:MountingHole_2.2mm_M2_DIN965_Pad
- NT1: footprint (none) -> NetTie:NetTie-2_SMD_Pad0.5mm
Changed lines of the file:
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@@
 			)
 		)
-		(property "Footprint" "MountingHole:MountingHole_3.5mm"
+		(property "Footprint" "MountingHole:MountingHole_2.2mm_M2_DIN965_Pad"
 			(at 228.6 153.67 0)
 			(effects
@@
 			)
 		)
-		(property "Footprint" ""
+		(property "Footprint" "NetTie:NetTie-2_SMD_Pad0.5mm"
 			(at 95.25 25.4 0)
 			(effects
@@
 			)
 		)
-		(property "Footprint" "MountingHole:MountingHole_3.5mm"
+		(property "Footprint" "MountingHole:MountingHole_2.2mm_M2_DIN965_Pad"
 			(at 228.6 139.7 0)
 			(effects

Commit message: Updated with traces, ground plane and change to stackup.
+ Changed to 2-Layer board.
+ Routed traces on layer 1
+ Added some silkscreen info
Parts:
- added C2: 22uF, Capacitor_SMD:C_0805_2012Metric, symbol Device:C
- added J3: Conn_01x02_Socket, Connector_Phoenix_MC:PhoenixContact_MCV_1,5_2-GF-3.81_1x02_P3.81mm_Vertical_ThreadedFlange_MountHole, symbol Connector:Conn_01x02_Socket
Connections:
- net +48V: now also J3.1 (Pin_1)
- net GND: now also C2.2
- new net: C2.1, J3.2 (Pin_2)
Other:
- note added: "48V Servo Power(Adapter --> Servo Motor)"
- note added: "Hardware(Mounting Holes)"
- note added: "Net Ties"
- note added: "Servo Power(External --> Adapter)"
- note removed: "Hardware"
- note removed: "Servo Power(Adapter --> Servo Motor)"
- moved on the sheet: J1, J4, NT1, U1, U2, U3, U4

Commit message: Added the 2pin power connector to servo adapter board and schematic.
Parts:
- removed J3: Conn_01x02_Socket, Connector_Phoenix_MC:PhoenixContact_MCV_1,5_2-GF-3.81_1x02_P3.81mm_Vertical_ThreadedFlange_MountHole, symbol Connector:Conn_01x02_Socket
- added J3: 1875425, servo_adapter_fp:CONN_1875425, symbol 1875425:1875425
Connections:
- net +48V: now also C2.1, J3.1, J3.2
- net GND: now also J3.3, J3.4
Changed lines of the file:
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@@
 	)
 	(junction
+		(at 241.3 29.21)
+		(diameter 0)
+		(color 0 0 0 0)
+	)
+	(junction
 		(at 241.3 86.36)
 		(diameter 0)
@@
 	)
 	(junction
+		(at 243.84 21.59)
+		(diameter 0)
+		(color 0 0 0 0)
+	)
+	(junction
 		(at 33.02 38.1)
 		(diameter 0)
@@
 	(wire
 		(pts
+			(xy 223.52 21.59) (xy 223.52 24.13)
+		)
+		(stroke
+			(width 0)
+			(type default)
+		)
+	)
+	(wire
+		(pts
 			(xy 228.6 50.8) (xy 228.6 48.26)
 		)
@@
 	(wire
 		(pts
+			(xy 241.3 26.67) (xy 241.3 29.21)
+		)
+		(stroke
+			(width 0)
+			(type default)
+		)
+	)
+	(wire
+		(pts
 			(xy 81.28 165.1) (xy 81.28 170.18)
 		)
@@
 	(wire
 		(pts
+			(xy 243.84 29.21) (xy 241.3 29.21)
+		)
+		(stroke
+			(width 0)
+			(type default)
+		)
+	)
+	(wire
+		(pts
 			(xy 228.6 78.74) (xy 228.6 86.36)
 		)
@@
 	(wire
 		(pts
+			(xy 223.52 21.59) (xy 243.84 21.59)
+		)
+		(stroke
+			(width 0)
+			(type default)
+		)
+	)
+	(wire
+		(pts
+			(xy 243.84 26.67) (xy 241.3 26.67)
+		)
+		(stroke
+			(width 0)
+			(type default)
+		)
+	)
+	(wire
+		(pts
 			(xy 25.4 30.48) (xy 38.1 30.48)
 		)
@@
 	(wire
 		(pts
-			(xy 38.1 35.56) (xy 33.02 35.56)
+			(xy 243.84 21.59) (xy 243.84 24.13)
 		)
 		(stroke
@@
 	(wire
 		(pts
-			(xy 261.62 71.12) (xy 228.6 71.12)
+			(xy 38.1 35.56) (xy 33.02 35.56)
 		)
 		(stroke
@@
 	(wire
 		(pts
-			(xy 38.1 38.1) (xy 33.02 38.1)
+			(xy 261.62 71.12) (xy 228.6 71.12)
 		)
 		(stroke
@@
 	(wire
 		(pts
-			(xy 30.48 78.74) (xy 46.99 78.74)
+			(xy 38.1 38.1) (xy 33.02 38.1)
 		)
 		(stroke
@@
 	(wire
 		(pts
-			(xy 223.52 24.13) (xy 241.3 24.13)
+			(xy 30.48 78.74) (xy 46.99 78.74)
 		)
 		(stroke
@@
 	)
 	(label "+48V"
-		(at 241.3 21.59 180)
+		(at 223.52 21.59 180)
 		(effects
 			(font
@@
 	)
 	(symbol
+		(lib_id "power:GND")
+		(at 241.3 29.21 0)
+		(unit 1)
+		(exclude_from_sim no)
+		(in_bom yes)
+		(on_board yes)
+		(dnp no)
+		(fields_autoplaced yes)
+		(property "Reference" "#PWR011"
+			(at 241.3 35.56 0)
+			(effects
+				(font
+					(size 1.27 1.27)
+				)
+				(hide yes)
+			)
+		)
+		(property "Value" "GND"
+			(at 241.3 34.29 0)
+			(effects
+				(font
+					(size 1.27 1.27)
+				)
+			)
+		)
+		(property "Footprint" ""
+			(at 241.3 29.21 0)
+			(effects
+				(font
+					(size 1.27 1.27)
+				)
+				(hide yes)
+			)
+		)
+		(property "Datasheet" ""
+			(at 241.3 29.21 0)
+			(effects
+				(font
+					(size 1.27 1.27)
+				)
+				(hide yes)
+			)
+		)
+		(property "Description" "Power symbol creates a global label with name \"GND\" , ground"
+			(at 241.3 29.21 0)
+			(effects
+				(font
+					(size 1.27 1.27)
+				)
+				(hide yes)
+			)
+		)
+		(pin "1"
+		)
+		(instances
+			(project "servo_adapter"
+				(path "/d2a6932a-1682-4170-bbbb-2fb2c0f935d7"
+					(reference "#PWR011")
+					(unit 1)
+				)
+			)
+		)
+	)
+	(symbol
 		(lib_id "Device:C")
 		(at 223.52 27.94 0)
@@
 	)
 	(symbol
-		(lib_id "Connector:Conn_01x02_Socket")
-		(at 246.38 21.59 0)
-		(unit 1)
-		(exclude_from_sim no)
-		(in_bom yes)
-		(on_board yes)
-		(dnp no)
-		(fields_autoplaced yes)
-		(property "Reference" "J3"
-			(at 247.65 21.5899 0)
-			(effects
-				(font
-					(size 1.27 1.27)
-				)
-				(justify left)
-			)
-		)
-		(property "Value" "Conn_01x02_Socket"
-			(at 247.65 24.1299 0)
-			(effects
-				(font
-					(size 1.27 1.27)
-				)
-				(justify left)
-			)
-		)
-		(property "Footprint" "Connector_Phoenix_MC:PhoenixContact_MCV_1,5_2-GF-3.81_1x02_P3.81mm_Vertical_ThreadedFlange_MountHole"
-			(at 246.38 21.59 0)
-			(effects
-				(font
-					(size 1.27 1.27)
-				)
-				(hide yes)
-			)
-		)
-		(property "Datasheet" "~"
-			(at 246.38 21.59 0)
-			(effects
-				(font
-					(size 1.27 1.27)
-				)
-				(hide yes)
-			)
-		)
-		(property "Description" "Generic connector, single row, 01x02, script generated"
-			(at 246.38 21.59 0)
-			(effects
-				(font
-					(size 1.27 1.27)
-				)
-				(hide yes)
-			)
-		)
-		(pin "2"
-		)
-		(pin "1"
-		)
-		(instances
-			(project ""
-				(path "/d2a6932a-1682-4170-bbbb-2fb2c0f935d7"
-					(reference "J3")
-					(unit 1)
-				)
-			)
-		)
-	)
-	(symbol
 		(lib_id "power:PWR_FLAG")
 		(at 54.61 72.39 180)
@@
 					(unit 1)
 				)
+			)
+		)
+	)
+	(symbol
+		(lib_id "1875425:1875425")
+		(at 243.84 21.59 0)
+		(unit 1)
+		(exclude_from_sim no)
+		(in_bom yes)
+		(on_board yes)
+		(dnp no)
+		(fields_autoplaced yes)
+		(property "Reference" "J3"
+			(at 257.81 24.1299 0)
+			(effects
+				(font
+					(size 1.524 1.524)
+				)
+				(justify left)
+			)
+		)
+		(property "Value" "1875425"
+			(at 257.81 26.6699 0)
+			(effects
+				(font
+					(size 1.524 1.524)
+				)
+				(justify left)
+			)
+		)
+		(property "Footprint" "servo_adapter_fp:CONN_1875425"
+			(at 243.84 21.59 0)
+			(effects
+				(font
+					(size 1.27 1.27)
+					(italic yes)
+				)
+				(hide yes)
+			)
+		)
+		(property "Datasheet" "1875425"
+			(at 243.84 21.59 0)
+			(effects
+				(font
+					(size 1.27 1.27)
+					(italic yes)
+				)
+				(hide yes)
+			)
+		)
+		(property "Description" ""
+			(at 243.84 21.59 0)
+			(effects
+				(font
+					(size 1.27 1.27)
+				)
+				(hide yes)
+			)
+		)
+		(pin "3"
+		)
+		(pin "2"
+		)
+		(pin "4"
+		)
+		(pin "1"
+		)
+		(instances
+			(project ""
+				(path "/d2a6932a-1682-4170-bbbb-2fb2c0f935d7"
+					(reference "J3")
+					(unit 1)
+				)

Commit message: Servo adapter, updated to using new 10 pin connector symbol in schematic.
Parts:
- removed C1: 22uF, Capacitor_SMD:C_0805_2012Metric, symbol Device:C
- removed J2: Conn_01x10_Socket, Connector_PinSocket_2.54mm:PinSocket_1x10_P2.54mm_Vertical, symbol Connector:Conn_01x10_Socket
- removed R1, R2: 3.5k, Resistor_SMD:R_0603_1608Metric, symbol Device:R
- added C3: 22uF, Capacitor_SMD:C_0805_2012Metric, symbol Device:C
- added J5: 5-535541-8, 5-535541-8_TYC, symbol TE_5-535541-8:5-535541-8
- added R3, R4: 3.5k, Resistor_SMD:R_0603_1608Metric, symbol Device:R
Connections:
- net +5V_Servo: now also C3.1, J5.A1, J5.A3, J5.A5, J5.A7, J5.A9
- net ALARM_OUT: now also J5.A10, R4.1
- net DIR-: now also J5.A4
- net ENA-: now also J5.A6
- net GND: now also C3.2, R3.2, R4.2
- net PED-: now also J5.A8, R3.1
- net PUL-: now also J5.A2

Commit message: Servo adapter, refactored new connector model and traces.
+ Re-routed the traces.
+ Chagned out the old 2.54mm connector.
+ Added copper fill for higher amprage on the +48V line.
Parts:
- renumbered C3 to C1, J4 to J1, J1 to J2, J5 to J3, J3 to J4, R3 to R1, R4 to R2
Changed lines of the file:
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@@
 		(dnp no)
 		(fields_autoplaced yes)
-		(property "Reference" "#FLG02"
+		(property "Reference" "#FLG01"
 			(at 25.4 32.385 0)
 			(effects
@@
 			(project "servo_adapter"
 				(path "/d2a6932a-1682-4170-bbbb-2fb2c0f935d7"
-					(reference "#FLG02")
+					(reference "#FLG01")
 					(unit 1)
 				)
@@
 		(dnp no)
 		(fields_autoplaced yes)
-		(property "Reference" "R4"
+		(property "Reference" "R2"
 			(at 274.32 81.2799 0)
 			(effects
@@
 			(project "servo_adapter"
 				(path "/d2a6932a-1682-4170-bbbb-2fb2c0f935d7"
-					(reference "R4")
+					(reference "R2")
 					(unit 1)
 				)
@@
 		(dnp no)
 		(fields_autoplaced yes)
-		(property "Reference" "#PWR04"
+		(property "Reference" "#PWR03"
 			(at 81.28 176.53 0)
 			(effects
@@
 			(project "servo_adapter"
 				(path "/d2a6932a-1682-4170-bbbb-2fb2c0f935d7"
-					(reference "#PWR04")
+					(reference "#PWR03")
 					(unit 1)
 				)
@@
 		(dnp no)
 		(fields_autoplaced yes)
-		(property "Reference" "#PWR01"
+		(property "Reference" "#PWR08"
 			(at 228.6 148.59 0)
 			(effects
@@
 			(project "servo_adapter"
 				(path "/d2a6932a-1682-4170-bbbb-2fb2c0f935d7"
-					(reference "#PWR01")
+					(reference "#PWR08")
 					(unit 1)
 				)
@@
 		(dnp no)
 		(fields_autoplaced yes)
-		(property "Reference" "#PWR012"
+		(property "Reference" "#PWR04"
 			(at 186.69 95.25 0)
 			(effects
@@
 			(project "servo_adapter"
 				(path "/d2a6932a-1682-4170-bbbb-2fb2c0f935d7"
-					(reference "#PWR012")
+					(reference "#PWR04")
 					(unit 1)
 				)
@@
 		(dnp no)
 		(fields_autoplaced yes)
-		(property "Reference" "R3"
+		(property "Reference" "R1"
 			(at 265.43 81.2799 0)
 			(effects
@@
 			(project "servo_adapter"
 				(path "/d2a6932a-1682-4170-bbbb-2fb2c0f935d7"
-					(reference "R3")
+					(reference "R1")
 					(unit 1)
 				)
@@
 		(dnp no)
 		(fields_autoplaced yes)
-		(property "Reference" "#PWR010"
+		(property "Reference" "#PWR05"
 			(at 223.52 38.1 0)
 			(effects
@@
 			(project "servo_adapter"
 				(path "/d2a6932a-1682-4170-bbbb-2fb2c0f935d7"
-					(reference "#PWR010")
+					(reference "#PWR05")
 					(unit 1)
 				)
@@
 		(dnp no)
 		(fields_autoplaced yes)
-		(property "Reference" "C3"
+		(property "Reference" "C1"
 			(at 190.5 81.2799 0)
 			(effects
@@
 			(project "servo_adapter"
 				(path "/d2a6932a-1682-4170-bbbb-2fb2c0f935d7"
-					(reference "C3")
+					(reference "C1")
 					(unit 1)
 				)
@@
 		(dnp no)
 		(fields_autoplaced yes)
-		(property "Reference" "J4"
+		(property "Reference" "J1"
 			(at 52.07 34.2899 0)
 			(effects
@@
 			(project ""
 				(path "/d2a6932a-1682-4170-bbbb-2fb2c0f935d7"
-					(reference "J4")
+					(reference "J1")
 					(unit 1)
 				)
@@
 		(dnp no)
 		(fields_autoplaced yes)
-		(property "Reference" "#PWR013"
+		(property "Reference" "#PWR012"
 			(at 271.78 96.52 0)
 			(effects
@@
 			(project "servo_adapter"
 				(path "/d2a6932a-1682-4170-bbbb-2fb2c0f935d7"
-					(reference "#PWR013")
+					(reference "#PWR012")
 					(unit 1)
 				)
@@
 		(dnp no)
 		(fields_autoplaced yes)
-		(property "Reference" "#PWR011"
+		(property "Reference" "#PWR010"
 			(at 241.3 35.56 0)
 			(effects
@@
 			(project "servo_adapter"
 				(path "/d2a6932a-1682-4170-bbbb-2fb2c0f935d7"
-					(reference "#PWR011")
+					(reference "#PWR010")
 					(unit 1)
 				)
@@
 		(dnp no)
 		(fields_autoplaced yes)
-		(property "Reference" "#PWR06"
+		(property "Reference" "#PWR07"
 			(at 228.6 134.62 0)
 			(effects
@@
 			(project "servo_adapter"
 				(path "/d2a6932a-1682-4170-bbbb-2fb2c0f935d7"
-					(reference "#PWR06")
+					(reference "#PWR07")
 					(unit 1)
 				)
@@
 		(on_board yes)
 		(dnp no)
-		(property "Reference" "J1"
+		(property "Reference" "J2"
 			(at 33.02 64.7699 0)
 			(effects
@@
 			(project ""
 				(path "/d2a6932a-1682-4170-bbbb-2fb2c0f935d7"
-					(reference "J1")
+					(reference "J2")
 					(unit 1)
 				)
@@
 		(dnp no)
 		(fields_autoplaced yes)
-		(property "Reference" "#FLG03"
+		(property "Reference" "#FLG02"
 			(at 28.575 78.74 0)
 			(effects
@@
 			(project "servo_adapter"
 				(path "/d2a6932a-1682-4170-bbbb-2fb2c0f935d7"
-					(reference "#FLG03")
+					(reference "#FLG02")
 					(unit 1)
 				)
@@
 		(dnp no)
 		(fields_autoplaced yes)
-		(property "Reference" "#PWR05"
+		(property "Reference" "#PWR06"
 			(at 228.6 119.38 0)
 			(effects
@@
 			(project "servo_adapter"
 				(path "/d2a6932a-1682-4170-bbbb-2fb2c0f935d7"
-					(reference "#PWR05")
+					(reference "#PWR06")
 					(unit 1)
 				)
@@
 		(dnp no)
 		(fields_autoplaced yes)
-		(property "Reference" "#PWR07"
+		(property "Reference" "#PWR011"
 			(at 265.43 132.08 0)
 			(effects
@@
 			(project "servo_adapter"
 				(path "/d2a6932a-1682-4170-bbbb-2fb2c0f935d7"
-					(reference "#PWR07")
+					(reference "#PWR011")
 					(unit 1)
 				)
@@
 		(dnp no)
 		(fields_autoplaced yes)
-		(property "Reference" "#FLG01"
+		(property "Reference" "#FLG03"
 			(at 54.61 74.295 0)
 			(effects
@@
 			(project ""
 				(path "/d2a6932a-1682-4170-bbbb-2fb2c0f935d7"
-					(reference "#FLG01")
+					(reference "#FLG03")
 					(unit 1)
 				)
@@
 		(dnp no)
 		(fields_autoplaced yes)
-		(property "Reference" "J5"
+		(property "Reference" "J3"
 			(at 226.06 58.42 0)
 			(effects
@@
 			(project ""
 				(path "/d2a6932a-1682-4170-bbbb-2fb2c0f935d7"
-					(reference "J5")
+					(reference "J3")
 					(unit 1)
 				)
@@
 		(dnp no)
 		(fields_autoplaced yes)
-		(property "Reference" "#PWR08"
+		(property "Reference" "#PWR01"
 			(at 33.02 46.99 0)
 			(effects
@@
 			(project "servo_adapter"
 				(path "/d2a6932a-1682-4170-bbbb-2fb2c0f935d7"
-					(reference "#PWR08")
+					(reference "#PWR01")
 					(unit 1)
 				)
@@
 		(dnp no)
 		(fields_autoplaced yes)
-		(property "Reference" "J3"
+		(property "Reference" "J4"
 			(at 257.81 24.1299 0)
 			(effects
@@
 			(project ""
 				(path "/d2a6932a-1682-4170-bbbb-2fb2c0f935d7"
-					(reference "J3")
-					(unit 1)
-				)
+					(reference "J4")
+					(unit 1)
+				)

Commit message: Servo adapter, refactored component selection and silkscreen
+ Added extra info to silkscreen
+ Updated/Changed capacitors
+ Added more copper fills.
+ Ran current trace calculations for +5V and +48V lines.
+ Ran and passed DRC.
Parts:
- C1: value 22uF -> 22uF/63v; footprint Capacitor_SMD:C_0805_2012Metric -> Capacitor_SMD:CP_Elec_6.3x7.7; JLCPCB C5674 -> C5246567
- C2: value 22uF -> 22uF/63V; footprint Capacitor_SMD:C_0805_2012Metric -> Capacitor_SMD:CP_Elec_6.3x7.7; JLCPCB C5674 -> C5246567
- R1, R2: footprint Resistor_SMD:R_0603_1608Metric -> Resistor_SMD:R_0805_2012Metric_Pad1.20x1.40mm_HandSolder; JLCPCB C1203 -> C4310
Changed lines of the file:
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@@
 			)
 		)
-		(property "Footprint" "Resistor_SMD:R_0603_1608Metric"
+		(property "Footprint" "Resistor_SMD:R_0805_2012Metric_Pad1.20x1.40mm_HandSolder"
 			(at 270.002 82.55 90)
 			(effects
@@
 			)
 		)
-		(property "JLCPCB" "C1203"
+		(property "JLCPCB" "C4310"
 			(at 271.78 82.55 0)
 			(effects
@@
 			)
 		)
-		(property "Footprint" "Resistor_SMD:R_0603_1608Metric"
+		(property "Footprint" "Resistor_SMD:R_0805_2012Metric_Pad1.20x1.40mm_HandSolder"
 			(at 261.112 82.55 90)
 			(effects
@@
 			)
 		)
-		(property "JLCPCB" "C1203"
+		(property "JLCPCB" "C4310"
 			(at 262.89 82.55 0)
 			(effects
@@
 			)
 		)
-		(property "Value" "22uF"
+		(property "Value" "22uF/63v"
 			(at 190.5 83.8199 0)
 			(effects
@@
 			)
 		)
-		(property "Footprint" "Capacitor_SMD:C_0805_2012Metric"
+		(property "Footprint" "Capacitor_SMD:CP_Elec_6.3x7.7"
 			(at 187.6552 86.36 0)
 			(effects
@@
 			)
 		)
-		(property "JLCPCB" "C5674"
+		(property "JLCPCB" "C5246567"
 			(at 186.69 82.55 0)
 			(effects
@@
 			)
 		)
-		(property "Value" "22uF"
+		(property "Value" "22uF/63V"
 			(at 227.33 29.2099 0)
 			(effects
@@
 			)
 		)
-		(property "Footprint" "Capacitor_SMD:C_0805_2012Metric"
+		(property "Footprint" "Capacitor_SMD:CP_Elec_6.3x7.7"
 			(at 224.4852 31.75 0)
 			(effects
@@
 			)
 		)
-		(property "JLCPCB" "C5674"
+		(property "JLCPCB" "C5246567"
 			(at 223.52 27.94 0)
 			(effects

Commit message: Servo adapter, added design comments / dimensions
+ Added dimensions to comments layer in pcb design.
+ Ran DRC again and confirmed passing.
Parts:
- removed H1, H2: MountingHole_Pad, MountingHole:MountingHole_3.5mm, symbol Mechanical:MountingHole_Pad
- added H1, H2: MountingHole, MountingHole:MountingHole_3.5mm, symbol Mechanical:MountingHole
