File: servo_adapter/servo_adapter.kicad_pcb (KiCad board)
At the start: 2 copper layers, 15 parts, among them J1 T4140012081-000, J2 Conn_01x10_Socket, J4 T4141012051-000, U1 MUN5233T1G, U2 MUN5233T1G, U3 MUN5233T1G, U4 MUN5233T1G

Commit message: Placed components related groups.
Parts:
- J2: moved to F.Cu
- moved U3 77.2 mm to (190.0, 79.5)
- moved J2 75.0 mm to (203.0, 77.5), turned to 0 degrees
- moved U4 71.8 mm to (190.0, 96.0)
- moved U2 68.8 mm to (190.0, 85.0)
- moved J4 67.6 mm to (164.0, 102.5)
- moved J1 63.1 mm to (166.3, 80.9)
- moved U1 61.6 mm to (190.0, 90.5)
- moved C1 49.0 mm to (179.8, 80.4)
- moved R2 29.1 mm to (197.5, 100.5), turned to 180 degrees
- moved H1 28.0 mm to (180.5, 51.5)
- moved H2 28.0 mm to (180.5, 58.5)
- moved R1 26.1 mm to (197.5, 95.5), turned to 180 degrees
- moved TP1 5.52 mm to (147.0, 85.5)
- moved TP2 5.52 mm to (147.0, 90.5)
- moved TP3 5.52 mm to (147.0, 95.5)

Commit message: Added board constraints, trace presets, and rules for working with jlcpcb manufacturing.
Parts:
- added H3: MountingHole_Pad, MountingHole:MountingHole_3.5mm, F.Cu at (267.8, 22.6)
- added H4: MountingHole_Pad, MountingHole:MountingHole_3.5mm, F.Cu at (267.8, 31.1)
- H1, H2: footprint MountingHole:MountingHole_2.7mm_M2.5 -> MountingHole:MountingHole_3.5mm
- moved C1 74.0 mm to (248.6, 53.0)
- moved H1 74.0 mm to (249.3, 24.2)
- moved H2 74.0 mm to (249.3, 31.1)
- moved J1 74.0 mm to (235.1, 53.5)
- moved TP1 74.0 mm to (215.8, 58.1)
- moved TP2 74.0 mm to (215.8, 63.1)
- moved TP3 74.0 mm to (215.8, 68.1)
- moved J2 74.0 mm to (271.8, 50.1)
- moved J4 74.0 mm to (232.7, 75.1)
- moved R1 74.0 mm to (266.3, 68.1)
- moved R2 74.0 mm to (266.3, 73.1)
- moved U1 74.0 mm to (258.8, 63.1)
- moved U2 74.0 mm to (258.8, 57.6)
- moved U3 74.0 mm to (258.8, 52.1)
- moved U4 74.0 mm to (258.8, 68.6)
Other:
- copper layers 2 -> 4

Commit message: Created edge cuts outline and rounded corners to 2mm.
Other:
- board outline added: 64 x 50 mm
Changed lines of the file:
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@@
 		)
+	)
+	(gr_arc
+		(start 164 98)
+		(mid 163.414214 99.414214)
+		(end 162 100)
+		(stroke
+			(width 0.05)
+			(type default)
+		)
+		(layer "Edge.Cuts")
+	)
+	(gr_arc
+		(start 102 100)
+		(mid 100.585786 99.414214)
+		(end 100 98)
+		(stroke
+			(width 0.05)
+			(type default)
+		)
+		(layer "Edge.Cuts")
+	)
+	(gr_line
+		(start 162 100)
+		(end 102 100)
+		(stroke
+			(width 0.05)
+			(type default)
+		)
+		(layer "Edge.Cuts")
+	)
+	(gr_line
+		(start 102 50)
+		(end 162 50)
+		(stroke
+			(width 0.05)
+			(type default)
+		)
+		(layer "Edge.Cuts")
+	)
+	(gr_arc
+		(start 100 52)
+		(mid 100.585786 50.585786)
+		(end 102 50)
+		(stroke
+			(width 0.05)
+			(type default)
+		)
+		(layer "Edge.Cuts")
+	)
+	(gr_line
+		(start 164 52)
+		(end 164 98)
+		(stroke
+			(width 0.05)
+			(type default)
+		)
+		(layer "Edge.Cuts")
+	)
+	(gr_arc
+		(start 162 50)
+		(mid 163.414214 50.585786)
+		(end 164 52)
+		(stroke
+			(width 0.05)
+			(type default)
+		)
+		(layer "Edge.Cuts")
+	)
+	(gr_line
+		(start 100 98)
+		(end 100 52)
+		(stroke
+			(width 0.05)
+			(type default)
+		)
+		(layer "Edge.Cuts")
 	)
 	(embedded_fonts no)

Commit message: Added date, title and version number to PCB.
Parts:
- moved H1 49.3 mm to (202.7, 40.4)
Changed lines of the file:
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@@
 	)
 	(paper "A4")
+	(title_block
+		(title "Servo Adapter PCB")
+		(date "2025-09-05")
+		(rev "0.1.0")
+	)
 	(layers
 		(0 "F.Cu" signal)
@@
 	(footprint "MountingHole:MountingHole_3.5mm"
 		(layer "F.Cu")
-		(at 249.2732 24.1673)
+		(at 202.692 40.386)
 		(descr "Mounting Hole 3.5mm, no annular, generated by kicad-footprint-generator mountinghole.py")
 		(tags "mountinghole")

Commit message: Added ground power plane for EMI resistance.
Routing:
- added copper zone on In2.Cu, net GND
Changed lines of the file:
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@@
 		(layer "Edge.Cuts")
+	)
+	(zone
+		(net 2)
+		(net_name "GND")
+		(layer "In2.Cu")
+		(hatch edge 0.5)
+		(connect_pads
+			(clearance 0.5)
+		)
+		(min_thickness 0.25)
+		(filled_areas_thickness no)
+		(fill yes
+			(thermal_gap 0.5)
+			(thermal_bridge_width 0.5)
+		)
+		(polygon
+			(pts
+				(xy 99.314 49.276) (xy 164.846 49.276) (xy 164.846 100.584) (xy 98.810981 100.584)
+			)
+		)
 	)
 	(embedded_fonts no)

Commit message: positioned the 2.54mm connector
Parts:
- moved J2 125.5 mm to (146.7, 59.6)
Changed lines of the file:
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@@
 	)
 	(footprint "Connector_PinSocket_2.54mm:PinSocket_1x10_P2.54mm_Vertical"
+		(locked yes)
 		(layer "F.Cu")
-		(at 271.7732 50.1173)
+		(at 146.674214 59.585787)
 		(descr "Through hole straight socket strip, 1x10, 2.54mm pitch, single row (from Kicad 4.0.7), script generated")
 		(tags "Through hole socket strip THT 1x10 2.54mm single row")
@@
 			(type default)
 		)
+		(locked yes)
 		(layer "Edge.Cuts")
 	)
@@
 			(type default)
 		)
+		(locked yes)
 		(layer "Edge.Cuts")
 	)
@@
 			(type default)
 		)
+		(locked yes)
 		(layer "Edge.Cuts")
 	)
@@
 			(type default)
 		)
+		(locked yes)
 		(layer "Edge.Cuts")
 	)
@@
 			(type default)
 		)
+		(locked yes)
 		(layer "Edge.Cuts")
 	)
@@
 			(type default)
 		)
+		(locked yes)
 		(layer "Edge.Cuts")
 	)
@@
 			(type default)
 		)
+		(locked yes)
 		(layer "Edge.Cuts")
 	)
@@
 			(type default)
 		)
+		(locked yes)
 		(layer "Edge.Cuts")
 	)

Commit message: placed and locked test points.
Parts:
- moved H4 165.4 mm to (107.9, 73.6)
- moved H3 164.0 mm to (108.0, 59.9)
- moved H2 130.9 mm to (125.3, 73.2)
- moved H1 79.6 mm to (125.5, 59.8)
- moved TP3 61.1 mm to (154.7, 68.8)
- moved TP2 61.1 mm to (154.7, 63.8)
- moved TP1 61.1 mm to (154.7, 58.8)
Changed lines of the file:
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@@
 	(net 15 "/AUX-")
 	(footprint "TestPoint:TestPoint_Pad_1.0x1.0mm"
+		(locked yes)
 		(layer "F.Cu")
-		(at 215.7732 58.1173)
+		(at 154.7 58.785787)
 		(descr "SMD rectangular pad as test Point, square 1.0mm side length")
 		(tags "test point SMD pad rectangle square")
@@
 	(footprint "MountingHole:MountingHole_3.5mm"
 		(layer "F.Cu")
-		(at 249.2732 31.1173)
+		(at 125.35 73.25)
 		(descr "Mounting Hole 3.5mm, no annular, generated by kicad-footprint-generator mountinghole.py")
 		(tags "mountinghole")
@@
 	(footprint "MountingHole:MountingHole_3.5mm"
 		(layer "F.Cu")
-		(at 202.692 40.386)
+		(at 125.45 59.75)
 		(descr "Mounting Hole 3.5mm, no annular, generated by kicad-footprint-generator mountinghole.py")
 		(tags "mountinghole")
@@
 	(footprint "MountingHole:MountingHole_3.5mm"
 		(layer "F.Cu")
-		(at 267.7732 31.1173)
+		(at 107.9 73.6)
 		(descr "Mounting Hole 3.5mm, no annular, generated by kicad-footprint-generator mountinghole.py")
 		(tags "mountinghole")
@@
 	)
 	(footprint "TestPoint:TestPoint_Pad_1.0x1.0mm"
+		(locked yes)
 		(layer "F.Cu")
-		(at 215.7732 68.1173)
+		(at 154.7 68.8)
 		(descr "SMD rectangular pad as test Point, square 1.0mm side length")
 		(tags "test point SMD pad rectangle square")
@@
 	(footprint "MountingHole:MountingHole_3.5mm"
 		(layer "F.Cu")
-		(at 267.7732 22.5673)
+		(at 108.05 59.85)
 		(descr "Mounting Hole 3.5mm, no annular, generated by kicad-footprint-generator mountinghole.py")
 		(tags "mountinghole")
@@
 	)
 	(footprint "TestPoint:TestPoint_Pad_1.0x1.0mm"
+		(locked yes)
 		(layer "F.Cu")
-		(at 215.7732 63.1173)
+		(at 154.7 63.792894)
 		(descr "SMD rectangular pad as test Point, square 1.0mm side length")
 		(tags "test point SMD pad rectangle square")

Commit message: placed and locked, resistors, test points and transistors.
Parts:
- moved U1 121.4 mm to (137.8, 73.8)
- moved U2 121.4 mm to (137.8, 68.3)
- moved U3 121.4 mm to (137.8, 62.8)
- moved U4 121.4 mm to (137.8, 79.3)
- moved R2 115.7 mm to (150.9, 82.5), turned to 0 degrees
- moved R1 115.7 mm to (150.9, 77.3), turned to 0 degrees
- moved J1 24.6 mm to (210.5, 55.1)
- moved J4 24.6 mm to (208.2, 76.7)
Routing:
- net GND: track 0.00 -> 24.8 mm, vias 0 -> 7
- net /ENA-: track 0.00 -> 8.52 mm
- net /+5V_Servo: track 0.00 -> 8.36 mm
- net /DIR-: track 0.00 -> 8.34 mm
- net /PUL-: track 0.00 -> 8.17 mm
- net /PED-: track 0.00 -> 3.46 mm
- net /ALARM_OUT: track 0.00 -> 3.45 mm
