File: servo_adapter/servo_adapter.kicad_pcb (KiCad board)
At the start: 4 copper layers, 64 x 50 mm, 17 parts, among them J1 T4140012081-000, J2 Conn_01x10_Socket, J4 T4141012051-000, U1 MUN5233T1G, U2 MUN5233T1G, U3 MUN5233T1G, U4 MUN5233T1G

Commit message: flipped the 2.54mm connectors.
Parts:
- J2: moved to B.Cu
- turned J2 to 180 degrees

Commit message: Refactored the dimensions and footprints
+ Re-dimensioned the step file.
+ Relocated the 2.54mm du-pont connector/socket.
+ Changed the MH3 and MH4 to use 2.2mm holes.(closest to 2.0mm).
+ Relocated MH1 and MH2
Parts:
- H3, H4: footprint MountingHole:MountingHole_3.5mm -> MountingHole:MountingHole_2.2mm_M2_DIN965_Pad
- moved TP1 51.1 mm to (104.0, 52.2), turned to 90 degrees
- moved TP2 47.1 mm to (109.0, 52.2), turned to 90 degrees
- moved TP3 43.9 mm to (114.0, 52.2), turned to 90 degrees
- moved J2 41.3 mm to (105.4, 59.7), turned to -90 degrees
- moved C1 41.1 mm to (102.1, 64.7), turned to -90 degrees
- moved H4 38.0 mm to (133.7, 61.7)
- moved H3 35.1 mm to (133.7, 57.7)
- moved R1 35.0 mm to (123.2, 56.0), turned to 90 degrees
- moved R2 34.9 mm to (128.2, 56.0), turned to 90 degrees
- moved J4 34.0 mm to (110.0, 97.0), turned to 90 degrees
- moved U3 30.3 mm to (107.6, 64.6), turned to 90 degrees
- moved H1 29.4 mm to (105.7, 81.5), turned to 90 degrees
- moved U2 25.0 mm to (113.1, 64.6), turned to 90 degrees
- moved J1 22.7 mm to (134.5, 95.0), turned to 90 degrees
- moved U1 21.3 mm to (118.6, 64.6), turned to 90 degrees
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Routing:
- net GND: track 24.8 -> 0.71 mm, vias 7 -> 0
- net /ENA-: track 8.52 -> 0.00 mm
- net /+5V_Servo: track 8.36 -> 0.00 mm
- net /DIR-: track 8.34 -> 0.00 mm
- net /PUL-: track 8.17 -> 0.00 mm
- net /ALARM_OUT: track 3.45 -> 0.01 mm
- net /PED-: track 3.46 -> 0.02 mm
Other:
- board size 64 x 50 mm -> 50 x 64 mm

Commit message: Updated with traces, ground plane and change to stackup.
+ Changed to 2-Layer board.
+ Routed traces on layer 1
+ Added some silkscreen info
Parts:
- added C2: 22uF, Capacitor_SMD:C_0805_2012Metric, F.Cu at (111.8, 72.4)
- added NT1: NetTie_2, NetTie:NetTie-2_SMD_Pad0.5mm, F.Cu at (137.5, 78.0)
Routing:
- net /+5V_Servo: track 0.00 -> 79.9 mm
- net /STEP_IN: track 0.00 -> 43.5 mm
- net /ALARM_OUT: track 0.01 -> 43.4 mm
- net /DIR_IN: track 0.00 -> 39.1 mm
- net /EN_IN: track 0.00 -> 38.8 mm
- net /AUX_IN: track 0.00 -> 32.7 mm
- net /PED-: track 0.02 -> 26.6 mm
- net /PED_OUT: track 0.00 -> 19.6 mm
- net GND: track 0.71 -> 20.1 mm, vias 0 -> 8
- net /ENA-: track 0.00 -> 4.10 mm
- net /PUL-: track 0.00 -> 4.07 mm
- net /DIR-: track 0.00 -> 3.93 mm
- added copper zone on B.Cu, net GND
- removed copper zone on In2.Cu, net GND
Other:
- copper layers 4 -> 2
- board text added: "+48V"
- board text added: "+5V"
- board text added: "1"
- board text added: "GND"
- board text added: "Servo Mega Conn"

Commit message: Added the 2pin power connector to servo adapter board and schematic.
Parts:
- added J3: 1875425, servo_adapter_fp:CONN_1875425, B.Cu at (110.0, 83.6)
- moved C2 4.42 mm to (112.2, 76.8), turned to 180 degrees
Connections:
- C2 pad 1: Net-(J3-Pin_2) -> /+48V

Commit message: Servo adapter, refactored new connector model and traces.
+ Re-routed the traces.
+ Chagned out the old 2.54mm connector.
+ Added copper fill for higher amprage on the +48V line.
Parts:
- removed the J2 at (105.4, 59.7)
- added J3: 5-535541-8, servo_adapter_fp:5-535541-8_TYC, B.Cu at (105.4, 59.7)
- moved C1 18.8 mm to (118.2, 55.1), turned to 90 degrees
- moved C2 2.34 mm to (112.6, 74.5)
- moved R1 0.60 mm to (123.2, 55.4)
- moved R2 0.60 mm to (128.2, 55.4)
- renumbered J4 to J1, J1 to J2, J3 to J4
Routing:
- net /+48V: track 0.00 -> 34.3 mm
- net GND: track 20.1 -> 24.5 mm
- net /STEP_IN: track 43.5 -> 44.5 mm
- net /ALARM_OUT: track 43.4 -> 44.0 mm
- net /PED-: track 26.6 -> 27.2 mm
- added copper zone on F.Cu, net /+48V

Commit message: Servo adapter, ran and passed derign rules check.
Other:
- board text added: "+5V_Servo"
- board text added: "ALARM_OUT"
- board text added: "DIR-"
- board text added: "ENA-"
- board text added: "PED-"
- board text added: "PUL-"
