File: servo_adapter/servo_adapter.kicad_pcb (KiCad board)
At the start: 2 copper layers, 50 x 64 mm, 20 parts, among them J1 T4141012051-000, J2 T4140012081-000, J3 5-535541-8, J4 1875425, U1 MUN5233T1G, U2 MUN5233T1G, U3 MUN5233T1G, U4 MUN5233T1G

Commit message: Servo adapter, refactored component selection and silkscreen
+ Added extra info to silkscreen
+ Updated/Changed capacitors
+ Added more copper fills.
+ Ran current trace calculations for +5V and +48V lines.
+ Ran and passed DRC.
Parts:
- C1: value 22uF -> 22uF/63v; footprint Capacitor_SMD:C_0805_2012Metric -> Capacitor_SMD:CP_Elec_6.3x7.7
- C2: value 22uF -> 22uF/63V; footprint Capacitor_SMD:C_0805_2012Metric -> Capacitor_SMD:CP_Elec_6.3x7.7
- R1, R2: footprint Resistor_SMD:R_0603_1608Metric -> Resistor_SMD:R_0805_2012Metric_Pad1.20x1.40mm_HandSolder
- moved C1 25.5 mm to (135.2, 74.2), turned to 0 degrees
- moved NT1 3.08 mm to (135.2, 80.1)
- moved C2 2.90 mm to (109.7, 74.2)
- moved R1 1.50 mm to (123.2, 53.9)
- moved R2 1.50 mm to (128.2, 53.9)
Routing:
- net GND: track 24.5 -> 16.1 mm, vias 8 -> 23
- net /PED-: track 27.2 -> 29.7 mm
- net /AUX_IN: track 32.7 -> 34.7 mm
- net /PED_OUT: track 19.6 -> 18.6 mm
- net /+48V: track 34.3 -> 33.6 mm
- net /ALARM_OUT: track 44.0 -> 44.6 mm
- added copper zone on F.Cu, net GND
Other:
- board text added: "Servo PWR Conn"

Commit message: Servo adapter, added design comments / dimensions
+ Added dimensions to comments layer in pcb design.
+ Ran DRC again and confirmed passing.
Parts:
- moved C2 2.96 mm to (109.1, 71.3)
- moved J4 2.52 mm to (110.0, 81.1)
- moved H1 2.44 mm to (105.7, 79.1)
- moved H2 2.44 mm to (118.5, 79.1)
Routing:
- net /+48V: track 33.6 -> 34.1 mm

Commit message: servo_adapter, updated with three alternate part numbers for the power to servo motor connector plug.
Parts:
- H1, H2: value MountingHole_Pad -> MountingHole
Changed lines of the file:
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@@
 			)
 		)
-		(property "Value" "MountingHole_Pad"
+		(property "Value" "MountingHole"
 			(at 0 4.45 90)
 			(layer "F.Fab")
@@
 			)
 		)
-		(property "Description" "Mounting Hole with connection"
+		(property "Description" "Mounting Hole without connection"
 			(at 0 0 90)
 			(layer "F.Fab")
@@
 			)
 		)
-		(property ki_fp_filters "MountingHole*Pad*")
+		(property ki_fp_filters "MountingHole*")
 		(sheetname "/")
 		(sheetfile "servo_adapter.kicad_sch")
@@
 			)
 		)
-		(property "Value" "MountingHole_Pad"
+		(property "Value" "MountingHole"
 			(at 0 4.45 90)
 			(layer "F.Fab")
@@
 			)
 		)
-		(property "Description" "Mounting Hole with connection"
+		(property "Description" "Mounting Hole without connection"
 			(at 0 0 90)
 			(layer "F.Fab")
@@
 			)
 		)
-		(property ki_fp_filters "MountingHole*Pad*")
+		(property ki_fp_filters "MountingHole*")
 		(sheetname "/")
 		(sheetfile "servo_adapter.kicad_sch")
@@
 		(sheetname "/")
 		(sheetfile "servo_adapter.kicad_sch")
-		(attr through_hole)
+		(attr through_hole exclude_from_bom dnp)
 		(fp_circle
 			(center -3.5 0)
@@
 					(thickness 0.15)
 				)
+				(justify mirror)
+			)
+		)
+		(property "JLCPCB" "C5189077"
+			(at 0 0 180)
+			(unlocked yes)
+			(layer "B.Fab")
+			(hide yes)
+			(effects
+				(font
+					(size 1 1)
+					(thickness 0.15)
+				)

Commit message: servo_adapter, updated PCB routing of traces.
Parts:
- J4: footprint servo_adapter_fp:CONN_1875425 -> servo_adapter_fp:PHOENIX_1875425
- moved R2 29.3 mm to (100.8, 64.1), turned to 0 degrees
- moved NT1 29.2 mm to (110.5, 64.7)
- moved R1 19.7 mm to (106.2, 64.1), turned to 180 degrees
- moved U3 18.2 mm to (125.7, 64.0)
- moved U4 16.2 mm to (140.2, 64.0)
- moved U2 7.62 mm to (120.7, 64.0)
- moved J4 6.47 mm to (116.3, 82.7)
- moved U1 3.06 mm to (115.6, 64.0)
- turned C2 to 0 degrees
Connections:
- J3 pad A1: /+5V_Servo -> /ALARM_OUT
- J3 pad A10: /ALARM_OUT -> /+5V_Servo
- J3 pad A2: /PUL- -> /+5V_Servo
- J3 pad A3: /+5V_Servo -> /PED-
- J3 pad A4: /DIR- -> /+5V_Servo
- J3 pad A5: /+5V_Servo -> /ENA-
- J3 pad A6: /ENA- -> /+5V_Servo
- J3 pad A7: /+5V_Servo -> /DIR-
- J3 pad A8: /PED- -> /+5V_Servo
- J3 pad A9: /+5V_Servo -> /PUL-
- J4 pad 1: /+48V -> GND
- J4 pad 2: /+48V -> GND
- J4 pad 3: GND -> /+48V
- J4 pad 4: GND -> /+48V
Routing:
- net /PED_OUT: track 18.6 -> 56.1 mm
- net /ALARM_OUT: track 44.6 -> 79.0 mm
- net /+5V_Servo: track 80.0 -> 112.8 mm
- net /PED-: track 29.7 -> 7.93 mm
- net /STEP_IN: track 44.5 -> 31.4 mm
- net GND: track 16.1 -> 25.3 mm, vias 23 -> 21
- net /EN_IN: track 38.8 -> 42.7 mm
- net /DIR_IN: track 39.1 -> 36.5 mm
- net /ENA-: track 4.10 -> 3.31 mm
- net /PUL-: track 4.07 -> 3.32 mm
- net /DIR-: track 3.93 -> 3.32 mm
- net /AUX_IN: track 34.7 -> 34.1 mm
