File: servo_adapter/servo_adapter.kicad_pcb (KiCad board)
At the start: 2 copper layers, 50 x 64 mm, 20 parts, among them J1 T4141012051-000, J2 T4140012081-000, J3 5-535541-8, J4 1875425, U1 MUN5233T1G, U2 MUN5233T1G, U3 MUN5233T1G, U4 MUN5233T1G

Commit message: Update of jlcpcb numbers of servo_adapter
Parts:
- C2: value 22uF/63V -> 22uF/63v
Routing:
- net /PED_OUT: track 56.1 -> 54.0 mm
Other:
- board text added: "ALM+"
- board text added: "DIR+"
- board text added: "ENA+"
- board text added: "PED+"
- board text added: "PUL+"
- board text removed: "+5V_Servo"
