File: ihss86-60-45_adapter/ihss86-60-45_adapter.kicad_pcb (KiCad board)
At the start: 2 copper layers, 0 parts

Commit message: Created the cuts layer of the PCB
Other:
- board outline added: 90 x 40 mm
Changed lines of the file:
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@@
 		)
+	)
+	(gr_line
+		(start 115 75)
+		(end 115 80)
+		(stroke
+			(width 0.05)
+			(type default)
+		)
+		(layer "Edge.Cuts")
+	)
+	(gr_line
+		(start 115 75)
+		(end 205 75)
+		(stroke
+			(width 0.05)
+			(type solid)
+		)
+		(layer "Edge.Cuts")
+	)
+	(gr_line
+		(start 115 80)
+		(end 120 80)
+		(stroke
+			(width 0.05)
+			(type default)
+		)
+		(layer "Edge.Cuts")
+	)
+	(gr_line
+		(start 115 110)
+		(end 120 110)
+		(stroke
+			(width 0.05)
+			(type default)
+		)
+		(layer "Edge.Cuts")
+	)
+	(gr_line
+		(start 115 115)
+		(end 115 110)
+		(stroke
+			(width 0.05)
+			(type default)
+		)
+		(layer "Edge.Cuts")
+	)
+	(gr_line
+		(start 120 110)
+		(end 120 80)
+		(stroke
+			(width 0.05)
+			(type default)
+		)
+		(layer "Edge.Cuts")
+	)
+	(gr_line
+		(start 200 80)
+		(end 200 110)
+		(stroke
+			(width 0.05)
+			(type solid)
+		)
+		(layer "Edge.Cuts")
+	)
+	(gr_line
+		(start 200 110)
+		(end 205 110)
+		(stroke
+			(width 0.05)
+			(type solid)
+		)
+		(layer "Edge.Cuts")
+	)
+	(gr_line
+		(start 205 75)
+		(end 205 80)
+		(stroke
+			(width 0.05)
+			(type solid)
+		)
+		(layer "Edge.Cuts")
+	)
+	(gr_line
+		(start 205 80)
+		(end 200 80)
+		(stroke
+			(width 0.05)
+			(type solid)
+		)
+		(layer "Edge.Cuts")
+	)
+	(gr_line
+		(start 205 110)
+		(end 205 115)
+		(stroke
+			(width 0.05)
+			(type solid)
+		)
+		(layer "Edge.Cuts")
+	)
+	(gr_line
+		(start 205 115)
+		(end 115 115)
+		(stroke
+			(width 0.05)
+			(type solid)
+		)
+		(layer "Edge.Cuts")
 	)
 	(embedded_fonts no)

Commit message: Placed components onto PCB
Parts:
- added C1: 22uF/63v, Capacitor_SMD:CP_Elec_6.3x7.7, F.Cu at (176.1, 104.9)
- added H1: MountingHole, MountingHole:MountingHole_3.5mm, F.Cu at (132.3, 80.4)
- added H2: MountingHole, MountingHole:MountingHole_3.5mm, F.Cu at (136.0, 109.0)
- added H3: MountingHole, MountingHole:MountingHole_3.5mm, F.Cu at (190.9, 79.4)
- added H4: MountingHole, MountingHole:MountingHole_3.5mm, F.Cu at (191.4, 111.0)
- added J2: T4140012081-000, servo_fp:TE_T4140012081-000, F.Cu at (189.6, 94.0)
- added J5: Conn_01x10_Socket, Connector_PinHeader_2.54mm:PinHeader_1x10_P2.54mm_Vertical, F.Cu at (145.0, 95.0)
- added NT1: NetTie_2, NetTie:NetTie-2_SMD_Pad0.5mm, F.Cu at (171.4, 82.0)
- added NT7: NetTie_2, NetTie:NetTie-2_SMD_Pad0.5mm, F.Cu at (171.4, 83.5)
- added R3: 3.5k, Resistor_SMD:R_0805_2012Metric_Pad1.20x1.40mm_HandSolder, F.Cu at (145.0, 99.7)
- added R4: 3.5k, Resistor_SMD:R_0805_2012Metric_Pad1.20x1.40mm_HandSolder, F.Cu at (150.1, 99.7)
- added TP1: +5V_Servo, TestPoint:TestPoint_Pad_1.0x1.0mm, F.Cu at (158.7, 109.7)
- added TP3: GND, TestPoint:TestPoint_Pad_1.0x1.0mm, F.Cu at (165.8, 110.2)
- added U1: MUN5233T1G, Package_TO_SOT_SMD:SOT-323_SC-70, F.Cu at (154.3, 89.3)
- added U2: MUN5233T1G, Package_TO_SOT_SMD:SOT-323_SC-70, F.Cu at (159.4, 89.3)
- added U3: MUN5233T1G, Package_TO_SOT_SMD:SOT-323_SC-70, F.Cu at (164.4, 89.3)
- added U4: MUN5233T1G, Package_TO_SOT_SMD:SOT-323_SC-70, F.Cu at (180.4, 82.2)

Commit message: Finished up basic PCB layout for the new servo adapter.
Parts:
- added NT2: NetTie_2, NetTie:NetTie-2_SMD_Pad0.5mm, F.Cu at (162.8, 91.5)
- added NT3: NetTie_2, NetTie:NetTie-2_SMD_Pad0.5mm, F.Cu at (167.9, 91.5)
- added NT4: NetTie_2, NetTie:NetTie-2_SMD_Pad0.5mm, F.Cu at (157.7, 91.5)
- added NT5: NetTie_2, NetTie:NetTie-2_SMD_Pad0.5mm, F.Cu at (152.6, 91.5)
- added NT6: NetTie_2, NetTie:NetTie-2_SMD_Pad0.5mm, F.Cu at (147.5, 98.3)
- J5: footprint Connector_PinHeader_2.54mm:PinHeader_1x10_P2.54mm_Vertical -> Connector_PinSocket_2.54mm:PinSocket_1x10_P2.54mm_Vertical; moved to B.Cu
- moved U4 27.9 mm to (181.8, 110.0), turned to 180 degrees
- moved NT7 27.6 mm to (145.0, 91.5), turned to -90 degrees
- moved C1 23.7 mm to (178.6, 81.3), turned to 90 degrees
- moved NT1 23.3 mm to (150.1, 91.5), turned to -90 degrees
- moved U1 15.1 mm to (156.0, 104.3), turned to 180 degrees
- moved U2 15.1 mm to (161.1, 104.3), turned to 180 degrees
- moved U3 15.1 mm to (166.2, 104.3), turned to 180 degrees
- moved H2 11.0 mm to (125.0, 110.0)
- moved H1 7.36 mm to (125.0, 80.0)
- moved H3 4.15 mm to (195.0, 80.0)
- moved H4 3.76 mm to (195.0, 110.0)
- moved TP3 2.04 mm to (167.9, 110.2)
- moved TP1 1.61 mm to (160.2, 110.2)
- moved J2 1.19 mm to (189.6, 95.2), turned to 90 degrees
- turned J5 to -90 degrees
Routing:
- net /+5V_Servo: track 0.00 -> 78.0 mm
- net /PED_OUT: track 0.00 -> 67.3 mm
- net /ALARM_OUT: track 0.00 -> 57.2 mm
- net /EN_IN: track 0.00 -> 37.3 mm
- net /DIR_IN: track 0.00 -> 29.7 mm
- net /STEP_IN: track 0.00 -> 24.9 mm
- net /AUX_IN: track 0.00 -> 24.6 mm
- net GND: track 0.00 -> 12.7 mm, vias 0 -> 11
- net /PUL-: track 0.00 -> 9.35 mm
- net /ENA-: track 0.00 -> 9.35 mm
- net /DIR-: track 0.00 -> 9.35 mm
- net /PED-: track 0.00 -> 6.72 mm
- net /ALM-: track 0.00 -> 6.72 mm
- net /PUL+: track 0.00 -> 3.05 mm
- net /PED+: track 0.00 -> 3.05 mm
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- added copper zone on B.Cu, net GND
- added copper zone on F.Cu, net GND
Other:
- board text added: "10: PUL+"
- board text added: "1: ALM-"
- board text added: "2: ALM+"
- board text added: "3: PED-"
- board text added: "4: PED+"
- board text added: "5: ENA-"
- board text added: "6: ALM+"
- board text added: "7: DIR-"
- board text added: "8: DIR+"
- board text added: "9: PUL-"

Commit message: Ran PCB DRC, updated to match current jlcpcb specs. Fixed silkscreen issue and added new info.
Other:
- board text added: "1"
- board text added: "2"
- board text added: "3"
- board text added: "4"
- board text added: "5"
- board text added: "6"
- board text added: "7"
- board text added: "8"
Changed lines of the file:
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@@
 		(tags "SOT TO_SOT_SMD SC-70 SOT-323")
 		(property "Reference" "U2"
-			(at 0 -1.8 0)
+			(at -0.0225 -2.2 0)
 			(layer "F.SilkS")
 			(effects
@@
 		(tags "SOT TO_SOT_SMD SC-70 SOT-323")
 		(property "Reference" "U3"
-			(at 0 -1.8 0)
+			(at 0.0325 -2.2 0)
 			(layer "F.SilkS")
 			(effects
@@
 		(tags "SOT TO_SOT_SMD SC-70 SOT-323")
 		(property "Reference" "U1"
-			(at 0 -1.8 0)
+			(at 0 -2.2 0)
 			(layer "F.SilkS")
 			(effects
@@
 		(tags "SOT TO_SOT_SMD SC-70 SOT-323")
 		(property "Reference" "U4"
-			(at 0 -1.8 0)
+			(at 0 -2.3 0)
 			(layer "F.SilkS")
 			(effects
@@
 	)
 	(gr_line
+		(start 191.075 88.825)
+		(end 189.95 94.15)
+		(stroke
+			(width 0.1)
+			(type default)
+		)
+		(layer "B.SilkS")
+	)
+	(gr_line
 		(start 115 75)
 		(end 115 80)
@@
 		)
 	)
-	(gr_text_box "Name: ihss86-60-45 Adapter\nVer: 0.1.0\nDate: 2026-08-07\n"
+	(gr_text "2"
+		(at 187.2 99.425 0)
+		(layer "B.SilkS")
+		(effects
+			(font
+				(size 1.25 1.25)
+				(thickness 0.15)
+			)
+			(justify left bottom mirror)
+		)
+	)
+	(gr_text "1"
+		(at 187.425 92.325 0)
+		(layer "B.SilkS")
+		(effects
+			(font
+				(size 1.25 1.25)
+				(thickness 0.15)
+			)
+			(justify left bottom mirror)
+		)
+	)
+	(gr_text "7"
+		(at 189.75 91.075 0)
+		(layer "B.SilkS")
+		(effects
+			(font
+				(size 1.25 1.25)
+				(thickness 0.15)
+			)
+			(justify left bottom mirror)
+		)
+	)
+	(gr_text "3"
+		(at 190 101.1 0)
+		(layer "B.SilkS")
+		(effects
+			(font
+				(size 1.25 1.25)
+				(thickness 0.15)
+			)
+			(justify left bottom mirror)
+		)
+	)
+	(gr_text "8"
+		(at 191.775 88.575 0)
+		(layer "B.SilkS")
+		(effects
+			(font
+				(size 1.25 1.25)
+				(thickness 0.15)
+			)
+			(justify left bottom mirror)
+		)
+	)
+	(gr_text "6"
+		(at 192.85 91.55 0)
+		(layer "B.SilkS")
+		(effects
+			(font
+				(size 1.25 1.25)
+				(thickness 0.15)
+			)
+			(justify left bottom mirror)
+		)
+	)
+	(gr_text "4"
+		(at 193.5 100.15 0)
+		(layer "B.SilkS")
+		(effects
+			(font
+				(size 1.25 1.25)
+				(thickness 0.15)
+			)
+			(justify left bottom mirror)
+		)
+	)
+	(gr_text "5"
+		(at 195.15 95.4 0)
+		(layer "B.SilkS")
+		(effects
+			(font
+				(size 1.25 1.25)
+				(thickness 0.15)
+			)
+			(justify left bottom mirror)
+		)
+	)
+	(gr_text_box "Name: ihss86-60-45 Adapter\nVer: 0.1.0\nDate: 2026-09-10\n"
 		(start 122 84.2375)
 		(end 138.03443 105.3)
@@
 		(border yes)
 		(stroke
-			(width 0.1)
+			(width 1.53)
 			(type solid)
 		)
