File: ihss86-60-45_adapter/ihss86-60-45_adapter.kicad_sch (KiCad schematic)
At the start: 0 parts

Commit message: Copied origial servo adapter schematic.
Parts:
- added C1, C2: 22uF/63v, Capacitor_SMD:CP_Elec_6.3x7.7, symbol Device:C
- added H1, H2: MountingHole, MountingHole:MountingHole_3.5mm, symbol Mechanical:MountingHole
- added H3, H4: MountingHole_Pad, MountingHole:MountingHole_2.2mm_M2_DIN965_Pad, symbol Mechanical:MountingHole_Pad
- added J1: T4141012051-000, servo_adapter_fp:CONN5_T4141012051, symbol T4141L12051-000:T4141012051-000
- added J2: T4140012081-000, servo_adapter_fp:TE_T4140012081-000, symbol T4140012081-000:T4140012081-000
- added J3: 5-535541-8, 5-535541-8_TYC, symbol TE_5-535541-8:5-535541-8
- added J4: 1875425, servo_adapter_fp:PHOENIX_1875425, symbol 1875425:1875425
- added NT1: NetTie_2, NetTie:NetTie-2_SMD_Pad0.5mm, symbol Device:NetTie_2
- added R1, R2: 3.5k, Resistor_SMD:R_0805_2012Metric_Pad1.20x1.40mm_HandSolder, symbol Device:R
- added TP1: +5V_Servo, TestPoint:TestPoint_Pad_1.0x1.0mm, symbol Connector:TestPoint
- added TP2: +48V, TestPoint:TestPoint_Pad_1.0x1.0mm, symbol Connector:TestPoint
- added TP3: GND, TestPoint:TestPoint_Pad_1.0x1.0mm, symbol Connector:TestPoint
- added U1, U2, U3, U4: MUN5233T1G, Package_TO_SOT_SMD:SOT-323_SC-70, symbol MUN5233T1G:MUN5233T1G
Connections:
- new net +48V: C2.1, J1.1, J1.2, J4.3, J4.4, TP2.1
- new net +5V_Servo: C1.1, J2.7, J3.A10, J3.A2, J3.A4, J3.A6, J3.A8, TP1.1
- new net ALARM_OUT: J2.5, J3.A1, R2.1
- new net AUX-: U4.3 (COLLECTOR)
- new net AUX_IN: J2.6, U4.1 (BASE)
- new net DIR-: J3.A7, U2.3 (COLLECTOR)
- new net DIR_IN: J2.2, U2.1 (BASE)
- new net ENA-: J3.A5, U1.3 (COLLECTOR)
- new net EN_IN: J2.3, U1.1 (BASE)
- new net GND: C1.2, C2.2, H3.1, H4.1, J1.3, J1.4, J2.8, J4.1, J4.2, R1.2, R2.2, TP3.1, U1.2 (EMITTER), U2.2 (EMITTER), U3.2 (EMITTER), U4.2 (EMITTER)
- new net PED-: J3.A3, NT1.2, R1.1
- new net PED_OUT: J2.4, NT1.1
- new net PUL-: J3.A9, U3.3 (COLLECTOR)
- new net STEP_IN: J2.1, U3.1 (BASE)
- no-connect marks 0 -> 1
Other:
- note added: "48V Servo Power(Adapter --> Servo Motor)"
- note added: "Hardware(Mounting Holes)"
- note added: "M12 8Pin Signal Connector(From Mega Shield)"
- note added: "Net Ties"
- note added: "Servo Driver Signals(Adapter --> Servo Motor)"
- note added: "Servo Driver Transistors"
- note added: "Servo Power(External --> Adapter)"
- note added: "Test Points"
- title: (none) -> IHSS86-60-45_adapter

Commit message: Added new 10 pin connector symbol and labels to match servo motor.
Parts:
- added J5: Conn_01x10_Socket, symbol Connector:Conn_01x10_Socket
Connections:
- net +5V_Servo: now also J5.10 (Pin_10), J5.4 (Pin_4), J5.6 (Pin_6), J5.8 (Pin_8)
- net DIR-: now also J5.7 (Pin_7)
- net ENA-: now also J5.5 (Pin_5)
- net PED-: now also J5.3 (Pin_3)
- net PUL-: now also J5.9 (Pin_9)
- new net ALM+: J5.2 (Pin_2)
- new net ALM-: J5.1 (Pin_1)
Changed lines of the file:
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@@
+	)
+	(label "DIR+"
+		(at 152.4 43.18 180)
+		(effects
+			(font
+				(size 1.27 1.27)
+			)
+			(justify right bottom)
+		)
+	)
+	(label "ENA+"
+		(at 152.4 38.1 180)
+		(effects
+			(font
+				(size 1.27 1.27)
+			)
+			(justify right bottom)
+		)
+	)
+	(label "ALM-"
+		(at 152.4 25.4 180)
+		(effects
+			(font
+				(size 1.27 1.27)
+			)
+			(justify right bottom)
+		)
 	)
 	(label "DIR+"
@@
 		)
 	)
+	(label "PED-"
+		(at 152.4 30.48 180)
+		(effects
+			(font
+				(size 1.27 1.27)
+			)
+			(justify right bottom)
+		)
+	)
 	(label "ENA-"
 		(at 71.12 101.6 0)
@@
 		)
 	)
+	(label "PUL-"
+		(at 152.4 45.72 180)
+		(effects
+			(font
+				(size 1.27 1.27)
+			)
+			(justify right bottom)
+		)
+	)
 	(label "PED+"
 		(at 198.12 76.2 180)
@@
 		)
 	)
+	(label "ENA-"
+		(at 152.4 35.56 180)
+		(effects
+			(font
+				(size 1.27 1.27)
+			)
+			(justify right bottom)
+		)
+	)
 	(label "ENA+"
 		(at 254 78.74 0)
@@
 		)
 	)
+	(label "DIR-"
+		(at 152.4 40.64 180)
+		(effects
+			(font
+				(size 1.27 1.27)
+			)
+			(justify right bottom)
+		)
+	)
+	(label "PED+"
+		(at 152.4 33.02 180)
+		(effects
+			(font
+				(size 1.27 1.27)
+			)
+			(justify right bottom)
+		)
+	)
 	(label "DIR_IN"
 		(at 20.32 121.92 180)
@@
 		)
 	)
+	(label "PUL+"
+		(at 152.4 48.26 180)
+		(effects
+			(font
+				(size 1.27 1.27)
+			)
+			(justify right bottom)
+		)
+	)
 	(label "PUL-"
 		(at 71.12 142.24 0)
@@
 	(label "PED-"
 		(at 198.12 73.66 180)
+		(effects
+			(font
+				(size 1.27 1.27)
+			)
+			(justify right bottom)
+		)
+	)
+	(label "ALM+"
+		(at 152.4 27.94 180)
 		(effects
 			(font
@@
 					(unit 1)
 				)
+			)
+		)
+	)
+	(symbol
+		(lib_id "Connector:Conn_01x10_Socket")
+		(at 157.48 35.56 0)
+		(unit 1)
+		(body_style 1)
+		(exclude_from_sim no)
+		(in_bom yes)
+		(on_board yes)
+		(in_pos_files yes)
+		(dnp no)
+		(fields_autoplaced yes)
+		(property "Reference" "J5"
+			(at 158.75 35.5599 0)
+			(show_name no)
+			(do_not_autoplace no)
+			(effects
+				(font
+					(size 1.27 1.27)
+				)
+				(justify left)
+			)
+		)
+		(property "Value" "Conn_01x10_Socket"
+			(at 158.75 38.0999 0)
+			(show_name no)
+			(do_not_autoplace no)
+			(effects
+				(font
+					(size 1.27 1.27)
+				)
+				(justify left)
+			)
+		)
+		(property "Footprint" ""
+			(at 157.48 35.56 0)
+			(hide yes)
+			(show_name no)
+			(do_not_autoplace no)
+			(effects
+				(font
+					(size 1.27 1.27)
+				)
+			)
+		)
+		(property "Datasheet" ""
+			(at 157.48 35.56 0)
+			(hide yes)
+			(show_name no)
+			(do_not_autoplace no)
+			(effects
+				(font
+					(size 1.27 1.27)
+				)
+			)
+		)
+		(property "Description" "Generic connector, single row, 01x10, script generated"
+			(at 157.48 35.56 0)
+			(hide yes)
+			(show_name no)
+			(do_not_autoplace no)
+			(effects
+				(font
+					(size 1.27 1.27)
+				)
+			)
+		)
+		(pin "8"
+		)
+		(pin "1"
+		)
+		(pin "2"
+		)
+		(pin "3"
+		)
+		(pin "4"
+		)
+		(pin "5"
+		)
+		(pin "9"
+		)
+		(pin "10"
+		)
+		(pin "6"
+		)
+		(pin "7"
+		)
+		(instances
+			(project "ihss86-60-45_adapter"
+				(path "/6ec498c9-9cf8-4ee4-aa81-f02f74425281"
+					(reference "J5")
+					(unit 1)
+				)

Commit message: Removed old style connector
Parts:
- removed J1: T4141012051-000, servo_adapter_fp:CONN5_T4141012051, symbol T4141L12051-000:T4141012051-000
- removed J4: 1875425, servo_adapter_fp:PHOENIX_1875425, symbol 1875425:1875425
- added J1: Conn_01x02_Pin, symbol Connector:Conn_01x02_Pin
Connections:
- net +48V: now also J1.1 (Pin_1)
- net GND: now also J1.2 (Pin_2)

Commit message: Updated schematic with new connectors
+ Added the 2.54mm connector 10 pin
+ Added the 2.54mm un-populated 10 pin connector.
+ Added note on the connection setup for the adapter --> servo signal.
Parts:
- removed C2: 22uF/63v, Capacitor_SMD:CP_Elec_6.3x7.7, symbol Device:C
- removed J1: Conn_01x02_Pin, symbol Connector:Conn_01x02_Pin
- removed J3: 5-535541-8, 5-535541-8_TYC, symbol TE_5-535541-8:5-535541-8
- removed R1, R2: 3.5k, Resistor_SMD:R_0805_2012Metric_Pad1.20x1.40mm_HandSolder, symbol Device:R
- removed TP2: +48V, TestPoint:TestPoint_Pad_1.0x1.0mm, symbol Connector:TestPoint
- added J6: Conn_01x10_Socket, symbol Connector:Conn_01x10_Socket
- added R3, R4: 3.5k, Resistor_SMD:R_0805_2012Metric_Pad1.20x1.40mm_HandSolder, symbol Device:R
Connections:
- net ALM+ is gone; now on net +5V_Servo: J5.2 (Pin_2)
- net ALM-: now also R3.1
- net GND: now also R3.2, R4.2
- net PED-: now also R4.1
- no-connect marks 1 -> 10
Other:
- note removed: "48V Servo Power(Adapter --> Servo Motor)"
- note removed: "Servo Power(External --> Adapter)"
- moved on the sheet: C1, J2, J5

Commit message: Updated M12 signal connection title.
Other:
- note added: "M12 8Pin A-Coded Signal Connector(From Mega Shield)"
- note removed: "M12 8Pin Signal Connector(From Mega Shield)"
Changed lines of the file:
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@@
 		)
 	)
-	(text "M12 8Pin Signal Connector(From Mega Shield)"
+	(text "M12 8Pin A-Coded Signal Connector(From Mega Shield)"
 		(exclude_from_sim no)
-		(at 48.26 24.384 0)
+		(at 25.4 24.384 0)
 		(effects
 			(font
 				(size 1.27 1.27)
 			)
+			(justify left)
 		)
 	)

Commit message: Updated all LCSC/JLCPCB numbers, refactored scheamtic connections.
Parts:
- removed H3, H4: MountingHole_Pad, MountingHole:MountingHole_2.2mm_M2_DIN965_Pad, symbol Mechanical:MountingHole_Pad
- added H3, H4: MountingHole, MountingHole:MountingHole_3.5mm, symbol Mechanical:MountingHole
- added NT2, NT3, NT4, NT5, NT6: NetTie_2, symbol Device:NetTie_2
- added NT7: NetTie_2, NetTie:NetTie-2_SMD_Pad0.5mm, symbol Device:NetTie_2
- J2: footprint servo_adapter_fp:TE_T4140012081-000 -> servo_fp:TE_T4140012081-000; LCSC (none) -> C45986647
- J5: footprint (none) -> Connector_PinHeader_2.54mm:PinHeader_1x10_P2.54mm_Vertical; LCSC (none) -> C5159939
- J6: footprint (none) -> Connector_PinHeader_2.54mm:PinHeader_1x10_P2.54mm_Vertical; LCSC (none) -> C2897373
Connections:
- net +5V_Servo: now also NT2.1, NT3.1, NT4.1, NT5.1, NT6.1; no longer J5.10 (Pin_10), J5.2 (Pin_2), J5.4 (Pin_4), J5.6 (Pin_6), J5.8 (Pin_8)
- net ALARM_OUT: now also NT7.1
- net ALM-: now also NT7.2
- new net ALM+: J5.2 (Pin_2), NT6.2
- new net DIR+: J5.8 (Pin_8), NT2.2
- new net ENA+: J5.6 (Pin_6), NT4.2
- new net PED+: J5.4 (Pin_4), NT5.2
- new net PUL+: J5.10 (Pin_10), NT3.2
Other:
- note added: "Round Female Header"
- note added: "Signal Name Net Ties"
- note added: "Square female Header"
- note removed: "Net Ties"
- moved on the sheet: H1, H2, NT1, TP1, TP3, U1, U2, U3, U4

Commit message: Finished up basic PCB layout for the new servo adapter.
Parts:
- J5: footprint Connector_PinHeader_2.54mm:PinHeader_1x10_P2.54mm_Vertical -> Connector_PinSocket_2.54mm:PinSocket_1x10_P2.54mm_Vertical
- NT2, NT3, NT4, NT5, NT6: footprint (none) -> NetTie:NetTie-2_SMD_Pad0.5mm
Changed lines of the file:
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@@
 			)
 		)
-		(property "Footprint" ""
+		(property "Footprint" "NetTie:NetTie-2_SMD_Pad0.5mm"
 			(at 203.2 63.5 0)
 			(hide yes)
@@
 			)
 		)
-		(property "Footprint" ""
+		(property "Footprint" "NetTie:NetTie-2_SMD_Pad0.5mm"
 			(at 203.2 43.18 0)
 			(hide yes)
@@
 			)
 		)
-		(property "Footprint" "Connector_PinHeader_2.54mm:PinHeader_1x10_P2.54mm_Vertical"
+		(property "Footprint" "Connector_PinSocket_2.54mm:PinSocket_1x10_P2.54mm_Vertical"
 			(at 217.17 50.8 0)
 			(hide yes)
@@
 			)
 		)
-		(property "Footprint" ""
+		(property "Footprint" "NetTie:NetTie-2_SMD_Pad0.5mm"
 			(at 203.2 53.34 0)
 			(hide yes)
@@
 			)
 		)
-		(property "Footprint" ""
+		(property "Footprint" "NetTie:NetTie-2_SMD_Pad0.5mm"
 			(at 203.2 48.26 0)
 			(hide yes)
@@
 			)
 		)
-		(property "Footprint" ""
+		(property "Footprint" "NetTie:NetTie-2_SMD_Pad0.5mm"
 			(at 203.2 58.42 0)
 			(hide yes)

Commit message: Updated number for the M12 8pin connector on the new motor interface.
The new part number is for the M12 8p connector with the PCB pins that
should be able to be assembled by JLCPCB.
Parts:
- J2: LCSC C45986647 -> C19171040; now fitted
Changed lines of the file:
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@@
 		(on_board yes)
 		(in_pos_files yes)
-		(dnp yes)
+		(dnp no)
 		(property "Reference" "J2"
 			(at 45.72 39.3699 0)
@@
 			)
 		)
-		(property "LCSC" "C45986647"
+		(property "LCSC" "C19171040"
 			(at 52.07 39.37 0)
 			(hide yes)
