File: ihss57-36-20_adapter/ihss57-36-20_adapter.kicad_pcb (KiCad board)
At the start: 2 copper layers, 50 x 64 mm, 20 parts, among them J1 T4141012051-000, J2 T4140012081-000, J3 5-535541-8, J4 1875425, U1 MUN5233T1G, U2 MUN5233T1G, U3 MUN5233T1G, U4 MUN5233T1G

Commit message: Updated the original servo adapter components/PCB design.
Parts:
- J3: value 5-535541-8 -> Conn_01x10_Socket; footprint servo_adapter_fp:5-535541-8_TYC -> Connector_PinSocket_2.54mm:PinSocket_1x10_P2.54mm_Vertical
- turned J3 to -90 degrees

Commit message: Updated routing using new net-ties.
Parts:
- added NT2: NetTie_2, NetTie:NetTie-2_SMD_Pad0.5mm, F.Cu at (105.4, 62.2)
- added NT3: NetTie_2, NetTie:NetTie-2_SMD_Pad0.5mm, F.Cu at (107.9, 57.2)
- added NT4: NetTie_2, NetTie:NetTie-2_SMD_Pad0.5mm, F.Cu at (113.0, 57.2)
- added NT5: NetTie_2, NetTie:NetTie-2_SMD_Pad0.5mm, F.Cu at (118.1, 57.2)
- added NT6: NetTie_2, NetTie:NetTie-2_SMD_Pad0.5mm, F.Cu at (123.2, 57.2)
- added NT7: NetTie_2, NetTie:NetTie-2_SMD_Pad0.5mm, F.Cu at (128.2, 57.2)
- moved R1 5.47 mm to (100.8, 64.1), turned to 0 degrees
- moved R2 5.47 mm to (106.2, 64.1), turned to 180 degrees
- moved NT1 2.21 mm to (110.5, 62.5)
- moved C1 0.15 mm to (135.2, 74.3), turned to 180 degrees
Connections:
- R1 pad 1: /PED- -> /ALM-
- R2 pad 1: /ALARM_OUT -> /PED-
Routing:
- net /+5V_Servo: track 112.8 -> 94.5 mm
- net /ALARM_OUT: track 79.0 -> 68.8 mm
- net /ALM-: track 0.00 -> 8.62 mm
- net GND: track 25.3 -> 18.7 mm, vias 21 -> 22
- net /PUL+: track 0.00 -> 1.96 mm
- net /PED+: track 0.00 -> 1.96 mm
- net /ENA+: track 0.00 -> 1.96 mm
- net /DIR+: track 0.00 -> 1.96 mm
- net /ALM+: track 0.00 -> 1.96 mm
- net /PED_OUT: track 54.0 -> 54.7 mm
