File: ihss57-36-20_adapter/ihss57-36-20_adapter.kicad_sch (KiCad schematic)
At the start: 20 parts, among them J1 T4141012051-000, J2 T4140012081-000, J3 5-535541-8, J4 1875425, U1 MUN5233T1G, U2 MUN5233T1G, U3 MUN5233T1G, U4 MUN5233T1G

Commit message: Updated the original servo adapter components/PCB design.
Parts:
- removed J3: 5-535541-8, 5-535541-8_TYC, symbol TE_5-535541-8:5-535541-8
- added J3, J5: Conn_01x10_Socket, Connector_PinSocket_2.54mm:PinSocket_1x10_P2.54mm_Vertical, symbol Connector:Conn_01x10_Socket
- added NT2: NetTie_2, NetTie:NetTie-2_SMD_Pad0.5mm, symbol Device:NetTie_2
- added NT3, NT4, NT5, NT6, NT7: NetTie_2, symbol Device:NetTie_2
- J1: LCSC (none) -> C7423411; now fitted
- J2: LCSC (none) -> C19171040; now fitted
Connections:
- net +5V_Servo: now also NT3.1, NT4.1, NT5.1, NT6.1, NT7.1
- net ALARM_OUT: now also NT2.1; no longer R2.1
- net DIR-: now also J3.7 (Pin_7)
- net ENA-: now also J3.5 (Pin_5)
- net PED-: now also R2.1, J3.3 (Pin_3); no longer R1.1
- net PUL-: now also J3.9 (Pin_9)
- new net ALM+: J3.2 (Pin_2), NT3.2
- new net ALM-: J3.1 (Pin_1), NT2.2, R1.1
- new net DIR+: J3.8 (Pin_8), NT6.2
- new net ENA+: J3.6 (Pin_6), NT5.2
- new net PED+: J3.4 (Pin_4), NT4.2
- new net PUL+: J3.10 (Pin_10), NT7.2
- no-connect marks 1 -> 11

Commit message: Updated routing using new net-ties.
Parts:
- NT3, NT4, NT5, NT6, NT7: footprint (none) -> NetTie:NetTie-2_SMD_Pad0.5mm
Changed lines of the file:
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@@
 			)
 		)
-		(property "Footprint" ""
+		(property "Footprint" "NetTie:NetTie-2_SMD_Pad0.5mm"
 			(at 203.2 76.2 0)
 			(hide yes)
@@
 			)
 		)
-		(property "Footprint" ""
+		(property "Footprint" "NetTie:NetTie-2_SMD_Pad0.5mm"
 			(at 203.2 81.28 0)
 			(hide yes)
@@
 			)
 		)
-		(property "Footprint" ""
+		(property "Footprint" "NetTie:NetTie-2_SMD_Pad0.5mm"
 			(at 203.2 71.12 0)
 			(hide yes)
@@
 			)
 		)
-		(property "Footprint" ""
+		(property "Footprint" "NetTie:NetTie-2_SMD_Pad0.5mm"
 			(at 203.2 66.04 0)
 			(hide yes)
@@
 			)
 		)
-		(property "Footprint" ""
+		(property "Footprint" "NetTie:NetTie-2_SMD_Pad0.5mm"
 			(at 203.2 86.36 0)
 			(hide yes)
